Commit message: 将realman的夹爪mimic关节改为仅在gazebo模式下启用

File: gripper/inspire_description/xacro/ros2_control/EG2-4C2.xacro (robot description, xacro)
@@ -3,4 +3,5 @@
   <!-- Inspire EG2-4C2夹爪完整接口定义宏 -->
   <xacro:macro name="eg2_4c2_interfaces" params="name">
+    <xacro:arg name="gazebo" default="false"/>
     <xacro:property name="prefix" value="${name + '_' if name else ''}"/>
     <!-- 夹爪主关节接口定义 -->
@@ -13,30 +14,32 @@
       <state_interface name="effort"/>
     </joint>
-    <!-- Inspire EG2-4C2夹爪的mimic关节接口 -->
-    <joint name="${prefix}left_inner_joint">
-      <state_interface name="position"/>
-      <state_interface name="velocity"/>
-      <state_interface name="effort"/>
-    </joint>
-    <joint name="${prefix}right_inner_joint">
-      <state_interface name="position"/>
-      <state_interface name="velocity"/>
-      <state_interface name="effort"/>
-    </joint>
-    <joint name="${prefix}right_outer_joint">
-      <state_interface name="position"/>
-      <state_interface name="velocity"/>
-      <state_interface name="effort"/>
-    </joint>
-    <joint name="${prefix}left_pad_joint">
-      <state_interface name="position"/>
-      <state_interface name="velocity"/>
-      <state_interface name="effort"/>
-    </joint>
-    <joint name="${prefix}right_pad_joint">
-      <state_interface name="position"/>
-      <state_interface name="velocity"/>
-      <state_interface name="effort"/>
-    </joint>
+    <xacro:if value="$(arg gazebo)">
+      <!-- Inspire EG2-4C2夹爪的mimic关节接口 (仅在Gazebo模式下启用) -->
+      <joint name="${prefix}left_inner_joint">
+        <state_interface name="position"/>
+        <state_interface name="velocity"/>
+        <state_interface name="effort"/>
+      </joint>
+      <joint name="${prefix}right_inner_joint">
+        <state_interface name="position"/>
+        <state_interface name="velocity"/>
+        <state_interface name="effort"/>
+      </joint>
+      <joint name="${prefix}right_outer_joint">
+        <state_interface name="position"/>
+        <state_interface name="velocity"/>
+        <state_interface name="effort"/>
+      </joint>
+      <joint name="${prefix}left_pad_joint">
+        <state_interface name="position"/>
+        <state_interface name="velocity"/>
+        <state_interface name="effort"/>
+      </joint>
+      <joint name="${prefix}right_pad_joint">
+        <state_interface name="position"/>
+        <state_interface name="velocity"/>
+        <state_interface name="effort"/>
+      </joint>
+    </xacro:if>
   </xacro:macro>
 </robot>
