Commit message: 修改关节命名错误

File: gripper/jodell_description/xacro/ros2_control/RG75-300.xacro (robot description, xacro)
@@ -16,5 +16,5 @@
     <xacro:if value="$(arg gazebo)">
       <!-- 右指 mimic 关节接口 (仅在Gazebo模式下启用) -->
-      <joint name="${prefix}right_driver_joint">
+      <joint name="${prefix}right_finger_joint">
         <state_interface name="position"/>
         <state_interface name="velocity"/>
