Commit message: swapped position for thumb_joint1 and thumb_joint2 to match modbus protocol

File: dexhands/linkerhand_description/xacro/l6.xacro (robot description, xacro)
@@ -88,5 +88,6 @@
 			</collision>
 		</link>
-		<joint name="${prefix}thumb_joint1" type="${joint_type}">
+		<joint name="${prefix}thumb_joint2" type="${joint_type}">
+			<!-- thumb_joint2: 大拇指横摆运动 (Current_Thumb_Yaw, Modbus Address 1) -->
 			<origin xyz="0.0078133 ${direction*-0.029898} 0.026692"/>
 			<parent link="${prefix}hand_base"/>
@@ -121,5 +122,6 @@
 			</collision>
 		</link>
-		<joint name="${prefix}thumb_joint2" type="${joint_type}">
+		<joint name="${prefix}thumb_joint1" type="${joint_type}">
+			<!-- thumb_joint1: 大拇指弯曲/伸直运动 (Current_Thumb_Pitch, Modbus Address 0) -->
 			<origin xyz="0.0050248 ${direction*-0.013602} 0.0066685"
 							rpy="${direction*1.2615} 0 ${direction*0.34907}"/>
@@ -162,5 +164,5 @@
 				<axis xyz="${direction*-1} 0 0"/>
 				<limit lower="0" upper="1.22" effort="100" velocity="1"/>
-				<mimic joint="${prefix}thumb_joint2" multiplier="1.23" offset="0"/>
+				<mimic joint="${prefix}thumb_joint1" multiplier="1.23" offset="0"/>
 			</xacro:unless>
 		</joint>

File: dexhands/linkerhand_description/xacro/o6.xacro (robot description, xacro)
@@ -92,5 +92,6 @@
 			</collision>
 		</link>
-		<joint name="${prefix}thumb_joint1" type="${joint_type}">
+		<joint name="${prefix}thumb_joint2" type="${joint_type}">
+			<!-- thumb_joint2: 大拇指横摆运动 (Current_Thumb_Yaw, Modbus Address 1) -->
 			<origin xyz="0.011508 ${direction*-0.022975} 0.032794"/>
 			<parent link="${prefix}hand_base"/>
@@ -127,5 +128,5 @@
 			</collision>
 		</link>
-		<joint name="${prefix}thumb_joint2" type="${joint_type}">
+		<joint name="${prefix}thumb_joint1" type="${joint_type}">
 			<origin xyz="0.0061649 ${direction*-0.010678} -0.004891" rpy="0 -1.1529 ${direction*2.0944}"/>
 			<parent link="${prefix}thumb_metacarpals_base2"/>
@@ -167,5 +168,5 @@
 				<axis xyz="0 1 0"/>
 				<limit lower="0" upper="1.08" effort="100" velocity="1"/>
-				<mimic joint="${prefix}thumb_joint2" multiplier="1.86" offset="0"/>
+				<mimic joint="${prefix}thumb_joint1" multiplier="1.86" offset="0"/>
 			</xacro:unless>
 		</joint>

File: dexhands/linkerhand_description/xacro/ros2_control/o6.xacro (robot description, xacro)
@@ -6,5 +6,6 @@
     <xacro:property name="prefix" value="${name + '_' if name else ''}"/>
     <!-- 6个主控关节接口定义 -->
-    <!-- 拇指关节 -->
+    <!-- 关节顺序与 Modbus 协议地址顺序一致 -->
+    <!-- Address 0: Current_Thumb_Pitch (大拇指弯曲) - thumb_joint1 是第一个关节 -->
     <joint name="${prefix}thumb_joint1">
       <command_interface name="position"/>
@@ -15,4 +16,5 @@
       <state_interface name="effort"/>
     </joint>
+    <!-- Address 1: Current_Thumb_Yaw (大拇指横摆) - thumb_joint2 是第二个关节 -->
     <joint name="${prefix}thumb_joint2">
       <command_interface name="position"/>

Commit message: migrate to glb mesh

File: dexhands/linkerhand_description/xacro/l6.xacro (robot description, xacro)
@@ -19,10 +19,10 @@
 				<visual>
 					<geometry>
-						<mesh filename="file://$(find changingtek_description)/meshes/AG2F90-C/visual/flange.obj"/>
+						<mesh filename="file://$(find changingtek_description)/meshes/AG2F90-C/visual/flange.glb"/>
 					</geometry>
 				</visual>
 				<visual>
 					<geometry>
-						<mesh filename="file://$(find linkerhand_description)/meshes/o6/flange.obj"/>
+						<mesh filename="file://$(find linkerhand_description)/meshes/o6/flange.glb"/>
 					</geometry>
 				</visual>
@@ -50,11 +50,11 @@
 			<visual>
 				<geometry>
-					<mesh filename="file://$(find linkerhand_description)/meshes/l6/base.obj"
-								scale="1 ${direction} 1"/>
-				</geometry>
-			</visual>
-			<collision>
-				<geometry>
-					<mesh filename="file://$(find linkerhand_description)/meshes/l6/base.obj"
+					<mesh filename="file://$(find linkerhand_description)/meshes/l6/base.glb"
+								scale="1 ${direction} 1"/>
+				</geometry>
+			</visual>
+			<collision>
+				<geometry>
+					<mesh filename="file://$(find linkerhand_description)/meshes/l6/base.glb"
 								scale="1 ${direction} 1"/>
 				</geometry>
@@ -77,11 +77,11 @@
 			<visual>
 				<geometry>
-					<mesh filename="file://$(find linkerhand_description)/meshes/l6/thumb_metacarpals_base.obj"
-								scale="1 ${direction} 1"/>
-				</geometry>
-			</visual>
-			<collision>
-				<geometry>
-					<mesh filename="file://$(find linkerhand_description)/meshes/l6/thumb_metacarpals_base.obj"
+					<mesh filename="file://$(find linkerhand_description)/meshes/l6/thumb_metacarpals_base.glb"
+								scale="1 ${direction} 1"/>
+				</geometry>
+			</visual>
+			<collision>
+				<geometry>
+					<mesh filename="file://$(find linkerhand_description)/meshes/l6/thumb_metacarpals_base.glb"
 								scale="1 ${direction} 1"/>
 				</geometry>
@@ -111,11 +111,11 @@
 			<visual>
 				<geometry>
-					<mesh filename="file://$(find linkerhand_description)/meshes/l6/thumb_metacarpals.obj"
-								scale="1 ${direction} 1"/>
-				</geometry>
-			</visual>
-			<collision>
-				<geometry>
-					<mesh filename="file://$(find linkerhand_description)/meshes/l6/thumb_metacarpals.obj"
+					<mesh filename="file://$(find linkerhand_description)/meshes/l6/thumb_metacarpals.glb"
+								scale="1 ${direction} 1"/>
+				</geometry>
+			</visual>
+			<collision>
+				<geometry>
+					<mesh filename="file://$(find linkerhand_description)/meshes/l6/thumb_metacarpals.glb"
 								scale="1 ${direction} 1"/>
 				</geometry>
@@ -146,11 +146,11 @@
 			<visual>
 				<geometry>
-					<mesh filename="file://$(find linkerhand_description)/meshes/l6/thumb_distal.obj"
-								scale="1 ${direction} 1"/>
-				</geometry>
-			</visual>
-			<collision>
-				<geometry>
-					<mesh filename="file://$(find linkerhand_description)/meshes/l6/thumb_distal.obj"
+					<mesh filename="file://$(find linkerhand_description)/meshes/l6/thumb_distal.glb"
+								scale="1 ${direction} 1"/>
+				</geometry>
+			</visual>
+			<collision>
+				<geometry>
+					<mesh filename="file://$(find linkerhand_description)/meshes/l6/thumb_distal.glb"
 								scale="1 ${direction} 1"/>
 				</geometry>
@@ -183,11 +183,11 @@
 			<visual>
 				<geometry>
-					<mesh filename="file://$(find linkerhand_description)/meshes/l6/index_proximal.obj"
-								scale="1 ${direction} 1"/>
-				</geometry>
-			</visual>
-			<collision>
-				<geometry>
-					<mesh filename="file://$(find linkerhand_description)/meshes/l6/index_proximal.obj"
+					<mesh filename="file://$(find linkerhand_description)/meshes/l6/index_proximal.glb"
+								scale="1 ${direction} 1"/>
+				</geometry>
+			</visual>
+			<collision>
+				<geometry>
+					<mesh filename="file://$(find linkerhand_description)/meshes/l6/index_proximal.glb"
 								scale="1 ${direction} 1"/>
 				</geometry>
@@ -216,10 +216,10 @@
 			<visual>
 				<geometry>
-					<mesh filename="file://$(find linkerhand_description)/meshes/l6/index_distal.obj"/>
-				</geometry>
-			</visual>
-			<collision>
-				<geometry>
-					<mesh filename="file://$(find linkerhand_description)/meshes/l6/index_distal.obj"/>
+					<mesh filename="file://$(find linkerhand_description)/meshes/l6/index_distal.glb"/>
+				</geometry>
+			</visual>
+			<collision>
+				<geometry>
+					<mesh filename="file://$(find linkerhand_description)/meshes/l6/index_distal.glb"/>
 				</geometry>
 			</collision>
@@ -251,10 +251,10 @@
 			<visual>
 				<geometry>
-					<mesh filename="file://$(find linkerhand_description)/meshes/l6/index_proximal.obj"/>
-				</geometry>
-			</visual>
-			<collision>
-				<geometry>
-					<mesh filename="file://$(find linkerhand_description)/meshes/l6/index_proximal.obj"/>
+					<mesh filename="file://$(find linkerhand_description)/meshes/l6/index_proximal.glb"/>
+				</geometry>
+			</visual>
+			<collision>
+				<geometry>
+					<mesh filename="file://$(find linkerhand_description)/meshes/l6/index_proximal.glb"/>
 				</geometry>
 			</collision>
@@ -282,10 +282,10 @@
 			<visual>
 				<geometry>
-					<mesh filename="file://$(find linkerhand_description)/meshes/l6/index_distal.obj"/>
-				</geometry>
-			</visual>
-			<collision>
-				<geometry>
-					<mesh filename="file://$(find linkerhand_description)/meshes/l6/index_distal.obj"/>
+					<mesh filename="file://$(find linkerhand_description)/meshes/l6/index_distal.glb"/>
+				</geometry>
+			</visual>
+			<collision>
+				<geometry>
+					<mesh filename="file://$(find linkerhand_description)/meshes/l6/index_distal.glb"/>
 				</geometry>
 			</collision>
@@ -317,10 +317,10 @@
 			<visual>
 				<geometry>
-					<mesh filename="file://$(find linkerhand_description)/meshes/l6/index_proximal.obj"/>
-				</geometry>
-			</visual>
-			<collision>
-				<geometry>
-					<mesh filename="file://$(find linkerhand_description)/meshes/l6/index_proximal.obj"/>
+					<mesh filename="file://$(find linkerhand_description)/meshes/l6/index_proximal.glb"/>
+				</geometry>
+			</visual>
+			<collision>
+				<geometry>
+					<mesh filename="file://$(find linkerhand_description)/meshes/l6/index_proximal.glb"/>
 				</geometry>
 			</collision>
@@ -348,10 +348,10 @@
 			<visual>
 				<geometry>
-					<mesh filename="file://$(find linkerhand_description)/meshes/l6/index_distal.obj"/>
-				</geometry>
-			</visual>
-			<collision>
-				<geometry>
-					<mesh filename="file://$(find linkerhand_description)/meshes/l6/index_distal.obj"/>
+					<mesh filename="file://$(find linkerhand_description)/meshes/l6/index_distal.glb"/>
+				</geometry>
+			</visual>
+			<collision>
+				<geometry>
+					<mesh filename="file://$(find linkerhand_description)/meshes/l6/index_distal.glb"/>
 				</geometry>
 			</collision>
@@ -383,10 +383,10 @@
 			<visual>
 				<geometry>
-					<mesh filename="file://$(find linkerhand_description)/meshes/l6/index_proximal.obj"/>
-				</geometry>
-			</visual>
-			<collision>
-				<geometry>
-					<mesh filename="file://$(find linkerhand_description)/meshes/l6/index_proximal.obj"/>
+					<mesh filename="file://$(find linkerhand_description)/meshes/l6/index_proximal.glb"/>
+				</geometry>
+			</visual>
+			<collision>
+				<geometry>
+					<mesh filename="file://$(find linkerhand_description)/meshes/l6/index_proximal.glb"/>
 				</geometry>
 			</collision>
@@ -414,10 +414,10 @@
 			<visual>
 				<geometry>
-					<mesh filename="file://$(find linkerhand_description)/meshes/l6/index_distal.obj"/>
-				</geometry>
-			</visual>
-			<collision>
-				<geometry>
-					<mesh filename="file://$(find linkerhand_description)/meshes/l6/index_distal.obj"/>
+					<mesh filename="file://$(find linkerhand_description)/meshes/l6/index_distal.glb"/>
+				</geometry>
+			</visual>
+			<collision>
+				<geometry>
+					<mesh filename="file://$(find linkerhand_description)/meshes/l6/index_distal.glb"/>
 				</geometry>
 			</collision>

File: dexhands/linkerhand_description/xacro/o6.xacro (robot description, xacro)
@@ -19,10 +19,10 @@
 				<visual>
 					<geometry>
-						<mesh filename="file://$(find changingtek_description)/meshes/AG2F90-C/visual/flange.obj"/>
+						<mesh filename="file://$(find changingtek_description)/meshes/AG2F90-C/visual/flange.glb"/>
 					</geometry>
 				</visual>
 				<visual>
 					<geometry>
-						<mesh filename="file://$(find linkerhand_description)/meshes/o6/flange.obj"/>
+						<mesh filename="file://$(find linkerhand_description)/meshes/o6/flange.glb"/>
 					</geometry>
 				</visual>
@@ -52,11 +52,11 @@
 			<visual>
 				<geometry>
-					<mesh filename="file://$(find linkerhand_description)/meshes/o6/hand_base.obj"
-								scale="1 ${direction} 1"/>
-				</geometry>
-			</visual>
-			<collision>
-				<geometry>
-					<mesh filename="file://$(find linkerhand_description)/meshes/o6/hand_base.obj"
+					<mesh filename="file://$(find linkerhand_description)/meshes/o6/hand_base.glb"
+								scale="1 ${direction} 1"/>
+				</geometry>
+			</visual>
+			<collision>
+				<geometry>
+					<mesh filename="file://$(find linkerhand_description)/meshes/o6/hand_base.glb"
 								scale="1 ${direction} 1"/>
 				</geometry>
@@ -81,11 +81,11 @@
 			<visual>
 				<geometry>
-					<mesh filename="file://$(find linkerhand_description)/meshes/o6/thumb_metacarpals_base.obj"
-								scale="1 ${direction} 1"/>
-				</geometry>
-			</visual>
-			<collision>
-				<geometry>
-					<mesh filename="file://$(find linkerhand_description)/meshes/o6/thumb_metacarpals_base.obj"
+					<mesh filename="file://$(find linkerhand_description)/meshes/o6/thumb_metacarpals_base.glb"
+								scale="1 ${direction} 1"/>
+				</geometry>
+			</visual>
+			<collision>
+				<geometry>
+					<mesh filename="file://$(find linkerhand_description)/meshes/o6/thumb_metacarpals_base.glb"
 								scale="1 ${direction} 1"/>
 				</geometry>
@@ -117,11 +117,11 @@
 			<visual>
 				<geometry>
-					<mesh filename="file://$(find linkerhand_description)/meshes/o6/thumb_metacarpals.obj"
-								scale="1 ${direction} 1"/>
-				</geometry>
-			</visual>
-			<collision>
-				<geometry>
-					<mesh filename="file://$(find linkerhand_description)/meshes/o6/thumb_metacarpals.obj"
+					<mesh filename="file://$(find linkerhand_description)/meshes/o6/thumb_metacarpals.glb"
+								scale="1 ${direction} 1"/>
+				</geometry>
+			</visual>
+			<collision>
+				<geometry>
+					<mesh filename="file://$(find linkerhand_description)/meshes/o6/thumb_metacarpals.glb"
 								scale="1 ${direction} 1"/>
 				</geometry>
@@ -152,10 +152,10 @@
 			<visual>
 				<geometry>
-					<mesh filename="file://$(find linkerhand_description)/meshes/o6/thumb_distal.obj"/>
-				</geometry>
-			</visual>
-			<collision>
-				<geometry>
-					<mesh filename="file://$(find linkerhand_description)/meshes/o6/thumb_distal.obj"/>
+					<mesh filename="file://$(find linkerhand_description)/meshes/o6/thumb_distal.glb"/>
+				</geometry>
+			</visual>
+			<collision>
+				<geometry>
+					<mesh filename="file://$(find linkerhand_description)/meshes/o6/thumb_distal.glb"/>
 				</geometry>
 			</collision>
@@ -189,10 +189,10 @@
 			<visual>
 				<geometry>
-					<mesh filename="file://$(find linkerhand_description)/meshes/o6/index_proximal.obj"/>
-				</geometry>
-			</visual>
-			<collision>
-				<geometry>
-					<mesh filename="file://$(find linkerhand_description)/meshes/o6/index_proximal.obj"/>
+					<mesh filename="file://$(find linkerhand_description)/meshes/o6/index_proximal.glb"/>
+				</geometry>
+			</visual>
+			<collision>
+				<geometry>
+					<mesh filename="file://$(find linkerhand_description)/meshes/o6/index_proximal.glb"/>
 				</geometry>
 			</collision>
@@ -222,10 +222,10 @@
 			<visual>
 				<geometry>
-					<mesh filename="file://$(find linkerhand_description)/meshes/o6/index_distal.obj"/>
-				</geometry>
-			</visual>
-			<collision>
-				<geometry>
-					<mesh filename="file://$(find linkerhand_description)/meshes/o6/index_distal.obj"/>
+					<mesh filename="file://$(find linkerhand_description)/meshes/o6/index_distal.glb"/>
+				</geometry>
+			</visual>
+			<collision>
+				<geometry>
+					<mesh filename="file://$(find linkerhand_description)/meshes/o6/index_distal.glb"/>
 				</geometry>
 			</collision>
@@ -259,10 +259,10 @@
 			<visual>
 				<geometry>
-					<mesh filename="file://$(find linkerhand_description)/meshes/o6/index_proximal.obj"/>
-				</geometry>
-			</visual>
-			<collision>
-				<geometry>
-					<mesh filename="file://$(find linkerhand_description)/meshes/o6/index_proximal.obj"/>
+					<mesh filename="file://$(find linkerhand_description)/meshes/o6/index_proximal.glb"/>
+				</geometry>
+			</visual>
+			<collision>
+				<geometry>
+					<mesh filename="file://$(find linkerhand_description)/meshes/o6/index_proximal.glb"/>
 				</geometry>
 			</collision>
@@ -292,10 +292,10 @@
 			<visual>
 				<geometry>
-					<mesh filename="file://$(find linkerhand_description)/meshes/o6/index_distal.obj"/>
-				</geometry>
-			</visual>
-			<collision>
-				<geometry>
-					<mesh filename="file://$(find linkerhand_description)/meshes/o6/index_distal.obj"/>
+					<mesh filename="file://$(find linkerhand_description)/meshes/o6/index_distal.glb"/>
+				</geometry>
+			</visual>
+			<collision>
+				<geometry>
+					<mesh filename="file://$(find linkerhand_description)/meshes/o6/index_distal.glb"/>
 				</geometry>
 			</collision>
@@ -329,10 +329,10 @@
 			<visual>
 				<geometry>
-					<mesh filename="file://$(find linkerhand_description)/meshes/o6/index_proximal.obj"/>
-				</geometry>
-			</visual>
-			<collision>
-				<geometry>
-					<mesh filename="file://$(find linkerhand_description)/meshes/o6/index_proximal.obj"/>
+					<mesh filename="file://$(find linkerhand_description)/meshes/o6/index_proximal.glb"/>
+				</geometry>
+			</visual>
+			<collision>
+				<geometry>
+					<mesh filename="file://$(find linkerhand_description)/meshes/o6/index_proximal.glb"/>
 				</geometry>
 			</collision>
@@ -362,10 +362,10 @@
 			<visual>
 				<geometry>
-					<mesh filename="file://$(find linkerhand_description)/meshes/o6/index_distal.obj"/>
-				</geometry>
-			</visual>
-			<collision>
-				<geometry>
-					<mesh filename="file://$(find linkerhand_description)/meshes/o6/index_distal.obj"/>
+					<mesh filename="file://$(find linkerhand_description)/meshes/o6/index_distal.glb"/>
+				</geometry>
+			</visual>
+			<collision>
+				<geometry>
+					<mesh filename="file://$(find linkerhand_description)/meshes/o6/index_distal.glb"/>
 				</geometry>
 			</collision>
@@ -399,10 +399,10 @@
 			<visual>
 				<geometry>
-					<mesh filename="file://$(find linkerhand_description)/meshes/o6/index_proximal.obj"/>
-				</geometry>
-			</visual>
-			<collision>
-				<geometry>
-					<mesh filename="file://$(find linkerhand_description)/meshes/o6/index_proximal.obj"/>
+					<mesh filename="file://$(find linkerhand_description)/meshes/o6/index_proximal.glb"/>
+				</geometry>
+			</visual>
+			<collision>
+				<geometry>
+					<mesh filename="file://$(find linkerhand_description)/meshes/o6/index_proximal.glb"/>
 				</geometry>
 			</collision>
@@ -432,10 +432,10 @@
 			<visual>
 				<geometry>
-					<mesh filename="file://$(find linkerhand_description)/meshes/o6/index_distal.obj"/>
-				</geometry>
-			</visual>
-			<collision>
-				<geometry>
-					<mesh filename="file://$(find linkerhand_description)/meshes/o6/index_distal.obj"/>
+					<mesh filename="file://$(find linkerhand_description)/meshes/o6/index_distal.glb"/>
+				</geometry>
+			</visual>
+			<collision>
+				<geometry>
+					<mesh filename="file://$(find linkerhand_description)/meshes/o6/index_distal.glb"/>
 				</geometry>
 			</collision>
