Commit message: migrate to glb mesh

File: dexhands/linkerhand_description/xacro/o7.xacro (robot description, xacro)
@@ -22,11 +22,11 @@
 			<visual>
 				<geometry>
-					<mesh filename="file://$(find linkerhand_description)/meshes/o7/base.obj"
-								scale="1 ${direction} 1"/>
-				</geometry>
-			</visual>
-			<collision>
-				<geometry>
-					<mesh filename="file://$(find linkerhand_description)/meshes/o7/base.obj"
+					<mesh filename="file://$(find linkerhand_description)/meshes/o7/base.glb"
+								scale="1 ${direction} 1"/>
+				</geometry>
+			</visual>
+			<collision>
+				<geometry>
+					<mesh filename="file://$(find linkerhand_description)/meshes/o7/base.glb"
 								scale="1 ${direction} 1"/>
 				</geometry>
@@ -51,11 +51,11 @@
 			<visual>
 				<geometry>
-					<mesh filename="file://$(find linkerhand_description)/meshes/o7/thumb_1.obj"
-								scale="1 ${direction} 1"/>
-				</geometry>
-			</visual>
-			<collision>
-				<geometry>
-					<mesh filename="file://$(find linkerhand_description)/meshes/o7/thumb_1.obj"
+					<mesh filename="file://$(find linkerhand_description)/meshes/o7/thumb_metacarpals_base2.glb"
+								scale="1 ${direction} 1"/>
+				</geometry>
+			</visual>
+			<collision>
+				<geometry>
+					<mesh filename="file://$(find linkerhand_description)/meshes/o7/thumb_metacarpals_base2.glb"
 								scale="1 ${direction} 1"/>
 				</geometry>
@@ -86,11 +86,11 @@
 			<visual>
 				<geometry>
-					<mesh filename="file://$(find linkerhand_description)/meshes/o7/thumb_2.obj"
-								scale="1 ${direction} 1"/>
-				</geometry>
-			</visual>
-			<collision>
-				<geometry>
-					<mesh filename="file://$(find linkerhand_description)/meshes/o7/thumb_2.obj"
+					<mesh filename="file://$(find linkerhand_description)/meshes/o7/thumb_metacarpals_base2.glb"
+								scale="1 ${direction} 1"/>
+				</geometry>
+			</visual>
+			<collision>
+				<geometry>
+					<mesh filename="file://$(find linkerhand_description)/meshes/o7/thumb_metacarpals_base2.glb"
 								scale="1 ${direction} 1"/>
 				</geometry>
@@ -121,11 +121,11 @@
 			<visual>
 				<geometry>
-					<mesh filename="file://$(find linkerhand_description)/meshes/o7/thumb_3.obj"
-								scale="1 ${direction} 1"/>
-				</geometry>
-			</visual>
-			<collision>
-				<geometry>
-					<mesh filename="file://$(find linkerhand_description)/meshes/o7/thumb_3.obj"
+					<mesh filename="file://$(find linkerhand_description)/meshes/o7/thumb_metacarpals.glb"
+								scale="1 ${direction} 1"/>
+				</geometry>
+			</visual>
+			<collision>
+				<geometry>
+					<mesh filename="file://$(find linkerhand_description)/meshes/o7/thumb_metacarpals.glb"
 								scale="1 ${direction} 1"/>
 				</geometry>
@@ -156,10 +156,10 @@
 			<visual>
 				<geometry>
-					<mesh filename="file://$(find linkerhand_description)/meshes/o7/thumb_4.obj"/>
-				</geometry>
-			</visual>
-			<collision>
-				<geometry>
-					<mesh filename="file://$(find linkerhand_description)/meshes/o7/thumb_4.obj"/>
+					<mesh filename="file://$(find linkerhand_description)/meshes/o7/thumb_proximal.glb"/>
+				</geometry>
+			</visual>
+			<collision>
+				<geometry>
+					<mesh filename="file://$(find linkerhand_description)/meshes/o7/thumb_proximal.glb"/>
 				</geometry>
 			</collision>
@@ -189,10 +189,10 @@
 			<visual>
 				<geometry>
-					<mesh filename="file://$(find linkerhand_description)/meshes/o7/thumb_5.obj"/>
-				</geometry>
-			</visual>
-			<collision>
-				<geometry>
-					<mesh filename="file://$(find linkerhand_description)/meshes/o7/thumb_5.obj"/>
+					<mesh filename="file://$(find linkerhand_description)/meshes/o7/thumb_distal.glb"/>
+				</geometry>
+			</visual>
+			<collision>
+				<geometry>
+					<mesh filename="file://$(find linkerhand_description)/meshes/o7/thumb_distal.glb"/>
 				</geometry>
 			</collision>
@@ -226,10 +226,10 @@
 			<visual>
 				<geometry>
-					<mesh filename="file://$(find linkerhand_description)/meshes/o7/index_1.obj"/>
-				</geometry>
-			</visual>
-			<collision>
-				<geometry>
-					<mesh filename="file://$(find linkerhand_description)/meshes/o7/index_1.obj"/>
+					<mesh filename="file://$(find linkerhand_description)/meshes/o7/index_proximal.glb"/>
+				</geometry>
+			</visual>
+			<collision>
+				<geometry>
+					<mesh filename="file://$(find linkerhand_description)/meshes/o7/index_proximal.glb"/>
 				</geometry>
 			</collision>
@@ -257,10 +257,10 @@
 			<visual>
 				<geometry>
-					<mesh filename="file://$(find linkerhand_description)/meshes/o7/index_2.obj"/>
-				</geometry>
-			</visual>
-			<collision>
-				<geometry>
-					<mesh filename="file://$(find linkerhand_description)/meshes/o7/index_2.obj"/>
+					<mesh filename="file://$(find linkerhand_description)/meshes/o7/index_middle.glb"/>
+				</geometry>
+			</visual>
+			<collision>
+				<geometry>
+					<mesh filename="file://$(find linkerhand_description)/meshes/o7/index_middle.glb"/>
 				</geometry>
 			</collision>
@@ -291,10 +291,10 @@
 			<visual>
 				<geometry>
-					<mesh filename="file://$(find linkerhand_description)/meshes/o7/index_3.obj"/>
-				</geometry>
-			</visual>
-			<collision>
-				<geometry>
-					<mesh filename="file://$(find linkerhand_description)/meshes/o7/index_3.obj"/>
+					<mesh filename="file://$(find linkerhand_description)/meshes/o7/index_distal.glb"/>
+				</geometry>
+			</visual>
+			<collision>
+				<geometry>
+					<mesh filename="file://$(find linkerhand_description)/meshes/o7/index_distal.glb"/>
 				</geometry>
 			</collision>
@@ -328,10 +328,10 @@
 			<visual>
 				<geometry>
-					<mesh filename="file://$(find linkerhand_description)/meshes/o7/index_1.obj"/>
-				</geometry>
-			</visual>
-			<collision>
-				<geometry>
-					<mesh filename="file://$(find linkerhand_description)/meshes/o7/index_1.obj"/>
+					<mesh filename="file://$(find linkerhand_description)/meshes/o7/index_proximal.glb"/>
+				</geometry>
+			</visual>
+			<collision>
+				<geometry>
+					<mesh filename="file://$(find linkerhand_description)/meshes/o7/index_proximal.glb"/>
 				</geometry>
 			</collision>
@@ -359,10 +359,10 @@
 			<visual>
 				<geometry>
-					<mesh filename="file://$(find linkerhand_description)/meshes/o7/index_2.obj"/>
-				</geometry>
-			</visual>
-			<collision>
-				<geometry>
-					<mesh filename="file://$(find linkerhand_description)/meshes/o7/index_2.obj"/>
+					<mesh filename="file://$(find linkerhand_description)/meshes/o7/index_middle.glb"/>
+				</geometry>
+			</visual>
+			<collision>
+				<geometry>
+					<mesh filename="file://$(find linkerhand_description)/meshes/o7/index_middle.glb"/>
 				</geometry>
 			</collision>
@@ -393,10 +393,10 @@
 			<visual>
 				<geometry>
-					<mesh filename="file://$(find linkerhand_description)/meshes/o7/index_3.obj"/>
-				</geometry>
-			</visual>
-			<collision>
-				<geometry>
-					<mesh filename="file://$(find linkerhand_description)/meshes/o7/index_3.obj"/>
+					<mesh filename="file://$(find linkerhand_description)/meshes/o7/index_distal.glb"/>
+				</geometry>
+			</visual>
+			<collision>
+				<geometry>
+					<mesh filename="file://$(find linkerhand_description)/meshes/o7/index_distal.glb"/>
 				</geometry>
 			</collision>
@@ -430,10 +430,10 @@
 			<visual>
 				<geometry>
-					<mesh filename="file://$(find linkerhand_description)/meshes/o7/index_1.obj"/>
-				</geometry>
-			</visual>
-			<collision>
-				<geometry>
-					<mesh filename="file://$(find linkerhand_description)/meshes/o7/index_1.obj"/>
+					<mesh filename="file://$(find linkerhand_description)/meshes/o7/index_proximal.glb"/>
+				</geometry>
+			</visual>
+			<collision>
+				<geometry>
+					<mesh filename="file://$(find linkerhand_description)/meshes/o7/index_proximal.glb"/>
 				</geometry>
 			</collision>
@@ -461,10 +461,10 @@
 			<visual>
 				<geometry>
-					<mesh filename="file://$(find linkerhand_description)/meshes/o7/index_2.obj"/>
-				</geometry>
-			</visual>
-			<collision>
-				<geometry>
-					<mesh filename="file://$(find linkerhand_description)/meshes/o7/index_2.obj"/>
+					<mesh filename="file://$(find linkerhand_description)/meshes/o7/index_middle.glb"/>
+				</geometry>
+			</visual>
+			<collision>
+				<geometry>
+					<mesh filename="file://$(find linkerhand_description)/meshes/o7/index_middle.glb"/>
 				</geometry>
 			</collision>
@@ -495,10 +495,10 @@
 			<visual>
 				<geometry>
-					<mesh filename="file://$(find linkerhand_description)/meshes/o7/index_3.obj"/>
-				</geometry>
-			</visual>
-			<collision>
-				<geometry>
-					<mesh filename="file://$(find linkerhand_description)/meshes/o7/index_3.obj"/>
+					<mesh filename="file://$(find linkerhand_description)/meshes/o7/index_distal.glb"/>
+				</geometry>
+			</visual>
+			<collision>
+				<geometry>
+					<mesh filename="file://$(find linkerhand_description)/meshes/o7/index_distal.glb"/>
 				</geometry>
 			</collision>
@@ -532,10 +532,10 @@
 			<visual>
 				<geometry>
-					<mesh filename="file://$(find linkerhand_description)/meshes/o7/index_1.obj"/>
-				</geometry>
-			</visual>
-			<collision>
-				<geometry>
-					<mesh filename="file://$(find linkerhand_description)/meshes/o7/index_1.obj"/>
+					<mesh filename="file://$(find linkerhand_description)/meshes/o7/index_proximal.glb"/>
+				</geometry>
+			</visual>
+			<collision>
+				<geometry>
+					<mesh filename="file://$(find linkerhand_description)/meshes/o7/index_proximal.glb"/>
 				</geometry>
 			</collision>
@@ -563,10 +563,10 @@
 			<visual>
 				<geometry>
-					<mesh filename="file://$(find linkerhand_description)/meshes/o7/index_2.obj"/>
-				</geometry>
-			</visual>
-			<collision>
-				<geometry>
-					<mesh filename="file://$(find linkerhand_description)/meshes/o7/index_2.obj"/>
+					<mesh filename="file://$(find linkerhand_description)/meshes/o7/index_middle.glb"/>
+				</geometry>
+			</visual>
+			<collision>
+				<geometry>
+					<mesh filename="file://$(find linkerhand_description)/meshes/o7/index_middle.glb"/>
 				</geometry>
 			</collision>
@@ -597,10 +597,10 @@
 			<visual>
 				<geometry>
-					<mesh filename="file://$(find linkerhand_description)/meshes/o7/index_3.obj"/>
-				</geometry>
-			</visual>
-			<collision>
-				<geometry>
-					<mesh filename="file://$(find linkerhand_description)/meshes/o7/index_3.obj"/>
+					<mesh filename="file://$(find linkerhand_description)/meshes/o7/index_distal.glb"/>
+				</geometry>
+			</visual>
+			<collision>
+				<geometry>
+					<mesh filename="file://$(find linkerhand_description)/meshes/o7/index_distal.glb"/>
 				</geometry>
 			</collision>
