Commit message: linkerhand o7 flange

File: dexhands/linkerhand_description/xacro/o7.xacro (robot description, xacro)
@@ -4,4 +4,29 @@
 		<xacro:property name="prefix" value="${name + '_' if name else ''}"/>
 		<xacro:property name="joint_type" value="${fixed_joints and 'fixed' or 'revolute'}"/>
+		<xacro:if value="${use_flange}">
+			<link name="${prefix}flange">
+				<inertial>
+					<origin xyz="-0.000388 0.002345 0.0"/>
+					<mass value="0.114"/>
+					<inertia
+							ixx="0.000040105"
+							ixy="0.000000214"
+							ixz="0.0"
+							iyy="0.000085776"
+							iyz="0.0"
+							izz="0.000054044"/>
+				</inertial>
+				<visual>
+					<geometry>
+						<mesh filename="file://$(find linkerhand_description)/meshes/o7/flange.glb"/>
+					</geometry>
+				</visual>
+			</link>
+			<joint name="${prefix}flange_joint" type="fixed">
+				<origin xyz="0 0 0.022"/>
+				<parent link="${prefix}flange"/>
+				<child link="${prefix}hand_base"/>
+			</joint>
+		</xacro:if>
 		<!-- ========================================== -->
 		<!-- 手掌基座 (Hand Base) -->

Commit message: fix linkerhand o7 joint order

File: dexhands/linkerhand_description/xacro/o7.xacro (robot description, xacro)
@@ -87,5 +87,5 @@
 			</collision>
 		</link>
-		<joint name="${prefix}thumb_joint1" type="${joint_type}">
+		<joint name="${prefix}thumb_joint3" type="${joint_type}">
 			<origin xyz="-0.0116 ${direction*-0.018174} 0.061651"/>
 			<parent link="${prefix}hand_base"/>
@@ -157,5 +157,5 @@
 			</collision>
 		</link>
-		<joint name="${prefix}thumb_joint3" type="${joint_type}">
+		<joint name="${prefix}thumb_joint1" type="${joint_type}">
 			<origin xyz="0.00456 ${direction*-0.015168} -0.0019302" rpy="0 -0.9163 ${direction*1.8628}"/>
 			<parent link="${prefix}thumb_metacarpals_base2"/>
@@ -197,5 +197,5 @@
 				<axis xyz="0 1 0"/>
 				<limit lower="0" upper="0.7152" effort="100" velocity="1"/>
-				<mimic joint="${prefix}thumb_joint3" multiplier="1.3898" offset="0"/>
+				<mimic joint="${prefix}thumb_joint1" multiplier="1.3898" offset="0"/>
 			</xacro:unless>
 		</joint>
@@ -230,5 +230,5 @@
 				<axis xyz="0 1 0"/>
 				<limit lower="0" upper="0.7763" effort="100" velocity="1"/>
-				<mimic joint="${prefix}thumb_joint3" multiplier="1.5085" offset="0"/>
+				<mimic joint="${prefix}thumb_joint1" multiplier="1.5085" offset="0"/>
 			</xacro:unless>
 		</joint>
