Commit message: Remove unused com parameters

File: dexhands/linkerhand_description/xacro/hand.xacro (robot description, xacro)
@@ -3,32 +3,17 @@
 	<xacro:arg name="type" default="o7"/>
 	<xacro:arg name="direction" default="1"/>
-	<!-- 质量中心偏移配置 (Center of Mass Offset) -->
-	<!-- 为不同类型的手设置质量中心偏移，用于调整惯性参数 -->
-	<!-- 单位: 米，默认值为 0 表示不偏移 -->
-	<!-- O7 手质量中心偏移 -->
-	<xacro:arg name="com_offset_o7_x" default="0"/>
-	<xacro:arg name="com_offset_o7_y" default="0"/>
-	<xacro:arg name="com_offset_o7_z" default="0"/>
-	<!-- O6 手质量中心偏移 -->
-	<xacro:arg name="com_offset_o6_x" default="0"/>
-	<xacro:arg name="com_offset_o6_y" default="0"/>
-	<xacro:arg name="com_offset_o6_z" default="0"/>
-	<!-- L6 手质量中心偏移 -->
-	<xacro:arg name="com_offset_l6_x" default="0"/>
-	<xacro:arg name="com_offset_l6_y" default="0"/>
-	<xacro:arg name="com_offset_l6_z" default="0"/>
 	<!-- 创建手部 (direction=1 为左手, direction=-1 为右手) -->
 	<!-- 支持 type: o7, o6, l6 -->
 	<xacro:if value="${'$(arg type)' == 'o7'}">
 		<xacro:include filename="$(find linkerhand_description)/xacro/o7.xacro"/>
-		<xacro:LinkerHandO7 name="" direction="$(arg direction)" com_offset_x="$(arg com_offset_o7_x)" com_offset_y="$(arg com_offset_o7_y)" com_offset_z="$(arg com_offset_o7_z)"/>
+		<xacro:LinkerHandO7 name="" direction="$(arg direction)"/>
 	</xacro:if>
 	<xacro:if value="${'$(arg type)' == 'o6'}">
 		<xacro:include filename="$(find linkerhand_description)/xacro/o6.xacro"/>
-		<xacro:LinkerHandO6 name="" direction="$(arg direction)" com_offset_x="$(arg com_offset_o6_x)" com_offset_y="$(arg com_offset_o6_y)" com_offset_z="$(arg com_offset_o6_z)"/>
+		<xacro:LinkerHandO6 name="" direction="$(arg direction)"/>
 	</xacro:if>
 	<xacro:if value="${'$(arg type)' == 'l6'}">
 		<xacro:include filename="$(find linkerhand_description)/xacro/l6.xacro"/>
-		<xacro:LinkerHandL6 name="" direction="$(arg direction)" com_offset_x="$(arg com_offset_l6_x)" com_offset_y="$(arg com_offset_l6_y)" com_offset_z="$(arg com_offset_l6_z)"/>
+		<xacro:LinkerHandL6 name="" direction="$(arg direction)"/>
 	</xacro:if>
 </robot>

File: dexhands/linkerhand_description/xacro/l6.xacro (robot description, xacro)
@@ -1,34 +1,7 @@
 <?xml version="1.0" encoding="utf-8"?>
 <robot xmlns:xacro="http://www.ros.org/wiki/xacro">
-	<!-- 定义 L6 手质量和转动惯量参数的宏 (用于生成 dyn_param) -->
-	<!-- dyn_param 格式 (10个值): [M, mx, my, mz, XX, XY, XZ, YY, YZ, ZZ] -->
-	<!-- M: 质量 (单位: kg) -->
-	<!-- mx, my, mz: 质心位置 (单位: mm) -->
-	<!-- XX, XY, XZ, YY, YZ, ZZ: 转动惯量 (6个值) -->
-	<xacro:macro name="LinkerHandL6_DynParams" params="direction com_offset_x:=0 com_offset_y:=0 com_offset_z:=0">
-		<!-- 质量中心位置 (单位: 米，考虑 direction 和偏移) -->
-		<xacro:property name="com_x_m" value="${0.00646140274510786 + com_offset_x}"/>
-		<xacro:property name="com_y_m" value="${direction*-0.0112810445470838 + com_offset_y}"/>
-		<xacro:property name="com_z_m" value="${0.0905307075615191 + com_offset_z}"/>
-		<!-- 转换为毫米 (乘以 1000) -->
-		<xacro:property name="com_x" value="${com_x_m * 1000}"/>
-		<xacro:property name="com_y" value="${com_y_m * 1000}"/>
-		<xacro:property name="com_z" value="${com_z_m * 1000}"/>
-		<!-- 质量 (单位: kg) -->
-		<xacro:property name="mass" value="0.989011744524491"/>
-		<!-- 转动惯量 -->
-		<xacro:property name="ixx" value="0.00478399523069539"/>
-		<xacro:property name="ixy" value="0.00035287455140517"/>
-		<xacro:property name="ixz" value="${direction*-0.000147692771617922}"/>
-		<xacro:property name="iyy" value="0.00333942627823233"/>
-		<xacro:property name="iyz" value="${direction*-0.000347763064470168}"/>
-		<xacro:property name="izz" value="0.00199340034930999"/>
-		<!-- 输出 dyn_param 数组格式: [M, mx, my, mz, XX, XY, XZ, YY, YZ, ZZ] -->
-		[${mass},${com_x},${com_y},${com_z},${ixx},${ixy},${ixz},${iyy},${iyz},${izz}]
-	</xacro:macro>
-	<xacro:macro name="LinkerHandL6" params="name direction:=1 use_flange:=false fixed_joints:=false com_offset_x:=0 com_offset_y:=0 com_offset_z:=0">
+	<xacro:macro name="LinkerHandL6" params="name direction:=1 use_flange:=false fixed_joints:=false">
 		<xacro:property name="prefix" value="${name + '_' if name else ''}"/>
 		<xacro:property name="joint_type" value="${fixed_joints and 'fixed' or 'revolute'}"/>
-		<!-- 质量中心偏移量 (单位: 米) -->
 		<xacro:if value="${use_flange}">
 			<link name="${prefix}flange">
@@ -66,6 +39,5 @@
 		<link name="${prefix}hand_base">
 			<inertial>
-				<!-- 质量中心位置 = 原始位置 + 偏移量 -->
-				<origin xyz="${0.00646140274510786 + com_offset_x} ${direction*-0.0112810445470838 + com_offset_y} ${0.0905307075615191 + com_offset_z}"/>
+				<origin xyz="0.00646140274510786 ${direction*-0.0112810445470838} 0.0905307075615191"/>
 				<mass value="0.989011744524491"/>
 				<inertia ixx="0.00478399523069539"

File: dexhands/linkerhand_description/xacro/o6.xacro (robot description, xacro)
@@ -1,34 +1,7 @@
 <?xml version="1.0" encoding="utf-8"?>
 <robot xmlns:xacro="http://www.ros.org/wiki/xacro">
-	<!-- 定义 O6 手质量和转动惯量参数的宏 (用于生成 dyn_param) -->
-	<!-- dyn_param 格式 (10个值): [M, mx, my, mz, XX, XY, XZ, YY, YZ, ZZ] -->
-	<!-- M: 质量 (单位: kg) -->
-	<!-- mx, my, mz: 质心位置 (单位: mm) -->
-	<!-- XX, XY, XZ, YY, YZ, ZZ: 转动惯量 (6个值) -->
-	<xacro:macro name="LinkerHandO6_DynParams" params="direction com_offset_x:=0 com_offset_y:=0 com_offset_z:=0">
-		<!-- 质量中心位置 (单位: 米，考虑 direction 和偏移) -->
-		<xacro:property name="com_x_m" value="${(direction == 1 and -0.00157788568070457 or -0.00160320773490556) + com_offset_x}"/>
-		<xacro:property name="com_y_m" value="${direction*-0.00034876725935859 + com_offset_y}"/>
-		<xacro:property name="com_z_m" value="${(direction == 1 and 0.0538452219801211 or 0.0538002704027215) + com_offset_z}"/>
-		<!-- 转换为毫米 (乘以 1000) -->
-		<xacro:property name="com_x" value="${com_x_m * 1000}"/>
-		<xacro:property name="com_y" value="${com_y_m * 1000}"/>
-		<xacro:property name="com_z" value="${com_z_m * 1000}"/>
-		<!-- 质量 (单位: kg) -->
-		<xacro:property name="mass" value="0.0672935238166485"/>
-		<!-- 转动惯量 -->
-		<xacro:property name="ixx" value="5.22525212160954E-05"/>
-		<xacro:property name="ixy" value="3.06955729584715E-07"/>
-		<xacro:property name="ixz" value="${direction*-3.90341166950521E-07}"/>
-		<xacro:property name="iyy" value="3.33522349207724E-05"/>
-		<xacro:property name="iyz" value="${direction*-7.76680063574627E-07}"/>
-		<xacro:property name="izz" value="2.28469461105385E-05"/>
-		<!-- 输出 dyn_param 数组格式: [M, mx, my, mz, XX, XY, XZ, YY, YZ, ZZ] -->
-		[${mass},${com_x},${com_y},${com_z},${ixx},${ixy},${ixz},${iyy},${iyz},${izz}]
-	</xacro:macro>
-	<xacro:macro name="LinkerHandO6" params="name direction:=1 use_flange:=false fixed_joints:=false com_offset_x:=0 com_offset_y:=0 com_offset_z:=0">
+	<xacro:macro name="LinkerHandO6" params="name direction:=1 use_flange:=false fixed_joints:=false">
 		<xacro:property name="prefix" value="${name + '_' if name else ''}"/>
 		<xacro:property name="joint_type" value="${fixed_joints and 'fixed' or 'revolute'}"/>
-		<!-- 质量中心偏移量 (单位: 米) -->
 		<xacro:if value="${use_flange}">
 			<link name="${prefix}flange">
@@ -66,7 +39,6 @@
 		<link name="${prefix}hand_base">
 			<inertial>
-				<!-- 质量中心位置 = 原始位置 + 偏移量 -->
-				<origin
-						xyz="${(direction == 1 and -0.00157788568070457 or -0.00160320773490556) + com_offset_x} ${(direction*-0.00034876725935859) + com_offset_y} ${(direction == 1 and 0.0538452219801211 or 0.0538002704027215) + com_offset_z}"
+				<origin
+						xyz="${direction == 1 and -0.00157788568070457 or -0.00160320773490556} ${direction*-0.00034876725935859} ${direction == 1 and 0.0538452219801211 or 0.0538002704027215}"
 				/>
 				<mass value="0.0672935238166485"/>

File: dexhands/linkerhand_description/xacro/o7.xacro (robot description, xacro)
@@ -1,34 +1,7 @@
 <?xml version="1.0" encoding="utf-8"?>
 <robot xmlns:xacro="http://www.ros.org/wiki/xacro">
-	<!-- 定义 O7 手质量和转动惯量参数的宏 (用于生成 dyn_param) -->
-	<!-- dyn_param 格式 (10个值): [M, mx, my, mz, XX, XY, XZ, YY, YZ, ZZ] -->
-	<!-- M: 质量 (单位: kg) -->
-	<!-- mx, my, mz: 质心位置 (单位: mm) -->
-	<!-- XX, XY, XZ, YY, YZ, ZZ: 转动惯量 (6个值) -->
-	<xacro:macro name="LinkerHandO7_DynParams" params="direction com_offset_x:=0 com_offset_y:=0 com_offset_z:=0">
-		<!-- 质量中心位置 (单位: 米，考虑 direction 和偏移) -->
-		<xacro:property name="com_x_m" value="${(direction == 1 and -0.000897326242450024 or -0.000635826168353301) + com_offset_x}"/>
-		<xacro:property name="com_y_m" value="${direction*-0.000912910200583317 + com_offset_y}"/>
-		<xacro:property name="com_z_m" value="${(direction == 1 and 0.0725139361953409 or 0.0808531524968522) + com_offset_z}"/>
-		<!-- 转换为毫米 (乘以 1000) -->
-		<xacro:property name="com_x" value="${com_x_m * 1000}"/>
-		<xacro:property name="com_y" value="${com_y_m * 1000}"/>
-		<xacro:property name="com_z" value="${com_z_m * 1000}"/>
-		<!-- 质量 (单位: kg) -->
-		<xacro:property name="mass" value="${direction == 1 and 0.0961317016824249 or 0.115532510357281}"/>
-		<!-- 转动惯量 -->
-		<xacro:property name="ixx" value="${direction == 1 and 0.000102695669168065 or 0.000103865728174833}"/>
-		<xacro:property name="ixy" value="${direction*-4.31409372592166E-07}"/>
-		<xacro:property name="ixz" value="-1.88110470378979E-06"/>
-		<xacro:property name="iyy" value="${direction == 1 and 6.48454975844519E-05 or 6.66546428907319E-05}"/>
-		<xacro:property name="iyz" value="${direction*8.30780063139162E-07}"/>
-		<xacro:property name="izz" value="${direction == 1 and 4.84048917293055E-05 or 4.97086581300188E-05}"/>
-		<!-- 输出 dyn_param 数组格式: [M, mx, my, mz, XX, XY, XZ, YY, YZ, ZZ] -->
-		[${mass},${com_x},${com_y},${com_z},${ixx},${ixy},${ixz},${iyy},${iyz},${izz}]
-	</xacro:macro>
-	<xacro:macro name="LinkerHandO7" params="name direction:=1 use_flange:=false fixed_joints:=false com_offset_x:=0 com_offset_y:=0 com_offset_z:=0">
+	<xacro:macro name="LinkerHandO7" params="name direction:=1 use_flange:=false fixed_joints:=false">
 		<xacro:property name="prefix" value="${name + '_' if name else ''}"/>
 		<xacro:property name="joint_type" value="${fixed_joints and 'fixed' or 'revolute'}"/>
-		<!-- 质量中心偏移量 (单位: 米) -->
 		<!-- ========================================== -->
 		<!-- 手掌基座 (Hand Base) -->
@@ -36,7 +9,6 @@
 		<link name="${prefix}hand_base">
 			<inertial>
-				<!-- 质量中心位置 = 原始位置 + 偏移量 -->
-				<origin
-						xyz="${(direction == 1 and -0.000897326242450024 or -0.000635826168353301) + com_offset_x} ${direction*-0.000912910200583317 + com_offset_y} ${(direction == 1 and 0.0725139361953409 or 0.0808531524968522) + com_offset_z}"
+				<origin
+						xyz="${direction == 1 and -0.000897326242450024 or -0.000635826168353301} ${direction*-0.000912910200583317} ${direction == 1 and 0.0725139361953409 or 0.0808531524968522}"
 				/>
 				<mass value="${direction == 1 and 0.0961317016824249 or 0.115532510357281}"/>

Commit message: add angellun omniwheel

File: dexhands/linkerhand_description/xacro/hand.xacro (robot description, xacro)
@@ -19,5 +19,5 @@
 	<xacro:if value="${'$(arg type)' == 'l10'}">
 		<xacro:include filename="$(find linkerhand_description)/xacro/l10.xacro"/>
-		<xacro:LinkerHandL10 name="" direction="$(arg direction)"/>
+		<xacro:LinkerHandL10 name="" direction="$(arg direction)" use_flange="true"/>
 	</xacro:if>
 </robot>

File: dexhands/linkerhand_description/xacro/l10.xacro (robot description, xacro)
@@ -4,4 +4,29 @@
 		<xacro:property name="prefix" value="${name + '_' if name else ''}"/>
 		<xacro:property name="joint_type" value="${fixed_joints and 'fixed' or 'revolute'}"/>
+		<xacro:if value="${use_flange}">
+			<link name="${prefix}flange">
+				<inertial>
+					<origin xyz="-0.000388 0.002345 0.0"/>
+					<mass value="0.114"/>
+					<inertia
+							ixx="0.000040105"
+							ixy="0.000000214"
+							ixz="0.0"
+							iyy="0.000085776"
+							iyz="0.0"
+							izz="0.000054044"/>
+				</inertial>
+				<visual>
+					<geometry>
+						<mesh filename="file://$(find linkerhand_description)/meshes/o7/flange.glb"/>
+					</geometry>
+				</visual>
+			</link>
+			<joint name="${prefix}flange_joint" type="fixed">
+				<origin xyz="0 0 0.022"/>
+				<parent link="${prefix}flange"/>
+				<child link="${prefix}hand_base"/>
+			</joint>
+		</xacro:if>
 		<!-- ========================================== -->
 		<!-- 手掌基座 (Hand Base) -->
