Commit message: add hand eef

File: dexhands/linkerhand_description/xacro/l10.xacro (robot description, xacro)
@@ -55,4 +55,10 @@
 			</collision>
 		</link>
+		<link name="${prefix}eef"/>
+		<joint name="${prefix}eef_joint" type="fixed">
+			<parent link="${prefix}hand_base"/>
+			<child link="${prefix}eef"/>
+			<origin xyz="0.03 0. 0.1"/>
+		</joint>
 		<!-- ========================================== -->
 		<!-- 拇指部分 (Thumb) -->

File: dexhands/linkerhand_description/xacro/l6.xacro (robot description, xacro)
@@ -61,4 +61,10 @@
 			</collision>
 		</link>
+		<link name="${prefix}eef"/>
+		<joint name="${prefix}eef_joint" type="fixed">
+			<parent link="${prefix}hand_base"/>
+			<child link="${prefix}eef"/>
+			<origin xyz="0.025 0. 0.08"/>
+		</joint>
 		<!-- ========================================== -->
 		<!-- 拇指部分 (Thumb) -->

File: dexhands/linkerhand_description/xacro/o6.xacro (robot description, xacro)
@@ -63,4 +63,10 @@
 			</collision>
 		</link>
+		<link name="${prefix}eef"/>
+		<joint name="${prefix}eef_joint" type="fixed">
+			<parent link="${prefix}hand_base"/>
+			<child link="${prefix}eef"/>
+			<origin xyz="0.02 0. 0.07"/>
+		</joint>
 		<!-- ========================================== -->
 		<!-- 拇指部分 (Thumb) -->

File: dexhands/linkerhand_description/xacro/o7.xacro (robot description, xacro)
@@ -58,4 +58,10 @@
 			</collision>
 		</link>
+		<link name="${prefix}eef"/>
+		<joint name="${prefix}eef_joint" type="fixed">
+			<parent link="${prefix}hand_base"/>
+			<child link="${prefix}eef"/>
+			<origin xyz="0.03 0. 0.1"/>
+		</joint>
 		<!-- ========================================== -->
 		<!-- 拇指部分 (Thumb) -->
