Commit message: add linkerhand o7

File: dexhands/brainco_description/xacro/revo2.xacro (robot description, xacro)
@@ -7,5 +7,5 @@
 			<link name="${prefix}flange">
 				<inertial>
-					<origin xyz="-0.00283400 0 0.00000145" rpy="0 0 0"/>
+					<origin xyz="-0.00283400 0 0.00000145" />
 					<mass value="0.02280635"/>
 					<inertia ixx="0.00000768" ixy="0.00000000" ixz="0.00000000" iyy="0.00000580" iyz="-0.00000000" izz="0.00000427"/>
@@ -67,5 +67,5 @@
 			</collision>
 		</link>
-		<joint name="${prefix}thumb_metacarpal_joint" type="${joint_type}">
+		<joint name="${prefix}thumb_joint1" type="${joint_type}">
 			<origin xyz="${direction == 1 and 0.0045 or 0.005619} ${direction == 1 and -0.019 or 0.019867} 0.027825"
 				  rpy="${1.5708 - direction * 1.5708} 0 ${direction == 1 and 0.16787 or 2.9637}"/>
@@ -95,5 +95,5 @@
 			</collision>
 		</link>
-		<joint name="${prefix}thumb_proximal_joint" type="${joint_type}">
+		<joint name="${prefix}thumb_joint2" type="${joint_type}">
 			<origin xyz="0 ${direction*-0.014227} 0"
 				  rpy="${direction == 1 and 0.17488 or -2.9667} -0.23736 2.9737"/>
@@ -133,5 +133,5 @@
 				<axis xyz="1 0 0"/>
 				<limit lower="0" upper="1.0472" effort="1.1" velocity="2.5303"/>
-				<mimic joint="${prefix}thumb_proximal_joint" multiplier="1" offset="0"/>
+				<mimic joint="${prefix}thumb_joint2" multiplier="1" offset="0"/>
 			</xacro:unless>
 		</joint>
@@ -190,5 +190,5 @@
 			</collision>
 		</link>
-		<joint name="${prefix}index_proximal_joint" type="${joint_type}">
+		<joint name="${prefix}index_joint" type="${joint_type}">
 			<origin xyz="-0.0021349 ${direction*-0.029578} 0.080876"
 				  rpy="${direction*0.11819} 0.14743 ${direction*0.17422}"/>
@@ -230,5 +230,5 @@
 				<axis xyz="0 1 0"/>
 				<limit lower="0" upper="1.693" effort="2" velocity="2.2685"/>
-				<mimic joint="${prefix}index_proximal_joint" multiplier="1.155" offset="0"/>
+				<mimic joint="${prefix}index_joint" multiplier="1.155" offset="0"/>
 			</xacro:unless>
 		</joint>
@@ -289,5 +289,5 @@
 			</collision>
 		</link>
-		<joint name="${prefix}middle_proximal_joint" type="${joint_type}">
+		<joint name="${prefix}middle_joint" type="${joint_type}">
 			<origin xyz="-0.0045935 ${direction*-0.010061} 0.084993"
 				  rpy="${direction*0.039468} 0.1483 ${direction*0.057975}"/>
@@ -329,5 +329,5 @@
 				<axis xyz="0 1 0"/>
 				<limit lower="0" upper="1.693" effort="2" velocity="2.2685"/>
-				<mimic joint="${prefix}middle_proximal_joint" multiplier="1.155" offset="0"/>
+				<mimic joint="${prefix}middle_joint" multiplier="1.155" offset="0"/>
 			</xacro:unless>
 		</joint>
@@ -393,5 +393,5 @@
 			</collision>
 		</link>
-		<joint name="${prefix}ring_proximal_joint" type="${joint_type}">
+		<joint name="${prefix}ring_joint" type="${joint_type}">
 			<origin xyz="-0.00468767815858587 ${direction*0.0100262714211602} 0.0839819548795939"
 				  rpy="${direction*-0.0394618478609065} 0.147209177132223 ${direction*-0.0579317909005277}"/>
@@ -443,5 +443,5 @@
 				<axis xyz="0 1 0"/>
 				<limit lower="0" upper="1.693" effort="2" velocity="2.2685"/>
-				<mimic joint="${prefix}ring_proximal_joint" multiplier="1.155" offset="0"/>
+				<mimic joint="${prefix}ring_joint" multiplier="1.155" offset="0"/>
 			</xacro:unless>
 		</joint>
@@ -497,5 +497,5 @@
 			</collision>
 		</link>
-		<joint name="${prefix}pinky_proximal_joint" type="${joint_type}">
+		<joint name="${prefix}pinky_joint" type="${joint_type}">
 			<origin xyz="-0.0023733 ${direction*0.029356} 0.078694"
 				  rpy="${direction*-0.11815} 0.14491 ${direction*-0.17392}"/>
@@ -547,5 +547,5 @@
 				<axis xyz="0 1 0"/>
 				<limit lower="0" upper="1.693" effort="2" velocity="2.2685"/>
-				<mimic joint="${prefix}pinky_proximal_joint" multiplier="1.155" offset="0"/>
+				<mimic joint="${prefix}pinky_joint" multiplier="1.155" offset="0"/>
 			</xacro:unless>
 		</joint>

Commit message: add ros2 control interfaces for brainco revo2

File: dexhands/brainco_description/xacro/revo2.xacro (robot description, xacro)
@@ -67,5 +67,5 @@
 			</collision>
 		</link>
-		<joint name="${prefix}thumb_joint1" type="${joint_type}">
+		<joint name="${prefix}thumb_joint2" type="${joint_type}">
 			<origin xyz="${direction == 1 and 0.0045 or 0.005619} ${direction == 1 and -0.019 or 0.019867} 0.027825"
 				  rpy="${1.5708 - direction * 1.5708} 0 ${direction == 1 and 0.16787 or 2.9637}"/>
@@ -95,5 +95,5 @@
 			</collision>
 		</link>
-		<joint name="${prefix}thumb_joint2" type="${joint_type}">
+		<joint name="${prefix}thumb_joint1" type="${joint_type}">
 			<origin xyz="0 ${direction*-0.014227} 0"
 				  rpy="${direction == 1 and 0.17488 or -2.9667} -0.23736 2.9737"/>
@@ -133,5 +133,5 @@
 				<axis xyz="1 0 0"/>
 				<limit lower="0" upper="1.0472" effort="1.1" velocity="2.5303"/>
-				<mimic joint="${prefix}thumb_joint2" multiplier="1" offset="0"/>
+				<mimic joint="${prefix}thumb_joint1" multiplier="1" offset="0"/>
 			</xacro:unless>
 		</joint>
