Commit message: update brainco hand to glb

File: dexhands/brainco_description/xacro/hand.xacro (robot description, xacro)
@@ -1,8 +1,8 @@
 <?xml version="1.0" encoding="utf-8"?>
-<robot name="BrainCo_$(arg type)" xmlns:xacro="http://www.ros.org/wiki/xacro">
+<robot name="BrainCo_$(arg type)_left" xmlns:xacro="http://www.ros.org/wiki/xacro">
 	<xacro:arg name="type" default="Revo2"/>
 	<xacro:arg name="direction" default="1"/>
 	<xacro:include filename="$(find brainco_description)/xacro/revo2.xacro"/>
 	<!-- 创建左手 (direction=1) -->
-	<xacro:BrainCoHand name="" direction="$(arg direction)"/>
+	<xacro:BrainCoHand name="left_hand" direction="$(arg direction)"/>
 </robot>

File: dexhands/brainco_description/xacro/revo2.xacro (robot description, xacro)
@@ -13,10 +13,10 @@
 				<visual>
 					<geometry>
-						<mesh filename="file://$(find brainco_description)/meshes/revo2/flange.obj"/>
+						<mesh filename="file://$(find brainco_description)/meshes/revo2/flange.glb"/>
 					</geometry>
 				</visual>
 				<collision>
 					<geometry>
-						<mesh filename="file://$(find brainco_description)/meshes/revo2/flange.obj"/>
+						<mesh filename="file://$(find brainco_description)/meshes/revo2/flange.glb"/>
 					</geometry>
 				</collision>
@@ -37,10 +37,10 @@
 			<visual>
 				<geometry>
-					<mesh filename="file://$(find brainco_description)/meshes/revo2/base_link.obj" scale="1 ${direction} 1"/>
-				</geometry>
-			</visual>
-			<collision>
-				<geometry>
-					<mesh filename="file://$(find brainco_description)/meshes/revo2/base_link.obj" scale="1 ${direction} 1"/>
+					<mesh filename="file://$(find brainco_description)/meshes/revo2/base_link.glb" scale="1 ${direction} 1"/>
+				</geometry>
+			</visual>
+			<collision>
+				<geometry>
+					<mesh filename="file://$(find brainco_description)/meshes/revo2/base_link.glb" scale="1 ${direction} 1"/>
 				</geometry>
 			</collision>
@@ -58,10 +58,10 @@
 			<visual>
 				<geometry>
-					<mesh filename="file://$(find brainco_description)/meshes/revo2/thumb_metacarpal.obj" scale="${direction} ${direction} ${direction}"/>
-				</geometry>
-			</visual>
-			<collision>
-				<geometry>
-					<mesh filename="file://$(find brainco_description)/meshes/revo2/thumb_metacarpal.obj" scale="${direction} ${direction} ${direction}"/>
+					<mesh filename="file://$(find brainco_description)/meshes/revo2/thumb_metacarpal.glb" scale="${direction} ${direction} ${direction}"/>
+				</geometry>
+			</visual>
+			<collision>
+				<geometry>
+					<mesh filename="file://$(find brainco_description)/meshes/revo2/thumb_metacarpal.glb" scale="${direction} ${direction} ${direction}"/>
 				</geometry>
 			</collision>
@@ -86,10 +86,10 @@
 			<visual>
 				<geometry>
-					<mesh filename="file://$(find brainco_description)/meshes/revo2/thumb_proximal.obj"/>
-				</geometry>
-			</visual>
-			<collision>
-				<geometry>
-					<mesh filename="file://$(find brainco_description)/meshes/revo2/thumb_proximal.obj"/>
+					<mesh filename="file://$(find brainco_description)/meshes/revo2/thumb_proximal.glb"/>
+				</geometry>
+			</visual>
+			<collision>
+				<geometry>
+					<mesh filename="file://$(find brainco_description)/meshes/revo2/thumb_proximal.glb"/>
 				</geometry>
 			</collision>
@@ -117,10 +117,10 @@
 			<visual>
 				<geometry>
-					<mesh filename="file://$(find brainco_description)/meshes/revo2/thumb_distal.obj"/>
-				</geometry>
-			</visual>
-			<collision>
-				<geometry>
-					<mesh filename="file://$(find brainco_description)/meshes/revo2/thumb_distal.obj"/>
+					<mesh filename="file://$(find brainco_description)/meshes/revo2/thumb_distal.glb"/>
+				</geometry>
+			</visual>
+			<collision>
+				<geometry>
+					<mesh filename="file://$(find brainco_description)/meshes/revo2/thumb_distal.glb"/>
 				</geometry>
 			</collision>
@@ -180,11 +180,11 @@
 				<geometry>
 					<mesh
-							filename="file://$(find brainco_description)/meshes/revo2/index_proximal.obj"/>
-				</geometry>
-			</visual>
-			<collision>
-				<geometry>
-					<mesh
-							filename="file://$(find brainco_description)/meshes/revo2/index_proximal.obj"/>
+							filename="file://$(find brainco_description)/meshes/revo2/index_proximal.glb"/>
+				</geometry>
+			</visual>
+			<collision>
+				<geometry>
+					<mesh
+							filename="file://$(find brainco_description)/meshes/revo2/index_proximal.glb"/>
 				</geometry>
 			</collision>
@@ -214,10 +214,10 @@
 			<visual>
 				<geometry>
-					<mesh filename="file://$(find brainco_description)/meshes/revo2/index_distal.obj"/>
-				</geometry>
-			</visual>
-			<collision>
-				<geometry>
-					<mesh filename="file://$(find brainco_description)/meshes/revo2/index_distal.obj"/>
+					<mesh filename="file://$(find brainco_description)/meshes/revo2/index_distal.glb"/>
+				</geometry>
+			</visual>
+			<collision>
+				<geometry>
+					<mesh filename="file://$(find brainco_description)/meshes/revo2/index_distal.glb"/>
 				</geometry>
 			</collision>
@@ -279,11 +279,11 @@
 				<geometry>
 					<mesh
-							filename="file://$(find brainco_description)/meshes/revo2/middle_proximal.obj"/>
-				</geometry>
-			</visual>
-			<collision>
-				<geometry>
-					<mesh
-							filename="file://$(find brainco_description)/meshes/revo2/middle_proximal.obj"/>
+							filename="file://$(find brainco_description)/meshes/revo2/middle_proximal.glb"/>
+				</geometry>
+			</visual>
+			<collision>
+				<geometry>
+					<mesh
+							filename="file://$(find brainco_description)/meshes/revo2/middle_proximal.glb"/>
 				</geometry>
 			</collision>
@@ -313,10 +313,10 @@
 			<visual>
 				<geometry>
-					<mesh filename="file://$(find brainco_description)/meshes/revo2/middle_distal.obj"/>
-				</geometry>
-			</visual>
-			<collision>
-				<geometry>
-					<mesh filename="file://$(find brainco_description)/meshes/revo2/middle_distal.obj"/>
+					<mesh filename="file://$(find brainco_description)/meshes/revo2/middle_distal.glb"/>
+				</geometry>
+			</visual>
+			<collision>
+				<geometry>
+					<mesh filename="file://$(find brainco_description)/meshes/revo2/middle_distal.glb"/>
 				</geometry>
 			</collision>
@@ -378,16 +378,11 @@
 				<geometry>
 					<mesh
-							filename="file://$(find brainco_description)/meshes/revo2/ring_proximal.obj"/>
-				</geometry>
-				<material
-						name="">
-					<color
-							rgba="1 1 1 1"/>
-				</material>
-			</visual>
-			<collision>
-				<geometry>
-					<mesh
-							filename="file://$(find brainco_description)/meshes/revo2/ring_proximal.obj"/>
+							filename="file://$(find brainco_description)/meshes/revo2/ring_proximal.glb"/>
+				</geometry>
+			</visual>
+			<collision>
+				<geometry>
+					<mesh
+							filename="file://$(find brainco_description)/meshes/revo2/ring_proximal.glb"/>
 				</geometry>
 			</collision>
@@ -421,16 +416,11 @@
 				<geometry>
 					<mesh
-							filename="file://$(find brainco_description)/meshes/revo2/ring_distal.obj"/>
-				</geometry>
-				<material
-						name="">
-					<color
-							rgba="1 1 1 1"/>
-				</material>
-			</visual>
-			<collision>
-				<geometry>
-					<mesh
-							filename="file://$(find brainco_description)/meshes/revo2/ring_distal.obj"/>
+							filename="file://$(find brainco_description)/meshes/revo2/ring_distal.glb"/>
+				</geometry>
+			</visual>
+			<collision>
+				<geometry>
+					<mesh
+							filename="file://$(find brainco_description)/meshes/revo2/ring_distal.glb"/>
 				</geometry>
 			</collision>
@@ -488,10 +478,10 @@
 			<visual>
 				<geometry>
-					<mesh filename="file://$(find brainco_description)/meshes/revo2/pinky_proximal.obj"/>
-				</geometry>
-			</visual>
-			<collision>
-				<geometry>
-					<mesh filename="file://$(find brainco_description)/meshes/revo2/pinky_proximal.obj"/>
+					<mesh filename="file://$(find brainco_description)/meshes/revo2/pinky_proximal.glb"/>
+				</geometry>
+			</visual>
+			<collision>
+				<geometry>
+					<mesh filename="file://$(find brainco_description)/meshes/revo2/pinky_proximal.glb"/>
 				</geometry>
 			</collision>
@@ -525,16 +515,11 @@
 				<geometry>
 					<mesh
-							filename="file://$(find brainco_description)/meshes/revo2/pinky_distal.obj"/>
-				</geometry>
-				<material
-						name="">
-					<color
-							rgba="1 1 1 1"/>
-				</material>
-			</visual>
-			<collision>
-				<geometry>
-					<mesh
-							filename="file://$(find brainco_description)/meshes/revo2/pinky_distal.obj"/>
+							filename="file://$(find brainco_description)/meshes/revo2/pinky_distal.glb"/>
+				</geometry>
+			</visual>
+			<collision>
+				<geometry>
+					<mesh
+							filename="file://$(find brainco_description)/meshes/revo2/pinky_distal.glb"/>
 				</geometry>
 			</collision>

Commit message: add linkerhand l10

File: dexhands/brainco_description/xacro/hand.xacro (robot description, xacro)
@@ -1,4 +1,4 @@
 <?xml version="1.0" encoding="utf-8"?>
-<robot name="BrainCo_$(arg type)_left" xmlns:xacro="http://www.ros.org/wiki/xacro">
+<robot name="BrainCo_$(arg type)" xmlns:xacro="http://www.ros.org/wiki/xacro">
 	<xacro:arg name="type" default="Revo2"/>
 	<xacro:arg name="direction" default="1"/>

File: dexhands/brainco_description/xacro/revo2.xacro (robot description, xacro)
@@ -149,13 +149,9 @@
 			</inertial>
 		</link>
-		<joint name="${prefix}thumb_tip_joint" type="${joint_type}">
+		<joint name="${prefix}thumb_tip_joint" type="fixed">
 			<origin xyz="0 0.026528781163583 -0.00177344281307927"
 				  rpy="${direction == 1 and 0.0667504507189052 or -0.06675} 0 ${direction == 1 and 3.14159265358979 or 0}"/>
 			<parent link="${prefix}thumb_distal_Link"/>
 			<child link="${prefix}thumb_tip_Link"/>
-			<xacro:unless value="${fixed_joints}">
-				<axis xyz="-1 0 0"/>
-				<limit lower="0" upper="0" effort="0" velocity="0"/>
-			</xacro:unless>
 		</joint>
 		<!-- ========================================== -->
@@ -249,12 +245,8 @@
 			</inertial>
 		</link>
-		<joint name="${prefix}index_tip_joint" type="${joint_type}">
+		<joint name="${prefix}index_tip_joint" type="fixed">
 			<origin xyz="0.011097 0 0.035739" rpy="0 0.48723 0"/>
 			<parent link="${prefix}index_distal_Link"/>
 			<child link="${prefix}index_tip_Link"/>
-			<xacro:unless value="${fixed_joints}">
-				<axis xyz="0 1 0"/>
-				<limit lower="1" upper="1" effort="1" velocity="1"/>
-			</xacro:unless>
 		</joint>
 		<!-- ========================================== -->
@@ -348,12 +340,8 @@
 			</inertial>
 		</link>
-		<joint name="${prefix}middle_tip_joint" type="${joint_type}">
+		<joint name="${prefix}middle_tip_joint" type="fixed">
 			<origin xyz="0.0073534 0 0.041703" rpy="0 0.34907 0"/>
 			<parent link="${prefix}middle_distal_Link"/>
 			<child link="${prefix}middle_tip_Link"/>
-			<xacro:unless value="${fixed_joints}">
-				<axis xyz="0 1 0"/>
-				<limit lower="1" upper="1" effort="1" velocity="1"/>
-			</xacro:unless>
 		</joint>
 		<!-- ========================================== -->
@@ -452,12 +440,8 @@
 			</inertial>
 		</link>
-		<joint name="${prefix}ring_tip_joint" type="${joint_type}">
+		<joint name="${prefix}ring_tip_joint" type="fixed">
 			<origin xyz="0.0071824 0 0.040734" rpy="0 0.34907 0"/>
 			<parent link="${prefix}ring_distal_Link"/>
 			<child link="${prefix}ring_tip_Link"/>
-			<xacro:unless value="${fixed_joints}">
-				<axis xyz="0 1 0"/>
-				<limit lower="1" upper="1" effort="1" velocity="1"/>
-			</xacro:unless>
 		</joint>
 		<!-- ========================================== -->
@@ -551,12 +535,8 @@
 			</inertial>
 		</link>
-		<joint name="${prefix}pinky_tip_joint" type="${joint_type}">
+		<joint name="${prefix}pinky_tip_joint" type="fixed">
 			<origin xyz="0.010221 0 0.032918" rpy="0 0.4756 0"/>
 			<parent link="${prefix}pinky_distal_Link"/>
 			<child link="${prefix}pinky_tip_Link"/>
-			<xacro:unless value="${fixed_joints}">
-				<axis xyz="0 1 0"/>
-				<limit lower="1" upper="1" effort="1" velocity="1"/>
-			</xacro:unless>
 		</joint>
 	</xacro:macro>

File: dexhands/linkerhand_description/xacro/hand.xacro (robot description, xacro)
@@ -4,5 +4,5 @@
 	<xacro:arg name="direction" default="1"/>
 	<!-- 创建手部 (direction=1 为左手, direction=-1 为右手) -->
-	<!-- 支持 type: o7, o6, l6 -->
+	<!-- 支持 type: o7, o6, l6, l10 -->
 	<xacro:if value="${'$(arg type)' == 'o7'}">
 		<xacro:include filename="$(find linkerhand_description)/xacro/o7.xacro"/>
@@ -17,3 +17,7 @@
 		<xacro:LinkerHandL6 name="" direction="$(arg direction)"/>
 	</xacro:if>
+	<xacro:if value="${'$(arg type)' == 'l10'}">
+		<xacro:include filename="$(find linkerhand_description)/xacro/l10.xacro"/>
+		<xacro:LinkerHandL10 name="" direction="$(arg direction)"/>
+	</xacro:if>
 </robot>

File: dexhands/linkerhand_description/xacro/o7.xacro (robot description, xacro)
@@ -76,11 +76,11 @@
 			<visual>
 				<geometry>
-					<mesh filename="file://$(find linkerhand_description)/meshes/o7/thumb_metacarpals_base2.glb"
-								scale="1 ${direction} 1"/>
-				</geometry>
-			</visual>
-			<collision>
-				<geometry>
-					<mesh filename="file://$(find linkerhand_description)/meshes/o7/thumb_metacarpals_base2.glb"
+					<mesh filename="file://$(find linkerhand_description)/meshes/o7/thumb_metacarpals_base1.glb"
+								scale="1 ${direction} 1"/>
+				</geometry>
+			</visual>
+			<collision>
+				<geometry>
+					<mesh filename="file://$(find linkerhand_description)/meshes/o7/thumb_metacarpals_base1.glb"
 								scale="1 ${direction} 1"/>
 				</geometry>

File: dexhands/linkerhand_description/xacro/ros2_control/hand.xacro (robot description, xacro)
@@ -36,5 +36,5 @@
             </xacro:if>
         </hardware>
-        <!-- Support type: o7, o6, l6 -->
+        <!-- Support type: o7, o6, l6, l10 -->
         <xacro:if value="${'$(arg type)' == 'o7'}">
             <xacro:include filename="$(find linkerhand_description)/xacro/ros2_control/o7.xacro"/>
@@ -44,4 +44,8 @@
             <xacro:include filename="$(find linkerhand_description)/xacro/ros2_control/o6.xacro"/>
             <xacro:linkerhand_o6_interfaces name=""/>
+        </xacro:if>
+        <xacro:if value="${'$(arg type)' == 'l10'}">
+            <xacro:include filename="$(find linkerhand_description)/xacro/ros2_control/l10.xacro"/>
+            <xacro:linkerhand_l10_interfaces name=""/>
         </xacro:if>
     </ros2_control>
