Commit message: add eef frame for eg2 4c2

File: gripper/inspire_description/xacro/EG2-4C2.xacro (robot description, xacro)
@@ -212,4 +212,10 @@
       <mimic joint="${prefix}gripper_joint" multiplier="1" offset="0"/>
     </joint>
+    <link name="${prefix}eef"/>
+    <joint name="${prefix}eef_joint" type="fixed">
+      <parent link="${prefix}gripper_base"/>
+      <child link="${prefix}eef"/>
+      <origin xyz="0 0 0.14"/>
+    </joint>
   </xacro:macro>
 </robot>
