Commit message: add inspire hand

File: gripper/inspire_description/xacro/hand.xacro (robot description, xacro)
@@ -8,3 +8,7 @@
     <xacro:InspireHandRH56E2 name="$(arg name)" direction="$(arg direction)" use_flange="true"/>
   </xacro:if>
+  <xacro:if value="${'$(arg type)' == 'RH56F2'}">
+    <xacro:include filename="$(find inspire_description)/xacro/hands/RH56F2.xacro"/>
+    <xacro:InspireHandRH56F2 name="$(arg name)" direction="$(arg direction)" use_flange="true"/>
+  </xacro:if>
 </robot>

File: gripper/inspire_description/xacro/hands/RH56E2.xacro (robot description, xacro)
@@ -804,5 +804,5 @@
       <child link="${prefix}ring_force_sensor_1" />
     </joint>
-    <link name="${prefix}little_1">
+    <link name="${prefix}pinky_1">
       <inertial>
         <origin xyz="-0.00219418424084009 ${dir*0.0127409391731467} -0.00664940009923338" />
@@ -830,9 +830,9 @@
       <origin xyz="0.025916 ${dir*0.00056467} 0.11815" rpy="${dir*1.4661} 0 ${dir*-1.5708}" />
       <parent link="${prefix}hand_base" />
-      <child link="${prefix}little_1" />
+      <child link="${prefix}pinky_1" />
       <axis xyz="0 0 ${dir}" />
       <limit lower="0" upper="1.4381" effort="10" velocity="1" />
     </joint>
-    <link name="${prefix}little_2">
+    <link name="${prefix}pinky_2">
       <inertial>
         <origin xyz="0.00142962322858008 ${dir*0.0206390061213492} -0.00609937271859847" />
@@ -848,10 +848,10 @@
       <visual>
         <geometry>
-          <mesh filename="file://$(find inspire_description)/meshes/RH56E2/little2.glb" scale="1 ${dir} 1" />
-        </geometry>
-      </visual>
-      <collision>
-        <geometry>
-          <mesh filename="file://$(find inspire_description)/meshes/RH56E2/little2.glb" scale="1 ${dir} 1" />
+          <mesh filename="file://$(find inspire_description)/meshes/RH56E2/pinky2.glb" scale="1 ${dir} 1" />
+        </geometry>
+      </visual>
+      <collision>
+        <geometry>
+          <mesh filename="file://$(find inspire_description)/meshes/RH56E2/pinky2.glb" scale="1 ${dir} 1" />
         </geometry>
       </collision>
@@ -859,6 +859,6 @@
     <joint name="${prefix}pinky_dip" type="revolute">
       <origin xyz="-0.0034259 ${dir*0.032596} -0.00055" />
-      <parent link="${prefix}little_1" />
-      <child link="${prefix}little_2" />
+      <parent link="${prefix}pinky_1" />
+      <child link="${prefix}pinky_2" />
       <axis xyz="0 0 ${dir}" />
       <limit lower="0" upper="3.14" effort="10" velocity="1" />
@@ -868,5 +868,5 @@
           offset="0" />
     </joint>
-    <link name="${prefix}little_force_sensor_2">
+    <link name="${prefix}pinky_force_sensor_2">
       <inertial>
         <origin xyz="1.83850807690782E-05 ${dir*-0.000118792499944516} -0.00077353663965421" />
@@ -882,22 +882,22 @@
       <visual>
         <geometry>
-          <mesh filename="file://$(find inspire_description)/meshes/RH56E2/sensors/little_force_sensor_2.STL" scale="1 ${dir} 1" />
-        </geometry>
-        <material name="">
-          <color rgba="0.411764705882353 0.411764705882353 0.411764705882353 1" />
-        </material>
-      </visual>
-      <collision>
-        <geometry>
-          <mesh filename="file://$(find inspire_description)/meshes/RH56E2/sensors/little_force_sensor_2.STL" scale="1 ${dir} 1" />
-        </geometry>
-      </collision>
-    </link>
-    <joint name="${prefix}little_force_sensor_2_joint" type="fixed">
+          <mesh filename="file://$(find inspire_description)/meshes/RH56E2/sensors/pinky_force_sensor_2.STL" scale="1 ${dir} 1" />
+        </geometry>
+        <material name="">
+          <color rgba="0.411764705882353 0.411764705882353 0.411764705882353 1" />
+        </material>
+      </visual>
+      <collision>
+        <geometry>
+          <mesh filename="file://$(find inspire_description)/meshes/RH56E2/sensors/pinky_force_sensor_2.STL" scale="1 ${dir} 1" />
+        </geometry>
+      </collision>
+    </link>
+    <joint name="${prefix}pinky_force_sensor_2_joint" type="fixed">
       <origin xyz="-0.00645123763174135 ${dir*0.0276833479200767} -0.00611719352979621" rpy="${dir*1.57079632679488} -1.45969392221055 ${dir*-1.22888814145719}" />
-      <parent link="${prefix}little_2" />
-      <child link="${prefix}little_force_sensor_2" />
-    </joint>
-    <link name="${prefix}little_force_sensor_3">
+      <parent link="${prefix}pinky_2" />
+      <child link="${prefix}pinky_force_sensor_2" />
+    </joint>
+    <link name="${prefix}pinky_force_sensor_3">
       <inertial>
         <origin xyz="6.36863053951123E-05 ${dir*-0.000437236774208316} -0.00112814037373121" />
@@ -913,22 +913,22 @@
       <visual>
         <geometry>
-          <mesh filename="file://$(find inspire_description)/meshes/RH56E2/sensors/little_force_sensor_3.STL" scale="1 ${dir} 1" />
-        </geometry>
-        <material name="">
-          <color rgba="0.411764705882353 0.411764705882353 0.411764705882353 1" />
-        </material>
-      </visual>
-      <collision>
-        <geometry>
-          <mesh filename="file://$(find inspire_description)/meshes/RH56E2/sensors/little_force_sensor_3.STL" scale="1 ${dir} 1" />
-        </geometry>
-      </collision>
-    </link>
-    <joint name="${prefix}little_force_sensor_3_joint" type="fixed">
+          <mesh filename="file://$(find inspire_description)/meshes/RH56E2/sensors/pinky_force_sensor_3.STL" scale="1 ${dir} 1" />
+        </geometry>
+        <material name="">
+          <color rgba="0.411764705882353 0.411764705882353 0.411764705882353 1" />
+        </material>
+      </visual>
+      <collision>
+        <geometry>
+          <mesh filename="file://$(find inspire_description)/meshes/RH56E2/sensors/pinky_force_sensor_3.STL" scale="1 ${dir} 1" />
+        </geometry>
+      </collision>
+    </link>
+    <joint name="${prefix}pinky_force_sensor_3_joint" type="fixed">
       <origin xyz="-0.00639723214432697 ${dir*0.042706921918282} -0.00611537168168175" rpy="${dir*1.5707963267949} -1.43362674619531 ${dir*-2.2760856926538}" />
-      <parent link="${prefix}little_2" />
-      <child link="${prefix}little_force_sensor_3" />
-    </joint>
-    <link name="${prefix}little_force_sensor_1">
+      <parent link="${prefix}pinky_2" />
+      <child link="${prefix}pinky_force_sensor_3" />
+    </joint>
+    <link name="${prefix}pinky_force_sensor_1">
       <inertial>
         <origin xyz="-1.2130080955873E-05 ${dir*0.000116026903212899} -0.00056744299424992" />
@@ -944,20 +944,20 @@
       <visual>
         <geometry>
-          <mesh filename="file://$(find inspire_description)/meshes/RH56E2/sensors/little_force_sensor_1.STL" scale="1 ${dir} 1" />
-        </geometry>
-        <material name="">
-          <color rgba="0.411764705882353 0.411764705882353 0.411764705882353 1" />
-        </material>
-      </visual>
-      <collision>
-        <geometry>
-          <mesh filename="file://$(find inspire_description)/meshes/RH56E2/sensors/little_force_sensor_1.STL" scale="1 ${dir} 1" />
-        </geometry>
-      </collision>
-    </link>
-    <joint name="${prefix}little_force_sensor_1_joint" type="fixed">
+          <mesh filename="file://$(find inspire_description)/meshes/RH56E2/sensors/pinky_force_sensor_1.STL" scale="1 ${dir} 1" />
+        </geometry>
+        <material name="">
+          <color rgba="0.411764705882353 0.411764705882353 0.411764705882353 1" />
+        </material>
+      </visual>
+      <collision>
+        <geometry>
+          <mesh filename="file://$(find inspire_description)/meshes/RH56E2/sensors/pinky_force_sensor_1.STL" scale="1 ${dir} 1" />
+        </geometry>
+      </collision>
+    </link>
+    <joint name="${prefix}pinky_force_sensor_1_joint" type="fixed">
       <origin xyz="-0.0120461582060113 ${dir*0.0196485471789908} -0.00665098451502223" rpy="${dir*1.5707963267949} -1.4636944932668 ${dir*-1.78288465285966}" />
-      <parent link="${prefix}little_1" />
-      <child link="${prefix}little_force_sensor_1" />
+      <parent link="${prefix}pinky_1" />
+      <child link="${prefix}pinky_force_sensor_1" />
     </joint>
   </xacro:macro>

File: gripper/inspire_description/xacro/ros2_control/hand.xacro (robot description, xacro)
@@ -26,4 +26,8 @@
       <xacro:inspire_rh56e2_interfaces name="$(arg name)" direction="$(arg direction)"/>
     </xacro:if>
+    <xacro:if value="${'$(arg type)' == 'RH56F2'}">
+      <xacro:include filename="$(find inspire_description)/xacro/ros2_control/RH56F2.xacro"/>
+      <xacro:inspire_rh56f2_interfaces name="$(arg name)" direction="$(arg direction)"/>
+    </xacro:if>
   </ros2_control>
   <xacro:if value="$(arg gazebo)">
