Commit message: 更新xacro文件，去掉多余stl

File: gripper/hitbot_description/xacro/Z-EFG-100.xacro (robot description, xacro)
@@ -24,7 +24,7 @@
   <xacro:macro name="Gripper"
     params="name collider_type:=simple">
-    <xacro:property name="prefix" value="${name + '_' if name else 'gripper_'}"/>
+    <xacro:property name="prefix" value="${name + '_' if name else ''}"/>
     <xacro:property name="M_PI" value="3.1415926535897931" />
-    <link name="${prefix}base">
+    <link name="${prefix}gripper_base">
       <inertial>
         <origin xyz="0.0828 0.03604 -7.000000000000001e-05" rpy="0 0 0" />
@@ -38,20 +38,11 @@
         </geometry>
       </visual>
-      <xacro:if value="${collider_type == 'convex_decomposition'}">
-        <collision>
-          <geometry>
-            <mesh filename="file://$(find hitbot_description)/meshes/Z-EFG-100/convex_decomposition/base_link_convex_decomposition.stl" />
-          </geometry>
-        </collision>
-      </xacro:if>
-      <xacro:if value="${collider_type == 'simple'}">
-        <collision>
-          <geometry>
-            <mesh filename="file://$(find hitbot_description)/meshes/Z-EFG-100/convex/base_link.stl" />
-          </geometry>
-        </collision>
-      </xacro:if>
-    </link>
-    <link name="${prefix}link1">
+      <collision>
+        <geometry>
+          <mesh filename="file://$(find hitbot_description)/meshes/Z-EFG-100/collision/base_link.stl" />
+        </geometry>
+      </collision>
+    </link>
+    <link name="${prefix}gripper_link1">
       <inertial>
         <origin xyz="0.01927 -0.00066 -0.00023999999999999998" rpy="0 0 0" />
@@ -65,29 +56,20 @@
         </geometry>
       </visual>
-      <xacro:if value="${collider_type == 'convex_decomposition'}">
-        <collision>
-          <geometry>
-            <mesh filename="file://$(find hitbot_description)/meshes/Z-EFG-100/convex_decomposition/gripper_link1_convex_decomposition.stl" />
-          </geometry>
-        </collision>
-      </xacro:if>
-      <xacro:if value="${collider_type == 'simple'}">
-        <collision>
-          <geometry>
-            <mesh filename="file://$(find hitbot_description)/meshes/Z-EFG-100/convex/gripper_link1.stl" />
-          </geometry>
-        </collision>
-      </xacro:if>
-    </link>
-    <joint name="${prefix}joint" type="revolute">
+      <collision>
+        <geometry>
+          <mesh filename="file://$(find hitbot_description)/meshes/Z-EFG-100/collision/gripper_link1.stl" />
+        </geometry>
+      </collision>
+    </link>
+    <joint name="${prefix}gripper_joint" type="revolute">
       <origin xyz="0.12183 -0.02 0" rpy="${M_PI} 0 ${-M_PI/4}" />
-      <parent link="${prefix}base" />
-      <child link="${prefix}link1" />
-      <axis xyz="0 0 -1" />
-      <limit lower="0" upper="0.75" velocity="3" effort="2" /> <!-- Tuned opening range
-      for
-      gripper -->
-    </joint>
-    <link name="${prefix}link2">
+      <parent link="${prefix}gripper_base" />
+      <child link="${prefix}gripper_link1" />
+      <axis xyz="0 0 -1" />
+      <limit lower="0" upper="0.75" velocity="3" effort="2" /> <!-- Tuned opening range
+      for
+      gripper -->
+    </joint>
+    <link name="${prefix}gripper_link2">
       <inertial>
         <origin xyz="0.02767 -0.0 -0.0" rpy="0 0 0" />
@@ -100,30 +82,21 @@
         </geometry>
       </visual>
-      <xacro:if value="${collider_type == 'convex_decomposition'}">
-        <collision>
-          <geometry>
-            <mesh filename="file://$(find hitbot_description)/meshes/Z-EFG-100/convex_decomposition/gripper_link2_convex_decomposition.stl" />
-          </geometry>
-        </collision>
-      </xacro:if>
-      <xacro:if value="${collider_type == 'simple'}">
-        <collision>
-          <geometry>
-            <mesh filename="file://$(find hitbot_description)/meshes/Z-EFG-100/convex/gripper_link2.stl" />
-          </geometry>
-        </collision>
-      </xacro:if>
-    </link>
-    <joint name="${prefix}joint2" type="revolute">
+      <collision>
+        <geometry>
+          <mesh filename="file://$(find hitbot_description)/meshes/Z-EFG-100/collision/gripper_link2.stl" />
+        </geometry>
+      </collision>
+    </link>
+    <joint name="${prefix}gripper_joint2" type="revolute">
       <origin xyz="0.1368 -0.01 0" rpy="${M_PI} 0 ${-M_PI/4}" />
-      <parent link="${prefix}base" />
-      <child link="${prefix}link2" />
-      <axis xyz="0 0 -1" />
-      <limit lower="0" upper="0.75" velocity="3" effort="2" /> <!-- Tuned opening range
-      for
-      gripper -->
-      <mimic joint="${prefix}joint" multiplier="1.0"/>
-    </joint>
-    <link name="${prefix}link3">
+      <parent link="${prefix}gripper_base" />
+      <child link="${prefix}gripper_link2" />
+      <axis xyz="0 0 -1" />
+      <limit lower="0" upper="0.75" velocity="3" effort="2" /> <!-- Tuned opening range
+      for
+      gripper -->
+      <mimic joint="${prefix}gripper_joint" multiplier="1.0"/>
+    </joint>
+    <link name="${prefix}gripper_link3">
       <inertial>
         <origin xyz="0.010320000000000001 -0.00034 0.0" rpy="0 0 0" />
@@ -137,30 +110,21 @@
         </geometry>
       </visual>
-      <xacro:if value="${collider_type == 'convex_decomposition'}">
-        <collision>
-          <geometry>
-            <mesh filename="file://$(find hitbot_description)/meshes/Z-EFG-100/convex_decomposition/gripper_link3_convex_decomposition.stl" />
-          </geometry>
-        </collision>
-      </xacro:if>
-      <xacro:if value="${collider_type == 'simple'}">
-        <collision>
-          <geometry>
-            <mesh filename="file://$(find hitbot_description)/meshes/Z-EFG-100/convex/gripper_link3.stl" />
-          </geometry>
-        </collision>
-      </xacro:if>
-    </link>
-    <joint name="${prefix}joint3" type="revolute">
+      <collision>
+        <geometry>
+          <mesh filename="file://$(find hitbot_description)/meshes/Z-EFG-100/collision/gripper_link3.stl" />
+        </geometry>
+      </collision>
+    </link>
+    <joint name="${prefix}gripper_joint3" type="revolute">
       <origin xyz="0.065 0 0" rpy="0 0 ${-M_PI/4}" />
-      <parent link="${prefix}link2" />
-      <child link="${prefix}link3" />
-      <axis xyz="0 0 -1" />
-      <limit lower="0" upper="0.75" velocity="3" effort="2" /> <!-- Tuned opening range
-      for
-      gripper -->
-      <mimic joint="${prefix}joint" multiplier="-1.0"/>
-    </joint>
-    <link name="${prefix}link4">
+      <parent link="${prefix}gripper_link2" />
+      <child link="${prefix}gripper_link3" />
+      <axis xyz="0 0 -1" />
+      <limit lower="0" upper="0.75" velocity="3" effort="2" /> <!-- Tuned opening range
+      for
+      gripper -->
+      <mimic joint="${prefix}gripper_joint" multiplier="-1.0"/>
+    </joint>
+    <link name="${prefix}gripper_link4">
       <inertial>
         <origin xyz="0.01927 0.00066 0.00023999999999999998" rpy="0 0 0" />
@@ -174,30 +138,21 @@
         </geometry>
       </visual>
-      <xacro:if value="${collider_type == 'convex_decomposition'}">
-        <collision>
-          <geometry>
-            <mesh filename="file://$(find hitbot_description)/meshes/Z-EFG-100/convex_decomposition/gripper_link4_convex_decomposition.stl" />
-          </geometry>
-        </collision>
-      </xacro:if>
-      <xacro:if value="${collider_type == 'simple'}">
-        <collision>
-          <geometry>
-            <mesh filename="file://$(find hitbot_description)/meshes/Z-EFG-100/convex/gripper_link4.stl" />
-          </geometry>
-        </collision>
-      </xacro:if>
-    </link>
-    <joint name="${prefix}joint4" type="revolute">
+      <collision>
+        <geometry>
+          <mesh filename="file://$(find hitbot_description)/meshes/Z-EFG-100/collision/gripper_link4.stl" />
+        </geometry>
+      </collision>
+    </link>
+    <joint name="${prefix}gripper_joint4" type="revolute">
       <origin xyz="0.121833370678203 0.0199999993241963 0" rpy="${M_PI} 0 ${M_PI/4}" />
-      <parent link="${prefix}base" />
-      <child link="${prefix}link4" />
-      <axis xyz="0 0 -1" />
-      <limit lower="0" upper="0.75" velocity="3" effort="2" /> <!-- Tuned opening range
-      for
-      gripper -->
-      <mimic joint="${prefix}joint" multiplier="-1.0"/>
-    </joint>
-    <link name="${prefix}link5">
+      <parent link="${prefix}gripper_base" />
+      <child link="${prefix}gripper_link4" />
+      <axis xyz="0 0 -1" />
+      <limit lower="0" upper="0.75" velocity="3" effort="2" /> <!-- Tuned opening range
+      for
+      gripper -->
+      <mimic joint="${prefix}gripper_joint" multiplier="-1.0"/>
+    </joint>
+    <link name="${prefix}gripper_link5">
       <inertial>
         <origin xyz="0.02767 0.0 0.0" rpy="0 0 0" />
@@ -210,30 +165,21 @@
         </geometry>
       </visual>
-      <xacro:if value="${collider_type == 'convex_decomposition'}">
-        <collision>
-          <geometry>
-            <mesh filename="file://$(find hitbot_description)/meshes/Z-EFG-100/convex_decomposition/gripper_link5_convex_decomposition.stl" />
-          </geometry>
-        </collision>
-      </xacro:if>
-      <xacro:if value="${collider_type == 'simple'}">
-        <collision>
-          <geometry>
-            <mesh filename="file://$(find hitbot_description)/meshes/Z-EFG-100/convex/gripper_link5.stl" />
-          </geometry>
-        </collision>
-      </xacro:if>
-    </link>
-    <joint name="${prefix}joint5" type="revolute">
+      <collision>
+        <geometry>
+          <mesh filename="file://$(find hitbot_description)/meshes/Z-EFG-100/collision/gripper_link5.stl" />
+        </geometry>
+      </collision>
+    </link>
+    <joint name="${prefix}gripper_joint5" type="revolute">
       <origin xyz="0.1368 0.01 0" rpy="${M_PI} 0 ${M_PI/4}" />
-      <parent link="${prefix}base" />
-      <child link="${prefix}link5" />
-      <axis xyz="0 0 -1" />
-      <limit lower="0" upper="0.75" velocity="3" effort="2" /> <!-- Tuned opening range
-      for
-      gripper -->
-      <mimic joint="${prefix}joint" multiplier="-1.0"/>
-    </joint>
-    <link name="${prefix}link6">
+      <parent link="${prefix}gripper_base" />
+      <child link="${prefix}gripper_link5" />
+      <axis xyz="0 0 -1" />
+      <limit lower="0" upper="0.75" velocity="3" effort="2" /> <!-- Tuned opening range
+      for
+      gripper -->
+      <mimic joint="${prefix}gripper_joint" multiplier="-1.0"/>
+    </joint>
+    <link name="${prefix}gripper_link6">
       <inertial>
         <origin xyz="0.010320000000000001 0.00034 -0.0" rpy="0 0 0" />
@@ -247,35 +193,26 @@
         </geometry>
       </visual>
-      <xacro:if value="${collider_type == 'convex_decomposition'}">
-        <collision>
-          <geometry>
-            <mesh filename="file://$(find hitbot_description)/meshes/Z-EFG-100/convex_decomposition/gripper_link6_convex_decomposition.stl" />
-          </geometry>
-        </collision>
-      </xacro:if>
-      <xacro:if value="${collider_type == 'simple'}">
-        <collision>
-          <geometry>
-            <mesh filename="file://$(find hitbot_description)/meshes/Z-EFG-100/convex/gripper_link6.stl" />
-          </geometry>
-        </collision>
-      </xacro:if>
-    </link>
-    <joint name="${prefix}joint6" type="revolute">
+      <collision>
+        <geometry>
+          <mesh filename="file://$(find hitbot_description)/meshes/Z-EFG-100/collision/gripper_link6.stl" />
+        </geometry>
+      </collision>
+    </link>
+    <joint name="${prefix}gripper_joint6" type="revolute">
       <origin xyz="0.065 0 0" rpy="0 0 ${M_PI/4}" />
-      <parent link="${prefix}link5" />
-      <child link="${prefix}link6" />
-      <axis xyz="0 0 -1" />
-      <limit lower="0" upper="0.75" velocity="3" effort="2" /> <!-- Tuned opening range
-      for
-      gripper -->
-      <mimic joint="${prefix}joint" multiplier="1.0"/>
+      <parent link="${prefix}gripper_link5" />
+      <child link="${prefix}gripper_link6" />
+      <axis xyz="0 0 -1" />
+      <limit lower="0" upper="0.75" velocity="3" effort="2" /> <!-- Tuned opening range
+      for
+      gripper -->
+      <mimic joint="${prefix}gripper_joint" multiplier="1.0"/>
     </joint>
     <!-- Tool Center Point -->
-    <link name="${prefix}tcp_link" />
-    <joint name="${prefix}tcp_joint" type="fixed">
+    <link name="${prefix}gripper_tcp_link" />
+    <joint name="${prefix}gripper_tcp_joint" type="fixed">
       <origin xyz="0.222892 0 0 " rpy="3.14 0 0" />
-      <parent link="${prefix}base" />
-      <child link="${prefix}tcp_link" />
+      <parent link="${prefix}gripper_base" />
+      <child link="${prefix}gripper_tcp_link" />
       <axis xyz="0 0 0" />
     </joint>

File: gripper/hitbot_description/xacro/ros2_control/Z-EFG-100.xacro (robot description, xacro)
@@ -1,15 +1,44 @@
 <?xml version="1.0"?>
 <robot xmlns:xacro="http://www.ros.org/wiki/xacro">
-  <xacro:macro name="hitbot_z_efg_100_interfaces" params="name initial_value:=0.75">
-    <joint name="${name}_joint">
+  <xacro:macro name="hitbot_z_efg_100_interfaces" params="name">
+    <xacro:arg name="gazebo" default="false"/>
+    <xacro:property name="prefix" value="${name + '_' if name else ''}"/>
+    <!-- Main driven joint interface -->
+    <joint name="${prefix}gripper_joint">
       <command_interface name="position"/>
       <state_interface name="position">
-        <param name="initial_value">${initial_value}</param>
+        <param name="initial_value">0.75</param>
       </state_interface>
-      <state_interface name="velocity">
-        <param name="initial_value">0.0</param>
-      </state_interface>
+      <state_interface name="velocity"/>
       <state_interface name="effort"/>
     </joint>
+    <xacro:if value="$(arg gazebo)">
+      <!-- Mimic joint interfaces, enabled only for Gazebo -->
+      <joint name="${prefix}gripper_joint2">
+        <state_interface name="position"/>
+        <state_interface name="velocity"/>
+        <state_interface name="effort"/>
+      </joint>
+      <joint name="${prefix}gripper_joint3">
+        <state_interface name="position"/>
+        <state_interface name="velocity"/>
+        <state_interface name="effort"/>
+      </joint>
+      <joint name="${prefix}gripper_joint4">
+        <state_interface name="position"/>
+        <state_interface name="velocity"/>
+        <state_interface name="effort"/>
+      </joint>
+      <joint name="${prefix}gripper_joint5">
+        <state_interface name="position"/>
+        <state_interface name="velocity"/>
+        <state_interface name="effort"/>
+      </joint>
+      <joint name="${prefix}gripper_joint6">
+        <state_interface name="position"/>
+        <state_interface name="velocity"/>
+        <state_interface name="effort"/>
+      </joint>
+    </xacro:if>
   </xacro:macro>
 </robot>

File: gripper/hitbot_description/xacro/ros2_control/gripper.xacro (robot description, xacro)
@@ -29,5 +29,5 @@
     <xacro:if value="${'$(arg type)' == 'Z-EFG-100'}">
       <xacro:include filename="$(find hitbot_description)/xacro/ros2_control/Z-EFG-100.xacro"/>
-      <xacro:hitbot_z_efg_100_interfaces name="gripper"/>
+      <xacro:hitbot_z_efg_100_interfaces name=""/>
     </xacro:if>
   </ros2_control>

Commit message: 去掉hitbot的stl文件

File: gripper/hitbot_description/xacro/Z-EFG-100.xacro (robot description, xacro)
@@ -35,10 +35,10 @@
       <visual>
         <geometry>
-          <mesh filename="file://$(find hitbot_description)/meshes/Z-EFG-100/visual/base.glb" />
-        </geometry>
-      </visual>
-      <collision>
-        <geometry>
-          <mesh filename="file://$(find hitbot_description)/meshes/Z-EFG-100/collision/base_link.stl" />
+          <mesh filename="file://$(find hitbot_description)/meshes/Z-EFG-100/base.glb" />
+        </geometry>
+      </visual>
+      <collision>
+        <geometry>
+          <mesh filename="file://$(find hitbot_description)/meshes/Z-EFG-100/base.glb" />
         </geometry>
       </collision>
@@ -53,10 +53,10 @@
       <visual>
         <geometry>
-          <mesh filename="file://$(find hitbot_description)/meshes/Z-EFG-100/visual/link1.glb" />
-        </geometry>
-      </visual>
-      <collision>
-        <geometry>
-          <mesh filename="file://$(find hitbot_description)/meshes/Z-EFG-100/collision/gripper_link1.stl" />
+          <mesh filename="file://$(find hitbot_description)/meshes/Z-EFG-100/link1.glb" />
+        </geometry>
+      </visual>
+      <collision>
+        <geometry>
+          <mesh filename="file://$(find hitbot_description)/meshes/Z-EFG-100/link1.glb" />
         </geometry>
       </collision>
@@ -79,10 +79,10 @@
       <visual>
         <geometry>
-          <mesh filename="file://$(find hitbot_description)/meshes/Z-EFG-100/visual/link2.glb" />
-        </geometry>
-      </visual>
-      <collision>
-        <geometry>
-          <mesh filename="file://$(find hitbot_description)/meshes/Z-EFG-100/collision/gripper_link2.stl" />
+          <mesh filename="file://$(find hitbot_description)/meshes/Z-EFG-100/link2.glb" />
+        </geometry>
+      </visual>
+      <collision>
+        <geometry>
+          <mesh filename="file://$(find hitbot_description)/meshes/Z-EFG-100/link2.glb" />
         </geometry>
       </collision>
@@ -107,10 +107,10 @@
       <visual>
         <geometry>
-          <mesh filename="file://$(find hitbot_description)/meshes/Z-EFG-100/visual/link3.glb" />
-        </geometry>
-      </visual>
-      <collision>
-        <geometry>
-          <mesh filename="file://$(find hitbot_description)/meshes/Z-EFG-100/collision/gripper_link3.stl" />
+          <mesh filename="file://$(find hitbot_description)/meshes/Z-EFG-100/link3.glb" />
+        </geometry>
+      </visual>
+      <collision>
+        <geometry>
+          <mesh filename="file://$(find hitbot_description)/meshes/Z-EFG-100/link3.glb" />
         </geometry>
       </collision>
@@ -135,10 +135,10 @@
       <visual>
         <geometry>
-          <mesh filename="file://$(find hitbot_description)/meshes/Z-EFG-100/visual/link4.glb" />
-        </geometry>
-      </visual>
-      <collision>
-        <geometry>
-          <mesh filename="file://$(find hitbot_description)/meshes/Z-EFG-100/collision/gripper_link4.stl" />
+          <mesh filename="file://$(find hitbot_description)/meshes/Z-EFG-100/link4.glb" />
+        </geometry>
+      </visual>
+      <collision>
+        <geometry>
+          <mesh filename="file://$(find hitbot_description)/meshes/Z-EFG-100/link4.glb" />
         </geometry>
       </collision>
@@ -162,10 +162,10 @@
       <visual>
         <geometry>
-          <mesh filename="file://$(find hitbot_description)/meshes/Z-EFG-100/visual/link5.glb" />
-        </geometry>
-      </visual>
-      <collision>
-        <geometry>
-          <mesh filename="file://$(find hitbot_description)/meshes/Z-EFG-100/collision/gripper_link5.stl" />
+          <mesh filename="file://$(find hitbot_description)/meshes/Z-EFG-100/link5.glb" />
+        </geometry>
+      </visual>
+      <collision>
+        <geometry>
+          <mesh filename="file://$(find hitbot_description)/meshes/Z-EFG-100/link5.glb" />
         </geometry>
       </collision>
@@ -190,10 +190,10 @@
       <visual>
         <geometry>
-          <mesh filename="file://$(find hitbot_description)/meshes/Z-EFG-100/visual/link6.glb" />
-        </geometry>
-      </visual>
-      <collision>
-        <geometry>
-          <mesh filename="file://$(find hitbot_description)/meshes/Z-EFG-100/collision/gripper_link6.stl" />
+          <mesh filename="file://$(find hitbot_description)/meshes/Z-EFG-100/link6.glb" />
+        </geometry>
+      </visual>
+      <collision>
+        <geometry>
+          <mesh filename="file://$(find hitbot_description)/meshes/Z-EFG-100/link6.glb" />
         </geometry>
       </collision>

Commit message: 改maintainer 去除多余注释

File: gripper/hitbot_description/xacro/Z-EFG-100.xacro (robot description, xacro)
@@ -67,7 +67,5 @@
       <child link="${prefix}gripper_link1" />
       <axis xyz="0 0 -1" />
-      <limit lower="0" upper="0.75" velocity="3" effort="2" /> <!-- Tuned opening range
-      for
-      gripper -->
+      <limit lower="0" upper="0.75" velocity="3" effort="2" />
     </joint>
     <link name="${prefix}gripper_link2">
@@ -93,7 +91,5 @@
       <child link="${prefix}gripper_link2" />
       <axis xyz="0 0 -1" />
-      <limit lower="0" upper="0.75" velocity="3" effort="2" /> <!-- Tuned opening range
-      for
-      gripper -->
+      <limit lower="0" upper="0.75" velocity="3" effort="2" />
       <mimic joint="${prefix}gripper_joint" multiplier="1.0"/>
     </joint>
@@ -121,7 +117,5 @@
       <child link="${prefix}gripper_link3" />
       <axis xyz="0 0 -1" />
-      <limit lower="0" upper="0.75" velocity="3" effort="2" /> <!-- Tuned opening range
-      for
-      gripper -->
+      <limit lower="0" upper="0.75" velocity="3" effort="2" />
       <mimic joint="${prefix}gripper_joint" multiplier="-1.0"/>
     </joint>
@@ -149,7 +143,5 @@
       <child link="${prefix}gripper_link4" />
       <axis xyz="0 0 -1" />
-      <limit lower="0" upper="0.75" velocity="3" effort="2" /> <!-- Tuned opening range
-      for
-      gripper -->
+      <limit lower="0" upper="0.75" velocity="3" effort="2" />
       <mimic joint="${prefix}gripper_joint" multiplier="-1.0"/>
     </joint>
@@ -176,7 +168,5 @@
       <child link="${prefix}gripper_link5" />
       <axis xyz="0 0 -1" />
-      <limit lower="0" upper="0.75" velocity="3" effort="2" /> <!-- Tuned opening range
-      for
-      gripper -->
+      <limit lower="0" upper="0.75" velocity="3" effort="2" />
       <mimic joint="${prefix}gripper_joint" multiplier="-1.0"/>
     </joint>
@@ -204,7 +194,5 @@
       <child link="${prefix}gripper_link6" />
       <axis xyz="0 0 -1" />
-      <limit lower="0" upper="0.75" velocity="3" effort="2" /> <!-- Tuned opening range
-      for
-      gripper -->
+      <limit lower="0" upper="0.75" velocity="3" effort="2" />
       <mimic joint="${prefix}gripper_joint" multiplier="1.0"/>
     </joint>
