Commit message: add common gripper side config

File: gripper/hitbot_description/xacro/Z-EFG-100.xacro (robot description, xacro)
@@ -23,7 +23,8 @@
 <robot xmlns:xacro="http://ros.org/wiki/xacro" name="hitbot_gripper">
   <xacro:macro name="Gripper"
-    params="name collider_type:=simple">
+    params="name collider_type:=simple kinematic_only:=false">
     <xacro:property name="prefix" value="${name + '_' if name else ''}"/>
     <xacro:property name="M_PI" value="3.1415926535897931" />
+    <xacro:property name="actuated_joint_type" value="${'fixed' if str(kinematic_only).lower() == 'true' else 'revolute'}"/>
     <link name="${prefix}gripper_base">
       <inertial>
@@ -62,5 +63,5 @@
       </collision>
     </link>
-    <joint name="${prefix}gripper_joint" type="revolute">
+    <joint name="${prefix}gripper_joint" type="${actuated_joint_type}">
       <origin xyz="0.12183 -0.02 0" rpy="${M_PI} 0 ${-M_PI/4}" />
       <parent link="${prefix}gripper_base" />
@@ -86,5 +87,5 @@
       </collision>
     </link>
-    <joint name="${prefix}gripper_joint2" type="revolute">
+    <joint name="${prefix}gripper_joint2" type="${actuated_joint_type}">
       <origin xyz="0.1368 -0.01 0" rpy="${M_PI} 0 ${-M_PI/4}" />
       <parent link="${prefix}gripper_base" />
@@ -92,5 +93,7 @@
       <axis xyz="0 0 -1" />
       <limit lower="0" upper="0.75" velocity="3" effort="2" />
+      <xacro:unless value="${str(kinematic_only).lower() == 'true'}">
       <mimic joint="${prefix}gripper_joint" multiplier="1.0"/>
+      </xacro:unless>
     </joint>
     <link name="${prefix}gripper_link3">
@@ -112,5 +115,5 @@
       </collision>
     </link>
-    <joint name="${prefix}gripper_joint3" type="revolute">
+    <joint name="${prefix}gripper_joint3" type="${actuated_joint_type}">
       <origin xyz="0.065 0 0" rpy="0 0 ${-M_PI/4}" />
       <parent link="${prefix}gripper_link2" />
@@ -118,5 +121,7 @@
       <axis xyz="0 0 -1" />
       <limit lower="0" upper="0.75" velocity="3" effort="2" />
+      <xacro:unless value="${str(kinematic_only).lower() == 'true'}">
       <mimic joint="${prefix}gripper_joint" multiplier="-1.0"/>
+      </xacro:unless>
     </joint>
     <link name="${prefix}gripper_link4">
@@ -138,5 +143,5 @@
       </collision>
     </link>
-    <joint name="${prefix}gripper_joint4" type="revolute">
+    <joint name="${prefix}gripper_joint4" type="${actuated_joint_type}">
       <origin xyz="0.121833370678203 0.0199999993241963 0" rpy="${M_PI} 0 ${M_PI/4}" />
       <parent link="${prefix}gripper_base" />
@@ -144,5 +149,7 @@
       <axis xyz="0 0 -1" />
       <limit lower="0" upper="0.75" velocity="3" effort="2" />
+      <xacro:unless value="${str(kinematic_only).lower() == 'true'}">
       <mimic joint="${prefix}gripper_joint" multiplier="-1.0"/>
+      </xacro:unless>
     </joint>
     <link name="${prefix}gripper_link5">
@@ -163,5 +170,5 @@
       </collision>
     </link>
-    <joint name="${prefix}gripper_joint5" type="revolute">
+    <joint name="${prefix}gripper_joint5" type="${actuated_joint_type}">
       <origin xyz="0.1368 0.01 0" rpy="${M_PI} 0 ${M_PI/4}" />
       <parent link="${prefix}gripper_base" />
@@ -169,5 +176,7 @@
       <axis xyz="0 0 -1" />
       <limit lower="0" upper="0.75" velocity="3" effort="2" />
+      <xacro:unless value="${str(kinematic_only).lower() == 'true'}">
       <mimic joint="${prefix}gripper_joint" multiplier="-1.0"/>
+      </xacro:unless>
     </joint>
     <link name="${prefix}gripper_link6">
@@ -189,5 +198,5 @@
       </collision>
     </link>
-    <joint name="${prefix}gripper_joint6" type="revolute">
+    <joint name="${prefix}gripper_joint6" type="${actuated_joint_type}">
       <origin xyz="0.065 0 0" rpy="0 0 ${M_PI/4}" />
       <parent link="${prefix}gripper_link5" />
@@ -195,5 +204,7 @@
       <axis xyz="0 0 -1" />
       <limit lower="0" upper="0.75" velocity="3" effort="2" />
+      <xacro:unless value="${str(kinematic_only).lower() == 'true'}">
       <mimic joint="${prefix}gripper_joint" multiplier="1.0"/>
+      </xacro:unless>
     </joint>
     <!-- Tool Center Point -->
