Commit message: 添加freedomv2

File: dexhands/freedom_description/xacro/freedomv1.xacro (robot description, xacro)
@@ -1,5 +1,5 @@
 <?xml version="1.0" encoding="utf-8"?>
 <robot xmlns:xacro="http://www.ros.org/wiki/xacro">
-	<xacro:macro name="FreedomHand" params="name direction:=1 fixed_joints:=false">
+	<xacro:macro name="FreedomHandV1" params="name direction:=1 fixed_joints:=false">
 		<xacro:property name="prefix" value="${name + '_' if name else ''}"/>
 		<xacro:property name="joint_type" value="${fixed_joints and 'fixed' or 'revolute'}"/>
@@ -12,13 +12,13 @@
 			<visual>
 				<geometry>
-					<mesh filename="file://$(find freedom_description)/meshes/freedom/base.glb" scale="${direction} 1 1"/>
-				</geometry>
-				<material name="">
-					<color rgba="0.52941 0.54902 0.54902 1"/>
-				</material>
-			</visual>
-			<collision>
-				<geometry>
-					<mesh filename="file://$(find freedom_description)/meshes/freedom/base.glb" scale="${direction} 1 1"/>
+					<mesh filename="file://$(find freedom_description)/meshes/freedomv1/base.glb" scale="${direction} 1 1"/>
+				</geometry>
+				<material name="">
+					<color rgba="0.52941 0.54902 0.54902 1"/>
+				</material>
+			</visual>
+			<collision>
+				<geometry>
+					<mesh filename="file://$(find freedom_description)/meshes/freedomv1/base.glb" scale="${direction} 1 1"/>
 				</geometry>
 			</collision>
@@ -32,13 +32,13 @@
 			<visual>
 				<geometry>
-					<mesh filename="file://$(find freedom_description)/meshes/freedom/l1.glb" scale="${direction} 1 1"/>
-				</geometry>
-				<material name="">
-					<color rgba="0.52941 0.54902 0.54902 1"/>
-				</material>
-			</visual>
-			<collision>
-				<geometry>
-					<mesh filename="file://$(find freedom_description)/meshes/freedom/l1.glb" scale="${direction} 1 1"/>
+					<mesh filename="file://$(find freedom_description)/meshes/freedomv1/l1.glb" scale="${direction} 1 1"/>
+				</geometry>
+				<material name="">
+					<color rgba="0.52941 0.54902 0.54902 1"/>
+				</material>
+			</visual>
+			<collision>
+				<geometry>
+					<mesh filename="file://$(find freedom_description)/meshes/freedomv1/l1.glb" scale="${direction} 1 1"/>
 				</geometry>
 			</collision>
@@ -52,13 +52,13 @@
 			<visual>
 				<geometry>
-					<mesh filename="file://$(find freedom_description)/meshes/freedom/l2.glb" scale="${direction} 1 1"/>
-				</geometry>
-				<material name="">
-					<color rgba="0.52941 0.54902 0.54902 1"/>
-				</material>
-			</visual>
-			<collision>
-				<geometry>
-					<mesh filename="file://$(find freedom_description)/meshes/freedom/l2.glb" scale="${direction} 1 1"/>
+					<mesh filename="file://$(find freedom_description)/meshes/freedomv1/l2.glb" scale="${direction} 1 1"/>
+				</geometry>
+				<material name="">
+					<color rgba="0.52941 0.54902 0.54902 1"/>
+				</material>
+			</visual>
+			<collision>
+				<geometry>
+					<mesh filename="file://$(find freedom_description)/meshes/freedomv1/l2.glb" scale="${direction} 1 1"/>
 				</geometry>
 			</collision>
@@ -72,5 +72,5 @@
 			<visual>
 				<geometry>
-					<mesh filename="file://$(find freedom_description)/meshes/freedom/l3.glb" scale="${direction} 1 1"/>
+					<mesh filename="file://$(find freedom_description)/meshes/freedomv1/l3.glb" scale="${direction} 1 1"/>
 				</geometry>
 				<material name="">
@@ -80,5 +80,5 @@
 			<collision>
 				<geometry>
-					<mesh filename="file://$(find freedom_description)/meshes/freedom/l3.glb" scale="${direction} 1 1"/>
+					<mesh filename="file://$(find freedom_description)/meshes/freedomv1/l3.glb" scale="${direction} 1 1"/>
 				</geometry>
 			</collision>
@@ -92,5 +92,5 @@
 			<visual>
 				<geometry>
-					<mesh filename="file://$(find freedom_description)/meshes/freedom/l4.glb" scale="${direction} 1 1"/>
+					<mesh filename="file://$(find freedom_description)/meshes/freedomv1/l4.glb" scale="${direction} 1 1"/>
 				</geometry>
 				<material name="">
@@ -100,5 +100,5 @@
 			<collision>
 				<geometry>
-					<mesh filename="file://$(find freedom_description)/meshes/freedom/l4.glb" scale="${direction} 1 1"/>
+					<mesh filename="file://$(find freedom_description)/meshes/freedomv1/l4.glb" scale="${direction} 1 1"/>
 				</geometry>
 			</collision>
@@ -112,5 +112,5 @@
 			<visual>
 				<geometry>
-					<mesh filename="file://$(find freedom_description)/meshes/freedom/l5.glb" scale="${direction} 1 1"/>
+					<mesh filename="file://$(find freedom_description)/meshes/freedomv1/l5.glb" scale="${direction} 1 1"/>
 				</geometry>
 				<material name="">
@@ -120,5 +120,5 @@
 			<collision>
 				<geometry>
-					<mesh filename="file://$(find freedom_description)/meshes/freedom/l5.glb" scale="${direction} 1 1"/>
+					<mesh filename="file://$(find freedom_description)/meshes/freedomv1/l5.glb" scale="${direction} 1 1"/>
 				</geometry>
 			</collision>
@@ -132,13 +132,13 @@
 			<visual>
 				<geometry>
-					<mesh filename="file://$(find freedom_description)/meshes/freedom/l4.glb" scale="${direction} 1 1"/>
-				</geometry>
-				<material name="">
-					<color rgba="0.52941 0.54902 0.54902 1"/>
-				</material>
-			</visual>
-			<collision>
-				<geometry>
-					<mesh filename="file://$(find freedom_description)/meshes/freedom/l4.glb" scale="${direction} 1 1"/>
+					<mesh filename="file://$(find freedom_description)/meshes/freedomv1/l4.glb" scale="${direction} 1 1"/>
+				</geometry>
+				<material name="">
+					<color rgba="0.52941 0.54902 0.54902 1"/>
+				</material>
+			</visual>
+			<collision>
+				<geometry>
+					<mesh filename="file://$(find freedom_description)/meshes/freedomv1/l4.glb" scale="${direction} 1 1"/>
 				</geometry>
 			</collision>
@@ -152,13 +152,13 @@
 			<visual>
 				<geometry>
-					<mesh filename="file://$(find freedom_description)/meshes/freedom/l5.glb" scale="${direction} 1 1"/>
-				</geometry>
-				<material name="">
-					<color rgba="0.52941 0.54902 0.54902 1"/>
-				</material>
-			</visual>
-			<collision>
-				<geometry>
-					<mesh filename="file://$(find freedom_description)/meshes/freedom/l5.glb" scale="${direction} 1 1"/>
+					<mesh filename="file://$(find freedom_description)/meshes/freedomv1/l5.glb" scale="${direction} 1 1"/>
+				</geometry>
+				<material name="">
+					<color rgba="0.52941 0.54902 0.54902 1"/>
+				</material>
+			</visual>
+			<collision>
+				<geometry>
+					<mesh filename="file://$(find freedom_description)/meshes/freedomv1/l5.glb" scale="${direction} 1 1"/>
 				</geometry>
 			</collision>
@@ -172,13 +172,13 @@
 			<visual>
 				<geometry>
-					<mesh filename="file://$(find freedom_description)/meshes/freedom/l4.glb" scale="${direction} 1 1"/>
-				</geometry>
-				<material name="">
-					<color rgba="0.52941 0.54902 0.54902 1"/>
-				</material>
-			</visual>
-			<collision>
-				<geometry>
-					<mesh filename="file://$(find freedom_description)/meshes/freedom/l4.glb" scale="${direction} 1 1"/>
+					<mesh filename="file://$(find freedom_description)/meshes/freedomv1/l4.glb" scale="${direction} 1 1"/>
+				</geometry>
+				<material name="">
+					<color rgba="0.52941 0.54902 0.54902 1"/>
+				</material>
+			</visual>
+			<collision>
+				<geometry>
+					<mesh filename="file://$(find freedom_description)/meshes/freedomv1/l4.glb" scale="${direction} 1 1"/>
 				</geometry>
 			</collision>
@@ -192,13 +192,13 @@
 			<visual>
 				<geometry>
-					<mesh filename="file://$(find freedom_description)/meshes/freedom/l5.glb" scale="${direction} 1 1"/>
-				</geometry>
-				<material name="">
-					<color rgba="0.52941 0.54902 0.54902 1"/>
-				</material>
-			</visual>
-			<collision>
-				<geometry>
-					<mesh filename="file://$(find freedom_description)/meshes/freedom/l5.glb" scale="${direction} 1 1"/>
+					<mesh filename="file://$(find freedom_description)/meshes/freedomv1/l5.glb" scale="${direction} 1 1"/>
+				</geometry>
+				<material name="">
+					<color rgba="0.52941 0.54902 0.54902 1"/>
+				</material>
+			</visual>
+			<collision>
+				<geometry>
+					<mesh filename="file://$(find freedom_description)/meshes/freedomv1/l5.glb" scale="${direction} 1 1"/>
 				</geometry>
 			</collision>
@@ -212,13 +212,13 @@
 			<visual>
 				<geometry>
-					<mesh filename="file://$(find freedom_description)/meshes/freedom/l4.glb" scale="${direction} 1 1"/>
-				</geometry>
-				<material name="">
-					<color rgba="0.52941 0.54902 0.54902 1"/>
-				</material>
-			</visual>
-			<collision>
-				<geometry>
-					<mesh filename="file://$(find freedom_description)/meshes/freedom/l4.glb" scale="${direction} 1 1"/>
+					<mesh filename="file://$(find freedom_description)/meshes/freedomv1/l4.glb" scale="${direction} 1 1"/>
+				</geometry>
+				<material name="">
+					<color rgba="0.52941 0.54902 0.54902 1"/>
+				</material>
+			</visual>
+			<collision>
+				<geometry>
+					<mesh filename="file://$(find freedom_description)/meshes/freedomv1/l4.glb" scale="${direction} 1 1"/>
 				</geometry>
 			</collision>
@@ -232,13 +232,13 @@
 			<visual>
 				<geometry>
-					<mesh filename="file://$(find freedom_description)/meshes/freedom/l5.glb" scale="${direction} 1 1"/>
-				</geometry>
-				<material name="">
-					<color rgba="0.52941 0.54902 0.54902 1"/>
-				</material>
-			</visual>
-			<collision>
-				<geometry>
-					<mesh filename="file://$(find freedom_description)/meshes/freedom/l5.glb" scale="${direction} 1 1"/>
+					<mesh filename="file://$(find freedom_description)/meshes/freedomv1/l5.glb" scale="${direction} 1 1"/>
+				</geometry>
+				<material name="">
+					<color rgba="0.52941 0.54902 0.54902 1"/>
+				</material>
+			</visual>
+			<collision>
+				<geometry>
+					<mesh filename="file://$(find freedom_description)/meshes/freedomv1/l5.glb" scale="${direction} 1 1"/>
 				</geometry>
 			</collision>
@@ -349,3 +349,6 @@
 		</joint>
 	</xacro:macro>
+	<xacro:macro name="FreedomHand" params="name direction:=1 fixed_joints:=false">
+		<xacro:FreedomHandV1 name="${name}" direction="${direction}" fixed_joints="${fixed_joints}"/>
+	</xacro:macro>
 </robot>

File: dexhands/freedom_description/xacro/hand.xacro (robot description, xacro)
@@ -1,7 +1,13 @@
 <?xml version="1.0" encoding="utf-8"?>
-<robot name="Freedom_$(arg type)" xmlns:xacro="http://www.ros.org/wiki/xacro">
-	<xacro:arg name="type" default="freedom"/>
+<robot name="Freedom" xmlns:xacro="http://www.ros.org/wiki/xacro">
+	<xacro:arg name="type" default="freedomv2"/>
 	<xacro:arg name="direction" default="1"/>
-	<xacro:include filename="$(find freedom_description)/xacro/freedom.xacro"/>
-	<xacro:FreedomHand name="" direction="$(arg direction)"/>
+	<xacro:if value="${'$(arg type)' == 'freedomv1' or '$(arg type)' == 'freedom_v1' or '$(arg type)' == 'freedom'}">
+		<xacro:include filename="$(find freedom_description)/xacro/freedomv1.xacro"/>
+		<xacro:FreedomHandV1 name="" direction="$(arg direction)"/>
+	</xacro:if>
+	<xacro:if value="${'$(arg type)' == 'freedomv2' or '$(arg type)' == 'freedom_v2'}">
+		<xacro:include filename="$(find freedom_description)/xacro/freedomv2.xacro"/>
+		<xacro:FreedomHandV2 name="" direction="$(arg direction)"/>
+	</xacro:if>
 </robot>

File: dexhands/freedom_description/xacro/ros2_control/freedomv1.xacro (robot description, xacro)
@@ -1,5 +1,5 @@
 <?xml version="1.0"?>
 <robot xmlns:xacro="http://www.ros.org/wiki/xacro">
-  <xacro:macro name="freedom_interfaces" params="name">
+  <xacro:macro name="freedomv1_interfaces" params="name">
     <xacro:property name="prefix" value="${name + '_' if name else ''}"/>
     <joint name="${prefix}thumb_joint1">
@@ -52,3 +52,6 @@
     </joint>
   </xacro:macro>
+  <xacro:macro name="freedom_interfaces" params="name">
+    <xacro:freedomv1_interfaces name="${name}"/>
+  </xacro:macro>
 </robot>

File: dexhands/freedom_description/xacro/ros2_control/hand.xacro (robot description, xacro)
@@ -1,5 +1,5 @@
 <?xml version="1.0"?>
-<robot name="Freedom_$(arg type)" xmlns:xacro="http://www.ros.org/wiki/xacro">
-    <xacro:arg name="type" default="freedom"/>
+<robot name="Freedom" xmlns:xacro="http://www.ros.org/wiki/xacro">
+    <xacro:arg name="type" default="freedomv2"/>
     <xacro:arg name="direction" default="1"/>
     <xacro:arg name="gazebo" default="false"/>
@@ -7,4 +7,5 @@
     <xacro:arg name="slave_id" default="auto"/>
     <xacro:arg name="baudrate" default="115200"/>
+    <xacro:arg name="command_speed" default="100"/>
     <xacro:arg name="can_interface" default="can0"/>
     <xacro:arg name="device_id" default="auto"/>
@@ -35,4 +36,5 @@
                 <param name="serial_port">$(arg serial_port)</param>
                 <param name="slave_id">$(arg slave_id)</param>
+                <param name="protocol_version">$(arg type)</param>
                 <xacro:if value="${'$(arg direction)' == '1'}">
                     <param name="hand_side">left</param>
@@ -42,6 +44,7 @@
                 </xacro:unless>
                 <param name="baudrate">$(arg baudrate)</param>
+                <param name="command_speed">$(arg command_speed)</param>
                 <param name="read_feedback">true</param>
-                <param name="feedback_timeout_ms">20</param>
+                <param name="feedback_timeout_ms">50</param>
             </xacro:if>
             <xacro:if value="${'$(arg ros2_control_hardware_type)' == 'real_can'}">
@@ -61,6 +64,12 @@
             </xacro:if>
         </hardware>
-        <xacro:include filename="$(find freedom_description)/xacro/ros2_control/freedom.xacro"/>
-        <xacro:freedom_interfaces name=""/>
+        <xacro:if value="${'$(arg type)' == 'freedomv1' or '$(arg type)' == 'freedom_v1' or '$(arg type)' == 'freedom'}">
+            <xacro:include filename="$(find freedom_description)/xacro/ros2_control/freedomv1.xacro"/>
+            <xacro:freedomv1_interfaces name=""/>
+        </xacro:if>
+        <xacro:if value="${'$(arg type)' == 'freedomv2' or '$(arg type)' == 'freedom_v2'}">
+            <xacro:include filename="$(find freedom_description)/xacro/ros2_control/freedomv2.xacro"/>
+            <xacro:freedomv2_interfaces name=""/>
+        </xacro:if>
     </ros2_control>
     <xacro:arg name="gazebo" default="false"/>

File: dexhands/freedom_description/xacro/ros2_control/side_systems.xacro (robot description, xacro)
@@ -1,7 +1,8 @@
 <?xml version="1.0"?>
 <robot xmlns:xacro="http://www.ros.org/wiki/xacro">
-  <xacro:include filename="$(find freedom_description)/xacro/ros2_control/freedom.xacro"/>
-  <xacro:macro name="freedom_rs485_side_system" params="side serial_port slave_id:=auto baudrate:=115200">
-    <ros2_control name="freedom_v1_${side}_system" type="system">
+  <xacro:include filename="$(find freedom_description)/xacro/ros2_control/freedomv1.xacro"/>
+  <xacro:include filename="$(find freedom_description)/xacro/ros2_control/freedomv2.xacro"/>
+  <xacro:macro name="freedom_rs485_side_system" params="side serial_port slave_id:=auto baudrate:=115200 type:=freedomv1 command_speed:=100">
+    <ros2_control name="${type}_${side}_system" type="system">
       <hardware>
         <plugin>modbus_ros2_control/FreedomRS485Hardware</plugin>
@@ -10,8 +11,15 @@
         <param name="slave_id">${slave_id}</param>
         <param name="baudrate">${baudrate}</param>
+        <param name="protocol_version">${type}</param>
+        <param name="command_speed">${command_speed}</param>
         <param name="read_feedback">true</param>
-        <param name="feedback_timeout_ms">20</param>
+        <param name="feedback_timeout_ms">50</param>
       </hardware>
-      <xacro:freedom_interfaces name="${side}_hand"/>
+      <xacro:if value="${type == 'freedomv2' or type == 'freedom_v2'}">
+        <xacro:freedomv2_interfaces name="${side}_hand"/>
+      </xacro:if>
+      <xacro:unless value="${type == 'freedomv2' or type == 'freedom_v2'}">
+        <xacro:freedom_interfaces name="${side}_hand"/>
+      </xacro:unless>
     </ros2_control>
   </xacro:macro>

Commit message: 添加inspireCANFD，修掉频率过低的问题

File: dexhands/freedom_description/xacro/freedomv1.xacro (robot description, xacro)
@@ -348,4 +348,10 @@
 			</xacro:unless>
 		</joint>
+		<link name="${prefix}eef"/>
+		<joint name="${prefix}eef_joint" type="fixed">
+			<parent link="${prefix}hand_base"/>
+			<child link="${prefix}eef"/>
+			<origin xyz="0 0.1074 0.001"/>
+		</joint>
 	</xacro:macro>
 	<xacro:macro name="FreedomHand" params="name direction:=1 fixed_joints:=false">

File: gripper/inspire_description/xacro/hands/RH56E2.xacro (robot description, xacro)
@@ -1,7 +1,8 @@
 <?xml version="1.0" encoding="utf-8"?>
 <robot xmlns:xacro="http://www.ros.org/wiki/xacro">
-  <xacro:macro name="InspireHandRH56E2" params="name:='' direction:=1 use_flange:=false ">
+  <xacro:macro name="InspireHandRH56E2" params="name:='' direction:=1 use_flange:=false fixed_joints:=false">
     <xacro:property name="prefix" value="${name + '_' if name else ''}"/>
     <xacro:property name="dir" value="${-1 * int(direction)}"/>
+    <xacro:property name="joint_type" value="${fixed_joints and 'fixed' or 'revolute'}"/>
     <xacro:if value="${use_flange}">
       <link name="${prefix}flange">
@@ -101,5 +102,5 @@
       </collision>
     </link>
-    <joint name="${prefix}thumb_joint1" type="revolute">
+    <joint name="${prefix}thumb_joint1" type="${joint_type}">
       <origin xyz="-0.0269 ${dir*0.02101} 0.0334" />
       <parent link="${prefix}hand_base" />
@@ -131,5 +132,5 @@
       </collision>
     </link>
-    <joint name="${prefix}thumb_joint2" type="revolute">
+    <joint name="${prefix}thumb_joint2" type="${joint_type}">
       <origin xyz="-0.0079252 ${dir*0.0090599} 0.0052" rpy="${dir*1.5708} 0 ${dir*2.8798}" />
       <parent link="${prefix}thumb_1" />
@@ -161,5 +162,5 @@
       </collision>
     </link>
-    <joint name="${prefix}thumb_joint3" type="revolute">
+    <joint name="${prefix}thumb_joint3" type="${joint_type}">
       <origin xyz="0.031403 ${dir*0.021069} 0.00095" />
       <parent link="${prefix}thumb_2" />
@@ -226,5 +227,5 @@
       </collision>
     </link>
-    <joint name="${prefix}thumb_joint4" type="revolute">
+    <joint name="${prefix}thumb_joint4" type="${joint_type}">
       <origin xyz="0.021903 ${dir*0.012816} -0.0003" />
       <parent link="${prefix}thumb_3" />
@@ -353,5 +354,5 @@
       </collision>
     </link>
-    <joint name="${prefix}index_joint" type="revolute">
+    <joint name="${prefix}index_joint" type="${joint_type}">
       <origin xyz="-0.038679 ${dir*0.00056467} 0.1209" rpy="${dir*1.6057} 0 ${dir*-1.5708}" />
       <parent link="${prefix}hand_base" />
@@ -383,5 +384,5 @@
       </collision>
     </link>
-    <joint name="${prefix}index_dip" type="revolute">
+    <joint name="${prefix}index_dip" type="${joint_type}">
       <origin xyz="-0.0034259 ${dir*0.032596} -0.00055" />
       <parent link="${prefix}index_1" />
@@ -510,5 +511,5 @@
       </collision>
     </link>
-    <joint name="${prefix}middle_joint" type="revolute">
+    <joint name="${prefix}middle_joint" type="${joint_type}">
       <origin xyz="-0.0171 ${dir*0.00056467} 0.1215" rpy="${dir*1.5708} 0 ${dir*-1.5708}" />
       <parent link="${prefix}hand_base" />
@@ -543,5 +544,5 @@
       </collision>
     </link>
-    <joint name="${prefix}middle_dip" type="revolute">
+    <joint name="${prefix}middle_dip" type="${joint_type}">
       <origin xyz="-0.0034259 ${dir*0.032596} -0.00055" />
       <parent link="${prefix}middle_1" />
@@ -670,5 +671,5 @@
       </collision>
     </link>
-    <joint name="${prefix}ring_joint" type="revolute">
+    <joint name="${prefix}ring_joint" type="${joint_type}">
       <origin xyz="0.0045302 ${dir*0.00056467} 0.12133" rpy="${dir*1.5184} 0 ${dir*-1.5708}" />
       <parent link="${prefix}hand_base" />
@@ -700,5 +701,5 @@
       </collision>
     </link>
-    <joint name="${prefix}ring_dip" type="revolute">
+    <joint name="${prefix}ring_dip" type="${joint_type}">
       <origin xyz="-0.0034259 ${dir*0.032596} -0.00055" />
       <parent link="${prefix}ring_1" />
@@ -827,5 +828,5 @@
       </collision>
     </link>
-    <joint name="${prefix}pinky_joint" type="revolute">
+    <joint name="${prefix}pinky_joint" type="${joint_type}">
       <origin xyz="0.025916 ${dir*0.00056467} 0.11815" rpy="${dir*1.4661} 0 ${dir*-1.5708}" />
       <parent link="${prefix}hand_base" />
@@ -857,5 +858,5 @@
       </collision>
     </link>
-    <joint name="${prefix}pinky_dip" type="revolute">
+    <joint name="${prefix}pinky_dip" type="${joint_type}">
       <origin xyz="-0.0034259 ${dir*0.032596} -0.00055" />
       <parent link="${prefix}pinky_1" />
@@ -961,4 +962,10 @@
       <child link="${prefix}pinky_force_sensor_1" />
     </joint>
+    <link name="${prefix}eef"/>
+    <joint name="${prefix}eef_joint" type="fixed">
+      <parent link="${prefix}hand_base"/>
+      <child link="${prefix}eef"/>
+      <origin xyz="-0.017 ${dir*0.0006} 0.1015"/>
+    </joint>
   </xacro:macro>
 </robot>
