Commit message: 更新freedomv2

File: dexhands/freedom_description/xacro/freedomv2.xacro (robot description, xacro)
@@ -1,5 +1,5 @@
 <?xml version="1.0" encoding="utf-8"?>
 <robot xmlns:xacro="http://www.ros.org/wiki/xacro">
-	<xacro:macro name="FreedomHandV2" params="name direction:=1 fixed_joints:=false">
+	<xacro:macro name="FreedomHandV2" params="name direction:=1 fixed_joints:=false enable_dip_joints:=false">
 		<xacro:property name="prefix" value="${name + '_' if name else ''}"/>
 		<xacro:property name="joint_type" value="${fixed_joints and 'fixed' or 'revolute'}"/>
@@ -263,15 +263,20 @@
 				</collision>
 			</link>
-			<joint name="${prefix}index_dip" type="${joint_type}">
-				<origin xyz="0.032003 -0.0025 0" rpy="0 0 0.41015"/>
-				<parent link="${prefix}f_link2_2"/>
-				<child link="${prefix}f_link2_3"/>
-				<xacro:unless value="${fixed_joints}">
-					<axis xyz="0 0 1"/>
-				</xacro:unless>
-				<xacro:unless value="${fixed_joints}">
+				<xacro:if value="${enable_dip_joints}">
+				<joint name="${prefix}index_joint2" type="revolute">
+					<origin xyz="0.032003 -0.0025 0" rpy="0 0 0.41015"/>
+					<parent link="${prefix}f_link2_2"/>
+					<child link="${prefix}f_link2_3"/>
+					<axis xyz="0 0 1"/>
 					<limit lower="0" upper="1.204" effort="10" velocity="1.5"/>
-				</xacro:unless>
-			</joint>
+				</joint>
+				</xacro:if>
+				<xacro:unless value="${enable_dip_joints}">
+				<joint name="${prefix}index_dip" type="fixed">
+					<origin xyz="0.032003 -0.0025 0" rpy="0 0 0.41015"/>
+					<parent link="${prefix}f_link2_2"/>
+					<child link="${prefix}f_link2_3"/>
+				</joint>
+				</xacro:unless>
 			<link name="${prefix}f_link3_1">
 				<inertial>
@@ -356,15 +361,20 @@
 				</collision>
 			</link>
-			<joint name="${prefix}middle_dip" type="${joint_type}">
-				<origin xyz="0.032003 -0.0025 0" rpy="0 0 0.41015"/>
-				<parent link="${prefix}f_link3_2"/>
-				<child link="${prefix}f_link3_3"/>
-				<xacro:unless value="${fixed_joints}">
-					<axis xyz="0 0 1"/>
-				</xacro:unless>
-				<xacro:unless value="${fixed_joints}">
+				<xacro:if value="${enable_dip_joints}">
+				<joint name="${prefix}middle_joint2" type="revolute">
+					<origin xyz="0.032003 -0.0025 0" rpy="0 0 0.41015"/>
+					<parent link="${prefix}f_link3_2"/>
+					<child link="${prefix}f_link3_3"/>
+					<axis xyz="0 0 1"/>
 					<limit lower="0" upper="1.204" effort="10" velocity="1.5"/>
-				</xacro:unless>
-			</joint>
+				</joint>
+				</xacro:if>
+				<xacro:unless value="${enable_dip_joints}">
+				<joint name="${prefix}middle_dip" type="fixed">
+					<origin xyz="0.032003 -0.0025 0" rpy="0 0 0.41015"/>
+					<parent link="${prefix}f_link3_2"/>
+					<child link="${prefix}f_link3_3"/>
+				</joint>
+				</xacro:unless>
 			<link name="${prefix}f_link4_1">
 				<inertial>
@@ -803,15 +813,20 @@
 				</collision>
 			</link>
-			<joint name="${prefix}index_dip" type="${joint_type}">
-				<origin xyz="0.032002535301686 -0.00250000000000612 0" rpy="0 0 0.410152374218668"/>
-				<parent link="${prefix}f_link2_2"/>
-				<child link="${prefix}f_link2_3"/>
-				<xacro:unless value="${fixed_joints}">
-					<axis xyz="0 0 1"/>
-				</xacro:unless>
-				<xacro:unless value="${fixed_joints}">
+				<xacro:if value="${enable_dip_joints}">
+				<joint name="${prefix}index_joint2" type="revolute">
+					<origin xyz="0.032002535301686 -0.00250000000000612 0" rpy="0 0 0.410152374218668"/>
+					<parent link="${prefix}f_link2_2"/>
+					<child link="${prefix}f_link2_3"/>
+					<axis xyz="0 0 1"/>
 					<limit lower="0" upper="1.204" effort="10" velocity="1.5"/>
-				</xacro:unless>
-			</joint>
+				</joint>
+				</xacro:if>
+				<xacro:unless value="${enable_dip_joints}">
+				<joint name="${prefix}index_dip" type="fixed">
+					<origin xyz="0.032002535301686 -0.00250000000000612 0" rpy="0 0 0.410152374218668"/>
+					<parent link="${prefix}f_link2_2"/>
+					<child link="${prefix}f_link2_3"/>
+				</joint>
+				</xacro:unless>
 			<link name="${prefix}f_link3_1">
 				<inertial>
@@ -896,15 +911,20 @@
 				</collision>
 			</link>
-			<joint name="${prefix}middle_dip" type="${joint_type}">
-				<origin xyz="0.0320025353016867 -0.00250000000000624 0" rpy="0 0 0.410152374218668"/>
-				<parent link="${prefix}f_link3_2"/>
-				<child link="${prefix}f_link3_3"/>
-				<xacro:unless value="${fixed_joints}">
-					<axis xyz="0 0 1"/>
-				</xacro:unless>
-				<xacro:unless value="${fixed_joints}">
+				<xacro:if value="${enable_dip_joints}">
+				<joint name="${prefix}middle_joint2" type="revolute">
+					<origin xyz="0.0320025353016867 -0.00250000000000624 0" rpy="0 0 0.410152374218668"/>
+					<parent link="${prefix}f_link3_2"/>
+					<child link="${prefix}f_link3_3"/>
+					<axis xyz="0 0 1"/>
 					<limit lower="0" upper="1.204" effort="10" velocity="1.5"/>
-				</xacro:unless>
-			</joint>
+				</joint>
+				</xacro:if>
+				<xacro:unless value="${enable_dip_joints}">
+				<joint name="${prefix}middle_dip" type="fixed">
+					<origin xyz="0.0320025353016867 -0.00250000000000624 0" rpy="0 0 0.410152374218668"/>
+					<parent link="${prefix}f_link3_2"/>
+					<child link="${prefix}f_link3_3"/>
+				</joint>
+				</xacro:unless>
 			<link name="${prefix}f_link4_1">
 				<inertial>

File: dexhands/freedom_description/xacro/hand.xacro (robot description, xacro)
@@ -3,4 +3,5 @@
 	<xacro:arg name="type" default="freedomv2"/>
 	<xacro:arg name="direction" default="1"/>
+	<xacro:arg name="enable_dip_joints" default="false"/>
 	<xacro:if value="${'$(arg type)' == 'freedomv1' or '$(arg type)' == 'freedom_v1' or '$(arg type)' == 'freedom'}">
 		<xacro:include filename="$(find freedom_description)/xacro/freedomv1.xacro"/>
@@ -9,5 +10,5 @@
 	<xacro:if value="${'$(arg type)' == 'freedomv2' or '$(arg type)' == 'freedom_v2'}">
 		<xacro:include filename="$(find freedom_description)/xacro/freedomv2.xacro"/>
-		<xacro:FreedomHandV2 name="" direction="$(arg direction)"/>
+		<xacro:FreedomHandV2 name="" direction="$(arg direction)" enable_dip_joints="$(arg enable_dip_joints)"/>
 	</xacro:if>
 </robot>

File: dexhands/freedom_description/xacro/ros2_control/freedomv2.xacro (robot description, xacro)
@@ -35,21 +35,5 @@
       <state_interface name="effort"/>
     </joint>
-    <joint name="${prefix}index_dip">
-      <command_interface name="position"/>
-      <state_interface name="position">
-        <param name="initial_value">0.0</param>
-      </state_interface>
-      <state_interface name="velocity"/>
-      <state_interface name="effort"/>
-    </joint>
     <joint name="${prefix}middle_joint">
-      <command_interface name="position"/>
-      <state_interface name="position">
-        <param name="initial_value">0.0</param>
-      </state_interface>
-      <state_interface name="velocity"/>
-      <state_interface name="effort"/>
-    </joint>
-    <joint name="${prefix}middle_dip">
       <command_interface name="position"/>
       <state_interface name="position">

Commit message: 修正marker

File: dexhands/freedom_description/xacro/freedomv2.xacro (robot description, xacro)
@@ -1104,4 +1104,10 @@
 			</joint>
 		</xacro:unless>
+		<link name="${prefix}eef"/>
+		<joint name="${prefix}eef_joint" type="fixed">
+			<parent link="${prefix}hand_base"/>
+			<child link="${prefix}eef"/>
+			<origin xyz="0.02 0 0.07"/>
+		</joint>
 	</xacro:macro>
 </robot>

Commit message: Add configuration files for Freedom V1 and update Freedom V2 parameters

File: dexhands/freedom_description/xacro/freedomv2.xacro (robot description, xacro)
@@ -82,5 +82,5 @@
 				<child link="${prefix}f_link1_1"/>
 				<xacro:unless value="${fixed_joints}">
-					<axis xyz="0 0 1"/>
+					<axis xyz="0 0 -1"/>
 				</xacro:unless>
 				<xacro:unless value="${fixed_joints}">
