Commit message: refactor freedom hand

File: dexhands/freedom_description/xacro/freedomv2.xacro (robot description, xacro)
@@ -1,1107 +1,486 @@
 <?xml version="1.0" encoding="utf-8"?>
 <robot xmlns:xacro="http://www.ros.org/wiki/xacro">
-	<xacro:macro name="FreedomHandV2" params="name direction:=1 fixed_joints:=false enable_dip_joints:=false">
+	<xacro:macro name="FreedomHandV2" params="name direction:=1 fixed_joints:=false">
 		<xacro:property name="prefix" value="${name + '_' if name else ''}"/>
 		<xacro:property name="joint_type" value="${fixed_joints and 'fixed' or 'revolute'}"/>
-		<xacro:if value="${direction == 1}">
-			<link name="${prefix}hand_base">
-				<inertial>
-					<origin xyz="1.72456639246921E-10 0.000159743547726118 0.00658240409197629" rpy="0 0 0"/>
-					<mass value="0.0176998254464378"/>
-					<inertia ixx="4.77814014865034E-06" ixy="-2.8287088790031E-15" ixz="-1.75792865725827E-14" iyy="4.84927762663746E-06" iyz="4.47414433687868E-09" izz="9.23717647630549E-06"/>
-				</inertial>
-				<visual>
-					<origin xyz="0 0 0" rpy="0 0 0"/>
-					<geometry>
-						<mesh filename="file://$(find freedom_description)/meshes/freedomv2/base.glb" scale="1 ${direction} 1"/>
-					</geometry>
-					<material name="">
-						<color rgba="0.752941176470588 1 0.752941176470588 1"/>
-					</material>
-				</visual>
-				<collision>
-					<origin xyz="0 0 0" rpy="0 0 0"/>
-					<geometry>
-						<mesh filename="file://$(find freedom_description)/meshes/freedomv2/base.glb" scale="1 ${direction} 1"/>
-					</geometry>
-				</collision>
-			</link>
-			<link name="${prefix}p_link1">
-				<inertial>
-					<origin xyz="-0.000806915097715849 0.00388610492404486 0.0525721443155858" rpy="0 0 0"/>
-					<mass value="3.09350498281211"/>
-					<inertia ixx="0.00483124658726801" ixy="-0.000120079243984059" ixz="2.7699838991495E-05" iyy="0.00363360625618824" iyz="0.000130624066360049" izz="0.00244702121245661"/>
-				</inertial>
-				<visual>
-					<origin xyz="0 0 0" rpy="0 0 0"/>
-					<geometry>
-						<mesh filename="file://$(find freedom_description)/meshes/freedomv2/l_p_link1.glb" scale="1 ${direction} 1"/>
-					</geometry>
-					<material name="">
-						<color rgba="0.529411764705882 0.549019607843137 0.549019607843137 1"/>
-					</material>
-				</visual>
-				<collision>
-					<origin xyz="0 0 0" rpy="0 0 0"/>
-					<geometry>
-						<mesh filename="file://$(find freedom_description)/meshes/freedomv2/l_p_link1.glb" scale="1 ${direction} 1"/>
-					</geometry>
-				</collision>
-			</link>
-			<joint name="${prefix}p_joint1" type="fixed">
-				<origin xyz="0 0 0.00899999999999999" rpy="0 0 0"/>
-				<parent link="${prefix}hand_base"/>
-				<child link="${prefix}p_link1"/>
-				<axis xyz="0 0 0"/>
-			</joint>
-			<link name="${prefix}f_link1_1">
-				<inertial>
-					<origin xyz="0.00145106672278547 0.000219751119078359 -0.000948786433616551" rpy="0 0 0"/>
-					<mass value="0.02293794994852"/>
-					<inertia ixx="1.34683661171916E-06" ixy="-2.07744949992747E-08" ixz="7.89788182035335E-08" iyy="1.55245577209657E-06" iyz="2.67848599029428E-08" izz="1.3933432603089E-06"/>
-				</inertial>
-				<visual>
-					<origin xyz="0 0 0" rpy="0 0 0"/>
-					<geometry>
-						<mesh filename="file://$(find freedom_description)/meshes/freedomv2/l_f_link1_1.glb" scale="1 1 ${direction}"/>
-					</geometry>
-					<material name="">
-						<color rgba="0.529411764705882 0.549019607843137 0.549019607843137 1"/>
-					</material>
-				</visual>
-				<collision>
-					<origin xyz="0 0 0" rpy="0 0 0"/>
-					<geometry>
-						<mesh filename="file://$(find freedom_description)/meshes/freedomv2/l_f_link1_1.glb" scale="1 1 ${direction}"/>
-					</geometry>
-				</collision>
-			</link>
-			<joint name="${prefix}thumb_joint1" type="${joint_type}">
-				<origin xyz="0.0019629 -0.02666 0.037173" rpy="-1.571 -0.001553 3.0223E-05"/>
-				<parent link="${prefix}p_link1"/>
-				<child link="${prefix}f_link1_1"/>
-				<xacro:unless value="${fixed_joints}">
-					<axis xyz="0 0 -1"/>
-				</xacro:unless>
-				<xacro:unless value="${fixed_joints}">
-					<limit lower="-0.4363" upper="0.43663" effort="10" velocity="1.5"/>
-				</xacro:unless>
-			</joint>
-			<link name="${prefix}f_link1_2">
-				<inertial>
-					<origin xyz="-0.017447784563969 0.0315995831691795 0.0162963928618926" rpy="0 0 0"/>
-					<mass value="0.341617867410056"/>
-					<inertia ixx="0.00012471975596469" ixy="2.83491215843258E-05" ixz="2.24006738785496E-05" iyy="8.89744452481692E-05" iyz="-4.06096513108848E-05" izz="9.75750752172789E-05"/>
-				</inertial>
-				<visual>
-					<origin xyz="0 0 0" rpy="0 0 0"/>
-					<geometry>
-						<mesh filename="file://$(find freedom_description)/meshes/freedomv2/l_f_link1_2.glb" scale="1 ${direction} 1"/>
-					</geometry>
-					<material name="">
-						<color rgba="0.529411764705882 0.549019607843137 0.549019607843137 1"/>
-					</material>
-				</visual>
-				<collision>
-					<origin xyz="0 0 0" rpy="0 0 0"/>
-					<geometry>
-						<mesh filename="file://$(find freedom_description)/meshes/freedomv2/l_f_link1_2.glb" scale="1 ${direction} 1"/>
-					</geometry>
-				</collision>
-			</link>
-			<joint name="${prefix}thumb_joint2" type="${joint_type}">
-				<origin xyz="0.010999 0 -0.001747" rpy="-1.5711 0 -3.1415"/>
-				<parent link="${prefix}f_link1_1"/>
-				<child link="${prefix}f_link1_2"/>
-				<xacro:unless value="${fixed_joints}">
-					<axis xyz="0 0 1"/>
-				</xacro:unless>
-				<xacro:unless value="${fixed_joints}">
-					<limit lower="0" upper="1.3786" effort="10" velocity="1.5"/>
-				</xacro:unless>
-			</joint>
-			<link name="${prefix}f_link1_3">
-				<inertial>
-					<origin xyz="0.013123608617489 -0.00699497111386572 -6.46545186624992E-08" rpy="0 0 0"/>
-					<mass value="0.0787286292541374"/>
-					<inertia ixx="4.50761163538385E-06" ixy="-6.41462388372337E-07" ixz="3.09811891080126E-12" iyy="7.81743380936836E-06" iyz="1.33295168138201E-10" izz="7.87624932256717E-06"/>
-				</inertial>
-				<visual>
-					<origin xyz="0 0 0" rpy="0 0 0"/>
-					<geometry>
-						<mesh filename="file://$(find freedom_description)/meshes/freedomv2/l_f_link1_3.glb" scale="1 1 ${direction}"/>
-					</geometry>
-					<material name="">
-						<color rgba="0.529411764705882 0.549019607843137 0.549019607843137 1"/>
-					</material>
-				</visual>
-				<collision>
-					<origin xyz="0 0 0" rpy="0 0 0"/>
-					<geometry>
-						<mesh filename="file://$(find freedom_description)/meshes/freedomv2/l_f_link1_3.glb" scale="1 1 ${direction}"/>
-					</geometry>
-				</collision>
-			</link>
-			<joint name="${prefix}thumb_joint3" type="${joint_type}">
-				<origin xyz="-0.027292 0.049447 0.045113" rpy="1.5708 -0.97827 2.0748"/>
-				<parent link="${prefix}f_link1_2"/>
-				<child link="${prefix}f_link1_3"/>
-				<xacro:unless value="${fixed_joints}">
-					<axis xyz="0 0 1"/>
-				</xacro:unless>
-				<xacro:unless value="${fixed_joints}">
-					<limit lower="0" upper="0.4537" effort="10" velocity="1.5"/>
-				</xacro:unless>
-			</joint>
-			<link name="${prefix}f_link1_4">
-				<inertial>
-					<origin xyz="0.013033714511231 0.00392466488779568 4.57210278786285E-08" rpy="0 0 0"/>
-					<mass value="0.0492559822656011"/>
-					<inertia ixx="1.83221974234297E-06" ixy="-2.92043601142965E-08" ixz="-1.24987758450123E-11" iyy="4.14827361187538E-06" iyz="-1.84821856863993E-13" izz="3.86182170639597E-06"/>
-				</inertial>
-				<visual>
-					<origin xyz="0 0 0" rpy="0 0 0"/>
-					<geometry>
-						<mesh filename="file://$(find freedom_description)/meshes/freedomv2/l_f_link1_4.glb" scale="1 1 ${direction}"/>
-					</geometry>
-					<material name="">
-						<color rgba="0.529411764705882 0.549019607843137 0.549019607843137 1"/>
-					</material>
-				</visual>
-				<collision>
-					<origin xyz="0 0 0" rpy="0 0 0"/>
-					<geometry>
-						<mesh filename="file://$(find freedom_description)/meshes/freedomv2/l_f_link1_4.glb" scale="1 1 ${direction}"/>
-					</geometry>
-				</collision>
-			</link>
-			<joint name="${prefix}thumb_dip" type="fixed">
-				<origin xyz="0.030304 -0.0075957 0" rpy="0 0 0.31426"/>
-				<parent link="${prefix}f_link1_3"/>
-				<child link="${prefix}f_link1_4"/>
-			</joint>
-			<link name="${prefix}f_link2_1">
-				<inertial>
-					<origin xyz="0.00431549531692989 -3.59544548608464E-05 -0.000293519581500933" rpy="0 0 0"/>
-					<mass value="0.01220067525638"/>
-					<inertia ixx="1.76157556392802E-07" ixy="-1.18013880311655E-11" ixz="5.1258189712677E-08" iyy="6.86901221323969E-07" iyz="-5.70496565074483E-13" izz="6.04592917607103E-07"/>
-				</inertial>
-				<visual>
-					<origin xyz="0 0 0" rpy="0 0 0"/>
-					<geometry>
-						<mesh filename="file://$(find freedom_description)/meshes/freedomv2/f_f_link2_1.glb" scale="1 1 ${direction}"/>
-					</geometry>
-					<material name="">
-						<color rgba="0.529411764705882 0.549019607843137 0.549019607843137 1"/>
-					</material>
-				</visual>
-				<collision>
-					<origin xyz="0 0 0" rpy="0 0 0"/>
-					<geometry>
-						<mesh filename="file://$(find freedom_description)/meshes/freedomv2/f_f_link2_1.glb" scale="1 1 ${direction}"/>
-					</geometry>
-				</collision>
-			</link>
-			<joint name="${prefix}index_spread" type="fixed">
-				<origin xyz="-0.00116057224596555 -0.0307705379422379 0.115175208614826" rpy="-0.672265009864131 -1.57073156717295 -2.46932794060801"/>
-				<parent link="${prefix}p_link1"/>
-				<child link="${prefix}f_link2_1"/>
-			</joint>
-			<link name="${prefix}f_link2_2">
-				<inertial>
-					<origin xyz="0.0104118354940718 0.000536686610708395 -1.76713780610308E-07" rpy="0 0 0"/>
-					<mass value="0.0784310054995946"/>
-					<inertia ixx="3.68968904398224E-06" ixy="3.62846908118645E-07" ixz="2.16090077515739E-10" iyy="1.11655087077302E-05" iyz="-8.17126072387152E-11" izz="1.11880378622959E-05"/>
-				</inertial>
-				<visual>
-					<origin xyz="0 0 0" rpy="0 0 0"/>
-					<geometry>
-						<mesh filename="file://$(find freedom_description)/meshes/freedomv2/f_f_link2_2.glb" scale="1 1 ${direction}"/>
-					</geometry>
-					<material name="">
-						<color rgba="0.792156862745098 0.819607843137255 0.933333333333333 1"/>
-					</material>
-				</visual>
-				<collision>
-					<origin xyz="0 0 0" rpy="0 0 0"/>
-					<geometry>
-						<mesh filename="file://$(find freedom_description)/meshes/freedomv2/f_f_link2_2.glb" scale="1 1 ${direction}"/>
-					</geometry>
-				</collision>
-			</link>
-			<joint name="${prefix}index_joint" type="${joint_type}">
-				<origin xyz="0.007 0 0.0021" rpy="1.5708 0 0"/>
-				<parent link="${prefix}f_link2_1"/>
-				<child link="${prefix}f_link2_2"/>
-				<xacro:unless value="${fixed_joints}">
-					<axis xyz="0 0 1"/>
-				</xacro:unless>
-				<xacro:unless value="${fixed_joints}">
-					<limit lower="0" upper="1.396" effort="10" velocity="1.5"/>
-				</xacro:unless>
-			</joint>
-			<link name="${prefix}f_link2_3">
-				<inertial>
-					<origin xyz="0.0254085981069671 0.00100288167736774 -1.01039098981967E-05" rpy="0 0 0"/>
-					<mass value="0.041685911200702"/>
-					<inertia ixx="1.69093305742986E-06" ixy="1.39625672092217E-06" ixz="-5.80269118862188E-09" iyy="1.03628643235447E-05" iyz="1.23011708787116E-09" izz="1.02474973432913E-05"/>
-				</inertial>
-				<visual>
-					<origin xyz="0 0 0" rpy="0 0 0"/>
-					<geometry>
-						<mesh filename="file://$(find freedom_description)/meshes/freedomv2/f_f_link2_3.glb" scale="1 1 ${direction}"/>
-					</geometry>
-					<material name="">
-						<color rgba="0.792156862745098 0.819607843137255 0.933333333333333 1"/>
-					</material>
-				</visual>
-				<collision>
-					<origin xyz="0 0 0" rpy="0 0 0"/>
-					<geometry>
-						<mesh filename="file://$(find freedom_description)/meshes/freedomv2/f_f_link2_3.glb" scale="1 1 ${direction}"/>
-					</geometry>
-				</collision>
-			</link>
-				<xacro:if value="${enable_dip_joints}">
-				<joint name="${prefix}index_joint2" type="revolute">
-					<origin xyz="0.032003 -0.0025 0" rpy="0 0 0.41015"/>
-					<parent link="${prefix}f_link2_2"/>
-					<child link="${prefix}f_link2_3"/>
-					<axis xyz="0 0 1"/>
-					<limit lower="0" upper="1.204" effort="10" velocity="1.5"/>
-				</joint>
-				</xacro:if>
-				<xacro:unless value="${enable_dip_joints}">
-				<joint name="${prefix}index_dip" type="fixed">
-					<origin xyz="0.032003 -0.0025 0" rpy="0 0 0.41015"/>
-					<parent link="${prefix}f_link2_2"/>
-					<child link="${prefix}f_link2_3"/>
-				</joint>
-				</xacro:unless>
-			<link name="${prefix}f_link3_1">
-				<inertial>
-					<origin xyz="0.00431549531692993 -3.59544548608516E-05 -0.000293519581500951" rpy="0 0 0"/>
-					<mass value="0.01220067525638"/>
-					<inertia ixx="1.76157556392802E-07" ixy="-1.18013880316246E-11" ixz="5.12581897126789E-08" iyy="6.86901221323972E-07" iyz="-5.70496565048013E-13" izz="6.04592917607106E-07"/>
-				</inertial>
-				<visual>
-					<origin xyz="0 0 0" rpy="0 0 0"/>
-					<geometry>
-						<mesh filename="file://$(find freedom_description)/meshes/freedomv2/f_f_link2_1.glb" scale="1 1 ${direction}"/>
-					</geometry>
-					<material name="">
-						<color rgba="0.529411764705882 0.549019607843137 0.549019607843137 1"/>
-					</material>
-				</visual>
-				<collision>
-					<origin xyz="0 0 0" rpy="0 0 0"/>
-					<geometry>
-						<mesh filename="file://$(find freedom_description)/meshes/freedomv2/f_f_link2_1.glb" scale="1 1 ${direction}"/>
-					</geometry>
-				</collision>
-			</link>
-			<joint name="${prefix}middle_spread" type="fixed">
-				<origin xyz="-0.0011607 -0.0087207 0.11685" rpy="-0.67227 -1.5707 -2.4693"/>
-				<parent link="${prefix}p_link1"/>
-				<child link="${prefix}f_link3_1"/>
-			</joint>
-			<link name="${prefix}f_link3_2">
-				<inertial>
-					<origin xyz="0.0104118354940713 0.000536686610708512 -1.76713780695309E-07" rpy="0 0 0"/>
-					<mass value="0.0784310054995923"/>
-					<inertia ixx="3.68968904398217E-06" ixy="3.62846908118472E-07" ixz="2.16090077641213E-10" iyy="1.11655087077294E-05" iyz="-8.17126072565028E-11" izz="1.1188037862295E-05"/>
-				</inertial>
-				<visual>
-					<origin xyz="0 0 0" rpy="0 0 0"/>
-					<geometry>
-						<mesh filename="file://$(find freedom_description)/meshes/freedomv2/f_f_link2_2.glb" scale="1 1 ${direction}"/>
-					</geometry>
-					<material name="">
-						<color rgba="0.792156862745098 0.819607843137255 0.933333333333333 1"/>
-					</material>
-				</visual>
-				<collision>
-					<origin xyz="0 0 0" rpy="0 0 0"/>
-					<geometry>
-						<mesh filename="file://$(find freedom_description)/meshes/freedomv2/f_f_link2_2.glb" scale="1 1 ${direction}"/>
-					</geometry>
-				</collision>
-			</link>
-			<joint name="${prefix}middle_joint" type="${joint_type}">
-				<origin xyz="0.007 0 0.0021" rpy="1.5708 0 0"/>
-				<parent link="${prefix}f_link3_1"/>
-				<child link="${prefix}f_link3_2"/>
-				<xacro:unless value="${fixed_joints}">
-					<axis xyz="0 0 1"/>
-				</xacro:unless>
-				<xacro:unless value="${fixed_joints}">
-					<limit lower="0" upper="1.396" effort="10" velocity="1.5"/>
-				</xacro:unless>
-			</joint>
-			<link name="${prefix}f_link3_3">
-				<inertial>
-					<origin xyz="0.025409 0.0010029 -1.0077E-05" rpy="0 0 0"/>
-					<mass value="0.041686"/>
-					<inertia ixx="1.6909E-06" ixy="1.3963E-06" ixz="-5.8025E-09" iyy="1.0363E-05" iyz="1.2305E-09" izz="1.0248E-05"/>
-				</inertial>
-				<visual>
-					<origin xyz="0 0 0" rpy="0 0 0"/>
-					<geometry>
-						<mesh filename="file://$(find freedom_description)/meshes/freedomv2/f_f_link2_3.glb" scale="1 1 ${direction}"/>
-					</geometry>
-					<material name="">
-						<color rgba="0.79216 0.81961 0.93333 1"/>
-					</material>
-				</visual>
-				<collision>
-					<origin xyz="0 0 0" rpy="0 0 0"/>
-					<geometry>
-						<mesh filename="file://$(find freedom_description)/meshes/freedomv2/f_f_link2_3.glb" scale="1 1 ${direction}"/>
-					</geometry>
-				</collision>
-			</link>
-				<xacro:if value="${enable_dip_joints}">
-				<joint name="${prefix}middle_joint2" type="revolute">
-					<origin xyz="0.032003 -0.0025 0" rpy="0 0 0.41015"/>
-					<parent link="${prefix}f_link3_2"/>
-					<child link="${prefix}f_link3_3"/>
-					<axis xyz="0 0 1"/>
-					<limit lower="0" upper="1.204" effort="10" velocity="1.5"/>
-				</joint>
-				</xacro:if>
-				<xacro:unless value="${enable_dip_joints}">
-				<joint name="${prefix}middle_dip" type="fixed">
-					<origin xyz="0.032003 -0.0025 0" rpy="0 0 0.41015"/>
-					<parent link="${prefix}f_link3_2"/>
-					<child link="${prefix}f_link3_3"/>
-				</joint>
-				</xacro:unless>
-			<link name="${prefix}f_link4_1">
-				<inertial>
-					<origin xyz="0.00431549531692992 -3.5954454860869E-05 -0.000293519581500958" rpy="0 0 0"/>
-					<mass value="0.01220067525638"/>
-					<inertia ixx="1.76157556392802E-07" ixy="-1.18013880314418E-11" ixz="5.12581897126789E-08" iyy="6.86901221323973E-07" iyz="-5.70496565100953E-13" izz="6.04592917607107E-07"/>
-				</inertial>
-				<visual>
-					<origin xyz="0 0 0" rpy="0 0 0"/>
-					<geometry>
-						<mesh filename="file://$(find freedom_description)/meshes/freedomv2/f_f_link2_1.glb" scale="1 1 ${direction}"/>
-					</geometry>
-					<material name="">
-						<color rgba="0.529411764705882 0.549019607843137 0.549019607843137 1"/>
-					</material>
-				</visual>
-				<collision>
-					<origin xyz="0 0 0" rpy="0 0 0"/>
-					<geometry>
-						<mesh filename="file://$(find freedom_description)/meshes/freedomv2/f_f_link2_1.glb" scale="1 1 ${direction}"/>
-					</geometry>
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
File: dexhands/freedom_description/xacro/hand.xacro (robot description, xacro)
@@ -3,5 +3,4 @@
 	<xacro:arg name="type" default="freedomv2"/>
 	<xacro:arg name="direction" default="1"/>
-	<xacro:arg name="enable_dip_joints" default="false"/>
 	<xacro:if value="${'$(arg type)' == 'freedomv1' or '$(arg type)' == 'freedom_v1' or '$(arg type)' == 'freedom'}">
 		<xacro:include filename="$(find freedom_description)/xacro/freedomv1.xacro"/>
@@ -10,5 +9,5 @@
 	<xacro:if value="${'$(arg type)' == 'freedomv2' or '$(arg type)' == 'freedom_v2'}">
 		<xacro:include filename="$(find freedom_description)/xacro/freedomv2.xacro"/>
-		<xacro:FreedomHandV2 name="" direction="$(arg direction)" enable_dip_joints="$(arg enable_dip_joints)"/>
+		<xacro:FreedomHandV2 name="" direction="$(arg direction)"/>
 	</xacro:if>
 </robot>
