Commit message: fix mimic problem

File: gripper/changingtek_description/xacro/AG2F120S.xacro (robot description, xacro)
@@ -176,5 +176,5 @@
       <axis xyz="0 0 -1"/>
       <limit lower="0" upper="1" effort="40"  velocity="${4*PI/3}"/>
-      <mimic joint="${prefix}left_2_joint" multiplier="1" offset="0"/>
+      <mimic joint="${prefix}gripper_joint" multiplier="1" offset="0"/>
     </joint>
     <link name="${prefix}right_1_link">
@@ -238,5 +238,5 @@
       <axis xyz="0 0 1"/>
       <limit lower="0" upper="1" effort="40"  velocity="${4*PI/3}"/>
-      <mimic joint="${prefix}right_1_joint" multiplier="1" offset="0"/>
+      <mimic joint="${prefix}gripper_joint" multiplier="1" offset="0"/>
     </joint>
     <link name="${prefix}right_pad_link">

File: gripper/changingtek_description/xacro/AG2F90-C.xacro (robot description, xacro)
@@ -264,5 +264,5 @@
 			<axis xyz="1 0 0"/>
 			<limit lower="0" upper="1" effort="50" velocity="${PI}"/>
-			<mimic joint="${prefix}left_2_Joint"/>
+			<mimic joint="${prefix}gripper_joint"/>
 		</joint>
 		<link name="${prefix}right_1_link">
@@ -326,5 +326,5 @@
 			<axis xyz="-1 0 0"/>
 			<limit lower="0" upper="1" effort="50" velocity="${PI}"/>
-			<mimic joint="${prefix}right_1_Joint" multiplier="0.1" offset="0"/>
+			<mimic joint="${prefix}gripper_joint" multiplier="0.1" offset="0"/>
 		</joint>
 		<link name="${prefix}right_up_link">
@@ -357,5 +357,5 @@
 			<axis xyz="-1 0 0"/>
 			<limit lower="0" upper="1" effort="50" velocity="${PI}"/>
-			<mimic joint="${prefix}right_1_Joint"/>
+			<mimic joint="${prefix}gripper_joint"/>
 		</joint>
 		<xacro:if value="${pad == 'soft'}">

Commit message: adapt more robots

File: gripper/changingtek_description/xacro/AG2F120S.xacro (robot description, xacro)
@@ -1,7 +1,8 @@
 <?xml version="1.0" ?>
 <robot xmlns:xacro="http://ros.org/wiki/xacro">
-  <xacro:macro name="AG2F120S" params="name">
+  <xacro:macro name="AG2F120S" params="name kinematic_only:=false">
     <xacro:property name="prefix" value="${name + '_' if name else ''}"/>
     <xacro:property name="PI" value="3.1415926535897931"/>
+    <xacro:property name="joint_type" value="${kinematic_only and 'fixed' or 'revolute'}"/>
     <link name="${prefix}gripper_base">
       <inertial>
@@ -50,10 +51,12 @@
       </collision>
     </link>
-    <joint name="${prefix}gripper_joint" type="revolute">
+    <joint name="${prefix}gripper_joint" type="${joint_type}">
       <origin xyz="-0.032553 0 0.10644" rpy="${PI/2} 0 ${PI}"/>
       <parent link="${prefix}gripper_base"/>
       <child link="${prefix}left_1_link"/>
-      <axis xyz="0 0 -1"/>
-      <limit lower="0" upper="1" effort="40" velocity="${4*PI/3}"/>
+      <xacro:unless value="${kinematic_only}">
+        <axis xyz="0 0 -1"/>
+        <limit lower="0" upper="1" effort="40" velocity="${4*PI/3}"/>
+      </xacro:unless>
     </joint>
     <link name="${prefix}left_support_link">
@@ -80,11 +83,13 @@
       </collision>
     </link>
-    <joint name="${prefix}left_support_joint" type="revolute">
+    <joint name="${prefix}left_support_joint" type="${joint_type}">
       <origin xyz="-0.0093594 0.056229 0"/>
       <parent link="${prefix}left_1_link"/>
       <child link="${prefix}left_support_link"/>
-      <axis xyz="0 0 1"/>
-      <limit lower="0" upper="1" effort="40"  velocity="${4*PI/3}"/>
-      <mimic joint="${prefix}gripper_joint" multiplier="1" offset="0"/>
+      <xacro:unless value="${kinematic_only}">
+        <axis xyz="0 0 1"/>
+        <limit lower="0" upper="1" effort="40"  velocity="${4*PI/3}"/>
+        <mimic joint="${prefix}gripper_joint" multiplier="1" offset="0"/>
+      </xacro:unless>
     </joint>
     <link name="${prefix}left_pad_link">
@@ -139,11 +144,13 @@
       </collision>
     </link>
-    <joint name="${prefix}left_2_joint" type="revolute">
+    <joint name="${prefix}left_2_joint" type="${joint_type}">
       <origin xyz="-0.017 0 0.122" rpy="${PI/2} 0 ${PI}"/>
       <parent link="${prefix}gripper_base"/>
       <child link="${prefix}left_2_link"/>
-      <axis xyz="0 0 -1"/>
-      <limit lower="0" upper="1" effort="40"  velocity="${4*PI/3}"/>
-      <mimic joint="${prefix}gripper_joint" multiplier="1" offset="0"/>
+      <xacro:unless value="${kinematic_only}">
+        <axis xyz="0 0 -1"/>
+        <limit lower="0" upper="1" effort="40"  velocity="${4*PI/3}"/>
+        <mimic joint="${prefix}gripper_joint" multiplier="1" offset="0"/>
+      </xacro:unless>
     </joint>
     <link name="${prefix}right_2_link">
@@ -170,11 +177,13 @@
       </collision>
     </link>
-    <joint name="${prefix}right_2_joint" type="revolute">
+    <joint name="${prefix}right_2_joint" type="${joint_type}">
       <origin xyz="0.017 0 0.122" rpy="${PI/2} 0 0"/>
       <parent link="${prefix}gripper_base"/>
       <child link="${prefix}right_2_link"/>
-      <axis xyz="0 0 -1"/>
-      <limit lower="0" upper="1" effort="40"  velocity="${4*PI/3}"/>
-      <mimic joint="${prefix}gripper_joint" multiplier="1" offset="0"/>
+      <xacro:unless value="${kinematic_only}">
+        <axis xyz="0 0 -1"/>
+        <limit lower="0" upper="1" effort="40"  velocity="${4*PI/3}"/>
+        <mimic joint="${prefix}gripper_joint" multiplier="1" offset="0"/>
+      </xacro:unless>
     </joint>
     <link name="${prefix}right_1_link">
@@ -201,11 +210,13 @@
       </collision>
     </link>
-    <joint name="${prefix}right_1_joint" type="revolute">
+    <joint name="${prefix}right_1_joint" type="${joint_type}">
       <origin xyz="0.032553 0 0.10644" rpy="${PI/2} 0 0"/>
       <parent link="${prefix}gripper_base"/>
       <child link="${prefix}right_1_link"/>
-      <axis xyz="0 0 -1"/>
-      <limit lower="0" upper="1" effort="40"  velocity="${4*PI/3}"/>
-      <mimic joint="${prefix}gripper_joint" multiplier="1" offset="0"/>
+      <xacro:unless value="${kinematic_only}">
+        <axis xyz="0 0 -1"/>
+        <limit lower="0" upper="1" effort="40"  velocity="${4*PI/3}"/>
+        <mimic joint="${prefix}gripper_joint" multiplier="1" offset="0"/>
+      </xacro:unless>
     </joint>
     <link name="${prefix}right_support_link">
@@ -232,11 +243,13 @@
       </collision>
     </link>
-    <joint name="${prefix}right_support_joint" type="revolute">
+    <joint name="${prefix}right_support_joint" type="${joint_type}">
       <origin xyz="-0.0093594 0.056229 0"/>
       <parent link="${prefix}right_1_link"/>
       <child link="${prefix}right_support_link"/>
-      <axis xyz="0 0 1"/>
-      <limit lower="0" upper="1" effort="40"  velocity="${4*PI/3}"/>
-      <mimic joint="${prefix}gripper_joint" multiplier="1" offset="0"/>
+      <xacro:unless value="${kinematic_only}">
+        <axis xyz="0 0 1"/>
+        <limit lower="0" upper="1" effort="40"  velocity="${4*PI/3}"/>
+        <mimic joint="${prefix}gripper_joint" multiplier="1" offset="0"/>
+      </xacro:unless>
     </joint>
     <link name="${prefix}right_pad_link">
@@ -274,4 +287,11 @@
     </joint>
     <link name="${prefix}gripper_center"/>
+    <!-- OCS2 end-effector frame (fixed_base.info eeFrame) -->
+    <link name="${prefix}eef"/>
+    <joint name="${prefix}eef_joint" type="fixed">
+      <origin xyz="0 0 0" rpy="0 0 0"/>
+      <parent link="${prefix}gripper_center"/>
+      <child link="${prefix}eef"/>
+    </joint>
   </xacro:macro>
 </robot>

Commit message: add 120s

File: gripper/changingtek_description/xacro/AG2F120S.xacro (robot description, xacro)
@@ -1,8 +1,52 @@
 <?xml version="1.0" ?>
 <robot xmlns:xacro="http://ros.org/wiki/xacro">
-  <xacro:macro name="AG2F120S" params="name kinematic_only:=false">
+  <xacro:arg name="collider" default="convex"/>
+  <xacro:property name="collider_type" value="$(arg collider)"/>
+  <!-- Simplified collision envelope (gripper_base +Z frame). -->
+  <xacro:macro name="AG2F120S_simple_collision">
+    <xacro:if value="${collider_type == 'simple'}">
+      <collision>
+        <origin xyz="0 0 0.05"/>
+        <geometry>
+          <cylinder length="0.15" radius="0.05"/>
+        </geometry>
+      </collision>
+      <collision>
+        <origin xyz="0 0 0.18"/>
+        <geometry>
+          <cylinder length="0.1" radius="0.025"/>
+        </geometry>
+      </collision>
+    </xacro:if>
+  </xacro:macro>
+  <xacro:macro name="AG2F120S" params="name use_flange:=false kinematic_only:=false">
     <xacro:property name="prefix" value="${name + '_' if name else ''}"/>
     <xacro:property name="PI" value="3.1415926535897931"/>
     <xacro:property name="joint_type" value="${kinematic_only and 'fixed' or 'revolute'}"/>
+    <xacro:if value="${use_flange}">
+      <link name="${prefix}flange">
+        <inertial>
+          <origin xyz="-0.000388 0.002345 0.0"/>
+          <mass value="0.114"/>
+          <inertia
+              ixx="0.000040105"
+              ixy="0.000000214"
+              ixz="0.0"
+              iyy="0.000085776"
+              iyz="0.0"
+              izz="0.000054044"/>
+        </inertial>
+        <visual>
+          <geometry>
+            <mesh filename="file://$(find changingtek_description)/meshes/AG2F90-C/visual/flange.glb"/>
+          </geometry>
+        </visual>
+      </link>
+      <joint name="${prefix}flange_joint" type="fixed">
+        <origin xyz="0 0 0.0258" rpy=" 0 0 ${PI/2}"/>
+        <parent link="${prefix}flange"/>
+        <child link="${prefix}gripper_base"/>
+      </joint>
+    </xacro:if>
     <link name="${prefix}gripper_base">
       <inertial>
@@ -19,12 +63,15 @@
       <visual>
         <geometry>
-          <mesh filename="file://$(find changingtek_description)/meshes/AG2F120S/visual/gripper_base.obj"/>
-        </geometry>
-      </visual>
-      <collision>
-        <geometry>
-          <mesh filename="file://$(find changingtek_description)/meshes/AG2F120S/collision/gripper_base.stl"/>
-        </geometry>
-      </collision>
+          <mesh filename="file://$(find changingtek_description)/meshes/AG2F120S/visual/base.glb"/>
+        </geometry>
+      </visual>
+      <xacro:if value="${collider_type == 'convex'}">
+        <collision>
+          <geometry>
+            <mesh filename="file://$(find changingtek_description)/meshes/AG2F120S/collision/gripper_base.stl"/>
+          </geometry>
+        </collision>
+      </xacro:if>
+      <xacro:AG2F120S_simple_collision/>
     </link>
     <link name="${prefix}left_1_link">
@@ -42,12 +89,14 @@
       <visual>
         <geometry>
-          <mesh filename="file://$(find changingtek_description)/meshes/AG2F120S/visual/link_1.obj"/>
-        </geometry>
-      </visual>
-      <collision>
-        <geometry>
-          <mesh filename="file://$(find changingtek_description)/meshes/AG2F120S/collision/link_1.stl"/>
-        </geometry>
-      </collision>
+          <mesh filename="file://$(find changingtek_description)/meshes/AG2F120S/visual/link1.glb"/>
+        </geometry>
+      </visual>
+      <xacro:if value="${collider_type == 'convex'}">
+        <collision>
+          <geometry>
+            <mesh filename="file://$(find changingtek_description)/meshes/AG2F120S/collision/link_1.stl"/>
+          </geometry>
+        </collision>
+      </xacro:if>
     </link>
     <joint name="${prefix}gripper_joint" type="${joint_type}">
@@ -74,12 +123,14 @@
       <visual>
         <geometry>
-          <mesh filename="file://$(find changingtek_description)/meshes/AG2F120S/visual/support_link.obj"/>
-        </geometry>
-      </visual>
-      <collision>
-        <geometry>
-          <mesh filename="file://$(find changingtek_description)/meshes/AG2F120S/collision/support_link.stl"/>
-        </geometry>
-      </collision>
+          <mesh filename="file://$(find changingtek_description)/meshes/AG2F120S/visual/support.glb"/>
+        </geometry>
+      </visual>
+      <xacro:if value="${collider_type == 'convex'}">
+        <collision>
+          <geometry>
+            <mesh filename="file://$(find changingtek_description)/meshes/AG2F120S/collision/support_link.stl"/>
+          </geometry>
+        </collision>
+      </xacro:if>
     </link>
     <joint name="${prefix}left_support_joint" type="${joint_type}">
@@ -107,12 +158,14 @@
       <visual>
         <geometry>
-          <mesh filename="file://$(find changingtek_description)/meshes/AG2F120S/visual/pad_link.obj"/>
-        </geometry>
-      </visual>
-      <collision>
-        <geometry>
-          <mesh filename="file://$(find changingtek_description)/meshes/AG2F120S/collision/pad_link.stl"/>
-        </geometry>
-      </collision>
+          <mesh filename="file://$(find changingtek_description)/meshes/AG2F120S/visual/pad.glb"/>
+        </geometry>
+      </visual>
+      <xacro:if value="${collider_type == 'convex'}">
+        <collision>
+          <geometry>
+            <mesh filename="file://$(find changingtek_description)/meshes/AG2F120S/collision/pad_link.stl"/>
+          </geometry>
+        </collision>
+      </xacro:if>
     </link>
     <joint name="${prefix}left_pad_joint" type="fixed">
@@ -135,12 +188,14 @@
       <visual>
         <geometry>
-          <mesh filename="file://$(find changingtek_description)/meshes/AG2F120S/visual/link_2.obj"/>
-        </geometry>
-      </visual>
-      <collision>
-        <geometry>
-          <mesh filename="file://$(find changingtek_description)/meshes/AG2F120S/collision/link_2.stl"/>
-        </geometry>
-      </collision>
+          <mesh filename="file://$(find changingtek_description)/meshes/AG2F120S/visual/link2.glb"/>
+        </geometry>
+      </visual>
+      <xacro:if value="${collider_type == 'convex'}">
+        <collision>
+          <geometry>
+            <mesh filename="file://$(find changingtek_description)/meshes/AG2F120S/collision/link_2.stl"/>
+          </geometry>
+        </collision>
+      </xacro:if>
     </link>
     <joint name="${prefix}left_2_joint" type="${joint_type}">
@@ -168,12 +223,14 @@
       <visual>
         <geometry>
-          <mesh filename="file://$(find changingtek_description)/meshes/AG2F120S/visual/link_2.obj"/>
-        </geometry>
-      </visual>
-      <collision>
-        <geometry>
-          <mesh filename="file://$(find changingtek_description)/meshes/AG2F120S/collision/link_2.stl"/>
-        </geometry>
-      </collision>
+          <mesh filename="file://$(find changingtek_description)/meshes/AG2F120S/visual/link2.glb"/>
+        </geometry>
+      </visual>
+      <xacro:if value="${collider_type == 'convex'}">
+        <collision>
+          <geometry>
+            <mesh filename="file://$(find changingtek_description)/meshes/AG2F120S/collision/link_2.stl"/>
+          </geometry>
+        </collision>
+      </xacro:if>
     </link>
     <joint name="${prefix}right_2_joint" type="${joint_type}">
@@ -201,12 +258,14 @@
       <visual>
         <geometry>
-          <mesh filename="file://$(find changingtek_description)/meshes/AG2F120S/visual/link_1.obj"/>
-        </geometry>
-      </visual>
-      <collision>
-        <geometry>
-          <mesh filename="file://$(find changingtek_description)/meshes/AG2F120S/collision/link_1.stl"/>
-        </geometry>
-      </collision>
+          <mesh filename="file://$(find changingtek_description)/meshes/AG2F120S/visual/link1.glb"/>
+        </geometry>
+      </visual>
+      <xacro:if value="${collider_type == 'convex'}">
+        <collision>
+          <geometry>
+            <mesh filename="file://$(find changingtek_description)/meshes/AG2F120S/collision/link_1.stl"/>
+          </geometry>
+        </collision>
+      </xacro:if>
     </link>
     <joint name="${prefix}right_1_joint" type="${joint_type}">
@@ -234,12 +293,14 @@
       <visual>
         <geometry>
-          <mesh filename="file://$(find changingtek_description)/meshes/AG2F120S/visual/support_link.obj"/>
-        </geometry>
-      </visual>
-      <collision>
-        <geometry>
-          <mesh filename="file://$(find changingtek_description)/meshes/AG2F120S/collision/support_link.stl"/>
-        </geometry>
-      </collision>
+          <mesh filename="file://$(find changingtek_description)/meshes/AG2F120S/visual/support.glb"/>
+        </geometry>
+      </visual>
+      <xacro:if value="${collider_type == 'convex'}">
+        <collision>
+          <geometry>
+            <mesh filename="file://$(find changingtek_description)/meshes/AG2F120S/collision/support_link.stl"/>
+          </geometry>
+        </collision>
+      </xacro:if>
     </link>
     <joint name="${prefix}right_support_joint" type="${joint_type}">
@@ -267,12 +328,14 @@
       <visual>
         <geometry>
-          <mesh filename="file://$(find changingtek_description)/meshes/AG2F120S/visual/pad_link.obj"/>
-        </geometry>
-      </visual>
-      <collision>
-        <geometry>
-          <mesh filename="file://$(find changingtek_description)/meshes/AG2F120S/collision/pad_link.stl"/>
-        </geometry>
-      </collision>
+          <mesh filename="file://$(find changingtek_description)/meshes/AG2F120S/visual/pad.glb"/>
+        </geometry>
+      </visual>
+      <xacro:if value="${collider_type == 'convex'}">
+        <collision>
+          <geometry>
+            <mesh filename="file://$(find changingtek_description)/meshes/AG2F120S/collision/pad_link.stl"/>
+          </geometry>
+        </collision>
+      </xacro:if>
     </link>
     <joint name="${prefix}right_pad_joint" type="fixed">
@@ -281,17 +344,10 @@
       <child link="${prefix}right_pad_link"/>
     </joint>
-    <joint name="${prefix}gripper_center_joint" type="fixed">
-      <origin xyz="0 0 0.2" rpy="${-PI/2} ${-PI/2} 0"/>
-      <parent link="${prefix}gripper_base"/>
-      <child link="${prefix}gripper_center"/>
-    </joint>
-    <link name="${prefix}gripper_center"/>
-    <!-- OCS2 end-effector frame (fixed_base.info eeFrame) -->
+    <joint name="${prefix}eef_joint" type="fixed">
+      <origin xyz="0 0 0.2" rpy="0 0 ${-PI/2}"/>
+      <parent link="${prefix}gripper_base"/>
+      <child link="${prefix}eef"/>
+    </joint>
     <link name="${prefix}eef"/>
-    <joint name="${prefix}eef_joint" type="fixed">
-      <origin xyz="0 0 0" rpy="0 0 0"/>
-      <parent link="${prefix}gripper_center"/>
-      <child link="${prefix}eef"/>
-    </joint>
   </xacro:macro>
 </robot>

File: gripper/changingtek_description/xacro/gripper.xacro (robot description, xacro)
@@ -19,3 +19,7 @@
     <xacro:AG2F120S name=""/>
   </xacro:if>
+  <xacro:if value="${'$(arg type)' == 'AG2F120'}">
+    <xacro:include filename="$(find changingtek_description)/xacro/AG2F120S.xacro"/>
+    <xacro:AG2F120S name="" use_flange="true"/>
+  </xacro:if>
 </robot>
