Commit message: update gripper lower limit

File: gripper/changingtek_description/xacro/AG2F90-C.xacro (robot description, xacro)
@@ -81,5 +81,5 @@
 			<axis xyz="1 0 0"/>
 			<xacro:if value="${pad == 'soft'}">
-				<limit lower="0.189" upper="1" effort="50" velocity="${PI}"/>
+				<limit lower="0.105" upper="1" effort="50" velocity="${PI}"/>
 			</xacro:if>
 			<xacro:if value="${pad == 'default'}">

Commit message: migrate to glb mesh

File: gripper/changingtek_description/xacro/AG2F90-C.xacro (robot description, xacro)
@@ -19,5 +19,5 @@
 				<visual>
 					<geometry>
-						<mesh filename="file://$(find changingtek_description)/meshes/AG2F90-C/visual/flange.obj"/>
+						<mesh filename="file://$(find changingtek_description)/meshes/AG2F90-C/visual/flange.glb"/>
 					</geometry>
 				</visual>
@@ -43,5 +43,5 @@
 			<visual>
 				<geometry>
-					<mesh filename="file://$(find changingtek_description)/meshes/AG2F90-C/visual/gripper_base.obj"/>
+					<mesh filename="file://$(find changingtek_description)/meshes/AG2F90-C/visual/gripper_base.glb"/>
 				</geometry>
 			</visual>
@@ -66,5 +66,5 @@
 			<visual>
 				<geometry>
-					<mesh filename="file://$(find changingtek_description)/meshes/AG2F90-C/visual/link_1.obj"/>
+					<mesh filename="file://$(find changingtek_description)/meshes/AG2F90-C/visual/link_1.glb"/>
 				</geometry>
 			</visual>
@@ -101,5 +101,5 @@
 			<visual>
 				<geometry>
-					<mesh filename="file://$(find changingtek_description)/meshes/AG2F90-C/visual/in_link.obj"/>
+					<mesh filename="file://$(find changingtek_description)/meshes/AG2F90-C/visual/in_link.glb"/>
 				</geometry>
 			</visual>
@@ -132,5 +132,5 @@
 			<visual>
 				<geometry>
-					<mesh filename="file://$(find changingtek_description)/meshes/AG2F90-C/visual/up_link.obj"/>
+					<mesh filename="file://$(find changingtek_description)/meshes/AG2F90-C/visual/up_link.glb"/>
 				</geometry>
 			</visual>
@@ -164,10 +164,10 @@
 				<visual>
 					<geometry>
-						<mesh filename="file://$(find changingtek_description)/meshes/AG2F90-C/visual/pad_link_soft.obj"/>
+						<mesh filename="file://$(find changingtek_description)/meshes/AG2F90-C/visual/pad_link_soft.glb"/>
 					</geometry>
 				</visual>
 				<collision>
 					<geometry>
-						<mesh filename="file://$(find changingtek_description)/meshes/AG2F90-C/visual/pad_link_soft.obj"/>
+						<mesh filename="file://$(find changingtek_description)/meshes/AG2F90-C/visual/pad_link_soft.glb"/>
 					</geometry>
 				</collision>
@@ -189,5 +189,5 @@
 				<visual>
 					<geometry>
-						<mesh filename="file://$(find changingtek_description)/meshes/AG2F90-C/visual/pad_link.obj"/>
+						<mesh filename="file://$(find changingtek_description)/meshes/AG2F90-C/visual/pad_link.glb"/>
 					</geometry>
 				</visual>
@@ -218,5 +218,5 @@
 			<visual>
 				<geometry>
-					<mesh filename="file://$(find changingtek_description)/meshes/AG2F90-C/visual/link_2.obj"/>
+					<mesh filename="file://$(find changingtek_description)/meshes/AG2F90-C/visual/link_2.glb"/>
 				</geometry>
 			</visual>
@@ -249,5 +249,5 @@
 			<visual>
 				<geometry>
-					<mesh filename="file://$(find changingtek_description)/meshes/AG2F90-C/visual/link_2.obj"/>
+					<mesh filename="file://$(find changingtek_description)/meshes/AG2F90-C/visual/link_2.glb"/>
 				</geometry>
 			</visual>
@@ -280,5 +280,5 @@
 			<visual>
 				<geometry>
-					<mesh filename="file://$(find changingtek_description)/meshes/AG2F90-C/visual/link_1.obj"/>
+					<mesh filename="file://$(find changingtek_description)/meshes/AG2F90-C/visual/link_1.glb"/>
 				</geometry>
 			</visual>
@@ -311,5 +311,5 @@
 			<visual>
 				<geometry>
-					<mesh filename="file://$(find changingtek_description)/meshes/AG2F90-C/visual/in_link.obj"/>
+					<mesh filename="file://$(find changingtek_description)/meshes/AG2F90-C/visual/in_link.glb"/>
 				</geometry>
 			</visual>
@@ -342,5 +342,5 @@
 			<visual>
 				<geometry>
-					<mesh filename="file://$(find changingtek_description)/meshes/AG2F90-C/visual/up_link.obj"/>
+					<mesh filename="file://$(find changingtek_description)/meshes/AG2F90-C/visual/up_link.glb"/>
 				</geometry>
 			</visual>
@@ -374,10 +374,10 @@
 				<visual>
 					<geometry>
-						<mesh filename="file://$(find changingtek_description)/meshes/AG2F90-C/visual/pad_link_soft.obj"/>
+						<mesh filename="file://$(find changingtek_description)/meshes/AG2F90-C/visual/pad_link_soft.glb"/>
 					</geometry>
 				</visual>
 				<collision>
 					<geometry>
-						<mesh filename="file://$(find changingtek_description)/meshes/AG2F90-C/visual/pad_link_soft.obj"/>
+						<mesh filename="file://$(find changingtek_description)/meshes/AG2F90-C/visual/pad_link_soft.glb"/>
 					</geometry>
 				</collision>
@@ -399,5 +399,5 @@
 				<visual>
 					<geometry>
-						<mesh filename="file://$(find changingtek_description)/meshes/AG2F90-C/visual/pad_link.obj"/>
+						<mesh filename="file://$(find changingtek_description)/meshes/AG2F90-C/visual/pad_link.glb"/>
 					</geometry>
 				</visual>

File: gripper/jodell_description/xacro/RG75-300.xacro (robot description, xacro)
@@ -18,10 +18,10 @@
             <visual>
                 <geometry>
-                    <mesh filename="file://$(find jodell_description)/meshes/RG75/base.obj"/>
+                    <mesh filename="file://$(find jodell_description)/meshes/RG75/base.glb"/>
                 </geometry>
             </visual>
             <collision>
                 <geometry>
-                    <mesh filename="file://$(find jodell_description)/meshes/RG75/base.obj"/>
+                    <mesh filename="file://$(find jodell_description)/meshes/RG75/base.glb"/>
                 </geometry>
             </collision>
@@ -42,10 +42,10 @@
                 <visual>
                     <geometry>
-                        <mesh filename="file://$(find jodell_description)/meshes/RG75/flange.obj"/>
-                    </geometry>
-                </visual>
-                <collision>
-                    <geometry>
-                        <mesh filename="file://$(find jodell_description)/meshes/RG75/flange.obj"/>
+                        <mesh filename="file://$(find jodell_description)/meshes/RG75/flange.glb"/>
+                    </geometry>
+                </visual>
+                <collision>
+                    <geometry>
+                        <mesh filename="file://$(find jodell_description)/meshes/RG75/flange.glb"/>
                     </geometry>
                 </collision>
@@ -70,10 +70,10 @@
             <visual>
                 <geometry>
-                    <mesh filename="file://$(find jodell_description)/meshes/RG75/finger.obj"/>
+                    <mesh filename="file://$(find jodell_description)/meshes/RG75/finger.glb"/>
                 </geometry>
             </visual>
             <collision>
                 <geometry>
-                    <mesh filename="file://$(find jodell_description)/meshes/RG75/finger.obj"/>
+                    <mesh filename="file://$(find jodell_description)/meshes/RG75/finger.glb"/>
                 </geometry>
             </collision>
@@ -100,10 +100,10 @@
             <visual>
                 <geometry>
-                    <mesh filename="file://$(find jodell_description)/meshes/RG75/finger.obj" scale="-1 -1 1"/>
+                    <mesh filename="file://$(find jodell_description)/meshes/RG75/finger.glb" scale="-1 -1 1"/>
                 </geometry>
             </visual>
             <collision>
                 <geometry>
-                    <mesh filename="file://$(find jodell_description)/meshes/RG75/finger.obj" scale="-1 -1 1"/>
+                    <mesh filename="file://$(find jodell_description)/meshes/RG75/finger.glb" scale="-1 -1 1"/>
                 </geometry>
             </collision>
@@ -132,10 +132,10 @@
                 <visual>
                     <geometry>
-                        <mesh filename="file://$(find jodell_description)/meshes/RG75/pad_fiveages.obj"/>
-                    </geometry>
-                </visual>
-                <collision>
-                    <geometry>
-                        <mesh filename="file://$(find jodell_description)/meshes/RG75/pad_fiveages.obj"/>
+                        <mesh filename="file://$(find jodell_description)/meshes/RG75/pad_fiveages.glb"/>
+                    </geometry>
+                </visual>
+                <collision>
+                    <geometry>
+                        <mesh filename="file://$(find jodell_description)/meshes/RG75/pad_fiveages.glb"/>
                     </geometry>
                 </collision>
@@ -160,11 +160,11 @@
                 <visual>
                     <geometry>
-                        <mesh filename="file://$(find jodell_description)/meshes/RG75/pad_fiveages.obj"
-                              scale="1 -1 1"/>
-                    </geometry>
-                </visual>
-                <collision>
-                    <geometry>
-                        <mesh filename="file://$(find jodell_description)/meshes/RG75/pad_fiveages.obj"
+                        <mesh filename="file://$(find jodell_description)/meshes/RG75/pad_fiveages.glb"
+                              scale="1 -1 1"/>
+                    </geometry>
+                </visual>
+                <collision>
+                    <geometry>
+                        <mesh filename="file://$(find jodell_description)/meshes/RG75/pad_fiveages.glb"
                               scale="1 -1 1"/>
                     </geometry>
@@ -198,10 +198,10 @@
                 <visual>
                     <geometry>
-                        <mesh filename="file://$(find jodell_description)/meshes/RG75/pad_leapmotor.obj"/>
-                    </geometry>
-                </visual>
-                <collision>
-                    <geometry>
-                        <mesh filename="file://$(find jodell_description)/meshes/RG75/pad_leapmotor.obj"/>
+                        <mesh filename="file://$(find jodell_description)/meshes/RG75/pad_leapmotor.glb"/>
+                    </geometry>
+                </visual>
+                <collision>
+                    <geometry>
+                        <mesh filename="file://$(find jodell_description)/meshes/RG75/pad_leapmotor.glb"/>
                     </geometry>
                 </collision>
@@ -226,11 +226,11 @@
                 <visual>
                     <geometry>
-                        <mesh filename="file://$(find jodell_description)/meshes/RG75/pad_leapmotor.obj"
-                              scale="1 -1 1"/>
-                    </geometry>
-                </visual>
-                <collision>
-                    <geometry>
-                        <mesh filename="file://$(find jodell_description)/meshes/RG75/pad_leapmotor.obj"
+                        <mesh filename="file://$(find jodell_description)/meshes/RG75/pad_leapmotor.glb"
+                              scale="1 -1 1"/>
+                    </geometry>
+                </visual>
+                <collision>
+                    <geometry>
+                        <mesh filename="file://$(find jodell_description)/meshes/RG75/pad_leapmotor.glb"
                               scale="1 -1 1"/>
                     </geometry>
