Commit message: remove planning urdf in launch

File: gripper/changingtek_description/xacro/AG2F90-C.xacro (robot description, xacro)
@@ -1,4 +1,6 @@
 <?xml version="1.0" ?>
 <robot xmlns:xacro="http://ros.org/wiki/xacro">
+	<xacro:arg name="collider" default="convex"/>
+	<xacro:property name="collider_type" value="$(arg collider)"/>
 	<xacro:macro name="AG2F90-C" params="name use_flange:=false pad:=default">
 		<xacro:property name="prefix" value="${name + '_' if name else ''}"/>
@@ -46,9 +48,11 @@
 				</geometry>
 			</visual>
-			<collision>
-				<geometry>
-					<mesh filename="file://$(find changingtek_description)/meshes/AG2F90-C/collision/base.stl"/>
-				</geometry>
-			</collision>
+			<xacro:if value="${collider_type == 'convex'}">
+				<collision>
+					<geometry>
+						<mesh filename="file://$(find changingtek_description)/meshes/AG2F90-C/collision/base.stl"/>
+					</geometry>
+				</collision>
+			</xacro:if>
 		</link>
 		<link name="${prefix}left_1_link">
@@ -69,9 +73,11 @@
 				</geometry>
 			</visual>
-			<collision>
-				<geometry>
-					<mesh filename="file://$(find changingtek_description)/meshes/AG2F90-C/collision/link_1.stl"/>
-				</geometry>
-			</collision>
+			<xacro:if value="${collider_type == 'convex'}">
+				<collision>
+					<geometry>
+						<mesh filename="file://$(find changingtek_description)/meshes/AG2F90-C/collision/link_1.stl"/>
+					</geometry>
+				</collision>
+			</xacro:if>
 		</link>
 		<joint name="${prefix}gripper_joint" type="revolute">
@@ -104,9 +110,11 @@
 				</geometry>
 			</visual>
-			<collision>
-				<geometry>
-					<mesh filename="file://$(find changingtek_description)/meshes/AG2F90-C/collision/in_link.stl"/>
-				</geometry>
-			</collision>
+			<xacro:if value="${collider_type == 'convex'}">
+				<collision>
+					<geometry>
+						<mesh filename="file://$(find changingtek_description)/meshes/AG2F90-C/collision/in_link.stl"/>
+					</geometry>
+				</collision>
+			</xacro:if>
 		</link>
 		<joint name="${prefix}left_in_Joint" type="revolute">
@@ -135,9 +143,11 @@
 				</geometry>
 			</visual>
-			<collision>
-				<geometry>
-					<mesh filename="file://$(find changingtek_description)/meshes/AG2F90-C/collision/up_link.stl"/>
-				</geometry>
-			</collision>
+			<xacro:if value="${collider_type == 'convex'}">
+				<collision>
+					<geometry>
+						<mesh filename="file://$(find changingtek_description)/meshes/AG2F90-C/collision/up_link.stl"/>
+					</geometry>
+				</collision>
+			</xacro:if>
 		</link>
 		<joint name="${prefix}left_up_Joint" type="revolute">
@@ -167,9 +177,11 @@
 					</geometry>
 				</visual>
-				<collision>
-					<geometry>
-						<mesh filename="file://$(find changingtek_description)/meshes/AG2F90-C/visual/pad_link_soft.glb"/>
-					</geometry>
-				</collision>
+				<xacro:if value="${collider_type == 'convex'}">
+					<collision>
+						<geometry>
+							<mesh filename="file://$(find changingtek_description)/meshes/AG2F90-C/visual/pad_link_soft.glb"/>
+						</geometry>
+					</collision>
+				</xacro:if>
 			</link>
 		</xacro:if>
@@ -192,9 +204,11 @@
 					</geometry>
 				</visual>
-				<collision>
-					<geometry>
-						<mesh filename="file://$(find changingtek_description)/meshes/AG2F90-C/collision/pad_link.stl"/>
-					</geometry>
-				</collision>
+				<xacro:if value="${collider_type == 'convex'}">
+					<collision>
+						<geometry>
+							<mesh filename="file://$(find changingtek_description)/meshes/AG2F90-C/collision/pad_link.stl"/>
+						</geometry>
+					</collision>
+				</xacro:if>
 			</link>
 		</xacro:if>
@@ -221,9 +235,11 @@
 				</geometry>
 			</visual>
-			<collision>
-				<geometry>
-					<mesh filename="file://$(find changingtek_description)/meshes/AG2F90-C/collision/link_2.stl"/>
-				</geometry>
-			</collision>
+			<xacro:if value="${collider_type == 'convex'}">
+				<collision>
+					<geometry>
+						<mesh filename="file://$(find changingtek_description)/meshes/AG2F90-C/collision/link_2.stl"/>
+					</geometry>
+				</collision>
+			</xacro:if>
 		</link>
 		<joint name="${prefix}left_2_Joint" type="revolute">
@@ -252,9 +268,11 @@
 				</geometry>
 			</visual>
-			<collision>
-				<geometry>
-					<mesh filename="file://$(find changingtek_description)/meshes/AG2F90-C/collision/link_2.stl"/>
-				</geometry>
-			</collision>
+			<xacro:if value="${collider_type == 'convex'}">
+				<collision>
+					<geometry>
+						<mesh filename="file://$(find changingtek_description)/meshes/AG2F90-C/collision/link_2.stl"/>
+					</geometry>
+				</collision>
+			</xacro:if>
 		</link>
 		<joint name="${prefix}right_2_Joint" type="revolute">
@@ -283,9 +301,11 @@
 				</geometry>
 			</visual>
-			<collision>
-				<geometry>
-					<mesh filename="file://$(find changingtek_description)/meshes/AG2F90-C/collision/link_1.stl"/>
-				</geometry>
-			</collision>
+			<xacro:if value="${collider_type == 'convex'}">
+				<collision>
+					<geometry>
+						<mesh filename="file://$(find changingtek_description)/meshes/AG2F90-C/collision/link_1.stl"/>
+					</geometry>
+				</collision>
+			</xacro:if>
 		</link>
 		<joint name="${prefix}right_1_Joint" type="revolute">
@@ -314,9 +334,11 @@
 				</geometry>
 			</visual>
-			<collision>
-				<geometry>
-					<mesh filename="file://$(find changingtek_description)/meshes/AG2F90-C/collision/in_link.stl"/>
-				</geometry>
-			</collision>
+			<xacro:if value="${collider_type == 'convex'}">
+				<collision>
+					<geometry>
+						<mesh filename="file://$(find changingtek_description)/meshes/AG2F90-C/collision/in_link.stl"/>
+					</geometry>
+				</collision>
+			</xacro:if>
 		</link>
 		<joint name="${prefix}right_in_Joint" type="revolute">
@@ -345,9 +367,11 @@
 				</geometry>
 			</visual>
-			<collision>
-				<geometry>
-					<mesh filename="file://$(find changingtek_description)/meshes/AG2F90-C/collision/up_link.stl"/>
-				</geometry>
-			</collision>
+			<xacro:if value="${collider_type == 'convex'}">
+				<collision>
+					<geometry>
+						<mesh filename="file://$(find changingtek_description)/meshes/AG2F90-C/collision/up_link.stl"/>
+					</geometry>
+				</collision>
+			</xacro:if>
 		</link>
 		<joint name="${prefix}right_up_Joint" type="revolute">
@@ -377,9 +401,11 @@
 					</geometry>
 				</visual>
-				<collision>
-					<geometry>
-						<mesh filename="file://$(find changingtek_description)/meshes/AG2F90-C/visual/pad_link_soft.glb"/>
-					</geometry>
-				</collision>
+				<xacro:if value="${collider_type == 'convex'}">
+					<collision>
+						<geometry>
+							<mesh filename="file://$(find changingtek_description)/meshes/AG2F90-C/visual/pad_link_soft.glb"/>
+						</geometry>
+					</collision>
+				</xacro:if>
 			</link>
 		</xacro:if>
@@ -402,9 +428,11 @@
 					</geometry>
 				</visual>
-				<collision>
-					<geometry>
-						<mesh filename="file://$(find changingtek_description)/meshes/AG2F90-C/collision/pad_link.stl"/>
-					</geometry>
-				</collision>
+				<xacro:if value="${collider_type == 'convex'}">
+					<collision>
+						<geometry>
+							<mesh filename="file://$(find changingtek_description)/meshes/AG2F90-C/collision/pad_link.stl"/>
+						</geometry>
+					</collision>
+				</xacro:if>
 			</link>
 		</xacro:if>

File: gripper/jodell_description/xacro/RG75-300.xacro (robot description, xacro)
@@ -1,4 +1,6 @@
 <?xml version="1.0"?>
 <robot xmlns:xacro="http://www.ros.org/wiki/xacro">
+    <xacro:arg name="collider" default="convex"/>
+    <xacro:property name="collider_type" value="$(arg collider)"/>
     <xacro:macro name="RG75-300" params="name use_flange:=false pad:=fiveages">
         <xacro:property name="prefix" value="${name + '_' if name else ''}"/>
@@ -21,9 +23,11 @@
                 </geometry>
             </visual>
-            <collision>
-                <geometry>
-                    <mesh filename="file://$(find jodell_description)/meshes/RG75/base.glb"/>
-                </geometry>
-            </collision>
+            <xacro:if value="${collider_type == 'convex'}">
+                <collision>
+                    <geometry>
+                        <mesh filename="file://$(find jodell_description)/meshes/RG75/base.glb"/>
+                    </geometry>
+                </collision>
+            </xacro:if>
         </link>
         <xacro:if value="${use_flange}">
@@ -45,9 +49,11 @@
                     </geometry>
                 </visual>
-                <collision>
-                    <geometry>
-                        <mesh filename="file://$(find jodell_description)/meshes/RG75/flange.glb"/>
-                    </geometry>
-                </collision>
+                <xacro:if value="${collider_type == 'convex'}">
+                    <collision>
+                        <geometry>
+                            <mesh filename="file://$(find jodell_description)/meshes/RG75/flange.glb"/>
+                        </geometry>
+                    </collision>
+                </xacro:if>
             </link>
             <joint name="${prefix}flange_joint" type="fixed">
@@ -73,9 +79,11 @@
                 </geometry>
             </visual>
-            <collision>
-                <geometry>
-                    <mesh filename="file://$(find jodell_description)/meshes/RG75/finger.glb"/>
-                </geometry>
-            </collision>
+            <xacro:if value="${collider_type == 'convex'}">
+                <collision>
+                    <geometry>
+                        <mesh filename="file://$(find jodell_description)/meshes/RG75/finger.glb"/>
+                    </geometry>
+                </collision>
+            </xacro:if>
         </link>
         <joint name="${prefix}gripper_joint" type="prismatic">
@@ -103,9 +111,11 @@
                 </geometry>
             </visual>
-            <collision>
-                <geometry>
-                    <mesh filename="file://$(find jodell_description)/meshes/RG75/finger.glb" scale="-1 -1 1"/>
-                </geometry>
-            </collision>
+            <xacro:if value="${collider_type == 'convex'}">
+                <collision>
+                    <geometry>
+                        <mesh filename="file://$(find jodell_description)/meshes/RG75/finger.glb" scale="-1 -1 1"/>
+                    </geometry>
+                </collision>
+            </xacro:if>
         </link>
         <joint name="${prefix}right_finger_joint" type="prismatic">
@@ -135,9 +145,11 @@
                     </geometry>
                 </visual>
-                <collision>
-                    <geometry>
-                        <mesh filename="file://$(find jodell_description)/meshes/RG75/pad_fiveages.glb"/>
-                    </geometry>
-                </collision>
+                <xacro:if value="${collider_type == 'convex'}">
+                    <collision>
+                        <geometry>
+                            <mesh filename="file://$(find jodell_description)/meshes/RG75/pad_fiveages.glb"/>
+                        </geometry>
+                    </collision>
+                </xacro:if>
             </link>
             <joint name="${prefix}left_finger_pad_joint" type="fixed">
@@ -164,10 +176,12 @@
                     </geometry>
                 </visual>
-                <collision>
-                    <geometry>
-                        <mesh filename="file://$(find jodell_description)/meshes/RG75/pad_fiveages.glb"
-                              scale="1 -1 1"/>
-                    </geometry>
-                </collision>
+                <xacro:if value="${collider_type == 'convex'}">
+                    <collision>
+                        <geometry>
+                            <mesh filename="file://$(find jodell_description)/meshes/RG75/pad_fiveages.glb"
+                                  scale="1 -1 1"/>
+                        </geometry>
+                    </collision>
+                </xacro:if>
             </link>
             <joint name="${prefix}right_finger_pad_joint" type="fixed">
@@ -201,9 +215,11 @@
                     </geometry>
                 </visual>
-                <collision>
-                    <geometry>
-                        <mesh filename="file://$(find jodell_description)/meshes/RG75/pad_leapmotor.glb"/>
-                    </geometry>
-                </collision>
+                <xacro:if value="${collider_type == 'convex'}">
+                    <collision>
+                        <geometry>
+                            <mesh filename="file://$(find jodell_description)/meshes/RG75/pad_leapmotor.glb"/>
+                        </geometry>
+                    </collision>
+                </xacro:if>
             </link>
             <joint name="${prefix}left_finger_pad_joint" type="fixed">
@@ -230,10 +246,12 @@
                     </geometry>
                 </visual>
-                <collision>
-                    <geometry>
-                        <mesh filename="file://$(find jodell_description)/meshes/RG75/pad_leapmotor.glb"
-                              scale="1 -1 1"/>
-                    </geometry>
-                </collision>
+                <xacro:if value="${collider_type == 'convex'}">
+                    <collision>
+                        <geometry>
+                            <mesh filename="file://$(find jodell_description)/meshes/RG75/pad_leapmotor.glb"
+                                  scale="1 -1 1"/>
+                        </geometry>
+                    </collision>
+                </xacro:if>
             </link>
             <joint name="${prefix}right_finger_pad_joint" type="fixed">
