Commit message: add none option for ag2f90

File: gripper/changingtek_description/xacro/AG2F90-C.xacro (robot description, xacro)
@@ -89,5 +89,5 @@
 				<limit lower="0.105" upper="1" effort="50" velocity="${PI}"/>
 			</xacro:if>
-			<xacro:if value="${pad == 'default'}">
+			<xacro:if value="${pad == 'default' or pad == 'none'}">
 				<limit lower="0" upper="1" effort="50" velocity="${PI}"/>
 			</xacro:if>
@@ -159,6 +159,176 @@
 			<mimic joint="${prefix}gripper_joint"/>
 		</joint>
+		<joint name="${prefix}left_Pad_Joint" type="fixed">
+			<origin xyz="0 0.04125 -0.02425"/>
+			<parent link="${prefix}left_up_link"/>
+			<child link="${prefix}left_Pad_link"/>
+		</joint>
+		<link name="${prefix}left_2_link">
+			<inertial>
+				<origin xyz="5.08224485200288E-06 0.0327050710040551 -0.00276963392800038"/>
+				<mass value="0.0188752657753052"/>
+				<inertia
+						ixx="3.4145090175335E-06"
+						ixy="-3.3317063785682E-22"
+						ixz="-8.3582474326843E-22"
+						iyy="2.86837057727488E-07"
+						iyz="2.64809197911117E-07"
+						izz="3.39111483394506E-06"/>
+			</inertial>
+			<visual>
+				<geometry>
+					<mesh filename="file://$(find changingtek_description)/meshes/AG2F90-C/visual/link_2.glb"/>
+				</geometry>
+			</visual>
+			<xacro:if value="${collider_type == 'convex'}">
+				<collision>
+					<geometry>
+						<mesh filename="file://$(find changingtek_description)/meshes/AG2F90-C/collision/link_2.stl"/>
+					</geometry>
+				</collision>
+			</xacro:if>
+		</link>
+		<joint name="${prefix}left_2_Joint" type="revolute">
+			<origin xyz="0 -0.016 0.107" rpy="${PI/2} 0 0"/>
+			<parent link="${prefix}gripper_base"/>
+			<child link="${prefix}left_2_link"/>
+			<axis xyz="1 0 0"/>
+			<limit lower="0" upper="1" effort="50" velocity="${PI}"/>
+			<mimic joint="${prefix}gripper_joint"/>
+		</joint>
+		<link name="${prefix}right_2_link">
+			<inertial>
+				<origin xyz="1.94651792710713E-17 0.0327174794493866 -0.00277053098700989"/>
+				<mass value="0.0188856364479881"/>
+				<inertia
+						ixx="3.41458781978465E-06"
+						ixy="2.85152078238725E-22"
+						ixz="9.8903086622122E-22"
+						iyy="2.86883124998043E-07"
+						iyz="2.64817198026894E-07"
+						izz="3.39114800103702E-06"/>
+			</inertial>
+			<visual>
+				<geometry>
+					<mesh filename="file://$(find changingtek_description)/meshes/AG2F90-C/visual/link_2.glb"/>
+				</geometry>
+			</visual>
+			<xacro:if value="${collider_type == 'convex'}">
+				<collision>
+					<geometry>
+						<mesh filename="file://$(find changingtek_description)/meshes/AG2F90-C/collision/link_2.stl"/>
+					</geometry>
+				</collision>
+			</xacro:if>
+		</link>
+		<joint name="${prefix}right_2_Joint" type="revolute">
+			<origin xyz="0 0.016 0.107" rpy="${PI/2} 0 ${PI}"/>
+			<parent link="${prefix}gripper_base"/>
+			<child link="${prefix}right_2_link"/>
+			<axis xyz="1 0 0"/>
+			<limit lower="0" upper="1" effort="50" velocity="${PI}"/>
+			<mimic joint="${prefix}gripper_joint"/>
+		</joint>
+		<link name="${prefix}right_1_link">
+			<inertial>
+				<origin xyz="-5.25233292439781E-19 0.0252734640095115 -0.00214040614650291"/>
+				<mass value="0.0129014357535444"/>
+				<inertia
+						ixx="3.35976482443235E-06"
+						ixy="-3.94978742494071E-23"
+						ixz="-2.72484926002331E-23"
+						iyy="1.65185846940368E-07"
+						iyz="2.63476012977044E-07"
+						izz="3.25394125032869E-06"/>
+			</inertial>
+			<visual>
+				<geometry>
+					<mesh filename="file://$(find changingtek_description)/meshes/AG2F90-C/visual/link_1.glb"/>
+				</geometry>
+			</visual>
+			<xacro:if value="${collider_type == 'convex'}">
+				<collision>
+					<geometry>
+						<mesh filename="file://$(find changingtek_description)/meshes/AG2F90-C/collision/link_1.stl"/>
+					</geometry>
+				</collision>
+			</xacro:if>
+		</link>
+		<joint name="${prefix}right_1_Joint" type="revolute">
+			<origin xyz="0 0.030141 0.090147" rpy="${PI/2} 0 ${PI}"/>
+			<parent link="${prefix}gripper_base"/>
+			<child link="${prefix}right_1_link"/>
+			<axis xyz="1 0 0"/>
+			<limit lower="0" upper="1" effort="50" velocity="${PI}"/>
+			<mimic joint="${prefix}gripper_joint"/>
+		</joint>
+		<link name="${prefix}right_in_link">
+			<inertial>
+				<origin xyz="-1.7568261982498E-11 -0.0108820145632292 -0.00405362317350229"/>
+				<mass value="0.0134557296415635"/>
+				<inertia
+						ixx="1.43307384392376E-06"
+						ixy="-1.06834687803419E-14"
+						ixz="-4.88548199727378E-15"
+						iyy="3.88838933230828E-07"
+						iyz="-4.1814613493025E-07"
+						izz="1.33747540965672E-06"/>
+			</inertial>
+			<visual>
+				<geometry>
+					<mesh filename="file://$(find changingtek_description)/meshes/AG2F90-C/visual/in_link.glb"/>
+				</geometry>
+			</visual>
+			<xacro:if value="${collider_type == 'convex'}">
+				<collision>
+					<geometry>
+						<mesh filename="file://$(find changingtek_description)/meshes/AG2F90-C/collision/in_link.stl"/>
+					</geometry>
+				</collision>
+			</xacro:if>
+		</link>
+		<joint name="${prefix}right_in_Joint" type="revolute">
+			<origin xyz="0 0.023914 -0.0020253"/>
+			<parent link="${prefix}right_1_link"/>
+			<child link="${prefix}right_in_link"/>
+			<axis xyz="-1 0 0"/>
+			<limit lower="0" upper="1" effort="50" velocity="${PI}"/>
+			<mimic joint="${prefix}gripper_joint" multiplier="0.1" offset="0"/>
+		</joint>
+		<link name="${prefix}right_up_link">
+			<inertial>
+				<origin xyz="8.69814518862609E-11 0.0124078988097266 -0.00725256147435587"/>
+				<mass value="0.014692561982481"/>
+				<inertia
+						ixx="2.35283034039115E-06"
+						ixy="3.49796366331572E-14"
+						ixz="-4.72158801523363E-15"
+						iyy="5.89429454773258E-07"
+						iyz="7.05860796343296E-07"
+						izz="2.07228020362137E-06"/>
+			</inertial>
+			<visual>
+				<geometry>
+					<mesh filename="file://$(find changingtek_description)/meshes/AG2F90-C/visual/up_link.glb"/>
+				</geometry>
+			</visual>
+			<xacro:if value="${collider_type == 'convex'}">
+				<collision>
+					<geometry>
+						<mesh filename="file://$(find changingtek_description)/meshes/AG2F90-C/collision/up_link.stl"/>
+					</geometry>
+				</collision>
+			</xacro:if>
+		</link>
+		<joint name="${prefix}right_up_Joint" type="revolute">
+			<origin xyz="0 0.054804 -0.0046413"/>
+			<parent link="${prefix}right_1_link"/>
+			<child link="${prefix}right_up_link"/>
+			<axis xyz="-1 0 0"/>
+			<limit lower="0" upper="1" effort="50" velocity="${PI}"/>
+			<mimic joint="${prefix}gripper_joint"/>
+		</joint>
 		<xacro:if value="${pad == 'soft'}">
-			<link name="${prefix}left_Pad_link">
+			<link name="${prefix}right_Pad_link">
 				<inertial>
 					<origin xyz="0 0.02438 0.00359"/>
@@ -185,204 +355,5 @@
 				</xacro:if>
 			</link>
-		</xacro:if>
-		<xacro:if value="${pad == 'default'}">
 			<link name="${prefix}left_Pad_link">
-				<inertial>
-					<origin xyz="-3.83777509579761E-08 0.00303135276101582 0.0028336970357949"/>
-					<mass value="0.0183171479595721"/>
-					<inertia
-							ixx="2.35683098270332E-06"
-							ixy="-4.7353365844279E-12"
-							ixz="-9.31433971475514E-13"
-							iyy="9.08136064346118E-07"
-							iyz="-1.55873132053129E-08"
-							izz="3.18448591439082E-06"/>
-				</inertial>
-				<visual>
-					<geometry>
-						<mesh filename="file://$(find changingtek_description)/meshes/AG2F90-C/visual/pad_link.glb"/>
-					</geometry>
-				</visual>
-				<xacro:if value="${collider_type == 'convex'}">
-					<collision>
-						<geometry>
-							<mesh filename="file://$(find changingtek_description)/meshes/AG2F90-C/collision/pad_link.stl"/>
-						</geometry>
-					</collision>
-				</xacro:if>
-			</link>
-		</xacro:if>
-		<joint name="${prefix}left_Pad_Joint" type="fixed">
-			<origin xyz="0 0.04125 -0.02425"/>
-			<parent link="${prefix}left_up_link"/>
-			<child link="${prefix}left_Pad_link"/>
-		</joint>
-		<link name="${prefix}left_2_link">
-			<inertial>
-				<origin xyz="5.08224485200288E-06 0.0327050710040551 -0.00276963392800038"/>
-				<mass value="0.0188752657753052"/>
-				<inertia
-						ixx="3.4145090175335E-06"
-						ixy="-3.3317063785682E-22"
-						ixz="-8.3582474326843E-22"
-						iyy="2.86837057727488E-07"
-						iyz="2.64809197911117E-07"
-						izz="3.39111483394506E-06"/>
-			</inertial>
-			<visual>
-				<geometry>
-					<mesh filename="file://$(find changingtek_description)/meshes/AG2F90-C/visual/link_2.glb"/>
-				</geometry>
-			</visual>
-			<xacro:if value="${collider_type == 'convex'}">
-				<collision>
-					<geometry>
-						<mesh filename="file://$(find changingtek_description)/meshes/AG2F90-C/collision/link_2.stl"/>
-					</geometry>
-				</collision>
-			</xacro:if>
-		</link>
-		<joint name="${prefix}left_2_Joint" type="revolute">
-			<origin xyz="0 -0.016 0.107" rpy="${PI/2} 0 0"/>
-			<parent link="${prefix}gripper_base"/>
-			<child link="${prefix}left_2_link"/>
-			<axis xyz="1 0 0"/>
-			<limit lower="0" upper="1" effort="50" velocity="${PI}"/>
-			<mimic joint="${prefix}gripper_joint"/>
-		</joint>
-		<link name="${prefix}right_2_link">
-			<inertial>
-				<origin xyz="1.94651792710713E-17 0.0327174794493866 -0.00277053098700989"/>
-				<mass value="0.0188856364479881"/>
-				<inertia
-						ixx="3.41458781978465E-06"
-						ixy="2.85152078238725E-22"
-						ixz="9.8903086622122E-22"
-						iyy="2.86883124998043E-07"
-						iyz="2.64817198026894E-07"
-						izz="3.39114800103702E-06"/>
-			</inertial>
-			<visual>
-				<geometry>
-					<mesh filename="file://$(find changingtek_description)/meshes/AG2F90-C/visual/link_2.glb"/>
-				</geometry>
-			</visual>
-			<xacro:if value="${collider_type == 'convex'}">
-				<collision>
-					<geometry>
-						<mesh filename="file://$(find changingtek_description)/meshes/AG2F90-C/collision/link_2.stl"/>
-					</geometry>
-				</collision>
-			</xacro:if>
-		</link>
-		<joint name="${prefix}right_2_Joint" type="revolute">
-			<origin xyz="0 0.016 0.107" rpy="${PI/2} 0 ${PI}"/>
-			<parent link="${prefix}gripper_base"/>
-			<child link="${prefix}right_2_link"/>
-			<axis xyz="1 0 0"/>
-			<limit lower="0" upper="1" effort="50" velocity="${PI}"/>
-			<mimic joint="${prefix}gripper_joint"/>
-		</joint>
-		<link name="${prefix}right_1_link">
-			<inertial>
-				<origin xyz="-5.25233292439781E-19 0.0252734640095115 -0.00214040614650291"/>
-				<mass value="0.0129014357535444"/>
-				<inertia
-						ixx="3.35976482443235E-06"
-						ixy="-3.94978742494071E-23"
-						ixz="-2.72484926002331E-23"
-						iyy="1.65185846940368E-07"
-						iyz="2.63476012977044E-07"
-						izz="3.25394125032869E-06"/>
-			</inertial>
-			<visual>
-				<geometry>
-					<mesh filename="file://$(find changingtek_description)/meshes/AG2F90-C/visual/link_1.glb"/>
-				</geometry>
-			</visual>
-			<xacro:if value="${collider_type == 'convex'}">
-				<collision>
-					<geometry>
-						<mesh filename="file://$(find changingtek_description)/meshes/AG2F90-C/collision/link_1.stl"/>
-					</geometry>
-				</collision>
-			</xacro:if>
-		</link>
-		<joint name="${prefix}right_1_Joint" type="revolute">
-			<origin xyz="0 0.030141 0.090147" rpy="${PI/2} 0 ${PI}"/>
-			<parent link="${prefix}gripper_base"/>
-			<child link="${prefix}right_1_link"/>
-			<axis xyz="1 0 0"/>
-			<limit lower="0" upper="1" effort="50" velocity="${PI}"/>
-			<mimic joint="${prefix}gripper_joint"/>
-		</joint>
-		<link name="${prefix}right_in_link">
-			<inertial>
-				<origin xyz="-1.7568261982498E-11 -0.0108820145632292 -0.00405362317350229"/>
-				<mass value="0.0134557296415635"/>
-				<inertia
-						ixx="1.43307384392376E-06"
-						ixy="-1.06834687803419E-14"
-						ixz="-4.88548199727378E-15"
-						iyy="3.88838933230828E-07"
-						iyz="-4.1814613493025E-07"
-						izz="1.33747540965672E-06"/>
-			</inertial>
-			<visual>
-				<geometry>
-					<mesh filename="file://$(find changingtek_description)/meshes/AG2F90-C/visual/in_link.glb"/>
-				</geometry>
-			</visual>
-			<xacro:if value="${collider_type == 'convex'}">
-				<collision>
-					<geometry>
-						<mesh filename="file://$(find changingtek_description)/meshes/AG2F90-C/collision/in_link.stl"/>
-					</geometry>
-				</collision>
-			</xacro:if>
-		</link>
-		<joint name="${prefix}right_in_Joint" type="revolute">
-			<origin xyz="0 0.023914 -0.0020253"/>
-			<parent link="${prefix}right_1_link"/>
-			<child link="${prefix}right_in_link"/>
-			<axis xyz="-1 0 0"/>
-			<limit lower="0" upper="1" effort="50" velocity="${PI}"/>
-			<mimic joint="${prefix}gripper_joint" multiplier="0.1" offset="0"/>
-		</joint>
-		<link name="${prefix}right_up_link">
-			<inertial>
-				<origin xyz="8.69814518862609E-11 0.0124078988097266 -0.00725256147435587"/>
-				<mass value="0.014692561982481"/>
-				<inertia
-						ixx="2.35283034039115E-06"
-						ixy="3.49796366331572E-14"
-						ixz="-4.72158801523363E-15"
-						iyy="5.89429454773258E-07"
-						iyz="7.05860796343296E-07"
-						izz="2.07228020362137E-06"/>
-			</inertial>
-			<visual>
-				<geometry>
-					<mesh filename="file://$(find changingtek_description)/meshes/AG2F90-C/visual/up_link.glb"/>
-				</geometry>
-			</visual>
-			<xacro:if value="${collider_type == 'convex'}">
-				<collision>
-					<geometry>
-						<mesh filename="file://$(find changingtek_description)/meshes/AG2F90-C/collision/up_link.stl"/>
-					</geometry>
-				</collision>
-			</xacro:if>
-		</link>
-		<joint name="${prefix}right_up_Joint" type="revolute">
-			<origin xyz="0 0.054804 -0.0046413"/>
-			<parent link="${prefix}right_1_link"/>
-			<child link="${prefix}right_up_link"/>
-			<axis xyz="-1 0 0"/>
-			<limit lower="0" upper="1" effort="50" velocity="${PI}"/>
-			<mimic joint="${prefix}gripper_joint"/>
-		</joint>
-		<xacro:if value="${pad == 'soft'}">
-			<link name="${prefix}right_Pad_link">
 				<inertial>
 					<origin xyz="0 0.02438 0.00359"/>
@@ -436,4 +407,33 @@
 				</xacro:if>
 			</link>
+			<link name="${prefix}left_Pad_link">
+				<inertial>
+					<origin xyz="-3.83777509579761E-08 0.00303135276101582 0.0028336970357949"/>
+					<mass value="0.0183171479595721"/>
+					<inertia
+							ixx="2.35683098270332E-06"
+							ixy="-4.7353365844279E-12"
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
File: gripper/changingtek_description/xacro/gripper.xacro (robot description, xacro)
@@ -6,4 +6,8 @@
     <xacro:include filename="$(find changingtek_description)/xacro/AG2F90-C.xacro"/>
     <xacro:AG2F90-C name=""/>
+  </xacro:if>
+  <xacro:if value="${'$(arg type)' == 'AG2F90'}">
+    <xacro:include filename="$(find changingtek_description)/xacro/AG2F90-C.xacro"/>
+    <xacro:AG2F90-C name="" pad="none" use_flange="true"/>
   </xacro:if>
   <xacro:if value="${'$(arg type)' == 'AG2F90-C-Soft'}">

Commit message: add diff eef support

File: gripper/changingtek_description/xacro/AG2F90-C.xacro (robot description, xacro)
@@ -3,5 +3,22 @@
 	<xacro:arg name="collider" default="convex"/>
 	<xacro:property name="collider_type" value="$(arg collider)"/>
-	<xacro:macro name="AG2F90-C" params="name use_flange:=false pad:=default">
+	<!-- Simplified collision envelope (migrated from m6_ccs arm link7; gripper_base +Z frame). -->
+	<xacro:macro name="AG2F90_simple_collision">
+		<xacro:if value="${collider_type == 'simple'}">
+			<collision>
+				<origin xyz="0 0 0.11"/>
+				<geometry>
+					<cylinder length="0.138392" radius="0.041707"/>
+				</geometry>
+			</collision>
+			<collision>
+				<origin xyz="0 0 0.22"/>
+				<geometry>
+					<cylinder length="0.08" radius="0.021707"/>
+				</geometry>
+			</collision>
+		</xacro:if>
+	</xacro:macro>
+	<xacro:macro name="AG2F90-C" params="name use_flange:=false pad:=default kinematic_only:=false">
 		<xacro:property name="prefix" value="${name + '_' if name else ''}"/>
 		<xacro:property name="PI" value="3.1415926535897931"/>
@@ -55,5 +72,7 @@
 				</collision>
 			</xacro:if>
-		</link>
+			<xacro:AG2F90_simple_collision/>
+		</link>
+		<xacro:unless value="${kinematic_only}">
 		<link name="${prefix}left_1_link">
 			<inertial>
@@ -442,4 +461,5 @@
 			<child link="${prefix}right_Pad_link"/>
 		</joint>
+		</xacro:unless>
 		<link name="${prefix}eef"/>
 		<joint name="${prefix}eef_joint" type="fixed">

File: gripper/jodell_description/xacro/RG75-300.xacro (robot description, xacro)
@@ -3,5 +3,32 @@
     <xacro:arg name="collider" default="convex"/>
     <xacro:property name="collider_type" value="$(arg collider)"/>
-    <xacro:macro name="RG75-300" params="name use_flange:=false pad:=default">
+    <!-- Simplified collision envelope (migrated from m6_ccs arm link7; gripper_base +Z frame). -->
+    <xacro:macro name="RG75_simple_collision" params="pad">
+        <xacro:if value="${collider_type == 'simple'}">
+            <collision>
+                <origin xyz="0 0 0.11"/>
+                <geometry>
+                    <cylinder length="0.138392" radius="0.05"/>
+                </geometry>
+            </collision>
+            <xacro:if value="${pad == 'heavy_carry'}">
+                <collision>
+                    <origin xyz="0 0 0.32"/>
+                    <geometry>
+                        <box size="0.1 0.1 0.08"/>
+                    </geometry>
+                </collision>
+            </xacro:if>
+            <xacro:if value="${pad == 'default' or pad == 'leapmotor' or pad == 'none' or pad == 'soft'}">
+                <collision>
+                    <origin xyz="0 0 0.22"/>
+                    <geometry>
+                        <cylinder length="0.08" radius="0.021707"/>
+                    </geometry>
+                </collision>
+            </xacro:if>
+        </xacro:if>
+    </xacro:macro>
+    <xacro:macro name="RG75-300" params="name use_flange:=false pad:=default kinematic_only:=false">
         <xacro:property name="prefix" value="${name + '_' if name else ''}"/>
         <xacro:property name="PI" value="3.1415926535897931"/>
@@ -31,4 +58,5 @@
                 </collision>
             </xacro:if>
+            <xacro:RG75_simple_collision pad="${pad}"/>
         </link>
         <xacro:if value="${use_flange}">
@@ -57,4 +85,12 @@
                     </collision>
                 </xacro:if>
+                <xacro:if value="${collider_type == 'simple'}">
+                    <collision>
+                        <origin xyz="0 0 0.015"/>
+                        <geometry>
+                            <cylinder length="0.03" radius="0.045"/>
+                        </geometry>
+                    </collision>
+                </xacro:if>
             </link>
             <joint name="${prefix}flange_joint" type="fixed">
@@ -63,4 +99,18 @@
             </joint>
         </xacro:if>
+        <xacro:if value="${kinematic_only}">
+            <link name="${prefix}eef"/>
+            <joint name="${prefix}eef_joint" type="fixed">
+                <parent link="${prefix}gripper_base"/>
+                <child link="${prefix}eef"/>
+                <xacro:if value="${pad == 'default' or pad == 'leapmotor' or pad == 'none'}">
+                    <origin xyz="0 0 0.22"/>
+                </xacro:if>
+                <xacro:if value="${pad == 'heavy_carry'}">
+                    <origin xyz="-0.2 0 0.42525" rpy="0 ${PI/2} ${PI}"/>
+                </xacro:if>
+            </joint>
+        </xacro:if>
+        <xacro:unless value="${kinematic_only}">
         <link name="${prefix}left_finger">
             <inertial>
@@ -422,4 +472,5 @@
             </joint>
         </xacro:if>
+        </xacro:unless>
     </xacro:macro>
 </robot>

Commit message: fix single arm type process

File: gripper/changingtek_description/xacro/AG2F90-C.xacro (robot description, xacro)
@@ -105,10 +105,5 @@
 			<child link="${prefix}left_1_link"/>
 			<axis xyz="1 0 0"/>
-			<xacro:if value="${pad == 'soft'}">
-				<limit lower="0.105" upper="1" effort="50" velocity="${PI}"/>
-			</xacro:if>
-			<xacro:if value="${pad == 'default' or pad == 'none'}">
-				<limit lower="0" upper="1" effort="50" velocity="${PI}"/>
-			</xacro:if>
+			<limit lower="0" upper="1" effort="50" velocity="${PI}"/>
 		</joint>
 		<link name="${prefix}left_in_link">
