Commit message: Update home position for xhand1 and add joint type parameterization

File: dexhands/xhand1_description/xacro/xhand1.xacro (robot description, xacro)
@@ -1,6 +1,7 @@
 <?xml version="1.0" encoding="utf-8"?>
 <robot xmlns:xacro="http://www.ros.org/wiki/xacro">
-  <xacro:macro name="XHand1" params="name direction:=1">
+  <xacro:macro name="XHand1" params="name direction:=1 fixed_joints:=false">
     <xacro:property name="prefix" value="${name + '_' if name else ''}"/>
+    <xacro:property name="joint_type" value="${fixed_joints and 'fixed' or 'revolute'}"/>
         <link
           name="${prefix}hand_base">
@@ -185,5 +186,5 @@
         <joint
           name="${prefix}thumb_joint1"
-          type="revolute">
+          type="${joint_type}">
           <origin
             xyz="0.0095 ${direction*-0.0228} 0.0305"
@@ -243,5 +244,5 @@
         <joint
           name="${prefix}thumb_joint2"
-          type="revolute">
+          type="${joint_type}">
           <origin
             xyz="0.0083177 ${direction*-0.028599} -0.00178"
@@ -354,5 +355,5 @@
         <joint
           name="${prefix}thumb_joint3"
-          type="revolute">
+          type="${joint_type}">
           <origin
             xyz="0 ${direction*-0.0553} 0"
@@ -518,5 +519,5 @@
         <joint
           name="${prefix}index_joint1"
-          type="revolute">
+          type="${joint_type}">
           <origin
             xyz="0.0065 ${direction*-0.0265} 0.0899"
@@ -576,5 +577,5 @@
         <joint
           name="${prefix}index_joint2"
-          type="revolute">
+          type="${joint_type}">
           <origin
             xyz="0 0 0.0178"
@@ -687,5 +688,5 @@
         <joint
           name="${prefix}index_joint3"
-          type="revolute">
+          type="${joint_type}">
           <origin
             xyz="0 0 0.0558"
@@ -851,5 +852,5 @@
         <joint
           name="${prefix}middle_joint1"
-          type="revolute">
+          type="${joint_type}">
           <origin
             xyz="0.0065 ${direction*-0.004} 0.1082"
@@ -962,5 +963,5 @@
         <joint
           name="${prefix}middle_joint2"
-          type="revolute">
+          type="${joint_type}">
           <origin
             xyz="0 0 0.0558"
@@ -1126,5 +1127,5 @@
         <joint
           name="${prefix}ring_joint1"
-          type="revolute">
+          type="${joint_type}">
           <origin
             xyz="0.0065 ${direction*0.016} 0.1052"
@@ -1237,5 +1238,5 @@
         <joint
           name="${prefix}ring_joint2"
-          type="revolute">
+          type="${joint_type}">
           <origin
             xyz="0 0 0.0558"
@@ -1401,5 +1402,5 @@
         <joint
           name="${prefix}pinky_joint1"
-          type="revolute">
+          type="${joint_type}">
           <origin
             xyz="0.0065 ${direction*0.036} 0.1022"
@@ -1512,5 +1513,5 @@
         <joint
           name="${prefix}pinky_joint2"
-          type="revolute">
+          type="${joint_type}">
           <origin
             xyz="0 0 0.0558"
