Commit message: fix xhand mesh

File: dexhands/xhand1_description/xacro/xhand1.xacro (robot description, xacro)
@@ -1,1250 +1,738 @@
 <?xml version="1.0" encoding="utf-8"?>
+<!--
+  XHAND1: single-tree + direction mirroring.
+  Meshes live in meshes/ (no left/right dirs).
+  hand_base: hand_link.glb (left) / hand_link_right.glb (right), no Y-scale.
+  Thumb / hand_back: left glb + Y-scale.
+  Index / middle / ring / pinky: shared meshes, no Y-scale.
+-->
 <robot xmlns:xacro="http://www.ros.org/wiki/xacro">
     <xacro:macro name="XHand1" params="name direction:=1 fixed_joints:=false">
         <xacro:property name="prefix" value="${name + '_' if name else ''}"/>
         <xacro:property name="joint_type" value="${fixed_joints and 'fixed' or 'revolute'}"/>
-        <link
-                name="${prefix}hand_base">
-            <inertial>
-                <origin
-                        xyz="0.0101781679017777 0.00332669287155701 0.0570610488181997"
-                />
-                <mass
-                        value="0.53930141"/>
-                <inertia
-                        ixx="0.00064456"
-                        ixy="-0.0000027"
-                        ixz="-0.00000218"
-                        iyy="0.00046462"
-                        iyz="-0.00005116"
-                        izz="0.00027776"/>
-            </inertial>
-            <visual>
-                <geometry>
-                    <mesh
-                            filename="file://$(find xhand1_description)/meshes/left/hand_link.glb"
-                            scale="1 ${direction} 1"/>
-                </geometry>
-            </visual>
-            <collision>
-                <geometry>
-                    <mesh
-                            filename="file://$(find xhand1_description)/meshes/left/hand_link.glb"
-                            scale="1 ${direction} 1"/>
-                </geometry>
-            </collision>
-        </link>
-        <link
-                name="${prefix}hand_ee_link">
-            <inertial>
-                <origin
-                        xyz="4.91746814101629E-21 6.73369254252873E-16 2.77555756156289E-17"
-                />
-                <mass
-                        value="0.00000565"/>
-                <inertia
-                        ixx="0.00000000001"
-                        ixy="0.00000000001"
-                        ixz="0.00000000001"
-                        iyy="0.00000000001"
-                        iyz="0.00000000001"
-                        izz="0.00000000001"/>
+        <xacro:property name="hand_link_mesh"
+                        value="${'hand_link_right.glb' if direction == -1 else 'hand_link.glb'}"/>
+        <link name="${prefix}hand_base">
+            <inertial>
+                <origin xyz="0.0101781679017777 0.00332669287155701 0.0570610488181997" rpy="0 0 0"/>
+                <mass value="0.53930141"/>
+                <inertia ixx="0.00064456" ixy="-0.0000027" ixz="-0.00000218"
+                         iyy="0.00046462" iyz="-0.00005116" izz="0.00027776"/>
+            </inertial>
+            <visual>
+                <geometry>
+                    <mesh filename="file://$(find xhand1_description)/meshes/${hand_link_mesh}"
+                          scale="1 1 1"/>
+                </geometry>
+            </visual>
+            <collision>
+                <geometry>
+                    <mesh filename="file://$(find xhand1_description)/meshes/${hand_link_mesh}"
+                          scale="1 1 1"/>
+                </geometry>
+            </collision>
+        </link>
+        <link name="${prefix}hand_ee_link">
+            <inertial>
+                <origin xyz="4.91746814101629E-21 6.73369254252873E-16 2.77555756156289E-17" rpy="0 0 0"/>
+                <mass value="0.00000565"/>
+                <inertia ixx="0.00000000001" ixy="0.00000000001" ixz="0.00000000001"
+                         iyy="0.00000000001" iyz="0.00000000001" izz="0.00000000001"/>
             </inertial>
         </link>
         <joint name="${prefix}eef_joint" type="fixed">
-            <origin xyz="0 0 0.065"/>
+            <origin xyz="0 0 0.065" rpy="0 0 0"/>
             <parent link="${prefix}hand_base"/>
             <child link="${prefix}hand_ee_link"/>
             <dynamics damping="0" friction="0"/>
         </joint>
-        <link
-                name="${prefix}hand_back_link">
-            <inertial>
-                <origin
-                        xyz="-0.014009233507471 0.00206609606832526 -0.000644386526891264"
-                />
-                <mass
-                        value="0.00000002"/>
-                <inertia
-                        ixx="0.00000000001"
-                        ixy="0.00000000001"
-                        ixz="0.00000000001"
-                        iyy="0.00000000001"
-                        iyz="0.00000000001"
-                        izz="0.00000000001"/>
-            </inertial>
-            <visual>
-                <geometry>
-                    <mesh
-                            filename="file://$(find xhand1_description)/meshes/left/hand_back.glb"
-                            scale="1 ${direction} 1"/>
-                </geometry>
-            </visual>
-            <collision>
-                <geometry>
-                    <mesh
-                            filename="file://$(find xhand1_description)/meshes/left/hand_back.glb"
-                            scale="1 ${direction} 1"/>
-                </geometry>
-            </collision>
-        </link>
-        <joint
-                name="${prefix}back_joint"
-                type="fixed">
-            <origin
-                    xyz="0 0 0.065"
-            />
-            <parent
-                    link="${prefix}hand_base"/>
-            <child
-                    link="${prefix}hand_back_link"/>
-        </joint>
-        <link
-                name="${prefix}hand_thumb_bend_link">
-            <inertial>
-                <origin
-                        xyz="-0.00116653621756009 -0.0144315029884419 6.50666001038684E-05"
-                />
-                <mass
-                        value="0.01151453"/>
-                <inertia
-                        ixx="0.00000155"
-                        ixy="0.00000003"
-                        ixz="0.00000000001"
-                        iyy="0.00000062"
-                        iyz="-0.00000007"
-                        izz="0.00000157"/>
-            </inertial>
-            <visual>
-                <geometry>
-                    <mesh
-                            filename="file://$(find xhand1_description)/meshes/left/thumb_bend.glb"
-                            scale="1 ${direction} 1"/>
-                </geometry>
-            </visual>
-            <collision>
-                <geometry>
-                    <mesh
-                            filename="file://$(find xhand1_description)/meshes/left/thumb_bend.glb"
-                            scale="1 ${direction} 1"/>
-                </geometry>
-            </collision>
-        </link>
-        <joint
-                name="${prefix}thumb_joint1"
-                type="${joint_type}">
-            <origin
-                    xyz="0.0095 ${direction*-0.0228} 0.0305"
-            />
-            <parent
-                    link="${prefix}hand_base"/>
-            <child
-                    link="${prefix}hand_thumb_bend_link"/>
-            <axis
-                    xyz="0 0 ${direction}"/>
-            <limit
-                    lower="0"
-                    upper="1.832"
-                    effort="1.1"
-                    velocity="8.63"/>
-        </joint>
-        <link
-                name="${prefix}hand_thumb_rota_link1">
-            <inertial>
-                <origin
-                        xyz="-0.00035301300459029 -0.028699400584612 0.00135210573795722"
-                />
-                <mass
-                        value="0.1322853"/>
-                <inertia
-                        ixx="0.00003665"
-                        ixy="0.00000788"
-                        ixz="0.00000198"
-                        iyy="0.00001694"
-                        iyz="-0.00000185"
-                        izz="0.00004358"/>
-            </inertial>
-            <visual>
-                <geometry>
-                    <mesh
-                            filename="file://$(find xhand1_description)/meshes/left/thumb_rota1.glb"
-                            scale="1 ${direction} 1"/>
-                </geometry>
-            </visual>
-            <collision>
-                <geometry>
-                    <mesh
-                            filename="file://$(find xhand1_description)/meshes/left/thumb_rota1.glb"
-                            scale="1 ${direction} 1"/>
-                </geometry>
-            </collision>
-        </link>
-        <joint
-                name="${prefix}thumb_joint2"
-                type="${joint_type}">
-            <origin
-                    xyz="0.0083177 ${direction*-0.028599} -0.00178"
+        <link name="${prefix}hand_back_link">
+            <inertial>
+                <origin xyz="-0.014009233507471 ${direction*0.00206609606832526} -0.000644386526891264" rpy="0 0 0"/>
+                <mass value="0.00000002"/>
+                <inertia ixx="0.00000000001" ixy="${direction*0.00000000001}" ixz="0.00000000001"
+                         iyy="0.00000000001" iyz="${direction*0.00000000001}" izz="0.00000000001"/>
+            </inertial>
+            <visual>
+                <geometry>
+                    <mesh filename="file://$(find xhand1_description)/meshes/hand_back.glb"
+                          scale="1 ${direction} 1"/>
+                </geometry>
+            </visual>
+            <collision>
+                <geometry>
+                    <mesh filename="file://$(find xhand1_description)/meshes/hand_back.glb"
+                          scale="1 ${direction} 1"/>
+                </geometry>
+            </collision>
+        </link>
+        <joint name="${prefix}back_joint" type="fixed">
+            <origin xyz="0 0 0.065" rpy="0 0 0"/>
+            <parent link="${prefix}hand_base"/>
+            <child link="${prefix}hand_back_link"/>
+        </joint>
+        <link name="${prefix}hand_thumb_bend_link">
+            <inertial>
+                <origin xyz="-0.00116653621756009 ${direction*-0.0144315029884419} 6.50666001038684E-05" rpy="0 0 0"/>
+                <mass value="0.01151453"/>
+                <inertia ixx="0.00000155" ixy="${direction*0.00000003}" ixz="0.00000000001"
+                         iyy="0.00000062" iyz="${direction*-0.00000007}" izz="0.00000157"/>
+            </inertial>
+            <visual>
+                <geometry>
+                    <mesh filename="file://$(find xhand1_description)/meshes/thumb_bend.glb"
+                          scale="1 ${direction} 1"/>
+                </geometry>
+            </visual>
+            <collision>
+                <geometry>
+                    <mesh filename="file://$(find xhand1_description)/meshes/thumb_bend.glb"
+                          scale="1 ${direction} 1"/>
+                </geometry>
+            </collision>
+        </link>
+        <joint name="${prefix}thumb_joint1" type="${joint_type}">
+            <origin xyz="0.0095 ${direction*-0.0228} 0.0305" rpy="0 0 0"/>
+            <parent link="${prefix}hand_base"/>
+            <child link="${prefix}hand_thumb_bend_link"/>
+            <xacro:unless value="${fixed_joints}">
+                <axis xyz="0 0 ${direction}"/>
+                <limit lower="0" upper="1.832" effort="1.1" velocity="8.63"/>
+            </xacro:unless>
+        </joint>
+        <link name="${prefix}hand_thumb_rota_link1">
+            <inertial>
+                <origin xyz="-0.00035301300459029 ${direction*-0.028699400584612} 0.00135210573795722" rpy="0 0 0"/>
+                <mass value="0.1322853"/>
+                <inertia ixx="0.00003665" ixy="${direction*0.00000788}" ixz="0.00000198"
+                         iyy="0.00001694" iyz="${direction*-0.00000185}" izz="0.00004358"/>
+            </inertial>
+            <visual>
+                <geometry>
+                    <mesh filename="file://$(find xhand1_description)/meshes/thumb_rota1.glb"
+                          scale="1 ${direction} 1"/>
+                </geometry>
+            </visual>
+            <collision>
+                <geometry>
+                    <mesh filename="file://$(find xhand1_description)/meshes/thumb_rota1.glb"
+                          scale="1 ${direction} 1"/>
+                </geometry>
+            </collision>
+        </link>
+        <joint name="${prefix}thumb_joint2" type="${joint_type}">
+            <origin xyz="0.0083177 ${direction*-0.028599} -0.00178"
                     rpy="0 0.2618 ${direction*0.0407}"/>
-            <parent
-                    link="${prefix}hand_thumb_bend_link"/>
-            <child
-                    link="${prefix}hand_thumb_rota_link1"/>
-            <axis
-                    xyz="${direction*-1} 0 0"/>
-            <limit
-                    lower="-0.698"
-                    upper="1.57"
-                    effort="1.1"
-                    velocity="8.63"/>
-        </joint>
-        <link
-                name="${prefix}hand_thumb_rotaback_link1">
-            <inertial>
-                <origin
-                        xyz="0.00145635345487377 0.0296284435379628 -0.00757347054072981"
-                />
-                <mass
-                        value="0.00000006"/>
-                <inertia
-                        ixx="0.00000000001"
-                        ixy="0.00000000001"
-                        ixz="0.00000000001"
-                        iyy="0.00000000001"
-                        iyz="0.00000000001"
-                        izz="0.00000000001"/>
-            </inertial>
-            <visual>
-                <geometry>
-                    <mesh
-                            filename="file://$(find xhand1_description)/meshes/left/thumb_rotaback1.glb"
-                            scale="1 ${direction} 1"/>
-                </geometry>
-            </visual>
-            <collision>
-                <geometry>
-                    <mesh
-                            filename="file://$(find xhand1_description)/meshes/left/thumb_rotaback1.glb"
-                            scale="1 ${direction} 1"/>
-                </geometry>
-            </collision>
-        </link>
-        <joint
-                name="${prefix}thumb_back_joint1"
-                type="fixed">
-            <origin
-                    xyz="0 ${direction*-0.0553000000000004} 0"
-            />
-            <parent
-                    link="${prefix}hand_thumb_rota_link1"/>
-            <child
-                    link="${prefix}hand_thumb_rotaback_link1"/>
-        </joint>
-        <link
-                name="${prefix}hand_thumb_rota_link2">
-            <inertial>
-                <origin
-                        xyz="-0.000460793967924878 -0.0228414268658243 0.000578251608109689"
-                />
-                <mass
-                        value="0.03516871"/>
-                <inertia
-                        ixx="0.00000779"
-                        ixy="-0.00000002"
-                        ixz="0.00000034"
-                        iyy="0.0000035"
-                        iyz="0.00000018"
-                        izz="0.00000896"/>
-            </inertial>
-            <visual>
-                <geometry>
-                    <mesh
-                            filename="file://$(find xhand1_description)/meshes/left/thumb_rota2.glb"
-                            scale="1 ${direction} 1"/>
-                </geometry>
-            </visual>
-            <collision>
-                <geometry>
-                    <mesh
-                            filename="file://$(find xhand1_description)/meshes/left/thumb_rota2.glb"
-                            scale="1 ${direction} 1"/>
-                </geometry>
-            </collision>
-        </link>
-        <joint
-                name="${prefix}thumb_joint3"
-                type="${joint_type}">
-            <origin
-                    xyz="0 ${direction*-0.0553} 0"
-            />
-            <parent
-                    link="${prefix}hand_thumb_rota_link1"/>
-            <child
-                    link="${prefix}hand_thumb_rota_link2"/>
-            <axis
-                    xyz="${direction*-1} 0 0"/>
-            <limit
-                    lower="0"
-                    upper="1.57"
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
Commit message: add flange for xhand

File: dexhands/xhand1_description/xacro/xhand1.xacro (robot description, xacro)
@@ -8,9 +8,39 @@
 -->
 <robot xmlns:xacro="http://www.ros.org/wiki/xacro">
-    <xacro:macro name="XHand1" params="name direction:=1 fixed_joints:=false">
+    <xacro:macro name="XHand1" params="name direction:=1 use_flange:=false fixed_joints:=false">
         <xacro:property name="prefix" value="${name + '_' if name else ''}"/>
         <xacro:property name="joint_type" value="${fixed_joints and 'fixed' or 'revolute'}"/>
         <xacro:property name="hand_link_mesh"
                         value="${'hand_link_right.glb' if direction == -1 else 'hand_link.glb'}"/>
+        <xacro:if value="${use_flange}">
+            <link name="${prefix}flange">
+                <inertial>
+                    <origin xyz="-0.000388 0.002345 0.0"/>
+                    <mass value="0.114"/>
+                    <inertia
+                            ixx="0.000040105"
+                            ixy="0.000000214"
+                            ixz="0.0"
+                            iyy="0.000085776"
+                            iyz="0.0"
+                            izz="0.000054044"/>
+                </inertial>
+                <visual>
+                    <geometry>
+                        <mesh filename="file://$(find changingtek_description)/meshes/AG2F90-C/visual/flange.glb"/>
+                    </geometry>
+                </visual>
+                <visual>
+                    <geometry>
+                        <mesh filename="file://$(find xhand1_description)/meshes/flange.glb"/>
+                    </geometry>
+                </visual>
+            </link>
+            <joint name="${prefix}flange_joint" type="fixed">
+                <origin xyz="0 0 0.024144"/>
+                <parent link="${prefix}flange"/>
+                <child link="${prefix}hand_base"/>
+            </joint>
+        </xacro:if>
         <link name="${prefix}hand_base">
             <inertial>
