Commit message: update mesh

File: dexhands/xhand1_description/xacro/hand.xacro (robot description, xacro)
@@ -1,4 +1,4 @@
 <?xml version="1.0" encoding="utf-8"?>
-<robot name="XHAND1_$(arg type)" xmlns:xacro="http://www.ros.org/wiki/xacro">
+<robot name="$(arg type)" xmlns:xacro="http://www.ros.org/wiki/xacro">
     <xacro:arg name="type" default="xhand1"/>
     <xacro:arg name="direction" default="1"/>

File: dexhands/xhand1_description/xacro/xhand1.xacro (robot description, xacro)
@@ -1,1641 +1,1251 @@
 <?xml version="1.0" encoding="utf-8"?>
 <robot xmlns:xacro="http://www.ros.org/wiki/xacro">
-  <xacro:macro name="XHand1" params="name direction:=1 fixed_joints:=false">
-    <xacro:property name="prefix" value="${name + '_' if name else ''}"/>
-    <xacro:property name="joint_type" value="${fixed_joints and 'fixed' or 'revolute'}"/>
-        <link
-          name="${prefix}hand_base">
-          <inertial>
-            <origin
-              xyz="0.0101781679017777 0.00332669287155701 0.0570610488181997"
-              rpy="0 0 0" />
-            <mass
-              value="0.53930141" />
-            <inertia
-              ixx="0.00064456"
-              ixy="-0.0000027"
-              ixz="-0.00000218"
-              iyy="0.00046462"
-              iyz="-0.00005116"
-              izz="0.00027776" />
-          </inertial>
-          <visual>
-            <origin
-              xyz="0 0 0"
-              rpy="0 0 0" />
-            <geometry>
-              <mesh
-                filename="package://xhand1_description/meshes/left/hand_link.glb"
-                scale="1 ${direction} 1" />
-            </geometry>
-          </visual>
-          <collision>
-            <origin
-              xyz="0 0 0"
-              rpy="0 0 0" />
-            <geometry>
-              <mesh
-                filename="package://xhand1_description/meshes/left/hand_link.glb"
-                scale="1 ${direction} 1" />
-            </geometry>
-          </collision>
-        </link>
-        <link
-          name="${prefix}hand_ee_link">
-          <inertial>
-            <origin
-              xyz="4.91746814101629E-21 6.73369254252873E-16 2.77555756156289E-17"
-              rpy="0 0 0" />
-            <mass
-              value="0.00000565" />
-            <inertia
-              ixx="0.00000000001"
-              ixy="0.00000000001"
-              ixz="0.00000000001"
-              iyy="0.00000000001"
-              iyz="0.00000000001"
-              izz="0.00000000001" />
-          </inertial>
-          <visual>
-            <origin
-              xyz="0 0 0"
-              rpy="0 0 0" />
-            <geometry>
-              <mesh
-                filename="package://xhand1_description/meshes/left/ee.glb"
-                scale="1 ${direction} 1" />
-            </geometry>
-          </visual>
-          <collision>
-            <origin
-              xyz="0 0 0"
-              rpy="0 0 0" />
-            <geometry>
-              <mesh
-                filename="package://xhand1_description/meshes/left/ee.glb"
-                scale="1 ${direction} 1" />
-            </geometry>
-          </collision>
-        </link>
-        <joint
-          name="${prefix}eef_joint"
-          type="fixed">
-          <origin
-            xyz="0 0 0.065"
-            rpy="0 0 0" />
-          <parent
-            link="${prefix}hand_base" />
-          <child
-            link="${prefix}hand_ee_link" />
-          <axis
-            xyz="0 0 0" />
-          <dynamics
-            damping="0"
-            friction="0" />
-        </joint>
-        <link
-          name="${prefix}hand_back_link">
-          <inertial>
-            <origin
-              xyz="-0.014009233507471 0.00206609606832526 -0.000644386526891264"
-              rpy="0 0 0" />
-            <mass
-              value="0.00000002" />
-            <inertia
-              ixx="0.00000000001"
-              ixy="0.00000000001"
-              ixz="0.00000000001"
-              iyy="0.00000000001"
-              iyz="0.00000000001"
-              izz="0.00000000001" />
-          </inertial>
-          <visual>
-            <origin
-              xyz="0 0 0"
-              rpy="0 0 0" />
-            <geometry>
-              <mesh
-                filename="package://xhand1_description/meshes/left/hand_back.glb"
-                scale="1 ${direction} 1" />
-            </geometry>
-          </visual>
-          <collision>
-            <origin
-              xyz="0 0 0"
-              rpy="0 0 0" />
-            <geometry>
-              <mesh
-                filename="package://xhand1_description/meshes/left/hand_back.glb"
-                scale="1 ${direction} 1" />
-            </geometry>
-          </collision>
-        </link>
-        <joint
-          name="${prefix}back_joint"
-          type="fixed">
-          <origin
-            xyz="0 0 0.065"
-            rpy="0 0 0" />
-          <parent
-            link="${prefix}hand_base" />
-          <child
-            link="${prefix}hand_back_link" />
-          <axis
-            xyz="0 0 0" />
-          <dynamics
-            damping="0"
-            friction="0" />
-        </joint>
-        <link
-          name="${prefix}hand_thumb_bend_link">
-          <inertial>
-            <origin
-              xyz="-0.00116653621756009 -0.0144315029884419 6.50666001038684E-05"
-              rpy="0 0 0" />
-            <mass
-              value="0.01151453" />
-            <inertia
-              ixx="0.00000155"
-              ixy="0.00000003"
-              ixz="0.00000000001"
-              iyy="0.00000062"
-              iyz="-0.00000007"
-              izz="0.00000157" />
-          </inertial>
-          <visual>
-            <origin
-              xyz="0 0 0"
-              rpy="0 0 0" />
-            <geometry>
-              <mesh
-                filename="package://xhand1_description/meshes/left/thumb_bend.glb"
-                scale="1 ${direction} 1" />
-            </geometry>
-          </visual>
-          <collision>
-            <origin
-              xyz="0 0 0"
-              rpy="0 0 0" />
-            <geometry>
-              <mesh
-                filename="package://xhand1_description/meshes/left/thumb_bend.glb"
-                scale="1 ${direction} 1" />
-            </geometry>
-          </collision>
-        </link>
-        <joint
-          name="${prefix}thumb_joint1"
-          type="${joint_type}">
-          <origin
-            xyz="0.0095 ${direction*-0.0228} 0.0305"
-            rpy="0 0 0" />
-          <parent
-            link="${prefix}hand_base" />
-          <child
-            link="${prefix}hand_thumb_bend_link" />
-          <axis
-            xyz="0 0 ${direction}" />
-          <limit
-            lower="0"
-            upper="1.832"
-            effort="1.1"
-            velocity="8.63" />
-          <dynamics
-            damping="0"
-            friction="0" />
-        </joint>
-        <link
-          name="${prefix}hand_thumb_rota_link1">
-          <inertial>
-            <origin
-              xyz="-0.00035301300459029 -0.028699400584612 0.00135210573795722"
-              rpy="0 0 0" />
-            <mass
-              value="0.1322853" />
-            <inertia
-              ixx="0.00003665"
-              ixy="0.00000788"
-              ixz="0.00000198"
-              iyy="0.00001694"
-              iyz="-0.00000185"
-              izz="0.00004358" />
-          </inertial>
-          <visual>
-            <origin
-              xyz="0 0 0"
-              rpy="0 0 0" />
-            <geometry>
-              <mesh
-                filename="package://xhand1_description/meshes/left/thumb_rota1.glb"
-                scale="1 ${direction} 1" />
-            </geometry>
-          </visual>
-          <collision>
-            <origin
-              xyz="0 0 0"
-              rpy="0 0 0" />
-            <geometry>
-              <mesh
-                filename="package://xhand1_description/meshes/left/thumb_rota1.glb"
-                scale="1 ${direction} 1" />
-            </geometry>
-          </collision>
-        </link>
-        <joint
-          name="${prefix}thumb_joint2"
-          type="${joint_type}">
-          <origin
-            xyz="0.0083177 ${direction*-0.028599} -0.00178"
-            rpy="0 0.2618 ${direction*0.0407}" />
-          <parent
-            link="${prefix}hand_thumb_bend_link" />
-          <child
-            link="${prefix}hand_thumb_rota_link1" />
-          <axis
-            xyz="${direction*-1} 0 0" />
-          <limit
-            lower="-0.698"
-            upper="1.57"
-            effort="1.1"
-            velocity="8.63" />
-          <dynamics
-            damping="0"
-            friction="0" />
-        </joint>
-        <link
-          name="${prefix}hand_thumb_rotaback_link1">
-          <inertial>
-            <origin
-              xyz="0.00145635345487377 0.0296284435379628 -0.00757347054072981"
-              rpy="0 0 0" />
-            <mass
-              value="0.00000006" />
-            <inertia
-              ixx="0.00000000001"
-              ixy="0.00000000001"
-              ixz="0.00000000001"
-              iyy="0.00000000001"
-              iyz="0.00000000001"
-              izz="0.00000000001" />
-          </inertial>
-          <visual>
-            <origin
-              xyz="0 0 0"
-              rpy="0 0 0" />
-            <geometry>
-              <mesh
-                filename="package://xhand1_description/meshes/left/thumb_rotaback1.glb"
-                scale="1 ${direction} 1" />
-            </geometry>
-          </visual>
-          <collision>
-            <origin
-              xyz="0 0 0"
-              rpy="0 0 0" />
-            <geometry>
-              <mesh
-                filename="package://xhand1_description/meshes/left/thumb_rotaback1.glb"
-                scale="1 ${direction} 1" />
-            </geometry>
-          </collision>
-        </link>
-        <joint
-          name="${prefix}thumb_back_joint1"
-          type="fixed">
-          <origin
-            xyz="0 ${direction*-0.0553000000000004} 0"
-            rpy="0 0 0" />
-          <parent
-            link="${prefix}hand_thumb_rota_link1" />
-          <child
-            link="${prefix}hand_thumb_rotaback_link1" />
-          <axis
-            xyz="0 0 0" />
-          <dynamics
-            damping="0"
-            friction="0" />
-        </joint>
-        <link
-          name="${prefix}hand_thumb_rota_link2">
-          <inertial>
-            <origin
-              xyz="-0.000460793967924878 -0.0228414268658243 0.000578251608109689"
-              rpy="0 0 0" />
-            <mass
-              value="0.03516871" />
-            <inertia
-              ixx="0.00000779"
-              ixy="-0.00000002"
-              ixz="0.00000034"
-              iyy="0.0000035"
-              iyz="0.00000018"
-              izz="0.00000896" />
-          </inertial>
-          <visual>
-            <origin
-              xyz="0 0 0"
-              rpy="0 0 0" />
-            <geometry>
-              <mesh
-                filename="package://xhand1_description/meshes/left/thumb_rota2.glb"
-                scale="1 ${direction} 1" />
-            </geometry>
-          </visual>
-          <collision>
-            <origin
-              xyz="0 0 0"
-              rpy="0 0 0" />
-            <geometry>
-              <mesh
-                filename="package://xhand1_description/meshes/left/thumb_rota2.glb"
-                scale="1 ${direction} 1" />
-            </geometry>
-          </collision>
-        </link>
-        <joint
-          name="${prefix}thumb_joint3"
-          type="${joint_type}">
-          <origin
-            xyz="0 ${direction*-0.0553} 0"
-            rpy="0 0 0" />
-          <parent
-            link="${prefix}hand_thumb_rota_link1" />
-          <child
-            link="${prefix}hand_thumb_rota_link2" />
-          <axis
-            xyz="${direction*-1} 0 0" />
-          <limit
-            lower="0"
-            upper="1.57"
-            effort="0.4"
-            velocity="14.38" />
-          <dynamics
-            damping="0"
-            friction="0" />
-        </joint>
-        <link
-          name="${prefix}hand_thumb_rotaback_link2">
-          <inertial>
-            <origin
-              xyz="-0.000513245945552355 0.0256681874022328 -0.00926148643045993"
-              rpy="0 0 0" />
-            <mass
-              value="0.00000004" />
-            <inertia
-              ixx="0.00000000001"
-              ixy="0.00000000001"
-              ixz="0.00000000001"
-              iyy="0.00000000001"
-              iyz="0.00000000001"
-              izz="0.00000000001" />
-          </inertial>
-          <visual>
-            <origin
-              xyz="0 0 0"
-              rpy="0 0 0" />
-            <geometry>
-              <mesh
-                filename="package://xhand1_description/meshes/left/thumb_rotaback2.glb"
-                scale="1 ${direction} 1" />
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