Commit message: add rg75 heavy config

File: gripper/jodell_description/xacro/RG75-300.xacro (robot description, xacro)
@@ -6,4 +6,5 @@
         <xacro:property name="prefix" value="${name + '_' if name else ''}"/>
         <xacro:property name="PI" value="3.1415926535897931"/>
+        <xacro:property name="is_heavy_carry" value="${pad == 'heavy carry' or pad == 'heavy_carry'}"/>
         <link name="${prefix}gripper_base">
             <inertial>
@@ -79,10 +80,10 @@
                 </geometry>
             </visual>
-            <xacro:if value="${collider_type == 'convex'}">
-                <collision>
-                    <geometry>
-                        <mesh filename="file://$(find jodell_description)/meshes/RG75/finger.glb"/>
-                    </geometry>
-                </collision>
+            <xacro:if value="${not is_heavy_carry}">
+                <visual>
+                    <geometry>
+                        <mesh filename="file://$(find jodell_description)/meshes/RG75/finger_support.glb"/>
+                    </geometry>
+                </visual>
             </xacro:if>
         </link>
@@ -108,13 +109,15 @@
             <visual>
                 <geometry>
-                    <mesh filename="file://$(find jodell_description)/meshes/RG75/finger.glb" scale="-1 -1 1"/>
+                    <mesh filename="file://$(find jodell_description)/meshes/RG75/finger.glb"/>
                 </geometry>
+                <origin rpy="0 0 ${PI}"/>
             </visual>
-            <xacro:if value="${collider_type == 'convex'}">
-                <collision>
-                    <geometry>
-                        <mesh filename="file://$(find jodell_description)/meshes/RG75/finger.glb" scale="-1 -1 1"/>
-                    </geometry>
-                </collision>
+            <xacro:if value="${not is_heavy_carry}">
+                <visual>
+                    <geometry>
+                        <mesh filename="file://$(find jodell_description)/meshes/RG75/finger_support.glb"/>
+                    </geometry>
+                    <origin rpy="0 0 ${PI}"/>
+                </visual>
             </xacro:if>
         </link>
@@ -127,4 +130,16 @@
             <mimic joint="${prefix}gripper_joint" multiplier="1" offset="0"/>
         </joint>
+        <xacro:if value="${not is_heavy_carry}">
+            <joint name="${prefix}left_finger_pad_joint" type="fixed">
+                <origin xyz="-0.014785 0.011478 0.0315"/>
+                <parent link="${prefix}left_finger"/>
+                <child link="${prefix}left_finger_pad"/>
+            </joint>
+            <joint name="${prefix}right_finger_pad_joint" type="fixed">
+                <origin xyz="0.014785 -0.011478 0.0315"/>
+                <parent link="${prefix}right_finger"/>
+                <child link="${prefix}right_finger_pad"/>
+            </joint>
+        </xacro:if>
         <xacro:if value="${pad == 'fiveages'}">
             <link name="${prefix}left_finger_pad">
@@ -153,9 +168,4 @@
                 </xacro:if>
             </link>
-            <joint name="${prefix}left_finger_pad_joint" type="fixed">
-                <origin xyz="-0.014715 0.011478 0.0315"/>
-                <parent link="${prefix}left_finger"/>
-                <child link="${prefix}left_finger_pad"/>
-            </joint>
             <link name="${prefix}right_finger_pad">
                 <inertial>
@@ -185,9 +195,4 @@
                 </xacro:if>
             </link>
-            <joint name="${prefix}right_finger_pad_joint" type="fixed">
-                <origin xyz="0.014785 -0.011478 0.03175"/>
-                <parent link="${prefix}right_finger"/>
-                <child link="${prefix}right_finger_pad"/>
-            </joint>
             <link name="${prefix}eef"/>
             <joint name="${prefix}eef_joint" type="fixed">
@@ -223,9 +228,4 @@
                 </xacro:if>
             </link>
-            <joint name="${prefix}left_finger_pad_joint" type="fixed">
-                <origin xyz="-0.02225 0.01245 0.0607500000000101"/>
-                <parent link="${prefix}left_finger"/>
-                <child link="${prefix}left_finger_pad"/>
-            </joint>
             <link name="${prefix}right_finger_pad">
                 <inertial>
@@ -255,9 +255,4 @@
                 </xacro:if>
             </link>
-            <joint name="${prefix}right_finger_pad_joint" type="fixed">
-                <origin xyz="0.00724999999998532 -0.01245 0.0607500000000101"/>
-                <parent link="${prefix}right_finger"/>
-                <child link="${prefix}right_finger_pad"/>
-            </joint>
             <link name="${prefix}eef"/>
             <joint name="${prefix}eef_joint" type="fixed">
@@ -267,4 +262,80 @@
             </joint>
         </xacro:if>
+        <xacro:if value="${pad == 'none'}">
+            <link name="${prefix}left_finger_pad"/>
+            <link name="${prefix}right_finger_pad"/>
+        </xacro:if>
+        <xacro:if value="${pad == 'heavy_carry'}">
+            <link name="${prefix}left_finger_pad">
+                <inertial>
+                    <origin xyz="-0.0273621671052904 -0.0115571775561825 0.131965151776638"/>
+                    <mass value="0.971848511966183"/>
+                    <inertia
+                            ixx="0.00567329523505055"
+                            ixy="-1.46176859453297E-08"
+                            ixz="0.00209826432464484"
+                            iyy="0.00798991806803702"
+                            iyz="-1.72430069472743E-06"
+                            izz="0.00233523656275322"/>
+                </inertial>
+                <visual>
+                    <geometry>
+                        <mesh filename="file://$(find jodell_description)/meshes/RG75/heavy_carry/${name}/left.glb"/>
+                    </geometry>
+                </visual>
+                <xacro:if value="${collider_type == 'convex'}">
+                    <collision>
+                        <geometry>
+                            <mesh filename="file://$(find jodell_description)/meshes/RG75/heavy_carry/${name}/left.glb"/>
+                        </geometry>
+                    </collision>
+                </xacro:if>
+            </link>
+            <joint name="${prefix}left_finger_pad_joint" type="fixed">
+                <origin xyz="0.01475 0.043263 0.13525"/>
+                <parent link="${prefix}gripper_base"/>
+                <child link="${prefix}left_finger_pad"/>
+            </joint>
+            <link name="${prefix}right_finger_pad">
+                <inertial>
+                    <origin xyz="-0.0273648226249448 0.0115580703720554 0.131965151776598"/>
+                    <mass value="0.971848511966211"/>
+                    <inertia
+                            ixx="0.00567329523505061"
+                            ixy="-1.46176859456687E-08"
+                            ixz="0.00209826432464498"
+                            iyy="0.00798991806803724"
+                            iyz="1.87585284859872E-06"
+                            izz="0.0023352365627534"/>
+                </inertial>
+                <visual>
+                    <geometry>
+                        <mesh filename="file://$(find jodell_description)/meshes/RG75/heavy_carry/${name}/right.glb"/>
+                    </geometry>
+                </visual>
+                <xacro:if value="${collider_type == 'convex'}">
+                    <collision>
+                        <geometry>
+                            <mesh filename="file://$(find jodell_description)/meshes/RG75/heavy_carry/${name}/right.glb"/>
+                        </geometry>
+                    </collision>
+                </xacro:if>
+            </link>
+            <joint name="${prefix}right_finger_pad_joint" type="fixed">
+                <parent link="${prefix}right_finger"/>
+                <child link="${prefix}right_finger_pad"/>
+            </joint>
+            <link name="${prefix}eef"/>
+            <joint name="${prefix}eef_joint" type="fixed">
+                <parent link="${prefix}gripper_base"/>
+                <child link="${prefix}eef"/>
+                <xacro:if value="${name == 'left'}">
+                    <origin xyz="0.06 0.07 0.16" rpy="${PI*17/9} 0 0"/>
+                </xacro:if>
+                <xacro:if value="${name == 'right'}">
+                    <origin xyz="-0.06 0.07 0.16" rpy="${PI*17/9} 0 0"/>
+                </xacro:if>
+            </joint>
+        </xacro:if>
     </xacro:macro>
 </robot>

File: gripper/jodell_description/xacro/gripper.xacro (robot description, xacro)
@@ -5,5 +5,5 @@
     <xacro:if value="${'$(arg type)' == 'RG75'}">
         <xacro:include filename="$(find jodell_description)/xacro/RG75-300.xacro"/>
-        <xacro:RG75-300 name="" use_flange="true"/>
+        <xacro:RG75-300 name="" use_flange="true" pad="none"/>
     </xacro:if>
     <xacro:if value="${'$(arg type)' == 'RG75-leapmotor'}">
@@ -11,3 +11,21 @@
         <xacro:RG75-300 name="" pad="leapmotor"/>
     </xacro:if>
+    <xacro:if value="${'$(arg type)' == 'heavy_carry_left'}">
+        <link name="gripper_base"/>
+        <joint name="base_joint" type="fixed">
+            <parent link="gripper_base"/>
+            <child link="left_gripper_base"/>
+        </joint>
+        <xacro:include filename="$(find jodell_description)/xacro/RG75-300.xacro"/>
+        <xacro:RG75-300 name="left" pad="heavy_carry"/>
+    </xacro:if>
+    <xacro:if value="${'$(arg type)' == 'heavy_carry_right'}">
+        <link name="gripper_base"/>
+        <joint name="base_joint" type="fixed">
+            <parent link="gripper_base"/>
+            <child link="right_gripper_base"/>
+        </joint>
+        <xacro:include filename="$(find jodell_description)/xacro/RG75-300.xacro"/>
+        <xacro:RG75-300 name="right" pad="heavy_carry"/>
+    </xacro:if>
 </robot>

Commit message: fix rg75

File: gripper/jodell_description/xacro/RG75-300.xacro (robot description, xacro)
@@ -3,5 +3,5 @@
     <xacro:arg name="collider" default="convex"/>
     <xacro:property name="collider_type" value="$(arg collider)"/>
-    <xacro:macro name="RG75-300" params="name use_flange:=false pad:=fiveages">
+    <xacro:macro name="RG75-300" params="name use_flange:=false pad:=default">
         <xacro:property name="prefix" value="${name + '_' if name else ''}"/>
         <xacro:property name="PI" value="3.1415926535897931"/>
@@ -142,5 +142,5 @@
             </joint>
         </xacro:if>
-        <xacro:if value="${pad == 'fiveages'}">
+        <xacro:if value="${pad == 'default'}">
             <link name="${prefix}left_finger_pad">
                 <inertial>
