Commit message: add macro for m6 ccs

File: gripper/inspire_description/xacro/hands/RH56F2.xacro (robot description, xacro)
@@ -1,8 +1,9 @@
 <?xml version="1.0" encoding="utf-8"?>
 <robot xmlns:xacro="http://www.ros.org/wiki/xacro">
-  <xacro:macro name="InspireHandRH56F2" params="name:='' direction:=1 use_flange:=false">
+  <xacro:macro name="InspireHandRH56F2" params="name:='' direction:=1 use_flange:=false fixed_joints:=false">
     <xacro:property name="prefix" value="${name + '_' if name else ''}"/>
     <!-- direction: 1=left (no mirror), -1=right (Y mirror); meshes from left hand -->
     <xacro:property name="dir" value="${int(direction)}"/>
+    <xacro:property name="joint_type" value="${fixed_joints and 'fixed' or 'revolute'}"/>
     <xacro:if value="${use_flange}">
       <link name="${prefix}flange">
@@ -508,5 +509,5 @@
       </collision>
     </link>
-    <joint name="${prefix}thumb_joint1" type="revolute">
+    <joint name="${prefix}thumb_joint1" type="${joint_type}">
       <origin xyz="0.018361 ${dir*-0.027493} 0.040054" rpy="0 0 0"/>
       <parent link="${prefix}hand_base"/>
@@ -515,5 +516,5 @@
       <limit lower="0" upper="2" effort="1" velocity="2"/>
     </joint>
-    <joint name="${prefix}thumb_joint2" type="revolute">
+    <joint name="${prefix}thumb_joint2" type="${joint_type}">
       <origin xyz="0.00903585558357 ${dir*-0.0124048110618} -0.00529612169302" rpy="${dir*1.57070938522} 0 ${dir*-1.48352986386}"/>
       <parent link="${prefix}thumb_1"/>
@@ -522,5 +523,5 @@
       <limit lower="0" upper="0.7854" effort="1" velocity="2"/>
     </joint>
-    <joint name="${prefix}thumb_joint3" type="revolute">
+    <joint name="${prefix}thumb_joint3" type="${joint_type}">
       <origin xyz="0.0437230821114 ${dir*0.0271075946182} -0.0025" rpy="0 0 0"/>
       <parent link="${prefix}thumb_2"/>
@@ -530,5 +531,5 @@
       <mimic joint="${prefix}thumb_joint2" multiplier="0.7222" offset="0"/>
     </joint>
-    <joint name="${prefix}thumb_joint4" type="revolute">
+    <joint name="${prefix}thumb_joint4" type="${joint_type}">
       <origin xyz="0.0117743449217 ${dir*0.00853690944054} 0.0023" rpy="0 0 0"/>
       <parent link="${prefix}thumb_3"/>
@@ -543,5 +544,5 @@
       <child link="${prefix}thumb_force_sensor"/>
     </joint>
-    <joint name="${prefix}index_joint" type="revolute">
+    <joint name="${prefix}index_joint" type="${joint_type}">
       <origin xyz="0.000707528417719 ${dir*-0.0343765200022} 0.105041789582" rpy="${dir*1.63188285056} 0 0"/>
       <parent link="${prefix}hand_base"/>
@@ -550,5 +551,5 @@
       <limit lower="0" upper="1.466" effort="1" velocity="2"/>
     </joint>
-    <joint name="${prefix}index_dip" type="revolute">
+    <joint name="${prefix}index_dip" type="${joint_type}">
       <origin xyz="0.00310563899528 ${dir*0.0328535387201} -0.001" rpy="0 0 0"/>
       <parent link="${prefix}index_1"/>
@@ -568,5 +569,5 @@
       <child link="${prefix}index_force_sensor"/>
     </joint>
-    <joint name="${prefix}middle_joint" type="revolute">
+    <joint name="${prefix}middle_joint" type="${joint_type}">
       <origin xyz="0.000707458100343 ${dir*-0.0157674860481} 0.105977715252" rpy="${dir*1.57079632675} 0 0"/>
       <parent link="${prefix}hand_base"/>
@@ -575,5 +576,5 @@
       <limit lower="0" upper="1.466" effort="1" velocity="2"/>
     </joint>
-    <joint name="${prefix}middle_dip" type="revolute">
+    <joint name="${prefix}middle_dip" type="${joint_type}">
       <origin xyz="0.00310557432106 ${dir*0.0328535448336} -0.001" rpy="0 0 0"/>
       <parent link="${prefix}middle_1"/>
@@ -593,5 +594,5 @@
       <child link="${prefix}middle_force_sensor"/>
     </joint>
-    <joint name="${prefix}ring_joint" type="revolute">
+    <joint name="${prefix}ring_joint" type="${joint_type}">
       <origin xyz="0.000707462370517 ${dir*0.00308760190729} 0.10592786535" rpy="${dir*1.51843644919} 0 0"/>
       <parent link="${prefix}hand_base"/>
@@ -600,5 +601,5 @@
       <limit lower="0" upper="1.466" effort="1" velocity="2"/>
     </joint>
-    <joint name="${prefix}ring_dip" type="revolute">
+    <joint name="${prefix}ring_dip" type="${joint_type}">
       <origin xyz="0.00310557506658 ${dir*0.0328535447632} -0.001" rpy="0 0 0"/>
       <parent link="${prefix}ring_1"/>
@@ -618,5 +619,5 @@
       <child link="${prefix}ring_force_sensor"/>
     </joint>
-    <joint name="${prefix}pinky_joint" type="revolute">
+    <joint name="${prefix}pinky_joint" type="${joint_type}">
       <origin xyz="0.000707528158212 ${dir*0.0210944782704} 0.104807160869" rpy="${dir*1.46607657163} 0 0"/>
       <parent link="${prefix}hand_base"/>
@@ -625,5 +626,5 @@
       <limit lower="0" upper="1.466" effort="1" velocity="2"/>
     </joint>
-    <joint name="${prefix}pinky_dip" type="revolute">
+    <joint name="${prefix}pinky_dip" type="${joint_type}">
       <origin xyz="0.00310565018524 ${dir*0.0328535376623} -0.00100000000001" rpy="0 0 0"/>
       <parent link="${prefix}pinky_1"/>
@@ -652,4 +653,10 @@
       <child link="${prefix}palm_casing"/>
     </joint>
+    <link name="${prefix}eef"/>
+    <joint name="${prefix}eef_joint" type="fixed">
+      <parent link="${prefix}hand_base"/>
+      <child link="${prefix}eef"/>
+      <origin xyz="0 ${dir*0} 0.106"/>
+    </joint>
   </xacro:macro>
 </robot>

File: gripper/inspire_description/xacro/ros2_control/side_systems.xacro (robot description, xacro)
@@ -2,6 +2,7 @@
 <robot xmlns:xacro="http://www.ros.org/wiki/xacro">
   <xacro:include filename="$(find inspire_description)/xacro/ros2_control/RH56E2.xacro"/>
-  <xacro:macro name="inspire_rs485_side_system" params="side serial_port baudrate:=115200 slave_id:=auto read_feedback:=true">
-    <ros2_control name="inspire_e2_${side}_system" type="system">
+  <xacro:include filename="$(find inspire_description)/xacro/ros2_control/RH56F2.xacro"/>
+  <xacro:macro name="inspire_rs485_side_system" params="side serial_port baudrate:=115200 slave_id:=auto read_feedback:=true hand_type:=inspire_e2">
+    <ros2_control name="${hand_type}_${side}_system" type="system">
       <hardware>
         <plugin>modbus_ros2_control/InspireHandHardware</plugin>
@@ -12,9 +13,14 @@
         <param name="read_feedback">${read_feedback}</param>
       </hardware>
-      <xacro:inspire_rh56e2_interfaces name="${side}_hand"/>
+      <xacro:if value="${hand_type == 'inspire_e2'}">
+        <xacro:inspire_rh56e2_interfaces name="${side}_hand"/>
+      </xacro:if>
+      <xacro:if value="${hand_type == 'inspire_f2'}">
+        <xacro:inspire_rh56f2_interfaces name="${side}_hand"/>
+      </xacro:if>
     </ros2_control>
   </xacro:macro>
-  <xacro:macro name="inspire_canfd_side_system" params="side can_interface hand_id:=auto read_feedback:=true">
-    <ros2_control name="inspire_e2_${side}_canfd_system" type="system">
+  <xacro:macro name="inspire_canfd_side_system" params="side can_interface hand_id:=auto read_feedback:=true hand_type:=inspire_e2">
+    <ros2_control name="${hand_type}_${side}_canfd_system" type="system">
       <hardware>
         <plugin>can_ros2_control/InspireCanfdHardware</plugin>
@@ -25,5 +31,10 @@
         <param name="feedback_timeout_ms">2</param>
       </hardware>
-      <xacro:inspire_rh56e2_interfaces name="${side}_hand"/>
+      <xacro:if value="${hand_type == 'inspire_e2'}">
+        <xacro:inspire_rh56e2_interfaces name="${side}_hand"/>
+      </xacro:if>
+      <xacro:if value="${hand_type == 'inspire_f2'}">
+        <xacro:inspire_rh56f2_interfaces name="${side}_hand"/>
+      </xacro:if>
     </ros2_control>
   </xacro:macro>
