Commit message: 添加 theo hand std16a hardware

File: dexhands/theohand_description/xacro/ros2_control/hand.xacro (robot description, xacro)
@@ -4,10 +4,9 @@
     <xacro:arg name="direction" default="1"/>
     <xacro:arg name="gazebo" default="false"/>
+    <xacro:arg name="ros2_control_hardware_type" default="real"/>
     <xacro:arg name="serial_port" default="/dev/ttyUSB0"/>
-    <xacro:arg name="slave_id" default="1"/>
+    <xacro:arg name="slave_id" default="auto"/>
     <xacro:arg name="baudrate" default="115200"/>
     <xacro:arg name="read_feedback" default="true"/>
-    <xacro:arg name="background_period_ms" default="200"/>
-    <xacro:arg name="feedback_quiet_after_write_ms" default="500"/>
     <link name="world"/>
     <joint name="world_fixed" type="fixed">
@@ -17,4 +16,5 @@
     </joint>
     <xacro:include filename="$(find theohand_description)/xacro/hand.xacro"/>
+    <xacro:property name="theohand_slave_id" value="${2 if '$(arg slave_id)' == 'auto' and '$(arg direction)' != '-1' else 1 if '$(arg slave_id)' == 'auto' else '$(arg slave_id)'}"/>
     <ros2_control name="theohand_system" type="system">
         <hardware>
@@ -35,9 +35,7 @@
                 <plugin>modbus_ros2_control/TheoHandModbusHardware</plugin>
                 <param name="serial_port">$(arg serial_port)</param>
-                <param name="slave_id">$(arg slave_id)</param>
+                <param name="slave_id">${theohand_slave_id}</param>
                 <param name="baudrate">$(arg baudrate)</param>
                 <param name="read_feedback">$(arg read_feedback)</param>
-                <param name="background_period_ms">$(arg background_period_ms)</param>
-                <param name="feedback_quiet_after_write_ms">$(arg feedback_quiet_after_write_ms)</param>
             </xacro:if>
         </hardware>

File: dexhands/theohand_description/xacro/std16a.xacro (robot description, xacro)
@@ -7,9 +7,7 @@
 			<parent link="${prefix}hand_base"/>
 			<child link="${prefix}base_link"/>
-			<origin xyz="0 0 0" rpy="0 0 0"/>
 		</joint>
 		<link name="${prefix}base_link">
 			<visual>
-				<origin xyz="0 0 0" rpy="0 0 0"/>
 				<geometry>
 					<mesh filename="file://$(find theohand_description)/meshes/std16a/base.glb"
@@ -18,5 +16,4 @@
 			</visual>
 			<collision>
-				<origin xyz="0 0 0" rpy="0 0 0"/>
 				<geometry>
 					<mesh filename="file://$(find theohand_description)/meshes/std16a/base.glb"
@@ -35,4 +32,10 @@
 			</inertial>
 		</link>
+		<link name="${prefix}eef"/>
+		<joint name="${prefix}eef_joint" type="fixed">
+			<parent link="${prefix}base_link"/>
+			<child link="${prefix}eef"/>
+			<origin xyz="0.03 0 0.1"/>
+		</joint>
 		<joint name="${prefix}thumb_joint1" type="prismatic">
 			<parent link="${prefix}base_link"/>
@@ -44,5 +47,4 @@
 		<link name="${prefix}thumb_link1">
 			<visual>
-				<origin xyz="0 0 0" rpy="0 0 0"/>
 				<geometry>
 					<mesh filename="file://$(find theohand_description)/meshes/std16a/thumb_link1.glb"
@@ -51,5 +53,4 @@
 			</visual>
 			<collision>
-				<origin xyz="0 0 0" rpy="0 0 0"/>
 				<geometry>
 					<mesh filename="file://$(find theohand_description)/meshes/std16a/thumb_link1.glb"
@@ -77,5 +78,4 @@
 		<link name="${prefix}thumb_link2">
 			<visual>
-				<origin xyz="0 0 0" rpy="0 0 0"/>
 				<geometry>
 					<mesh filename="file://$(find theohand_description)/meshes/std16a/thumb_link2.glb"
@@ -84,5 +84,4 @@
 			</visual>
 			<collision>
-				<origin xyz="0 0 0" rpy="0 0 0"/>
 				<geometry>
 					<mesh filename="file://$(find theohand_description)/meshes/std16a/thumb_link2.glb"
@@ -143,5 +142,4 @@
 		<link name="${prefix}thumb_link4">
 			<visual>
-				<origin xyz="0 0 0" rpy="0 0 0"/>
 				<geometry>
 					<mesh filename="file://$(find theohand_description)/meshes/std16a/thumb_link4.glb"/>
@@ -149,5 +147,4 @@
 			</visual>
 			<collision>
-				<origin xyz="0 0 0" rpy="0 0 0"/>
 				<geometry>
 					<mesh filename="file://$(find theohand_description)/meshes/std16a/thumb_link4.glb"/>
@@ -174,12 +171,10 @@
 		<link name="${prefix}index_link1">
 			<visual>
-				<origin xyz="0 0 0" rpy="0 0 0"/>
-				<geometry>
-					<mesh filename="file://$(find theohand_description)/meshes/std16a/index_link1.glb"
-								scale="1 1 ${-direction}"/>
-				</geometry>
-			</visual>
-			<collision>
-				<origin xyz="0 0 0" rpy="0 0 0"/>
+				<geometry>
+					<mesh filename="file://$(find theohand_description)/meshes/std16a/index_link1.glb"
+								scale="1 1 ${-direction}"/>
+				</geometry>
+			</visual>
+			<collision>
 				<geometry>
 					<mesh filename="file://$(find theohand_description)/meshes/std16a/index_link1.glb"
@@ -207,12 +202,10 @@
 		<link name="${prefix}index_link2">
 			<visual>
-				<origin xyz="0 0 0" rpy="0 0 0"/>
-				<geometry>
-					<mesh filename="file://$(find theohand_description)/meshes/std16a/index_link2.glb"
-								scale="1 1 ${-direction}"/>
-				</geometry>
-			</visual>
-			<collision>
-				<origin xyz="0 0 0" rpy="0 0 0"/>
+				<geometry>
+					<mesh filename="file://$(find theohand_description)/meshes/std16a/index_link2.glb"
+								scale="1 1 ${-direction}"/>
+				</geometry>
+			</visual>
+			<collision>
 				<geometry>
 					<mesh filename="file://$(find theohand_description)/meshes/std16a/index_link2.glb"
@@ -240,11 +233,9 @@
 		<link name="${prefix}index_link3">
 			<visual>
-				<origin xyz="0 0 0" rpy="0 0 0"/>
-				<geometry>
-					<mesh filename="file://$(find theohand_description)/meshes/std16a/index_link3.glb"/>
-				</geometry>
-			</visual>
-			<collision>
-				<origin xyz="0 0 0" rpy="0 0 0"/>
+				<geometry>
+					<mesh filename="file://$(find theohand_description)/meshes/std16a/index_link3.glb"/>
+				</geometry>
+			</visual>
+			<collision>
 				<geometry>
 					<mesh filename="file://$(find theohand_description)/meshes/std16a/index_link3.glb"/>
@@ -271,12 +262,10 @@
 		<link name="${prefix}middle_link1">
 			<visual>
-				<origin xyz="0 0 0" rpy="0 0 0"/>
-				<geometry>
-					<mesh filename="file://$(find theohand_description)/meshes/std16a/index_link1.glb"
-								scale="1 1 ${-direction}"/>
-				</geometry>
-			</visual>
-			<collision>
-				<origin xyz="0 0 0" rpy="0 0 0"/>
+				<geometry>
+					<mesh filename="file://$(find theohand_description)/meshes/std16a/index_link1.glb"
+								scale="1 1 ${-direction}"/>
+				</geometry>
+			</visual>
+			<collision>
 				<geometry>
 					<mesh filename="file://$(find theohand_description)/meshes/std16a/index_link1.glb"
@@ -304,12 +293,10 @@
 		<link name="${prefix}middle_link2">
 			<visual>
-				<origin xyz="0 0 0" rpy="0 0 0"/>
-				<geometry>
-					<mesh filename="file://$(find theohand_description)/meshes/std16a/index_link2.glb"
-								scale="1 1 ${-direction}"/>
-				</geometry>
-			</visual>
-			<collision>
-				<origin xyz="0 0 0" rpy="0 0 0"/>
+				<geometry>
+					<mesh filename="file://$(find theohand_description)/meshes/std16a/index_link2.glb"
+								scale="1 1 ${-direction}"/>
+				</geometry>
+			</visual>
+			<collision>
 				<geometry>
 					<mesh filename="file://$(find theohand_description)/meshes/std16a/index_link2.glb"
@@ -337,11 +324,9 @@
 		<link name="${prefix}middle_link3">
 			<visual>
-				<origin xyz="0 0 0" rpy="0 0 0"/>
-				<geometry>
-					<mesh filename="file://$(find theohand_description)/meshes/std16a/index_link3.glb"/>
-				</geometry>
-			</visual>
-			<collision>
-				<origin xyz="0 0 0" rpy="0 0 0"/>
+				<geometry>
+					<mesh filename="file://$(find theohand_description)/meshes/std16a/index_link3.glb"/>
+				</geometry>
+			</visual>
+			<collision>
 				<geometry>
 					<mesh filename="file://$(find theohand_description)/meshes/std16a/index_link3.glb"/>
@@ -368,12 +353,10 @@
 		<link name="${prefix}ring_link1">
 			<visual>
-				<origin xyz="0 0 0" rpy="0 0 0"/>
-				<geometry>
-					<mesh filename="file://$(find theohand_description)/meshes/std16a/index_link1.glb"
-								scale="1 1 ${-direction}"/>
-				</geometry>
-			</visual>
-			<collision>
-				<origin xyz="0 0 0" rpy="0 0 0"/>
+				<geometry>
+					<mesh filename="file://$(find theohand_description)/meshes/std16a/index_link1.glb"
+								scale="1 1 ${-direction}"/>
+				</geometry>
+			</visual>
+			<collision>
 				<geometry>
 					<mesh filename="file://$(find theohand_description)/meshes/std16a/index_link1.glb"
@@ -401,12 +384,10 @@
 		<link name="${prefix}ring_link2">
 			<visual>
-				<origin xyz="0 0 0" rpy="0 0 0"/>
-				<geometry>
-					<mesh filename="file://$(find theohand_description)/meshes/std16a/index_link2.glb"
-								scale="1 1 ${-direction}"/>
-				</geometry>
-			</visual>
-			<collision>
-				<origin xyz="0 0 0" rpy="0 0 0"/>
+				<geometry>
+					<mesh filename="file://$(find theohand_description)/meshes/std16a/index_link2.glb"
+								scale="1 1 ${-direction}"/>
+				</geometry>
+			</visual>
+			<collision>
 				<geometry>
 					<mesh filename="file://$(find theohand_description)/meshes/std16a/index_link2.glb"
@@ -434,11 +415,9 @@
 		<link name="${prefix}ring_link3">
 			<visual>
-				<origin xyz="0 0 0" rpy="0 0 0"/>
-				<geometry>
-					<mesh filename="file://$(find theohand_description)/meshes/std16a/index_link3.glb"/>
-				</geometry>
-			</visual>
-			<collision>
-				<origin xyz="0 0 0" rpy="0 0 0"/>
+				<geometry>
+					<mesh filename="file://$(find theohand_description)/meshes/std16a/index_link3.glb"/>
+				</geometry>
+			</visual>
+			<collision>
 				<geometry>
 					<mesh filename="file://$(find theohand_description)/meshes/std16a/index_link3.glb"/>
@@ -465,12 +444,10 @@
 		<link name="${prefix}pinky_link1">
 			<visual>
-				<origin xyz="0 0 0" rpy="0 0 0"/>
-				<geometry>
-					<mesh filename="file://$(find theohand_description)/meshes/std16a/index_link1.glb"
-								scale="1 1 ${-direction}"/>
-				</geometry>
-			</visual>
-			<collision>
-				<origin xyz="0 0 0" rpy="0 0 0"/>
+				<geometry>
+					<mesh filename="file://$(find theohand_description)/meshes/std16a/index_link1.glb"
+								scale="1 1 ${-direction}"/>
+				</geometry>
+			</visual>
+			<collision>
 				<geometry>
 					<mesh filename="file://$(find theohand_description)/meshes/std16a/index_link1.glb"
@@ -498,12 +475,10 @@
 		<link name="${prefix}pinky_link2">
 			<visual>
-				<origin xyz="0 0 0" rpy="0 0 0"/>
-				<geometry>
-					<mesh filename="file://$(find theohand_description)/meshes/std16a/index_link2.glb"
-								scale="1 1 ${-direction}"/>
-				</geometry>
-			</visual>
-			<collision>
-				<origin xyz="0 0 0" rpy="0 0 0"/>
+				<geometry>
+					<mesh filename="file://$(find theohand_description)/meshes/std16a/index_link2.glb"
+								scale="1 1 ${-direction}"/>
+				</geometry>
+			</visual>
+			<collision>
 				<geometry>
 					<mesh filename="file://$(find theohand_description)/meshes/std16a/index_link2.glb"
@@ -531,11 +506,9 @@
 		<link name="${prefix}pinky_link3">
 			<visual>
-				<origin xyz="0 0 0" rpy="0 0 0"/>
-				<geometry>
-					<mesh filename="file://$(find theohand_description)/meshes/std16a/index_link3.glb"/>
-				</geometry>
-			</visual>
-			<collision>
-				<origin xyz="0 0 0" rpy="0 0 0"/>
+				<geometry>
+					<mesh filename="file://$(find theohand_description)/meshes/std16a/index_link3.glb"/>
+				</geometry>
+			</visual>
+			<collision>
 				<geometry>
 					<mesh filename="file://$(find theohand_description)/meshes/std16a/index_link3.glb"/>
