Commit message: 修改xacro增加flange

File: dexhands/theohand_description/xacro/std16a.xacro (robot description, xacro)
@@ -1,7 +1,60 @@
 <?xml version="1.0" encoding="utf-8"?>
 <robot xmlns:xacro="http://www.ros.org/wiki/xacro">
-	<xacro:macro name="TheoHandStd16A" params="name direction:=1 fixed_joints:=false">
+	<xacro:arg name="collider" default="simple"/>
+	<xacro:property name="collider_type" value="$(arg collider)"/>
+	<xacro:macro name="TheoHandStd16A_flange_simple_collision">
+		<xacro:if value="${collider_type == 'simple'}">
+			<collision>
+				<origin xyz="0 0 0.015"/>
+				<geometry>
+					<cylinder length="0.03" radius="0.045"/>
+				</geometry>
+			</collision>
+		</xacro:if>
+	</xacro:macro>
+	<xacro:macro name="TheoHandStd16A_base_simple_collision">
+		<xacro:if value="${collider_type == 'simple'}">
+			<collision>
+				<origin xyz="0.0 0.0 0.075"/>
+				<geometry>
+					<box size="0.11 0.095 0.12"/>
+				</geometry>
+			</collision>
+			<collision>
+				<origin xyz="-0.004 0.0 0.19"/>
+				<geometry>
+					<box size="0.09 0.06 0.13"/>
+				</geometry>
+			</collision>
+		</xacro:if>
+	</xacro:macro>
+	<xacro:macro name="TheoHandStd16A" params="name direction:=1 use_flange:=false fixed_joints:=false">
 		<xacro:property name="prefix" value="${name + '_' if name else ''}"/>
 		<xacro:property name="joint_type" value="${fixed_joints and 'fixed' or 'revolute'}"/>
+		<xacro:property name="PI" value="3.141592653589793"/>
+		<xacro:if value="${use_flange}">
+			<link name="${prefix}flange">
+				<inertial>
+					<origin xyz="-0.000388 0.002345 0.0"/>
+					<mass value="0.114"/>
+					<inertia ixx="0.000040105"
+									 ixy="0.0"
+									 ixz="0.0"
+									 iyy="0.000085776"
+									 iyz="0.0"
+									 izz="0.000054044"/>
+				</inertial>
+				<visual>
+					<geometry>
+					<mesh filename="file://$(find theohand_description)/meshes/std16a/flange.glb"/>
+					</geometry>
+				</visual>
+				<xacro:TheoHandStd16A_flange_simple_collision/>
+			</link>
+			<joint name="${prefix}flange_joint" type="fixed">
+				<parent link="${prefix}flange"/>
+				<child link="${prefix}hand_base"/>
+			</joint>
+		</xacro:if>
 		<link name="${prefix}hand_base"/>
 		<joint name="${prefix}hand_base_fixed" type="fixed">
@@ -16,12 +69,15 @@
 				</geometry>
 			</visual>
-			<collision>
-				<geometry>
+			<xacro:if value="${collider_type == 'convex'}">
+				<collision>
+					<geometry>
 					<mesh filename="file://$(find theohand_description)/meshes/std16a/base.glb"
 								scale="1 ${-direction} 1"/>
-				</geometry>
-			</collision>
-			<inertial>
-				<origin xyz="-0.00381424636269485 0.00207802750628399 0.0762957680404765" rpy="0 0 0"/>
+					</geometry>
+				</collision>
+			</xacro:if>
+			<xacro:TheoHandStd16A_base_simple_collision/>
+			<inertial>
+				<origin xyz="-0.00381424636269485 0.00207802750628399 0.0762957680404765"/>
 				<mass value="0.57109497006203"/>
 				<inertia ixx="0.000373948529416664"
@@ -42,5 +98,5 @@
 			<parent link="${prefix}base_link"/>
 			<child link="${prefix}thumb_link1"/>
-			<origin xyz="0.0305 ${direction*0.0002} ${0.049825 + direction*0.001475}" rpy="-1.5708 0 -1.5708"/>
+			<origin xyz="0.0305 ${direction*0.0002} ${0.049825 + direction*0.001475}" rpy="${-PI/2} 0 ${-PI/2}"/>
 			<xacro:unless value="${fixed_joints}">
 				<axis xyz="0 0 -1"/>
@@ -55,12 +111,14 @@
 				</geometry>
 			</visual>
-			<collision>
-				<geometry>
+			<xacro:if value="${collider_type == 'convex'}">
+				<collision>
+					<geometry>
 					<mesh filename="file://$(find theohand_description)/meshes/std16a/thumb_link1.glb"
 								scale="1 1 ${-direction}"/>
-				</geometry>
-			</collision>
-			<inertial>
-				<origin xyz="-0.00302015619783484 0.00158556016884966 0.00010450052403644" rpy="0 0 0"/>
+					</geometry>
+				</collision>
+			</xacro:if>
+			<inertial>
+				<origin xyz="-0.00302015619783484 0.00158556016884966 0.00010450052403644"/>
 				<mass value="0.00536774508646078"/>
 				<inertia ixx="1.62182890325478E-07"
@@ -75,8 +133,8 @@
 			<parent link="${prefix}thumb_link1"/>
 			<child link="${prefix}thumb_link2"/>
-			<origin xyz="0 0 0" rpy="1.5708 ${direction*1.5708} 0"/>
+			<origin xyz="0 0 0" rpy="${PI/2} ${direction*PI/2} 0"/>
 			<xacro:unless value="${fixed_joints}">
 				<axis xyz="0 0 ${direction}"/>
-				<limit lower="0" upper="1.5708" effort="0" velocity="0"/>
+				<limit lower="0" upper="${PI/2}" effort="0" velocity="0"/>
 			</xacro:unless>
 		</joint>
@@ -88,12 +146,14 @@
 				</geometry>
 			</visual>
-			<collision>
-				<geometry>
+			<xacro:if value="${collider_type == 'convex'}">
+				<collision>
+					<geometry>
 					<mesh filename="file://$(find theohand_description)/meshes/std16a/thumb_link2.glb"
 								scale="${-direction} 1 1"/>
-				</geometry>
-			</collision>
-			<inertial>
-				<origin xyz="0.00803208062854856 0.000160364028669376 -0.000106935756475329" rpy="0 0 0"/>
+					</geometry>
+				</collision>
+			</xacro:if>
+			<inertial>
+				<origin xyz="0.00803208062854856 0.000160364028669376 -0.000106935756475329"/>
 				<mass value="0.0623877025966598"/>
 				<inertia ixx="6.01468694889977E-06"
@@ -108,27 +168,27 @@
 			<parent link="${prefix}thumb_link2"/>
 			<child link="${prefix}thumb_link3"/>
-			<origin xyz="${direction*-0.0305} 0 0.00995" rpy="${direction*1.5708} ${(direction+1)*-0.7854} 0"/>
-			<xacro:unless value="${fixed_joints}">
-				<axis xyz="0 0 -1"/>
-				<limit lower="0" upper="1.5708" effort="0" velocity="0"/>
+			<origin xyz="${direction*-0.0305} 0 0.00995" rpy="${direction*PI/2} ${(direction+1)*-PI/4} 0"/>
+			<xacro:unless value="${fixed_joints}">
+				<axis xyz="0 0 -1"/>
+				<limit lower="0" upper="${PI/2}" effort="0" velocity="0"/>
 			</xacro:unless>
 		</joint>
 		<link name="${prefix}thumb_link3">
 			<visual>
-				<origin xyz="0 0 0" rpy="0 0 ${(direction+1)*0.7854}"/>
-				<geometry>
-					<mesh filename="file://$(find theohand_description)/meshes/std16a/thumb_link3.glb"
-								scale="1 1 ${-direction}"/>
-				</geometry>
-			</visual>
+				<origin xyz="0 0 0" rpy="0 0 ${(direction+1)*PI/4}"/>
+				<geometry>
+					<mesh filename="file://$(find theohand_description)/meshes/std16a/thumb_link3.glb"/>
+				</geometry>
+			</visual>
+			<xacro:if value="${collider_type == 'convex'}">
 			<collision>
-				<origin xyz="0 0 0" rpy="0 0 ${(direction+1)*0.7854}"/>
-				<geometry>
-					<mesh filename="file://$(find theohand_description)/meshes/std16a/thumb_link3.glb"
-								scale="1 1 ${-direction}"/>
-				</geometry>
-			</collision>
-			<inertial>
-				<origin xyz="0.0256802161872409 0.00960068824062393 1.30290134271738E-08" rpy="0 0 0"/>
+				<origin xyz="0 0 0" rpy="0 0 ${(direction+1)*PI/4}"/>
+				<geometry>
+					<mesh filename="file://$(find theohand_description)/meshes/std16a/thumb_link3.glb"/>
+					</geometry>
+				</collision>
+			</xacro:if>
+			<inertial>
+				<origin xyz="0.0256802161872409 0.00960068824062393 1.30290134271738E-08"/>
 				<mass value="0.0542172777399717"/>
 				<inertia ixx="3.35658095569514E-06"
@@ -143,8 +203,8 @@
 			<parent link="${prefix}thumb_link3"/>
 			<child link="${prefix}thumb_link4"/>
-			<origin xyz="${(1-direction)*0.02755} ${(direction+1)*0.02755} 0" rpy="0 0 ${(1-direction)*-0.7854}"/>
-			<xacro:unless value="${fixed_joints}">
-				<axis xyz="0 0 -1"/>
-				<limit lower="-0.610865" upper="1.48353" effort="0" velocity="0"/>
+			<origin xyz="${(1-direction)*0.02755} ${(direction+1)*0.02755} 0" rpy="0 0 ${(1-direction)*-PI/4}"/>
+			<xacro:unless value="${fixed_joints}">
+				<axis xyz="0 0 -1"/>
+				<limit lower="${-35*PI/180}" upper="${85*PI/180}" effort="0" velocity="0"/>
 			</xacro:unless>
 		</joint>
@@ -155,11 +215,13 @@
 				</geometry>
 			</visual>
-			<collision>
-				<geometry>
+			<xacro:if value="${collider_type == 'convex'}">
+				<collision>
+					<geometry>
 					<mesh filename="file://$(find theohand_description)/meshes/std16a/thumb_link4.glb"/>
-				</geometry>
-			</collision>
-			<inertial>
-				<origin xyz="-0.012255014618924 0.0137954013291241 2.15840115913926E-07" rpy="0 0 0"/>
+					</geometry>
+				</collision>
+			</xacro:if>
+			<inertial>
+				<origin xyz="-0.012255014618924 0.0137954013291241 2.15840115913926E-07"/>
 				<mass value="0.0231445815777574"/>
 				<inertia ixx="1.76157653282557E-06"
@@ -174,8 +236,8 @@
 			<parent link="${prefix}base_link"/>
 			<child link="${prefix}index_link1"/>
-			<origin xyz="${0.0306745 + direction*0.0001745} ${direction*0.008} 0.12775" rpy="1.5708 0 ${direction*1.5708}"/>
-			<xacro:unless value="${fixed_joints}">
-				<axis xyz="0 0 -1"/>
-				<limit lower="0" upper="1.5708" effort="0" velocity="0"/>
+			<origin xyz="${0.0306745 + direction*0.0001745} ${direction*0.008} 0.12775" rpy="${PI/2} 0 ${direction*PI/2}"/>
+			<xacro:unless value="${fixed_joints}">
+				<axis xyz="0 0 -1"/>
+				<limit lower="0" upper="${PI/2}" effort="0" velocity="0"/>
 			</xacro:unless>
 		</joint>
@@ -183,16 +245,16 @@
 			<visual>
 				<geometry>
-					<mesh filename="file://$(find theohand_description)/meshes/std16a/index_link1.glb"
-								scale="1 1 ${-direction}"/>
-				</geometry>
-			</visual>
-			<collision>
-				<geometry>
-					<mesh filename="file://$(find theohand_description)/meshes/std16a/index_link1.glb"
-								scale="1 1 ${-direction}"/>
-				</geometry>
-			</collision>
-			<inertial>
-				<origin xyz="-0.00968074774266574 0.02323760004207 2.33146973810383E-07" rpy="0 0 0"/>
+					<mesh filename="file://$(find theohand_description)/meshes/std16a/index_link1.glb"/>
+				</geometry>
+			</visual>
+			<xacro:if value="${collider_type == 'convex'}">
+				<collision>
+					<geometry>
+					<mesh filename="file://$(find theohand_description)/meshes/std16a/index_link1.glb"/>
+					</geometry>
+				</collision>
+			</xacro:if>
+			<inertial>
+				<origin xyz="-0.00968074774266574 0.02323760004207 2.33146973810383E-07"/>
 				<mass value="0.0482246598938861"/>
 				<inertia ixx="8.42297253866219E-06"
@@ -207,8 +269,8 @@
 			<parent link="${prefix}index_link1"/>
 			<child link="${prefix}index_link2"/>
-			<origin xyz="0 0.04435 ${(direction+1)*-0.0001743}" rpy="0 0 0"/>
-			<xacro:unless value="${fixed_joints}">
-				<axis xyz="0 0 -1"/>
-				<limit lower="0" upper="1.5708" effort="0" velocity="0"/>
+			<origin xyz="0 0.04435 ${(direction+1)*-0.0001743}"/>
+			<xacro:unless value="${fixed_joints}">
+				<axis xyz="0 0 -1"/>
+				<limit lower="0" upper="${PI/2}" effort="0" velocity="0"/>
 			</xacro:unless>
 		</joint>
@@ -216,16 +278,16 @@
 			<visual>
 				<geometry>
-					<mesh filename="file://$(find theohand_description)/meshes/std16a/index_link2.glb"
-								scale="1 1 ${-direction}"/>
-				</geometry>
-			</visual>
-			<collision>
-				<geometry>
-					<mesh filename="file://$(find theohand_description)/meshes/std16a/index_link2.glb"
-								scale="1 1 ${-direction}"/>
-				</geometry>
-			</collision>
-			<inertial>
-				<origin xyz="-0.00968074774266556 0.02323760004207 2.33146973845078E-07" rpy="0 0 0"/>
+					<mesh filename="file://$(find theohand_description)/meshes/std16a/index_link2.glb"/>
+				</geometry>
+			</visual>
+			<xacro:if value="${collider_type == 'convex'}">
+				<collision>
+					<geometry>
+					<mesh filename="file://$(find theohand_description)/meshes/std16a/index_link2.glb"/>
+					</geometry>
+				</collision>
+			</xacro:if>
+			<inertial>
+				<origin xyz="-0.00968074774266556 0.02323760004207 2.33146973845078E-07"/>
 				<mass value="0.048224659893886"/>
 				<inertia ixx="8.42297253866218E-06"
@@ -240,8 +302,8 @@
 			<parent link="${prefix}index_link2"/>
 			<child link="${prefix}index_link3"/>
-			<origin xyz="0 0.04435 0" rpy="0 0 0"/>
-			<xacro:unless value="${fixed_joints}">
-				<axis xyz="0 0 -1"/>
-				<limit lower="0" upper="1.5708" effort="0" velocity="0"/>
+			<origin xyz="0 0.04435 0"/>
+			<xacro:unless value="${fixed_joints}">
+				<axis xyz="0 0 -1"/>
+				<limit lower="0" upper="${PI/2}" effort="0" velocity="0"/>
 			</xacro:unless>
 		</joint>
@@ -252,11 +314,13 @@
 				</geometry>
 			</visual>
-			<collision>
-				<geometry>
-					<mesh filename="file://$(find theohand_description)/meshes/std16a/index_link3.glb"/>
-				</geometry>
-			</collision>
-			<inertial>
-				<origin xyz="-0.0122550144033681 0.0137954015029786 2.15837223926929E-07" rpy="0 0 0"/>
+			<xacro:if value="${collider_type == 'convex'}">
+				<collision>
+					<geometry>
+					<mesh filename="file://$(find theohand_description)/meshes/std16a/index_link3.glb"/>
+					</geometry>
+				</collision>
+			</xacro:if>
+			<inertial>
+				<origin xyz="-0.0122550144033681 0.0137954015029786 2.15837223926929E-07"/>
 				<mass value="0.0231445815514515"/>
 				<inertia ixx="1.76157653952119E-06"
@@ -271,8 +335,8 @@
 			<parent link="${prefix}base_link"/>
 			<child link="${prefix}middle_link1"/>
-			<origin xyz="0.0075 ${direction*0.008} 0.12775" rpy="1.5708 0 ${direction*1.5708}"/>
-			<xacro:unless value="${fixed_joints}">
-				<axis xyz="0 0 -1"/>
-				<limit lower="0" upper="1.5708" effort="0" velocity="0"/>
+			<origin xyz="0.0075 ${direction*0.008} 0.12775" rpy="${PI/2} 0 ${direction*PI/2}"/>
+			<xacro:unless value="${fixed_joints}">
+				<axis xyz="0 0 -1"/>
+				<limit lower="0" upper="${PI/2}" effort="0" velocity="0"/>
 			</xacro:unless>
 		</joint>
@@ -280,16 +344,16 @@
 			<visual>
 				<geometry>
-					<mesh filename="file://$(find theohand_description)/meshes/std16a/index_link1.glb"
-								scale="1 1 ${-direction}"/>
-				</geometry>
-			</visual>
-			<collision>
-				<geometry>
-					<mesh filename="file://$(find theohand_description)/meshes/std16a/index_link1.glb"
-								scale="1 1 ${-direction}"/>
-				</geometry>
-			</collision>
-			<inertial>
-				<origin xyz="-0.00968074774266573 0.0232376000420838 2.33146966274744E-07" rpy="0 0 0"/>
+					<mesh filename="file://$(find theohand_description)/meshes/std16a/index_link1.glb"/>
+				</geometry>
+			</visual>
+			<xacro:if value="${collider_type == 'convex'}">
+				<collision>
+					<geometry>
+					<mesh filename="file://$(find theohand_description)/meshes/std16a/index_link1.glb"/>
+					</geometry>
+				</collision>
+			</xacro:if>
+			<inertial>
+				<origin xyz="-0.00968074774266573 0.0232376000420838 2.33146966274744E-07"/>
 				<mass value="0.048224659893886"/>
 				<inertia ixx="8.42297253866217E-06"
@@ -304,8 +368,8 @@
 			<parent link="${prefix}middle_link1"/>
 			<child link="${prefix}middle_link2"/>
-			<origin xyz="0 0.04435 0" rpy="0 0 0"/>
-			<xacro:unless value="${fixed_joints}">
-				<axis xyz="0 0 -1"/>
-				<limit lower="0" upper="1.5708" effort="0" velocity="0"/>
+			<origin xyz="0 0.04435 0"/>
+			<xacro:unless value="${fixed_joints}">
+				<axis xyz="0 0 -1"/>
+				<limit lower="0" upper="${PI/2}" effort="0" velocity="0"/>
 			</xacro:unless>
 		</joint>
@@ -313,16 +377,16 @@
 			<visual>
 				<geometry>
-					<mesh filename="file://$(find theohand_description)/meshes/std16a/index_link2.glb"
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