Commit message: fix the mesh filename path

File: dexhands/wuji_description/xacro/hand1.xacro (robot description, xacro)
@@ -21,14 +21,14 @@
         <origin xyz="0 0 0" rpy="0 0 0"/>
         <geometry>
-          <mesh filename="package://wuji_description/meshes/hand1/${mesh_side}/${mesh_side}_palm_link.STL"/>
-        </geometry>
-        <material name="">
-          <color rgba="0.627451 0.627451 0.627451 1"/>
-        </material>
-      </visual>
-      <collision>
-        <origin xyz="0 0 0" rpy="0 0 0"/>
-        <geometry>
-          <mesh filename="package://wuji_description/meshes/hand1/${mesh_side}/${mesh_side}_palm_link.STL"/>
+          <mesh filename="file://$(find wuji_description)/meshes/hand1/${mesh_side}/${mesh_side}_palm_link.STL"/>
+        </geometry>
+        <material name="">
+          <color rgba="0.627451 0.627451 0.627451 1"/>
+        </material>
+      </visual>
+      <collision>
+        <origin xyz="0 0 0" rpy="0 0 0"/>
+        <geometry>
+          <mesh filename="file://$(find wuji_description)/meshes/hand1/${mesh_side}/${mesh_side}_palm_link.STL"/>
         </geometry>
       </collision>
@@ -43,14 +43,14 @@
         <origin xyz="0 0 0" rpy="0 0 0"/>
         <geometry>
-          <mesh filename="package://wuji_description/meshes/hand1/${mesh_side}/${mesh_side}_finger1_link1.STL"/>
-        </geometry>
-        <material name="">
-          <color rgba="0.627451 0.627451 0.627451 1"/>
-        </material>
-      </visual>
-      <collision>
-        <origin xyz="0 0 0" rpy="0 0 0"/>
-        <geometry>
-          <mesh filename="package://wuji_description/meshes/hand1/${mesh_side}/${mesh_side}_finger1_link1.STL"/>
+          <mesh filename="file://$(find wuji_description)/meshes/hand1/${mesh_side}/${mesh_side}_finger1_link1.STL"/>
+        </geometry>
+        <material name="">
+          <color rgba="0.627451 0.627451 0.627451 1"/>
+        </material>
+      </visual>
+      <collision>
+        <origin xyz="0 0 0" rpy="0 0 0"/>
+        <geometry>
+          <mesh filename="file://$(find wuji_description)/meshes/hand1/${mesh_side}/${mesh_side}_finger1_link1.STL"/>
         </geometry>
       </collision>
@@ -74,14 +74,14 @@
         <origin xyz="0 0 0" rpy="0 0 0"/>
         <geometry>
-          <mesh filename="package://wuji_description/meshes/hand1/${mesh_side}/${mesh_side}_finger1_link2.STL"/>
-        </geometry>
-        <material name="">
-          <color rgba="0.627451 0.627451 0.627451 1"/>
-        </material>
-      </visual>
-      <collision>
-        <origin xyz="0 0 0" rpy="0 0 0"/>
-        <geometry>
-          <mesh filename="package://wuji_description/meshes/hand1/${mesh_side}/${mesh_side}_finger1_link2.STL"/>
+          <mesh filename="file://$(find wuji_description)/meshes/hand1/${mesh_side}/${mesh_side}_finger1_link2.STL"/>
+        </geometry>
+        <material name="">
+          <color rgba="0.627451 0.627451 0.627451 1"/>
+        </material>
+      </visual>
+      <collision>
+        <origin xyz="0 0 0" rpy="0 0 0"/>
+        <geometry>
+          <mesh filename="file://$(find wuji_description)/meshes/hand1/${mesh_side}/${mesh_side}_finger1_link2.STL"/>
         </geometry>
       </collision>
@@ -105,14 +105,14 @@
         <origin xyz="0 0 0" rpy="0 0 0"/>
         <geometry>
-          <mesh filename="package://wuji_description/meshes/hand1/${mesh_side}/${mesh_side}_finger1_link3.STL"/>
-        </geometry>
-        <material name="">
-          <color rgba="0.627451 0.627451 0.627451 1"/>
-        </material>
-      </visual>
-      <collision>
-        <origin xyz="0 0 0" rpy="0 0 0"/>
-        <geometry>
-          <mesh filename="package://wuji_description/meshes/hand1/${mesh_side}/${mesh_side}_finger1_link3.STL"/>
+          <mesh filename="file://$(find wuji_description)/meshes/hand1/${mesh_side}/${mesh_side}_finger1_link3.STL"/>
+        </geometry>
+        <material name="">
+          <color rgba="0.627451 0.627451 0.627451 1"/>
+        </material>
+      </visual>
+      <collision>
+        <origin xyz="0 0 0" rpy="0 0 0"/>
+        <geometry>
+          <mesh filename="file://$(find wuji_description)/meshes/hand1/${mesh_side}/${mesh_side}_finger1_link3.STL"/>
         </geometry>
       </collision>
@@ -136,14 +136,14 @@
         <origin xyz="0 0 0" rpy="0 0 0"/>
         <geometry>
-          <mesh filename="package://wuji_description/meshes/hand1/${mesh_side}/${mesh_side}_finger1_link4.STL"/>
-        </geometry>
-        <material name="">
-          <color rgba="0.5294118 0.5490196 0.5490196 1"/>
-        </material>
-      </visual>
-      <collision>
-        <origin xyz="0 0 0" rpy="0 0 0"/>
-        <geometry>
-          <mesh filename="package://wuji_description/meshes/hand1/${mesh_side}/${mesh_side}_finger1_link4.STL"/>
+          <mesh filename="file://$(find wuji_description)/meshes/hand1/${mesh_side}/${mesh_side}_finger1_link4.STL"/>
+        </geometry>
+        <material name="">
+          <color rgba="0.5294118 0.5490196 0.5490196 1"/>
+        </material>
+      </visual>
+      <collision>
+        <origin xyz="0 0 0" rpy="0 0 0"/>
+        <geometry>
+          <mesh filename="file://$(find wuji_description)/meshes/hand1/${mesh_side}/${mesh_side}_finger1_link4.STL"/>
         </geometry>
       </collision>
@@ -167,14 +167,14 @@
         <origin xyz="0 0 0" rpy="0 0 0"/>
         <geometry>
-          <mesh filename="package://wuji_description/meshes/hand1/${mesh_side}/${mesh_side}_finger1_tip_link.STL"/>
-        </geometry>
-        <material name="">
-          <color rgba="0.5294118 0.5490196 0.5490196 1"/>
-        </material>
-      </visual>
-      <collision>
-        <origin xyz="0 0 0" rpy="0 0 0"/>
-        <geometry>
-          <mesh filename="package://wuji_description/meshes/hand1/${mesh_side}/${mesh_side}_finger1_tip_link.STL"/>
+          <mesh filename="file://$(find wuji_description)/meshes/hand1/${mesh_side}/${mesh_side}_finger1_tip_link.STL"/>
+        </geometry>
+        <material name="">
+          <color rgba="0.5294118 0.5490196 0.5490196 1"/>
+        </material>
+      </visual>
+      <collision>
+        <origin xyz="0 0 0" rpy="0 0 0"/>
+        <geometry>
+          <mesh filename="file://$(find wuji_description)/meshes/hand1/${mesh_side}/${mesh_side}_finger1_tip_link.STL"/>
         </geometry>
       </collision>
@@ -194,14 +194,14 @@
         <origin xyz="0 0 0" rpy="0 0 0"/>
         <geometry>
-          <mesh filename="package://wuji_description/meshes/hand1/${mesh_side}/${mesh_side}_digit_link1.STL"/>
-        </geometry>
-        <material name="">
-          <color rgba="0.627451 0.627451 0.627451 1"/>
-        </material>
-      </visual>
-      <collision>
-        <origin xyz="0 0 0" rpy="0 0 0"/>
-        <geometry>
-          <mesh filename="package://wuji_description/meshes/hand1/${mesh_side}/${mesh_side}_digit_link1.STL"/>
+          <mesh filename="file://$(find wuji_description)/meshes/hand1/${mesh_side}/${mesh_side}_digit_link1.STL"/>
+        </geometry>
+        <material name="">
+          <color rgba="0.627451 0.627451 0.627451 1"/>
+        </material>
+      </visual>
+      <collision>
+        <origin xyz="0 0 0" rpy="0 0 0"/>
+        <geometry>
+          <mesh filename="file://$(find wuji_description)/meshes/hand1/${mesh_side}/${mesh_side}_digit_link1.STL"/>
         </geometry>
       </collision>
@@ -225,14 +225,14 @@
         <origin xyz="0 0 0" rpy="0 0 0"/>
         <geometry>
-          <mesh filename="package://wuji_description/meshes/hand1/${mesh_side}/${mesh_side}_digit_link2.STL"/>
-        </geometry>
-        <material name="">
-          <color rgba="0.627451 0.627451 0.627451 1"/>
-        </material>
-      </visual>
-      <collision>
-        <origin xyz="0 0 0" rpy="0 0 0"/>
-        <geometry>
-          <mesh filename="package://wuji_description/meshes/hand1/${mesh_side}/${mesh_side}_digit_link2.STL"/>
+          <mesh filename="file://$(find wuji_description)/meshes/hand1/${mesh_side}/${mesh_side}_digit_link2.STL"/>
+        </geometry>
+        <material name="">
+          <color rgba="0.627451 0.627451 0.627451 1"/>
+        </material>
+      </visual>
+      <collision>
+        <origin xyz="0 0 0" rpy="0 0 0"/>
+        <geometry>
+          <mesh filename="file://$(find wuji_description)/meshes/hand1/${mesh_side}/${mesh_side}_digit_link2.STL"/>
         </geometry>
       </collision>
@@ -256,14 +256,14 @@
         <origin xyz="0 0 0" rpy="0 0 0"/>
         <geometry>
-          <mesh filename="package://wuji_description/meshes/hand1/${mesh_side}/${mesh_side}_digit_link3.STL"/>
-        </geometry>
-        <material name="">
-          <color rgba="0.627451 0.627451 0.627451 1"/>
-        </material>
-      </visual>
-      <collision>
-        <origin xyz="0 0 0" rpy="0 0 0"/>
-        <geometry>
-          <mesh filename="package://wuji_description/meshes/hand1/${mesh_side}/${mesh_side}_digit_link3.STL"/>
+          <mesh filename="file://$(find wuji_description)/meshes/hand1/${mesh_side}/${mesh_side}_digit_link3.STL"/>
+        </geometry>
+        <material name="">
+          <color rgba="0.627451 0.627451 0.627451 1"/>
+        </material>
+      </visual>
+      <collision>
+        <origin xyz="0 0 0" rpy="0 0 0"/>
+        <geometry>
+          <mesh filename="file://$(find wuji_description)/meshes/hand1/${mesh_side}/${mesh_side}_digit_link3.STL"/>
         </geometry>
       </collision>
@@ -287,14 +287,14 @@
         <origin xyz="0 0 0" rpy="0 0 0"/>
         <geometry>
-          <mesh filename="package://wuji_description/meshes/hand1/${mesh_side}/${mesh_side}_digit_link4.STL"/>
-        </geometry>
-        <material name="">
-          <color rgba="0.5294118 0.5490196 0.5490196 1"/>
-        </material>
-      </visual>
-      <collision>
-        <origin xyz="0 0 0" rpy="0 0 0"/>
-        <geometry>
-          <mesh filename="package://wuji_description/meshes/hand1/${mesh_side}/${mesh_side}_digit_link4.STL"/>
+          <mesh filename="file://$(find wuji_description)/meshes/hand1/${mesh_side}/${mesh_side}_digit_link4.STL"/>
+        </geometry>
+        <material name="">
+          <color rgba="0.5294118 0.5490196 0.5490196 1"/>
+        </material>
+      </visual>
+      <collision>
+        <origin xyz="0 0 0" rpy="0 0 0"/>
+        <geometry>
+          <mesh filename="file://$(find wuji_description)/meshes/hand1/${mesh_side}/${mesh_side}_digit_link4.STL"/>
         </geometry>
       </collision>
@@ -318,14 +318,14 @@
         <origin xyz="0 0 0" rpy="0 0 0"/>
         <geometry>
-          <mesh filename="package://wuji_description/meshes/hand1/${mesh_side}/${mesh_side}_digit_tip_link.STL"/>
-        </geometry>
-        <material name="">
-          <color rgba="0.5294118 0.5490196 0.5490196 1"/>
-        </material>
-      </visual>
-      <collision>
-        <origin xyz="0 0 0" rpy="0 0 0"/>
-        <geometry>
-          <mesh filename="package://wuji_description/meshes/hand1/${mesh_side}/${mesh_side}_digit_tip_link.STL"/>
+          <mesh filename="file://$(find wuji_description)/meshes/hand1/${mesh_side}/${mesh_side}_digit_tip_link.STL"/>
+        </geometry>
+        <material name="">
+          <color rgba="0.5294118 0.5490196 0.5490196 1"/>
+        </material>
+      </visual>
+      <collision>
+        <origin xyz="0 0 0" rpy="0 0 0"/>
+        <geometry>
+          <mesh filename="file://$(find wuji_description)/meshes/hand1/${mesh_side}/${mesh_side}_digit_tip_link.STL"/>
         </geometry>
       </collision>
@@ -345,14 +345,14 @@
         <origin xyz="0 0 0" rpy="0 0 0"/>
         <geometry>
-          <mesh filename="package://wuji_description/meshes/hand1/${mesh_side}/${mesh_side}_digit_link1.STL"/>
-        </geometry>
-        <material name="">
-          <color rgba="0.627451 0.627451 0.627451 1"/>
-        </material>
-      </visual>
-      <collision>
-        <origin xyz="0 0 0" rpy="0 0 0"/>
-        <geometry>
-          <mesh filename="package://wuji_description/meshes/hand1/${mesh_side}/${mesh_side}_digit_link1.STL"/>
+          <mesh filename="file://$(find wuji_description)/meshes/hand1/${mesh_side}/${mesh_side}_digit_link1.STL"/>
+        </geometry>
+        <material name="">
+          <color rgba="0.627451 0.627451 0.627451 1"/>
+        </material>
+      </visual>
+      <collision>
+        <origin xyz="0 0 0" rpy="0 0 0"/>
+        <geometry>
+          <mesh filename="file://$(find wuji_description)/meshes/hand1/${mesh_side}/${mesh_side}_digit_link1.STL"/>
         </geometry>
       </collision>
@@ -376,14 +376,14 @@
         <origin xyz="0 0 0" rpy="0 0 0"/>
         <geometry>
-          <mesh filename="package://wuji_description/meshes/hand1/${mesh_side}/${mesh_side}_digit_link2.STL"/>
-        </geometry>
-        <material name="">
-          <color rgba="0.627451 0.627451 0.627451 1"/>
-        </material>
-      </visual>
-      <collision>
-        <origin xyz="0 0 0" rpy="0 0 0"/>
-        <geometry>
-          <mesh filename="package://wuji_description/meshes/hand1/${mesh_side}/${mesh_side}_digit_link2.STL"/>
+          <mesh filename="file://$(find wuji_description)/meshes/hand1/${mesh_side}/${mesh_side}_digit_link2.STL"/>
+        </geometry>
+        <material name="">
+          <color rgba="0.627451 0.627451 0.627451 1"/>
+        </material>
+      </visual>
+      <collision>
+        <origin xyz="0 0 0" rpy="0 0 0"/>
+        <geometry>
+          <mesh filename="file://$(find wuji_description)/meshes/hand1/${mesh_side}/${mesh_side}_digit_link2.STL"/>
         </geometry>
       </collision>
@@ -407,14 +407,14 @@
         <origin xyz="0 0 0" rpy="0 0 0"/>
         <geometry>
-          <mesh filename="package://wuji_description/meshes/hand1/${mesh_side}/${mesh_side}_digit_link3.STL"/>
-        </geometry>
-        <material name="">
-          <color rgba="0.627451 0.627451 0.627451 1"/>
-        </material>
-      </visual>
-      <collision>
-        <origin xyz="0 0 0" rpy="0 0 0"/>
-        <geometry>
-          <mesh filename="package://wuji_description/meshes/hand1/${mesh_side}/${mesh_side}_digit_link3.STL"/>
+          <mesh filename="file://$(find wuji_description)/meshes/hand1/${mesh_side}/${mesh_side}_digit_link3.STL"/>
+        </geometry>
+        <material name="">
+          <color rgba="0.627451 0.627451 0.627451 1"/>
+        </material>
+      </visual>
+      <collision>
+        <origin xyz="0 0 0" rpy="0 0 0"/>
+        <geometry>
+          <mesh filename="file://$(find wuji_description)/meshes/hand1/${mesh_side}/${mesh_side}_digit_link3.STL"/>
         </geometry>
       </collision>
@@ -438,14 +438,14 @@
         <origin xyz="0 0 0" rpy="0 0 0"/>
         <geometry>
-          <mesh filename="package://wuji_description/meshes/hand1/${mesh_side}/${mesh_side}_digit_link4.STL"/>
-        </geometry>
-        <material name="">
-          <color rgba="0.5294118 0.5490196 0.5490196 1"/>
-        </material>
-      </visual>
-      <collision>
-        <origin xyz="0 0 0" rpy="0 0 0"/>
-        <geometry>
-          <mesh filename="package://wuji_description/meshes/hand1/${mesh_side}/${mesh_side}_digit_link4.STL"/>
+          <mesh filename="file://$(find wuji_description)/meshes/hand1/${mesh_side}/${mesh_side}_digit_link4.STL"/>
+        </geometry>
+        <material name="">
+          <color rgba="0.5294118 0.5490196 0.5490196 1"/>
+        </material>
+      </visual>
+      <collision>
+        <origin xyz="0 0 0" rpy="0 0 0"/>
+        <geometry>
+          <mesh filename="file://$(find wuji_description)/meshes/hand1/${mesh_side}/${mesh_side}_digit_link4.STL"/>
         </geometry>
       </collision>
@@ -469,14 +469,14 @@
         <origin xyz="0 0 0" rpy="0 0 0"/>
         <geometry>
-          <mesh filename="package://wuji_description/meshes/hand1/${mesh_side}/${mesh_side}_digit_tip_link.STL"/>
-        </geometry>
-        <material name="">
-          <color rgba="0.5294118 0.5490196 0.5490196 1"/>
-        </material>
-      </visual>
-      <collision>
-        <origin xyz="0 0 0" rpy="0 0 0"/>
-        <geometry>
-          <mesh filename="package://wuji_description/meshes/hand1/${mesh_side}/${mesh_side}_digit_tip_link.STL"/>
+          <mesh filename="file://$(find wuji_description)/meshes/hand1/${mesh_side}/${mesh_side}_digit_tip_link.STL"/>
+        </geometry>
+        <material name="">
+          <color rgba="0.5294118 0.5490196 0.5490196 1"/>
+        </material>
+      </visual>
+      <collision>
+        <origin xyz="0 0 0" rpy="0 0 0"/>
+        <geometry>
+          <mesh filename="file://$(find wuji_description)/meshes/hand1/${mesh_side}/${mesh_side}_digit_tip_link.STL"/>
         </geometry>
       </collision>
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