Commit message: fix the mesh filename path

File: dexhands/wuji_description/xacro/hand2.xacro (robot description, xacro)
@@ -25,5 +25,5 @@
         <origin xyz="0 0 0" rpy="0 0 0"/>
         <geometry>
-          <mesh filename="package://wuji_description/meshes/hand2/left/l_mount.STL" scale="1 ${direction} 1"/>
+          <mesh filename="file://$(find wuji_description)/meshes/hand2/left/l_mount.STL" scale="1 ${direction} 1"/>
         </geometry>
         <material name="">
@@ -34,5 +34,5 @@
         <origin xyz="0 0 0" rpy="0 0 0"/>
         <geometry>
-          <mesh filename="package://wuji_description/meshes/hand2/left/l_mount.STL" scale="1 ${direction} 1"/>
+          <mesh filename="file://$(find wuji_description)/meshes/hand2/left/l_mount.STL" scale="1 ${direction} 1"/>
         </geometry>
       </collision>
@@ -68,5 +68,5 @@
         <origin xyz="0 0 0" rpy="0 0 0"/>
         <geometry>
-          <mesh filename="package://wuji_description/meshes/hand2/left/l_wrist.STL" scale="1 ${direction} 1"/>
+          <mesh filename="file://$(find wuji_description)/meshes/hand2/left/l_wrist.STL" scale="1 ${direction} 1"/>
         </geometry>
         <material name="">
@@ -77,5 +77,5 @@
         <origin xyz="0 0 0" rpy="0 0 0"/>
         <geometry>
-          <mesh filename="package://wuji_description/meshes/hand2/left/l_wrist.STL" scale="1 ${direction} 1"/>
+          <mesh filename="file://$(find wuji_description)/meshes/hand2/left/l_wrist.STL" scale="1 ${direction} 1"/>
         </geometry>
       </collision>
@@ -90,5 +90,5 @@
         <origin xyz="0 0 0" rpy="0 0 0"/>
         <geometry>
-          <mesh filename="package://wuji_description/meshes/hand2/left/l_thumb_proximal.STL" scale="1 ${direction} 1"/>
+          <mesh filename="file://$(find wuji_description)/meshes/hand2/left/l_thumb_proximal.STL" scale="1 ${direction} 1"/>
         </geometry>
         <material name="">
@@ -99,5 +99,5 @@
         <origin xyz="0 0 0" rpy="0 0 0"/>
         <geometry>
-          <mesh filename="package://wuji_description/meshes/hand2/left/l_thumb_proximal.STL" scale="1 ${direction} 1"/>
+          <mesh filename="file://$(find wuji_description)/meshes/hand2/left/l_thumb_proximal.STL" scale="1 ${direction} 1"/>
         </geometry>
       </collision>
@@ -121,5 +121,5 @@
         <origin xyz="0 0 0" rpy="0 0 0"/>
         <geometry>
-          <mesh filename="package://wuji_description/meshes/hand2/left/l_thumb_proximal_abd.STL" scale="1 ${direction} 1"/>
+          <mesh filename="file://$(find wuji_description)/meshes/hand2/left/l_thumb_proximal_abd.STL" scale="1 ${direction} 1"/>
         </geometry>
         <material name="">
@@ -130,5 +130,5 @@
         <origin xyz="0 0 0" rpy="0 0 0"/>
         <geometry>
-          <mesh filename="package://wuji_description/meshes/hand2/left/l_thumb_proximal_abd.STL" scale="1 ${direction} 1"/>
+          <mesh filename="file://$(find wuji_description)/meshes/hand2/left/l_thumb_proximal_abd.STL" scale="1 ${direction} 1"/>
         </geometry>
       </collision>
@@ -152,5 +152,5 @@
         <origin xyz="0 0 0" rpy="0 0 0"/>
         <geometry>
-          <mesh filename="package://wuji_description/meshes/hand2/left/l_thumb_middle.STL" scale="1 ${direction} 1"/>
+          <mesh filename="file://$(find wuji_description)/meshes/hand2/left/l_thumb_middle.STL" scale="1 ${direction} 1"/>
         </geometry>
         <material name="">
@@ -161,5 +161,5 @@
         <origin xyz="0 0 0" rpy="0 0 0"/>
         <geometry>
-          <mesh filename="package://wuji_description/meshes/hand2/left/l_thumb_middle.STL" scale="1 ${direction} 1"/>
+          <mesh filename="file://$(find wuji_description)/meshes/hand2/left/l_thumb_middle.STL" scale="1 ${direction} 1"/>
         </geometry>
       </collision>
@@ -183,5 +183,5 @@
         <origin xyz="0 0 0" rpy="0 0 0"/>
         <geometry>
-          <mesh filename="package://wuji_description/meshes/hand2/left/l_thumb_distal.STL" scale="1 ${direction} 1"/>
+          <mesh filename="file://$(find wuji_description)/meshes/hand2/left/l_thumb_distal.STL" scale="1 ${direction} 1"/>
         </geometry>
         <material name="">
@@ -192,5 +192,5 @@
         <origin xyz="0 0 0" rpy="0 0 0"/>
         <geometry>
-          <mesh filename="package://wuji_description/meshes/hand2/left/l_thumb_distal.STL" scale="1 ${direction} 1"/>
+          <mesh filename="file://$(find wuji_description)/meshes/hand2/left/l_thumb_distal.STL" scale="1 ${direction} 1"/>
         </geometry>
       </collision>
@@ -220,5 +220,5 @@
         <origin xyz="0 0 0" rpy="0 0 0"/>
         <geometry>
-          <mesh filename="package://wuji_description/meshes/hand2/left/l_thumb_tip_sensor_frame.STL" scale="1 ${direction} 1"/>
+          <mesh filename="file://$(find wuji_description)/meshes/hand2/left/l_thumb_tip_sensor_frame.STL" scale="1 ${direction} 1"/>
         </geometry>
         <material name="">
@@ -229,5 +229,5 @@
         <origin xyz="0 0 0" rpy="0 0 0"/>
         <geometry>
-          <mesh filename="package://wuji_description/meshes/hand2/left/l_thumb_tip_sensor_frame.STL" scale="1 ${direction} 1"/>
+          <mesh filename="file://$(find wuji_description)/meshes/hand2/left/l_thumb_tip_sensor_frame.STL" scale="1 ${direction} 1"/>
         </geometry>
       </collision>
@@ -247,14 +247,14 @@
         <origin xyz="0 0 0" rpy="0 0 0"/>
         <geometry>
-          <mesh filename="package://wuji_description/meshes/hand2/left/l_digit_proximal.STL" scale="1 ${direction} 1"/>
-        </geometry>
-        <material name="">
-          <color rgba="1 1 1 1"/>
-        </material>
-      </visual>
-      <collision>
-        <origin xyz="0 0 0" rpy="0 0 0"/>
-        <geometry>
-          <mesh filename="package://wuji_description/meshes/hand2/left/l_digit_proximal.STL" scale="1 ${direction} 1"/>
+          <mesh filename="file://$(find wuji_description)/meshes/hand2/left/l_digit_proximal.STL" scale="1 ${direction} 1"/>
+        </geometry>
+        <material name="">
+          <color rgba="1 1 1 1"/>
+        </material>
+      </visual>
+      <collision>
+        <origin xyz="0 0 0" rpy="0 0 0"/>
+        <geometry>
+          <mesh filename="file://$(find wuji_description)/meshes/hand2/left/l_digit_proximal.STL" scale="1 ${direction} 1"/>
         </geometry>
       </collision>
@@ -278,14 +278,14 @@
         <origin xyz="0 0 0" rpy="0 0 0"/>
         <geometry>
-          <mesh filename="package://wuji_description/meshes/hand2/left/l_digit_proximal_abd.STL" scale="1 ${direction} 1"/>
-        </geometry>
-        <material name="">
-          <color rgba="1 1 1 1"/>
-        </material>
-      </visual>
-      <collision>
-        <origin xyz="0 0 0" rpy="0 0 0"/>
-        <geometry>
-          <mesh filename="package://wuji_description/meshes/hand2/left/l_digit_proximal_abd.STL" scale="1 ${direction} 1"/>
+          <mesh filename="file://$(find wuji_description)/meshes/hand2/left/l_digit_proximal_abd.STL" scale="1 ${direction} 1"/>
+        </geometry>
+        <material name="">
+          <color rgba="1 1 1 1"/>
+        </material>
+      </visual>
+      <collision>
+        <origin xyz="0 0 0" rpy="0 0 0"/>
+        <geometry>
+          <mesh filename="file://$(find wuji_description)/meshes/hand2/left/l_digit_proximal_abd.STL" scale="1 ${direction} 1"/>
         </geometry>
       </collision>
@@ -309,14 +309,14 @@
         <origin xyz="0 0 0" rpy="0 0 0"/>
         <geometry>
-          <mesh filename="package://wuji_description/meshes/hand2/left/l_digit_middle.STL" scale="1 ${direction} 1"/>
-        </geometry>
-        <material name="">
-          <color rgba="1 1 1 1"/>
-        </material>
-      </visual>
-      <collision>
-        <origin xyz="0 0 0" rpy="0 0 0"/>
-        <geometry>
-          <mesh filename="package://wuji_description/meshes/hand2/left/l_digit_middle.STL" scale="1 ${direction} 1"/>
+          <mesh filename="file://$(find wuji_description)/meshes/hand2/left/l_digit_middle.STL" scale="1 ${direction} 1"/>
+        </geometry>
+        <material name="">
+          <color rgba="1 1 1 1"/>
+        </material>
+      </visual>
+      <collision>
+        <origin xyz="0 0 0" rpy="0 0 0"/>
+        <geometry>
+          <mesh filename="file://$(find wuji_description)/meshes/hand2/left/l_digit_middle.STL" scale="1 ${direction} 1"/>
         </geometry>
       </collision>
@@ -340,5 +340,5 @@
         <origin xyz="0 0 0" rpy="0 0 0"/>
         <geometry>
-          <mesh filename="package://wuji_description/meshes/hand2/left/l_digit_distal.STL" scale="1 ${direction} 1"/>
+          <mesh filename="file://$(find wuji_description)/meshes/hand2/left/l_digit_distal.STL" scale="1 ${direction} 1"/>
         </geometry>
         <material name="">
@@ -349,5 +349,5 @@
         <origin xyz="0 0 0" rpy="0 0 0"/>
         <geometry>
-          <mesh filename="package://wuji_description/meshes/hand2/left/l_digit_distal.STL" scale="1 ${direction} 1"/>
+          <mesh filename="file://$(find wuji_description)/meshes/hand2/left/l_digit_distal.STL" scale="1 ${direction} 1"/>
         </geometry>
       </collision>
@@ -377,5 +377,5 @@
         <origin xyz="0 0 0" rpy="0 0 0"/>
         <geometry>
-          <mesh filename="package://wuji_description/meshes/hand2/left/l_digit_tip_sensor_frame.STL" scale="1 ${direction} 1"/>
+          <mesh filename="file://$(find wuji_description)/meshes/hand2/left/l_digit_tip_sensor_frame.STL" scale="1 ${direction} 1"/>
         </geometry>
         <material name="">
@@ -386,5 +386,5 @@
         <origin xyz="0 0 0" rpy="0 0 0"/>
         <geometry>
-          <mesh filename="package://wuji_description/meshes/hand2/left/l_digit_tip_sensor_frame.STL" scale="1 ${direction} 1"/>
+          <mesh filename="file://$(find wuji_description)/meshes/hand2/left/l_digit_tip_sensor_frame.STL" scale="1 ${direction} 1"/>
         </geometry>
       </collision>
@@ -404,14 +404,14 @@
         <origin xyz="0 0 0" rpy="0 0 0"/>
         <geometry>
-          <mesh filename="package://wuji_description/meshes/hand2/left/l_digit_proximal.STL" scale="1 ${direction} 1"/>
-        </geometry>
-        <material name="">
-          <color rgba="1 1 1 1"/>
-        </material>
-      </visual>
-      <collision>
-        <origin xyz="0 0 0" rpy="0 0 0"/>
-        <geometry>
-          <mesh filename="package://wuji_description/meshes/hand2/left/l_digit_proximal.STL" scale="1 ${direction} 1"/>
+          <mesh filename="file://$(find wuji_description)/meshes/hand2/left/l_digit_proximal.STL" scale="1 ${direction} 1"/>
+        </geometry>
+        <material name="">
+          <color rgba="1 1 1 1"/>
+        </material>
+      </visual>
+      <collision>
+        <origin xyz="0 0 0" rpy="0 0 0"/>
+        <geometry>
+          <mesh filename="file://$(find wuji_description)/meshes/hand2/left/l_digit_proximal.STL" scale="1 ${direction} 1"/>
         </geometry>
       </collision>
@@ -435,14 +435,14 @@
         <origin xyz="0 0 0" rpy="0 0 0"/>
         <geometry>
-          <mesh filename="package://wuji_description/meshes/hand2/left/l_digit_proximal_abd.STL" scale="1 ${direction} 1"/>
-        </geometry>
-        <material name="">
-          <color rgba="1 1 1 1"/>
-        </material>
-      </visual>
-      <collision>
-        <origin xyz="0 0 0" rpy="0 0 0"/>
-        <geometry>
-          <mesh filename="package://wuji_description/meshes/hand2/left/l_digit_proximal_abd.STL" scale="1 ${direction} 1"/>
+          <mesh filename="file://$(find wuji_description)/meshes/hand2/left/l_digit_proximal_abd.STL" scale="1 ${direction} 1"/>
+        </geometry>
+        <material name="">
+          <color rgba="1 1 1 1"/>
+        </material>
+      </visual>
+      <collision>
+        <origin xyz="0 0 0" rpy="0 0 0"/>
+        <geometry>
+          <mesh filename="file://$(find wuji_description)/meshes/hand2/left/l_digit_proximal_abd.STL" scale="1 ${direction} 1"/>
         </geometry>
       </collision>
@@ -466,14 +466,14 @@
         <origin xyz="0 0 0" rpy="0 0 0"/>
         <geometry>
-          <mesh filename="package://wuji_description/meshes/hand2/left/l_digit_middle.STL" scale="1 ${direction} 1"/>
-        </geometry>
-        <material name="">
-          <color rgba="1 1 1 1"/>
-        </material>
-      </visual>
-      <collision>
-        <origin xyz="0 0 0" rpy="0 0 0"/>
-        <geometry>
-          <mesh filename="package://wuji_description/meshes/hand2/left/l_digit_middle.STL" scale="1 ${direction} 1"/>
+          <mesh filename="file://$(find wuji_description)/meshes/hand2/left/l_digit_middle.STL" scale="1 ${direction} 1"/>
+        </geometry>
+        <material name="">
+          <color rgba="1 1 1 1"/>
+        </material>
+      </visual>
+      <collision>
+        <origin xyz="0 0 0" rpy="0 0 0"/>
+        <geometry>
+          <mesh filename="file://$(find wuji_description)/meshes/hand2/left/l_digit_middle.STL" scale="1 ${direction} 1"/>
         </geometry>
       </collision>
@@ -497,5 +497,5 @@
         <origin xyz="0 0 0" rpy="0 0 0"/>
         <geometry>
-          <mesh filename="package://wuji_description/meshes/hand2/left/l_digit_distal.STL" scale="1 ${direction} 1"/>
+          <mesh filename="file://$(find wuji_description)/meshes/hand2/left/l_digit_distal.STL" scale="1 ${direction} 1"/>
         </geometry>
         <material name="">
@@ -506,5 +506,5 @@
         <origin xyz="0 0 0" rpy="0 0 0"/>
         <geometry>
-          <mesh filename="package://wuji_description/meshes/hand2/left/l_digit_distal.STL" scale="1 ${direction} 1"/>
+          <mesh filename="file://$(find wuji_description)/meshes/hand2/left/l_digit_distal.STL" scale="1 ${direction} 1"/>
         </geometry>
       </collision>
@@ -534,5 +534,5 @@
         <origin xyz="0 0 0" rpy="0 0 0"/>
         <geometry>
-          <mesh filename="package://wuji_description/meshes/hand2/left/l_digit_tip_sensor_frame.STL" scale="1 ${direction} 1"/>
+          <mesh filename="file://$(find wuji_description)/meshes/hand2/left/l_digit_tip_sensor_frame.STL" scale="1 ${direction} 1"/>
         </geometry>
         <material name="">
@@ -543,5 +543,5 @@
         <origin xyz="0 0 0" rpy="0 0 0"/>
         <geometry>
-          <mesh filename="package://wuji_description/meshes/hand2/left/l_digit_tip_sensor_frame.STL" scale="1 ${direction} 1"/>
+          <mesh filename="file://$(find wuji_description)/meshes/hand2/left/l_digit_tip_sensor_frame.STL" scale="1 ${direction} 1"/>
         </geometry>
       </collision>
@@ -561,14 +561,14 @@
         <origin xyz="0 0 0" rpy="0 0 0"/>
         <geometry>
-          <mesh filename="package://wuji_description/meshes/hand2/left/l_digit_proximal.STL" scale="1 ${direction} 1"/>
-        </geometry>
-        <material name="">
-          <color rgba="1 1 1 1"/>
-        </material>
-      </visual>
-      <collision>
-        <origin xyz="0 0 0" rpy="0 0 0"/>
-        <geometry>
-          <mesh filename="package://wuji_description/meshes/hand2/left/l_digit_proximal.STL" scale="1 ${direction} 1"/>
+          <mesh filename="file://$(find wuji_description)/meshes/hand2/left/l_digit_proximal.STL" scale="1 ${direction} 1"/>
+        </geometry>
+        <material name="">
+          <color rgba="1 1 1 1"/>
+        </material>
+      </visual>
+      <collision>
+        <origin xyz="0 0 0" rpy="0 0 0"/>
+        <geometry>
+          <mesh filename="file://$(find wuji_description)/meshes/hand2/left/l_digit_proximal.STL" scale="1 ${direction} 1"/>
         </geometry>
       </collision>
@@ -592,14 +592,14 @@
         <origin xyz="0 0 0" rpy="0 0 0"/>
         <geometry>
-          <mesh filename="package://wuji_description/meshes/hand2/left/l_digit_proximal_abd.STL" scale="1 ${direction} 1"/>
-        </geometry>
-        <material name="">
-          <color rgba="1 1 1 1"/>
-        </material>
-      </visual>
-      <collision>
-        <origin xyz="0 0 0" rpy="0 0 0"/>
-        <geometry>
-          <mesh filename="package://wuji_description/meshes/hand2/left/l_digit_proximal_abd.STL" scale="1 ${direction} 1"/>
+          <mesh filename="file://$(find wuji_description)/meshes/hand2/left/l_digit_proximal_abd.STL" scale="1 ${direction} 1"/>
+        </geometry>
+        <material name="">
+          <color rgba="1 1 1 1"/>
+        </material>
+      </visual>
+      <collision>
+        <origin xyz="0 0 0" rpy="0 0 0"/>
+        <geometry>
+          <mesh filename="file://$(find wuji_description)/meshes/hand2/left/l_digit_proximal_abd.STL" scale="1 ${direction} 1"/>
         </geometry>
       </collision>
@@ -623,14 +623,14 @@
         <origin xyz="0 0 0" rpy="0 0 0"/>
         <geometry>
-          <mesh filename="package://wuji_description/meshes/hand2/left/l_digit_middle.STL" scale="1 ${direction} 1"/>
-        </geometry>
-        <material name="">
-          <color rgba="1 1 1 1"/>
-        </material>
-      </visual>
-      <collision>
-        <origin xyz="0 0 0" rpy="0 0 0"/>
-        <geometry>
-          <mesh filename="package://wuji_description/meshes/hand2/left/l_digit_middle.STL" scale="1 ${direction} 1"/>
+          <mesh filename="file://$(find wuji_description)/meshes/hand2/left/l_digit_middle.STL" scale="1 ${direction} 1"/>
+        </geometry>
+        <material name="">
+          <color rgba="1 1 1 1"/>
+        </material>
+      </visual>
+      <collision>
+        <origin xyz="0 0 0" rpy="0 0 0"/>
+        <geometry>
+          <mesh filename="file://$(find wuji_description)/meshes/hand2/left/l_digit_middle.STL" scale="1 ${direction} 1"/>
         </geometry>
       </collision>
@@ -654,5 +654,5 @@
         <origin xyz="0 0 0" rpy="0 0 0"/>
         <geometry>
-          <mesh filename="package://wuji_description/meshes/hand2/left/l_digit_distal.STL" scale="1 ${direction} 1"/>
+          <mesh filename="file://$(find wuji_description)/meshes/hand2/left/l_digit_distal.STL" scale="1 ${direction} 1"/>
         </geometry>
         <material name="">
@@ -663,5 +663,5 @@
         <origin xyz="0 0 0" rpy="0 0 0"/>
         <geometry>
-          <mesh filename="package://wuji_description/meshes/hand2/left/l_digit_distal.STL" scale="1 ${direction} 1"/>
+          <mesh filename="file://$(find wuji_description)/meshes/hand2/left/l_digit_distal.STL" scale="1 ${direction} 1"/>
         </geometry>
       </collision>
@@ -691,5 +691,5 @@
         <origin xyz="0 0 0" rpy="0 0 0"/>
         <geometry>
-          <mesh filename="package://wuji_description/meshes/hand2/left/l_digit_tip_sensor_frame.STL" scale="1 ${direction} 1"/>
+          <mesh filename="file://$(find wuji_description)/meshes/hand2/left/l_digit_tip_sensor_frame.STL" scale="1 ${direction} 1"/>
         </geometry>
         <material name="">
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