Commit message: fix wuji hand xacro

File: dexhands/wuji_description/xacro/hand.xacro (robot description, xacro)
@@ -3,5 +3,5 @@
 	<xacro:arg name="type" default="hand2"/>
 	<xacro:arg name="direction" default="1"/>
-	<xacro:arg name="use_mount" default="false"/>
+	<xacro:arg name="use_mount" default="true"/>
 	<!-- type: hand1 (gen1), hand2 (beta2, default) -->
 	<xacro:if value="${'$(arg type)' == 'hand2'}">

File: dexhands/wuji_description/xacro/hand1.xacro (robot description, xacro)
@@ -7,792 +7,749 @@
 -->
 <robot xmlns:xacro="http://www.ros.org/wiki/xacro">
-  <xacro:macro name="WujiHand" params="name direction:=1 use_mount:=false fixed_joints:=false">
-    <xacro:property name="prefix" value="${name + '_' if name else ''}"/>
-    <xacro:property name="joint_type" value="${fixed_joints and 'fixed' or 'revolute'}"/>
-    <xacro:property name="mesh_side" value="${'left' if direction == 1 else 'right'}"/>
-    <!-- use_mount ignored: gen1 has no mount link; meshes: side STL, no Y-scale -->
-    <link name="${prefix}hand_base">
-      <inertial>
-        <origin xyz="-0.002979471 ${direction*-0.0004557176} 0.03665409" rpy="0 0 0"/>
-        <mass value="0.16914"/>
-        <inertia ixx="0.00014" ixy="${direction*-2.54e-06}" ixz="6.9100000000e-06" iyy="9.4700000000e-05" iyz="${direction*6.63e-06}" izz="6.0000000000e-05"/>
-      </inertial>
-      <visual>
-        <origin xyz="0 0 0" rpy="0 0 0"/>
-        <geometry>
-          <mesh filename="file://$(find wuji_description)/meshes/hand1/${mesh_side}/${mesh_side}_palm_link.STL"/>
-        </geometry>
-        <material name="">
-          <color rgba="0.627451 0.627451 0.627451 1"/>
-        </material>
-      </visual>
-      <collision>
-        <origin xyz="0 0 0" rpy="0 0 0"/>
-        <geometry>
-          <mesh filename="file://$(find wuji_description)/meshes/hand1/${mesh_side}/${mesh_side}_palm_link.STL"/>
-        </geometry>
-      </collision>
-    </link>
-    <link name="${prefix}finger1_link1">
-      <inertial>
-        <origin xyz="-0.002466361 ${direction*0.001243356} 0.007796453" rpy="0 0 0"/>
-        <mass value="0.0075"/>
-        <inertia ixx="3.2e-07" ixy="${direction*-2e-08}" ixz="0" iyy="3e-07" iyz="${direction*4e-08}" izz="2.3e-07"/>
-      </inertial>
-      <visual>
-        <origin xyz="0 0 0" rpy="0 0 0"/>
-        <geometry>
-          <mesh filename="file://$(find wuji_description)/meshes/hand1/${mesh_side}/${mesh_side}_finger1_link1.STL"/>
-        </geometry>
-        <material name="">
-          <color rgba="0.627451 0.627451 0.627451 1"/>
-        </material>
-      </visual>
-      <collision>
-        <origin xyz="0 0 0" rpy="0 0 0"/>
-        <geometry>
-          <mesh filename="file://$(find wuji_description)/meshes/hand1/${mesh_side}/${mesh_side}_finger1_link1.STL"/>
-        </geometry>
-      </collision>
-    </link>
-    <joint name="${prefix}finger1_joint1" type="${joint_type}">
-      <origin xyz="0.0084399 ${direction*-0.020587} 0.028893" rpy="${direction*1.328} -0.37161 ${direction*0.7307}"/>
-      <parent link="${prefix}hand_base"/>
-      <child link="${prefix}finger1_link1"/>
-      <xacro:unless value="${fixed_joints}">
-        <axis xyz="0 1 0"/>
-        <limit lower="0.0475" upper="1.6033" effort="0.4452" velocity="8.587"/>
-      </xacro:unless>
-    </joint>
-    <link name="${prefix}finger1_link2">
-      <inertial>
-        <origin xyz="0.001165924 ${direction*1.466029e-05} 0.01565596" rpy="0 0 0"/>
-        <mass value="0.0248"/>
-        <inertia ixx="2.76e-06" ixy="${direction*2e-08}" ixz="1e-08" iyy="2.81e-06" iyz="${direction*2e-08}" izz="6.8e-07"/>
-      </inertial>
-      <visual>
-        <origin xyz="0 0 0" rpy="0 0 0"/>
-        <geometry>
-          <mesh filename="file://$(find wuji_description)/meshes/hand1/${mesh_side}/${mesh_side}_finger1_link2.STL"/>
-        </geometry>
-        <material name="">
-          <color rgba="0.627451 0.627451 0.627451 1"/>
-        </material>
-      </visual>
-      <collision>
-        <origin xyz="0 0 0" rpy="0 0 0"/>
-        <geometry>
-          <mesh filename="file://$(find wuji_description)/meshes/hand1/${mesh_side}/${mesh_side}_finger1_link2.STL"/>
-        </geometry>
-      </collision>
-    </link>
-    <joint name="${prefix}finger1_joint2" type="${joint_type}">
-      <origin xyz="-0.0047549 ${direction*0.0058191} 0.014132" rpy="${direction==1 and '0.57428 -0.23677 -1.8034' or '0.57428 0.23677 -1.3382'}"/>
-      <parent link="${prefix}finger1_link1"/>
-      <child link="${prefix}finger1_link2"/>
-      <xacro:unless value="${fixed_joints}">
-        <axis xyz="0 ${-direction} 0"/>
-        <limit lower="-0.1387" upper="0.9324" effort="0.4259" velocity="11.1"/>
-      </xacro:unless>
-    </joint>
-    <link name="${prefix}finger1_link3">
-      <inertial>
-        <origin xyz="-0.001123197 ${direction*1.572991e-05} 0.01305658" rpy="0 0 0"/>
-        <mass value="0.0165"/>
-        <inertia ixx="1.46e-06" ixy="0" ixz="-2e-08" iyy="1.42e-06" iyz="0" izz="4.5e-07"/>
-      </inertial>
-      <visual>
-        <origin xyz="0 0 0" rpy="0 0 0"/>
-        <geometry>
-          <mesh filename="file://$(find wuji_description)/meshes/hand1/${mesh_side}/${mesh_side}_finger1_link3.STL"/>
-        </geometry>
-        <material name="">
-          <color rgba="0.627451 0.627451 0.627451 1"/>
-        </material>
-      </visual>
-      <collision>
-        <origin xyz="0 0 0" rpy="0 0 0"/>
-        <geometry>
-          <mesh filename="file://$(find wuji_description)/meshes/hand1/${mesh_side}/${mesh_side}_finger1_link3.STL"/>
-        </geometry>
-      </collision>
-    </link>
-    <joint name="${prefix}finger1_joint3" type="${joint_type}">
-      <origin xyz="${direction*0.00026671} 0.0009915 0.034666" rpy="${direction==1 and '-0.049049 0.017311 1.9085' or '0.04904945 0.01731124 1.233052'}"/>
-      <parent link="${prefix}finger1_link2"/>
-      <child link="${prefix}finger1_link3"/>
-      <xacro:unless value="${fixed_joints}">
-        <axis xyz="0 1 0"/>
-        <limit lower="-0.4642" upper="1.5623" effort="0.1888" velocity="12.863"/>
-      </xacro:unless>
-    </joint>
-    <link name="${prefix}finger1_link4">
-      <inertial>
-        <origin xyz="-0.0011922 ${direction*0.00021414} 0.0082113" rpy="0 0 0"/>
-        <mass value="0.0165"/>
-        <inertia ixx="1.18e-06" ixy="0" ixz="1.2e-07" iyy="1.25e-06" iyz="0" izz="5.1e-07"/>
-      </inertial>
-      <visual>
-        <origin xyz="0 0 0" rpy="0 0 0"/>
-        <geometry>
-          <mesh filename="file://$(find wuji_description)/meshes/hand1/${mesh_side}/${mesh_side}_finger1_link4.STL"/>
-        </geometry>
-        <material name="">
-          <color rgba="0.5294118 0.5490196 0.5490196 1"/>
-        </material>
-      </visual>
-      <collision>
-        <origin xyz="0 0 0" rpy="0 0 0"/>
-        <geometry>
-          <mesh filename="file://$(find wuji_description)/meshes/hand1/${mesh_side}/${mesh_side}_finger1_link4.STL"/>
-        </geometry>
-      </collision>
-    </link>
-    <joint name="${prefix}finger1_joint4" type="${joint_type}">
-      <origin xyz="0 ${direction*-0.0002} 0.0295" rpy="0 0 0"/>
-      <parent link="${prefix}finger1_link3"/>
-      <child link="${prefix}finger1_link4"/>
-      <xacro:unless value="${fixed_joints}">
-        <axis xyz="0 1 0"/>
-        <limit lower="-0.4699" upper="1.5568" effort="0.1468" velocity="13.578"/>
-      </xacro:unless>
-    </joint>
-    <link name="${prefix}finger1_tip_link">
-      <inertial>
-        <origin xyz="-0.00017019 ${direction*1.7524e-05} -0.0071779" rpy="0 0 0"/>
-        <mass value="0.0041"/>
-        <inertia ixx="5.5e-07" ixy="0" ixz="2e-08" iyy="5.2e-07" iyz="0" izz="2.7e-07"/>
-      </inertial>
-      <visual>
-        <origin xyz="0 0 0" rpy="0 0 0"/>
-        <geometry>
-          <mesh filename="file://$(find wuji_description)/meshes/hand1/${mesh_side}/${mesh_side}_finger1_tip_link.STL"/>
-        </geometry>
-        <material name="">
-          <color rgba="0.5294118 0.5490196 0.5490196 1"/>
-        </material>
-      </visual>
-      <collision>
-        <origin xyz="0 0 0" rpy="0 0 0"/>
-        <geometry>
-          <mesh filename="file://$(find wuji_description)/meshes/hand1/${mesh_side}/${mesh_side}_finger1_tip_link.STL"/>
-        </geometry>
-      </collision>
-    </link>
-    <joint name="${prefix}finger1_tip_fixed" type="fixed">
-      <origin xyz="-0.00105 0.0002 0.0313" rpy="0 0 0"/>
-      <parent link="${prefix}finger1_link4"/>
-      <child link="${prefix}finger1_tip_link"/>
-    </joint>
-    <link name="${prefix}finger2_link1">
-      <inertial>
-        <origin xyz="-0.0013291 ${direction*-5.6587e-09} 0.00031994" rpy="0 0 0"/>
-        <mass value="0.0032"/>
-        <inertia ixx="8e-08" ixy="0" ixz="-3e-08" iyy="7e-08" iyz="0" izz="8e-08"/>
-      </inertial>
-      <visual>
-        <origin xyz="0 0 0" rpy="0 0 0"/>
-        <geometry>
-          <mesh filename="file://$(find wuji_description)/meshes/hand1/${mesh_side}/${mesh_side}_digit_link1.STL"/>
-        </geometry>
-        <material name="">
-          <color rgba="0.627451 0.627451 0.627451 1"/>
-        </material>
-      </visual>
-      <collision>
-        <origin xyz="0 0 0" rpy="0 0 0"/>
-        <geometry>
-          <mesh filename="file://$(find wuji_description)/meshes/hand1/${mesh_side}/${mesh_side}_digit_link1.STL"/>
-        </geometry>
-      </collision>
-    </link>
-    <joint name="${prefix}finger2_joint1" type="${joint_type}">
-      <origin xyz="-0.0058701 ${direction*-0.029434} 0.091917" rpy="${direction*0.11071} -0.071139 ${direction*0.21822}"/>
-      <parent link="${prefix}hand_base"/>
-      <child link="${prefix}finger2_link1"/>
-      <xacro:unless value="${fixed_joints}">
-        <axis xyz="0 1 0"/>
-        <limit lower="-0.1585" upper="1.5604" effort="0.6188" velocity="8.203"/>
-      </xacro:unless>
-    </joint>
-    <link name="${prefix}finger2_link2">
-      <inertial>
-        <origin xyz="4.378686e-07 ${direction*0.006157522} 0.02091104" rpy="0 0 0"/>
-        <mass value="0.033"/>
-        <inertia ixx="6.31e-06" ixy="0" ixz="-1.6e-07" iyy="6.34e-06" iyz="0" izz="8.9e-07"/>
-      </inertial>
-      <visual>
-        <origin xyz="0 0 0" rpy="0 0 0"/>
-        <geometry>
-          <mesh filename="file://$(find wuji_description)/meshes/hand1/${mesh_side}/${mesh_side}_digit_link2.STL"/>
-        </geometry>
-        <material name="">
-          <color rgba="0.627451 0.627451 0.627451 1"/>
-        </material>
-      </visual>
-      <collision>
-        <origin xyz="0 0 0" rpy="0 0 0"/>
-        <geometry>
-          <mesh filename="file://$(find wuji_description)/meshes/hand1/${mesh_side}/${mesh_side}_digit_link2.STL"/>
-        </geometry>
-      </collision>
-    </link>
-    <joint name="${prefix}finger2_joint2" type="${joint_type}">
-      <origin xyz="0.0022 0 0.004000006" rpy="0 0 1.570796"/>
-      <parent link="${prefix}finger2_link1"/>
-      <child link="${prefix}finger2_link2"/>
-      <xacro:unless value="${fixed_joints}">
-        <axis xyz="0 1 0"/>
-        <limit lower="-0.3700" upper="0.3700" effort="0.1822" velocity="8.115"/>
-      </xacro:unless>
-    </joint>
-    <link name="${prefix}finger2_link3">
-      <inertial>
-        <origin xyz="-0.001121873 ${direction*3.276186e-05} 0.01571884" rpy="0 0 0"/>
-        <mass value="0.0165"/>
-        <inertia ixx="1.47e-06" ixy="0" ixz="3e-08" iyy="1.44e-06" iyz="0" izz="4.5e-07"/>
-      </inertial>
-      <visual>
-        <origin xyz="0 0 0" rpy="0 0 0"/>
-        <geometry>
-          <mesh filename="file://$(find wuji_description)/meshes/hand1/${mesh_side}/${mesh_side}_digit_link3.STL"/>
-        </geometry>
-        <material name="">
-          <color rgba="0.627451 0.627451 0.627451 1"/>
-        </material>
-      </visual>
-      <collision>
-        <origin xyz="0 0 0" rpy="0 0 0"/>
-        <geometry>
-          <mesh filename="file://$(find wuji_description)/meshes/hand1/${mesh_side}/${mesh_side}_digit_link3.STL"/>
-        </geometry>
-      </collision>
-    </link>
-    <joint name="${prefix}finger2_joint3" type="${joint_type}">
-      <origin xyz="0 0.004749999 0.04361769" rpy="0 0 -1.570528"/>
-      <parent link="${prefix}finger2_link2"/>
-      <child link="${prefix}finger2_link3"/>
-      <xacro:unless value="${fixed_joints}">
-        <axis xyz="0 1 0"/>
-        <limit lower="-0.4777" upper="1.5485" effort="0.2251" velocity="12.863"/>
-      </xacro:unless>
-    </joint>
-    <link name="${prefix}finger2_link4">
-      <inertial>
-        <origin xyz="-0.0008943786 ${direction*0.0002170653} 0.005351759" rpy="0 0 0"/>
-        <mass value="0.014"/>
-        <inertia ixx="9.5e-07" ixy="0" ixz="1.4e-07" iyy="8.6e-07" iyz="${direction*-1e-08}" izz="3e-07"/>
-      </inertial>
-      <visual>
-        <origin xyz="0 0 0" rpy="0 0 0"/>
-        <geometry>
-          <mesh filename="file://$(find wuji_description)/meshes/hand1/${mesh_side}/${mesh_side}_digit_link4.STL"/>
-        </geometry>
-        <material name="">
-          <color rgba="0.5294118 0.5490196 0.5490196 1"/>
-        </material>
-      </visual>
-      <collision>
-        <origin xyz="0 0 0" rpy="0 0 0"/>
-        <geometry>
-          <mesh filename="file://$(find wuji_description)/meshes/hand1/${mesh_side}/${mesh_side}_digit_link4.STL"/>
-        </geometry>
-      </collision>
-    </link>
-    <joint name="${prefix}finger2_joint4" type="${joint_type}">
-      <origin xyz="0 -0.0002 0.0295" rpy="0 0 0"/>
-      <parent link="${prefix}finger2_link3"/>
-      <child link="${prefix}finger2_link4"/>
-      <xacro:unless value="${fixed_joints}">
-        <axis xyz="0 1 0"/>
-        <limit lower="-0.4683" upper="1.5753" effort="0.2170" velocity="13.578"/>
-      </xacro:unless>
-    </joint>
-    <link name="${prefix}finger2_tip_link">
-      <inertial>
-        <origin xyz="-0.0001897323 ${direction*3.534942e-06} -0.009137204" rpy="0 0 0"/>
-        <mass value="0.00318"/>
-        <inertia ixx="2e-07" ixy="0" ixz="0" iyy="2.1e-07" iyz="0" izz="1.3e-07"/>
-      </inertial>
-      <visual>
-        <origin xyz="0 0 0" rpy="0 0 0"/>
-        <geometry>
-          <mesh filename="file://$(find wuji_description)/meshes/hand1/${mesh_side}/${mesh_side}_digit_tip_link.STL"/>
-        </geometry>
-        <material name="">
-          <color rgba="0.5294118 0.5490196 0.5490196 1"/>
-        </material>
-      </visual>
-      <collision>
-        <origin xyz="0 0 0" rpy="0 0 0"/>
-        <geometry>
-          <mesh filename="file://$(find wuji_description)/meshes/hand1/${mesh_side}/${mesh_side}_digit_tip_link.STL"/>
-        </geometry>
-      </collision>
-    </link>
-    <joint name="${prefix}finger2_tip_fixed" type="fixed">
-      <origin xyz="-0.0010521 0.0002108692 0.0267" rpy="0 0 0"/>
-      <parent link="${prefix}finger2_link4"/>
-      <child link="${prefix}finger2_tip_link"/>
-    </joint>
-    <link name="${prefix}finger3_link1">
-      <inertial>
-        <origin xyz="-0.0013291 ${direction*-1.4994e-08} 0.0003199" rpy="0 0 0"/>
-        <mass value="0.0032"/>
-        <inertia ixx="8e-08" ixy="0" ixz="-3e-08" iyy="7e-08" iyz="0" izz="8e-08"/>
-      </inertial>
-      <visual>
-        <origin xyz="0 0 0" rpy="0 0 0"/>
-        <geometry>
-          <mesh filename="file://$(find wuji_description)/meshes/hand1/${mesh_side}/${mesh_side}_digit_link1.STL"/>
-        </geometry>
-        <material name="">
-          <color rgba="0.627451 0.627451 0.627451 1"/>
-        </material>
-      </visual>
-      <collision>
-        <origin xyz="0 0 0" rpy="0 0 0"/>
-        <geometry>
-          <mesh filename="file://$(find wuji_description)/meshes/hand1/${mesh_side}/${mesh_side}_digit_link1.STL"/>
-        </geometry>
-      </collision>
-    </link>
-    <joint name="${prefix}finger3_joint1" type="${joint_type}">
-      <origin xyz="-0.01046 ${direction*-0.0074615} 0.089544" rpy="${direction*5.0894e-05} -0.087266 ${direction*-0.00058387}"/>
-      <parent link="${prefix}hand_base"/>
-      <child link="${prefix}finger3_link1"/>
-      <xacro:unless value="${fixed_joints}">
-        <axis xyz="0 1 0"/>
-        <limit lower="-0.1644" upper="1.5516" effort="0.6494" velocity="8.203"/>
-      </xacro:unless>
-    </joint>
-    <link name="${prefix}finger3_link2">
-      <inertial>
-        <origin xyz="4.38062e-07 ${direction*0.006157535} 0.02091104" rpy="0 0 0"/>
-        <mass value="0.033"/>
-        <inertia ixx="6.31e-06" ixy="0" ixz="-1.6e-07" iyy="6.34e-06" iyz="0" izz="8.9e-07"/>
-      </inertial>
-      <visual>
-        <origin xyz="0 0 0" rpy="0 0 0"/>
-        <geometry>
-          <mesh filename="file://$(find wuji_description)/meshes/hand1/${mesh_side}/${mesh_side}_digit_link2.STL"/>
-        </geometry>
-        <material name="">
-          <color rgba="0.627451 0.627451 0.627451 1"/>
-        </material>
-      </visual>
-      <collision>
-        <origin xyz="0 0 0" rpy="0 0 0"/>
-        <geometry>
-          <mesh filename="file://$(find wuji_description)/meshes/hand1/${mesh_side}/${mesh_side}_digit_link2.STL"/>
-        </geometry>
-      </collision>
-    </link>
-    <joint name="${prefix}finger3_joint2" type="${joint_type}">
-      <origin xyz="0.0022 0 0.004000006" rpy="0 0 1.570796"/>
-      <parent link="${prefix}finger3_link1"/>
-      <child link="${prefix}finger3_link2"/>
-      <xacro:unless value="${fixed_joints}">
-        <axis xyz="0 1 0"/>
-        <limit lower="-0.3700" upper="0.3700" effort="0.1827" velocity="8.115"/>
-      </xacro:unless>
-    </joint>
-    <link name="${prefix}finger3_link3">
-      <inertial>
-        <origin xyz="-0.001121872 ${direction*3.278072e-05} 0.01571884" rpy="0 0 0"/>
-        <mass value="0.0165"/>
-        <inertia ixx="1.47e-06" ixy="0" ixz="3e-08" iyy="1.44e-06" iyz="0" izz="4.5e-07"/>
-      </inertial>
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