Commit message: fix wuji hand xacro

File: dexhands/wuji_description/xacro/hand.xacro (robot description, xacro)
@@ -4,12 +4,5 @@
 	<xacro:arg name="direction" default="1"/>
 	<xacro:arg name="use_mount" default="true"/>
-	<!-- type: hand1 (gen1), hand2 (beta2, default) -->
-	<xacro:if value="${'$(arg type)' == 'hand2'}">
-		<xacro:include filename="$(find wuji_description)/xacro/hand2.xacro"/>
-		<xacro:WujiHand2 name="" direction="$(arg direction)" use_mount="$(arg use_mount)"/>
-	</xacro:if>
-	<xacro:if value="${'$(arg type)' == 'hand1'}">
-		<xacro:include filename="$(find wuji_description)/xacro/hand1.xacro"/>
-		<xacro:WujiHand name="" direction="$(arg direction)" use_mount="$(arg use_mount)"/>
-	</xacro:if>
+	<xacro:include filename="$(find wuji_description)/xacro/hand2.xacro"/>
+	<xacro:WujiHand2 name="" direction="$(arg direction)" use_mount="$(arg use_mount)"/>
 </robot>

File: dexhands/wuji_description/xacro/hand2.xacro (robot description, xacro)
@@ -26,5 +26,5 @@
                 <visual>
                     <geometry>
-                        <mesh filename="file://$(find wuji_description)/meshes/hand2/left/l_mount.glb"
+                        <mesh filename="file://$(find wuji_description)/meshes/hand2/l_mount.glb"
                               scale="1 ${direction} 1"/>
                     </geometry>
@@ -32,5 +32,5 @@
                 <collision>
                     <geometry>
-                        <mesh filename="file://$(find wuji_description)/meshes/hand2/left/l_mount.glb"
+                        <mesh filename="file://$(find wuji_description)/meshes/hand2/l_mount.glb"
                               scale="1 ${direction} 1"/>
                     </geometry>
@@ -66,11 +66,11 @@
             <visual>
                 <geometry>
-                    <mesh filename="file://$(find wuji_description)/meshes/hand2/left/l_wrist.glb"
-                          scale="1 ${direction} 1"/>
-                </geometry>
-            </visual>
-            <collision>
-                <geometry>
-                    <mesh filename="file://$(find wuji_description)/meshes/hand2/left/l_wrist.glb"
+                    <mesh filename="file://$(find wuji_description)/meshes/hand2/l_wrist.glb"
+                          scale="1 ${direction} 1"/>
+                </geometry>
+            </visual>
+            <collision>
+                <geometry>
+                    <mesh filename="file://$(find wuji_description)/meshes/hand2/l_wrist.glb"
                           scale="1 ${direction} 1"/>
                 </geometry>
@@ -86,11 +86,11 @@
             <visual>
                 <geometry>
-                    <mesh filename="file://$(find wuji_description)/meshes/hand2/left/l_thumb_proximal.glb"
-                          scale="1 ${direction} 1"/>
-                </geometry>
-            </visual>
-            <collision>
-                <geometry>
-                    <mesh filename="file://$(find wuji_description)/meshes/hand2/left/l_thumb_proximal.glb"
+                    <mesh filename="file://$(find wuji_description)/meshes/hand2/l_thumb_proximal.glb"
+                          scale="1 ${direction} 1"/>
+                </geometry>
+            </visual>
+            <collision>
+                <geometry>
+                    <mesh filename="file://$(find wuji_description)/meshes/hand2/l_thumb_proximal.glb"
                           scale="1 ${direction} 1"/>
                 </geometry>
@@ -116,11 +116,11 @@
             <visual>
                 <geometry>
-                    <mesh filename="file://$(find wuji_description)/meshes/hand2/left/l_thumb_proximal_abd.glb"
-                          scale="1 ${direction} 1"/>
-                </geometry>
-            </visual>
-            <collision>
-                <geometry>
-                    <mesh filename="file://$(find wuji_description)/meshes/hand2/left/l_thumb_proximal_abd.glb"
+                    <mesh filename="file://$(find wuji_description)/meshes/hand2/l_thumb_proximal_abd.glb"
+                          scale="1 ${direction} 1"/>
+                </geometry>
+            </visual>
+            <collision>
+                <geometry>
+                    <mesh filename="file://$(find wuji_description)/meshes/hand2/l_thumb_proximal_abd.glb"
                           scale="1 ${direction} 1"/>
                 </geometry>
@@ -146,11 +146,11 @@
             <visual>
                 <geometry>
-                    <mesh filename="file://$(find wuji_description)/meshes/hand2/left/l_thumb_middle.glb"
-                          scale="1 ${direction} 1"/>
-                </geometry>
-            </visual>
-            <collision>
-                <geometry>
-                    <mesh filename="file://$(find wuji_description)/meshes/hand2/left/l_thumb_middle.glb"
+                    <mesh filename="file://$(find wuji_description)/meshes/hand2/l_thumb_middle.glb"
+                          scale="1 ${direction} 1"/>
+                </geometry>
+            </visual>
+            <collision>
+                <geometry>
+                    <mesh filename="file://$(find wuji_description)/meshes/hand2/l_thumb_middle.glb"
                           scale="1 ${direction} 1"/>
                 </geometry>
@@ -176,11 +176,11 @@
             <visual>
                 <geometry>
-                    <mesh filename="file://$(find wuji_description)/meshes/hand2/left/l_thumb_distal.glb"
-                          scale="1 ${direction} 1"/>
-                </geometry>
-            </visual>
-            <collision>
-                <geometry>
-                    <mesh filename="file://$(find wuji_description)/meshes/hand2/left/l_thumb_distal.glb"
+                    <mesh filename="file://$(find wuji_description)/meshes/hand2/l_thumb_distal.glb"
+                          scale="1 ${direction} 1"/>
+                </geometry>
+            </visual>
+            <collision>
+                <geometry>
+                    <mesh filename="file://$(find wuji_description)/meshes/hand2/l_thumb_distal.glb"
                           scale="1 ${direction} 1"/>
                 </geometry>
@@ -211,11 +211,11 @@
             <visual>
                 <geometry>
-                    <mesh filename="file://$(find wuji_description)/meshes/hand2/left/l_thumb_tip_sensor_frame.glb"
-                          scale="1 ${direction} 1"/>
-                </geometry>
-            </visual>
-            <collision>
-                <geometry>
-                    <mesh filename="file://$(find wuji_description)/meshes/hand2/left/l_thumb_tip_sensor_frame.glb"
+                    <mesh filename="file://$(find wuji_description)/meshes/hand2/l_thumb_tip_sensor_frame.glb"
+                          scale="1 ${direction} 1"/>
+                </geometry>
+            </visual>
+            <collision>
+                <geometry>
+                    <mesh filename="file://$(find wuji_description)/meshes/hand2/l_thumb_tip_sensor_frame.glb"
                           scale="1 ${direction} 1"/>
                 </geometry>
@@ -235,11 +235,11 @@
             <visual>
                 <geometry>
-                    <mesh filename="file://$(find wuji_description)/meshes/hand2/left/l_digit_proximal.glb"
-                          scale="1 ${direction} 1"/>
-                </geometry>
-            </visual>
-            <collision>
-                <geometry>
-                    <mesh filename="file://$(find wuji_description)/meshes/hand2/left/l_digit_proximal.glb"
+                    <mesh filename="file://$(find wuji_description)/meshes/hand2/l_digit_proximal.glb"
+                          scale="1 ${direction} 1"/>
+                </geometry>
+            </visual>
+            <collision>
+                <geometry>
+                    <mesh filename="file://$(find wuji_description)/meshes/hand2/l_digit_proximal.glb"
                           scale="1 ${direction} 1"/>
                 </geometry>
@@ -265,11 +265,11 @@
             <visual>
                 <geometry>
-                    <mesh filename="file://$(find wuji_description)/meshes/hand2/left/l_digit_proximal_abd.glb"
-                          scale="1 ${direction} 1"/>
-                </geometry>
-            </visual>
-            <collision>
-                <geometry>
-                    <mesh filename="file://$(find wuji_description)/meshes/hand2/left/l_digit_proximal_abd.glb"
+                    <mesh filename="file://$(find wuji_description)/meshes/hand2/l_digit_proximal_abd.glb"
+                          scale="1 ${direction} 1"/>
+                </geometry>
+            </visual>
+            <collision>
+                <geometry>
+                    <mesh filename="file://$(find wuji_description)/meshes/hand2/l_digit_proximal_abd.glb"
                           scale="1 ${direction} 1"/>
                 </geometry>
@@ -294,11 +294,11 @@
             <visual>
                 <geometry>
-                    <mesh filename="file://$(find wuji_description)/meshes/hand2/left/l_digit_middle.glb"
-                          scale="1 ${direction} 1"/>
-                </geometry>
-            </visual>
-            <collision>
-                <geometry>
-                    <mesh filename="file://$(find wuji_description)/meshes/hand2/left/l_digit_middle.glb"
+                    <mesh filename="file://$(find wuji_description)/meshes/hand2/l_digit_middle.glb"
+                          scale="1 ${direction} 1"/>
+                </geometry>
+            </visual>
+            <collision>
+                <geometry>
+                    <mesh filename="file://$(find wuji_description)/meshes/hand2/l_digit_middle.glb"
                           scale="1 ${direction} 1"/>
                 </geometry>
@@ -323,11 +323,11 @@
             <visual>
                 <geometry>
-                    <mesh filename="file://$(find wuji_description)/meshes/hand2/left/l_digit_distal.glb"
-                          scale="1 ${direction} 1"/>
-                </geometry>
-            </visual>
-            <collision>
-                <geometry>
-                    <mesh filename="file://$(find wuji_description)/meshes/hand2/left/l_digit_distal.glb"
+                    <mesh filename="file://$(find wuji_description)/meshes/hand2/l_digit_distal.glb"
+                          scale="1 ${direction} 1"/>
+                </geometry>
+            </visual>
+            <collision>
+                <geometry>
+                    <mesh filename="file://$(find wuji_description)/meshes/hand2/l_digit_distal.glb"
                           scale="1 ${direction} 1"/>
                 </geometry>
@@ -358,11 +358,11 @@
             <visual>
                 <geometry>
-                    <mesh filename="file://$(find wuji_description)/meshes/hand2/left/l_digit_tip_sensor_frame.glb"
-                          scale="1 ${direction} 1"/>
-                </geometry>
-            </visual>
-            <collision>
-                <geometry>
-                    <mesh filename="file://$(find wuji_description)/meshes/hand2/left/l_digit_tip_sensor_frame.glb"
+                    <mesh filename="file://$(find wuji_description)/meshes/hand2/l_digit_tip_sensor_frame.glb"
+                          scale="1 ${direction} 1"/>
+                </geometry>
+            </visual>
+            <collision>
+                <geometry>
+                    <mesh filename="file://$(find wuji_description)/meshes/hand2/l_digit_tip_sensor_frame.glb"
                           scale="1 ${direction} 1"/>
                 </geometry>
@@ -382,11 +382,11 @@
             <visual>
                 <geometry>
-                    <mesh filename="file://$(find wuji_description)/meshes/hand2/left/l_digit_proximal.glb"
-                          scale="1 ${direction} 1"/>
-                </geometry>
-            </visual>
-            <collision>
-                <geometry>
-                    <mesh filename="file://$(find wuji_description)/meshes/hand2/left/l_digit_proximal.glb"
+                    <mesh filename="file://$(find wuji_description)/meshes/hand2/l_digit_proximal.glb"
+                          scale="1 ${direction} 1"/>
+                </geometry>
+            </visual>
+            <collision>
+                <geometry>
+                    <mesh filename="file://$(find wuji_description)/meshes/hand2/l_digit_proximal.glb"
                           scale="1 ${direction} 1"/>
                 </geometry>
@@ -412,11 +412,11 @@
             <visual>
                 <geometry>
-                    <mesh filename="file://$(find wuji_description)/meshes/hand2/left/l_digit_proximal_abd.glb"
-                          scale="1 ${direction} 1"/>
-                </geometry>
-            </visual>
-            <collision>
-                <geometry>
-                    <mesh filename="file://$(find wuji_description)/meshes/hand2/left/l_digit_proximal_abd.glb"
+                    <mesh filename="file://$(find wuji_description)/meshes/hand2/l_digit_proximal_abd.glb"
+                          scale="1 ${direction} 1"/>
+                </geometry>
+            </visual>
+            <collision>
+                <geometry>
+                    <mesh filename="file://$(find wuji_description)/meshes/hand2/l_digit_proximal_abd.glb"
                           scale="1 ${direction} 1"/>
                 </geometry>
@@ -441,11 +441,11 @@
             <visual>
                 <geometry>
-                    <mesh filename="file://$(find wuji_description)/meshes/hand2/left/l_digit_middle.glb"
-                          scale="1 ${direction} 1"/>
-                </geometry>
-            </visual>
-            <collision>
-                <geometry>
-                    <mesh filename="file://$(find wuji_description)/meshes/hand2/left/l_digit_middle.glb"
+                    <mesh filename="file://$(find wuji_description)/meshes/hand2/l_digit_middle.glb"
+                          scale="1 ${direction} 1"/>
+                </geometry>
+            </visual>
+            <collision>
+                <geometry>
+                    <mesh filename="file://$(find wuji_description)/meshes/hand2/l_digit_middle.glb"
                           scale="1 ${direction} 1"/>
                 </geometry>
@@ -470,11 +470,11 @@
             <visual>
                 <geometry>
-                    <mesh filename="file://$(find wuji_description)/meshes/hand2/left/l_digit_distal.glb"
-                          scale="1 ${direction} 1"/>
-                </geometry>
-            </visual>
-            <collision>
-                <geometry>
-                    <mesh filename="file://$(find wuji_description)/meshes/hand2/left/l_digit_distal.glb"
+                    <mesh filename="file://$(find wuji_description)/meshes/hand2/l_digit_distal.glb"
+                          scale="1 ${direction} 1"/>
+                </geometry>
+            </visual>
+            <collision>
+                <geometry>
+                    <mesh filename="file://$(find wuji_description)/meshes/hand2/l_digit_distal.glb"
                           scale="1 ${direction} 1"/>
                 </geometry>
@@ -505,11 +505,11 @@
             <visual>
                 <geometry>
-                    <mesh filename="file://$(find wuji_description)/meshes/hand2/left/l_digit_tip_sensor_frame.glb"
-                          scale="1 ${direction} 1"/>
-                </geometry>
-            </visual>
-            <collision>
-                <geometry>
-                    <mesh filename="file://$(find wuji_description)/meshes/hand2/left/l_digit_tip_sensor_frame.glb"
+                    <mesh filename="file://$(find wuji_description)/meshes/hand2/l_digit_tip_sensor_frame.glb"
+                          scale="1 ${direction} 1"/>
+                </geometry>
+            </visual>
+            <collision>
+                <geometry>
+                    <mesh filename="file://$(find wuji_description)/meshes/hand2/l_digit_tip_sensor_frame.glb"
                           scale="1 ${direction} 1"/>
                 </geometry>
@@ -529,11 +529,11 @@
             <visual>
                 <geometry>
-                    <mesh filename="file://$(find wuji_description)/meshes/hand2/left/l_digit_proximal.glb"
-                          scale="1 ${direction} 1"/>
-                </geometry>
-            </visual>
-            <collision>
-                <geometry>
-                    <mesh filename="file://$(find wuji_description)/meshes/hand2/left/l_digit_proximal.glb"
+                    <mesh filename="file://$(find wuji_description)/meshes/hand2/l_digit_proximal.glb"
+                          scale="1 ${direction} 1"/>
+                </geometry>
+            </visual>
+            <collision>
+                <geometry>
+                    <mesh filename="file://$(find wuji_description)/meshes/hand2/l_digit_proximal.glb"
                           scale="1 ${direction} 1"/>
                 </geometry>
@@ -559,11 +559,11 @@
             <visual>
                 <geometry>
-                    <mesh filename="file://$(find wuji_description)/meshes/hand2/left/l_digit_proximal_abd.glb"
-                          scale="1 ${direction} 1"/>
-                </geometry>
-            </visual>
-            <collision>
-                <geometry>
-                    <mesh filename="file://$(find wuji_description)/meshes/hand2/left/l_digit_proximal_abd.glb"
+                    <mesh filename="file://$(find wuji_description)/meshes/hand2/l_digit_proximal_abd.glb"
+                          scale="1 ${direction} 1"/>
+                </geometry>
+            </visual>
+            <collision>
+                <geometry>
+                    <mesh filename="file://$(find wuji_description)/meshes/hand2/l_digit_proximal_abd.glb"
                           scale="1 ${direction} 1"/>
                 </geometry>
@@ -588,11 +588,11 @@
             <visual>
                 <geometry>
-                    <mesh filename="file://$(find wuji_description)/meshes/hand2/left/l_digit_middle.glb"
-                          scale="1 ${direction} 1"/>
-                </geometry>
-            </visual>
-            <collision>
-                <geometry>
-                    <mesh filename="file://$(find wuji_description)/meshes/hand2/left/l_digit_middle.glb"
+                    <mesh filename="file://$(find wuji_description)/meshes/hand2/l_digit_middle.glb"
+                          scale="1 ${direction} 1"/>
+                </geometry>
+            </visual>
+            <collision>
+                <geometry>
+                    <mesh filename="file://$(find wuji_description)/meshes/hand2/l_digit_middle.glb"
                           scale="1 ${direction} 1"/>
                 </geometry>
@@ -617,11 +617,11 @@
             <visual>
                 <geometry>
-                    <mesh filename="file://$(find wuji_description)/meshes/hand2/left/l_digit_distal.glb"
-                          scale="1 ${direction} 1"/>
-                </geometry>
-            </visual>
-            <collision>
-                <geometry>
-                    <mesh filename="file://$(find wuji_description)/meshes/hand2/left/l_digit_distal.glb"
+                    <mesh filename="file://$(find wuji_description)/meshes/hand2/l_digit_distal.glb"
+                          scale="1 ${direction} 1"/>
+                </geometry>
+            </visual>
+            <collision>
+                <geometry>
+                    <mesh filename="file://$(find wuji_description)/meshes/hand2/l_digit_distal.glb"
                           scale="1 ${direction} 1"/>
                 </geometry>
@@ -652,11 +652,11 @@
             <visual>
                 <geometry>
-                    <mesh filename="file://$(find wuji_description)/meshes/hand2/left/l_digit_tip_sensor_frame.glb"
-                          scale="1 ${direction} 1"/>
-                </geometry>
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
File: dexhands/wuji_description/xacro/ros2_control/hand.xacro (robot description, xacro)
@@ -9,9 +9,8 @@
     <joint name="world_fixed" type="fixed">
         <parent link="world"/>
-        <!-- mount exists only for hand2 -->
-        <xacro:if value="${'$(arg type)' == 'hand2' and '$(arg use_mount)' == 'true'}">
+        <xacro:if value="${'$(arg use_mount)' == 'true'}">
             <child link="mount"/>
         </xacro:if>
-        <xacro:unless value="${'$(arg type)' == 'hand2' and '$(arg use_mount)' == 'true'}">
+        <xacro:unless value="${'$(arg use_mount)' == 'true'}">
             <child link="hand_base"/>
         </xacro:unless>
@@ -48,12 +47,6 @@
             </xacro:if>
         </hardware>
-        <xacro:if value="${'$(arg type)' == 'hand2'}">
-            <xacro:include filename="$(find wuji_description)/xacro/ros2_control/hand2.xacro"/>
-            <xacro:wuji_hand2_interfaces name=""/>
-        </xacro:if>
-        <xacro:if value="${'$(arg type)' == 'hand1'}">
-            <xacro:include filename="$(find wuji_description)/xacro/ros2_control/hand1.xacro"/>
-            <xacro:wuji_hand1_interfaces name=""/>
-        </xacro:if>
+        <xacro:include filename="$(find wuji_description)/xacro/ros2_control/hand2.xacro"/>
+        <xacro:wuji_hand2_interfaces name=""/>
     </ros2_control>
     <xacro:if value="$(arg gazebo)">
