Commit message: fix hand2 z direction

File: dexhands/wuji_description/xacro/hand2.xacro (robot description, xacro)
@@ -5,4 +5,9 @@
   thumb_mcp / pinky_mcp_flex: forced mirror (motion-control; ~1-3 mm tip FK vs official right).
   Meshes: left STL + Y-scale; four-finger digit_* share (pinky proximal_abd/middle unique).
+  Frame convention (fa_w2 / dexhands-aligned):
+    hand_base  — external wrist; +Z = finger extension (like LinkerHand O6)
+    wrist      — official beta2 wrist geometry/kinematics (−Z fingers in that frame)
+    wrist_align — fixed R_x(pi) maps official −Z onto hand_base +Z
+  Joint angles / ros2_control names are unchanged (HI ↔ SDK still joint-space).
 -->
 <robot xmlns:xacro="http://www.ros.org/wiki/xacro">
@@ -33,11 +38,26 @@
       </collision>
     </link>
+    <!-- Official mount→wrist = Trans(t); with wrist_align=R_x(pi): mount→hand_base = Trans(t)*R_x(pi). -->
     <joint name="${prefix}wrist_fixed" type="fixed">
-      <origin xyz="0.003 -0.00030011 -0.0285" rpy="0 0 0"/>
+      <origin xyz="0.003 -0.00030011 -0.0285" rpy="${radians(180)} 0 0"/>
       <parent link="${prefix}mount"/>
       <child link="${prefix}hand_base"/>
     </joint>
     </xacro:if>
+    <!-- External wrist frame: +Z along fingers (dexhands / fa_w2). -->
     <link name="${prefix}hand_base">
+      <inertial>
+        <origin xyz="0 0 0" rpy="0 0 0"/>
+        <mass value="0.001"/>
+        <inertia ixx="1e-9" ixy="0" ixz="0" iyy="1e-9" iyz="0" izz="1e-9"/>
+      </inertial>
+    </link>
+    <joint name="${prefix}wrist_align" type="fixed">
+      <origin xyz="0 0 0" rpy="${radians(180)} 0 0"/>
+      <parent link="${prefix}hand_base"/>
+      <child link="${prefix}wrist"/>
+    </joint>
+    <!-- Official beta2 wrist (mesh + finger parents); fingers extend in −Z of this frame. -->
+    <link name="${prefix}wrist">
       <inertial>
         <origin xyz="-0.00354846481181 ${direction*0.00346683963964} -0.0356860644391" rpy="0 0 0"/>
@@ -85,5 +105,5 @@
     <joint name="${prefix}thumb_cmc_flex" type="${joint_type}">
       <origin xyz="0.017208 ${direction*-0.008138} -0.01646" rpy="${direction*1.6615} -1.0591 ${direction*-1.9919}"/>
-      <parent link="${prefix}hand_base"/>
+      <parent link="${prefix}wrist"/>
       <child link="${prefix}thumb_proximal"/>
       <xacro:unless value="${fixed_joints}">
@@ -242,5 +262,5 @@
     <joint name="${prefix}index_finger_mcp_flex" type="${joint_type}">
       <origin xyz="0.0226524150577 ${direction*0.00332515884505} -0.0699780241478" rpy="${direction*0.0397801377023} -0.136929341253 ${direction*-0.10040392464}"/>
-      <parent link="${prefix}hand_base"/>
+      <parent link="${prefix}wrist"/>
       <child link="${prefix}index_finger_proximal"/>
       <xacro:unless value="${fixed_joints}">
@@ -399,5 +419,5 @@
     <joint name="${prefix}middle_finger_mcp_flex" type="${joint_type}">
       <origin xyz="0.000943093646039 ${direction*0.00830301349135} -0.0739154421481" rpy="${direction*0.0339135947071} 0.0111579717229 ${direction*0.000715284906568}"/>
-      <parent link="${prefix}hand_base"/>
+      <parent link="${prefix}wrist"/>
       <child link="${prefix}middle_finger_proximal"/>
       <xacro:unless value="${fixed_joints}">
@@ -556,5 +576,5 @@
     <joint name="${prefix}ring_mcp_flex" type="${joint_type}">
       <origin xyz="-0.019752 ${direction*0.0055929} -0.065397" rpy="${direction*0.016663} 0.14175 ${direction*0.068321}"/>
-      <parent link="${prefix}hand_base"/>
+      <parent link="${prefix}wrist"/>
       <child link="${prefix}ring_proximal"/>
       <xacro:unless value="${fixed_joints}">
@@ -713,5 +733,5 @@
     <joint name="${prefix}pinky_mcp_flex" type="${joint_type}">
       <origin xyz="-0.0373572872886 ${direction*0.000733759922595} -0.0552917010368" rpy="${direction*0.00981701706873} 0.24897582673 ${direction*0.13602514716}"/>
-      <parent link="${prefix}hand_base"/>
+      <parent link="${prefix}wrist"/>
       <child link="${prefix}pinky_proximal"/>
       <xacro:unless value="${fixed_joints}">
@@ -848,5 +868,5 @@
     <link name="${prefix}eef"/>
     <joint name="${prefix}eef_joint" type="fixed">
-      <origin xyz="0 0 0" rpy="0 0 0"/>
+      <origin xyz="0 0 0.07" rpy="0 0 0"/>
       <parent link="${prefix}hand_base"/>
       <child link="${prefix}eef"/>

Commit message: add wuji hand2 glb

File: dexhands/wuji_description/xacro/hand2.xacro (robot description, xacro)
@@ -4,5 +4,6 @@
   Source: wuji-description/hand2/hand2_beta2 left/right ROS URDFs.
   thumb_mcp / pinky_mcp_flex: forced mirror (motion-control; ~1-3 mm tip FK vs official right).
-  Meshes: left STL + Y-scale; four-finger digit_* share (pinky proximal_abd/middle unique).
+  Meshes: left glb + Y-scale; index/middle/ring share digit_* ;
+  pinky uses l_pinky_proximal + unique proximal_abd/middle; distal/tip_sensor share digit_*.
   Frame convention (fa_w2 / dexhands-aligned):
     hand_base  — external wrist; +Z = finger extension (like LinkerHand O6)
@@ -25,14 +26,11 @@
         <origin xyz="0 0 0" rpy="0 0 0"/>
         <geometry>
-          <mesh filename="file://$(find wuji_description)/meshes/hand2/left/l_mount.STL" scale="1 ${direction} 1"/>
-        </geometry>
-        <material name="">
-          <color rgba="0.627450980392157 0.627450980392157 0.627450980392157 1"/>
-        </material>
-      </visual>
-      <collision>
-        <origin xyz="0 0 0" rpy="0 0 0"/>
-        <geometry>
-          <mesh filename="file://$(find wuji_description)/meshes/hand2/left/l_mount.STL" scale="1 ${direction} 1"/>
+          <mesh filename="package://wuji_description/meshes/hand2/left/l_mount.glb" scale="1 ${direction} 1"/>
+        </geometry>
+      </visual>
+      <collision>
+        <origin xyz="0 0 0" rpy="0 0 0"/>
+        <geometry>
+          <mesh filename="package://wuji_description/meshes/hand2/left/l_mount.glb" scale="1 ${direction} 1"/>
         </geometry>
       </collision>
@@ -68,14 +66,11 @@
         <origin xyz="0 0 0" rpy="0 0 0"/>
         <geometry>
-          <mesh filename="file://$(find wuji_description)/meshes/hand2/left/l_wrist.STL" scale="1 ${direction} 1"/>
-        </geometry>
-        <material name="">
-          <color rgba="0.792156862745098 0.819607843137255 0.933333333333333 1"/>
-        </material>
-      </visual>
-      <collision>
-        <origin xyz="0 0 0" rpy="0 0 0"/>
-        <geometry>
-          <mesh filename="file://$(find wuji_description)/meshes/hand2/left/l_wrist.STL" scale="1 ${direction} 1"/>
+          <mesh filename="package://wuji_description/meshes/hand2/left/l_wrist.glb" scale="1 ${direction} 1"/>
+        </geometry>
+      </visual>
+      <collision>
+        <origin xyz="0 0 0" rpy="0 0 0"/>
+        <geometry>
+          <mesh filename="package://wuji_description/meshes/hand2/left/l_wrist.glb" scale="1 ${direction} 1"/>
         </geometry>
       </collision>
@@ -90,14 +85,11 @@
         <origin xyz="0 0 0" rpy="0 0 0"/>
         <geometry>
-          <mesh filename="file://$(find wuji_description)/meshes/hand2/left/l_thumb_proximal.STL" scale="1 ${direction} 1"/>
-        </geometry>
-        <material name="">
-          <color rgba="0.627450980392157 0.627450980392157 0.627450980392157 1"/>
-        </material>
-      </visual>
-      <collision>
-        <origin xyz="0 0 0" rpy="0 0 0"/>
-        <geometry>
-          <mesh filename="file://$(find wuji_description)/meshes/hand2/left/l_thumb_proximal.STL" scale="1 ${direction} 1"/>
+          <mesh filename="package://wuji_description/meshes/hand2/left/l_thumb_proximal.glb" scale="1 ${direction} 1"/>
+        </geometry>
+      </visual>
+      <collision>
+        <origin xyz="0 0 0" rpy="0 0 0"/>
+        <geometry>
+          <mesh filename="package://wuji_description/meshes/hand2/left/l_thumb_proximal.glb" scale="1 ${direction} 1"/>
         </geometry>
       </collision>
@@ -121,14 +113,11 @@
         <origin xyz="0 0 0" rpy="0 0 0"/>
         <geometry>
-          <mesh filename="file://$(find wuji_description)/meshes/hand2/left/l_thumb_proximal_abd.STL" scale="1 ${direction} 1"/>
-        </geometry>
-        <material name="">
-          <color rgba="0.627450980392157 0.627450980392157 0.627450980392157 1"/>
-        </material>
-      </visual>
-      <collision>
-        <origin xyz="0 0 0" rpy="0 0 0"/>
-        <geometry>
-          <mesh filename="file://$(find wuji_description)/meshes/hand2/left/l_thumb_proximal_abd.STL" scale="1 ${direction} 1"/>
+          <mesh filename="package://wuji_description/meshes/hand2/left/l_thumb_proximal_abd.glb" scale="1 ${direction} 1"/>
+        </geometry>
+      </visual>
+      <collision>
+        <origin xyz="0 0 0" rpy="0 0 0"/>
+        <geometry>
+          <mesh filename="package://wuji_description/meshes/hand2/left/l_thumb_proximal_abd.glb" scale="1 ${direction} 1"/>
         </geometry>
       </collision>
@@ -152,14 +141,11 @@
         <origin xyz="0 0 0" rpy="0 0 0"/>
         <geometry>
-          <mesh filename="file://$(find wuji_description)/meshes/hand2/left/l_thumb_middle.STL" scale="1 ${direction} 1"/>
-        </geometry>
-        <material name="">
-          <color rgba="0.627450980392157 0.627450980392157 0.627450980392157 1"/>
-        </material>
-      </visual>
-      <collision>
-        <origin xyz="0 0 0" rpy="0 0 0"/>
-        <geometry>
-          <mesh filename="file://$(find wuji_description)/meshes/hand2/left/l_thumb_middle.STL" scale="1 ${direction} 1"/>
+          <mesh filename="package://wuji_description/meshes/hand2/left/l_thumb_middle.glb" scale="1 ${direction} 1"/>
+        </geometry>
+      </visual>
+      <collision>
+        <origin xyz="0 0 0" rpy="0 0 0"/>
+        <geometry>
+          <mesh filename="package://wuji_description/meshes/hand2/left/l_thumb_middle.glb" scale="1 ${direction} 1"/>
         </geometry>
       </collision>
@@ -183,14 +169,11 @@
         <origin xyz="0 0 0" rpy="0 0 0"/>
         <geometry>
-          <mesh filename="file://$(find wuji_description)/meshes/hand2/left/l_thumb_distal.STL" scale="1 ${direction} 1"/>
-        </geometry>
-        <material name="">
-          <color rgba="0.792156862745098 0.819607843137255 0.933333333333333 1"/>
-        </material>
-      </visual>
-      <collision>
-        <origin xyz="0 0 0" rpy="0 0 0"/>
-        <geometry>
-          <mesh filename="file://$(find wuji_description)/meshes/hand2/left/l_thumb_distal.STL" scale="1 ${direction} 1"/>
+          <mesh filename="package://wuji_description/meshes/hand2/left/l_thumb_distal.glb" scale="1 ${direction} 1"/>
+        </geometry>
+      </visual>
+      <collision>
+        <origin xyz="0 0 0" rpy="0 0 0"/>
+        <geometry>
+          <mesh filename="package://wuji_description/meshes/hand2/left/l_thumb_distal.glb" scale="1 ${direction} 1"/>
         </geometry>
       </collision>
@@ -220,14 +203,11 @@
         <origin xyz="0 0 0" rpy="0 0 0"/>
         <geometry>
-          <mesh filename="file://$(find wuji_description)/meshes/hand2/left/l_thumb_tip_sensor_frame.STL" scale="1 ${direction} 1"/>
-        </geometry>
-        <material name="">
-          <color rgba="0.55 0.78 0.95 1"/>
-        </material>
-      </visual>
-      <collision>
-        <origin xyz="0 0 0" rpy="0 0 0"/>
-        <geometry>
-          <mesh filename="file://$(find wuji_description)/meshes/hand2/left/l_thumb_tip_sensor_frame.STL" scale="1 ${direction} 1"/>
+          <mesh filename="package://wuji_description/meshes/hand2/left/l_thumb_tip_sensor_frame.glb" scale="1 ${direction} 1"/>
+        </geometry>
+      </visual>
+      <collision>
+        <origin xyz="0 0 0" rpy="0 0 0"/>
+        <geometry>
+          <mesh filename="package://wuji_description/meshes/hand2/left/l_thumb_tip_sensor_frame.glb" scale="1 ${direction} 1"/>
         </geometry>
       </collision>
@@ -247,14 +227,11 @@
         <origin xyz="0 0 0" rpy="0 0 0"/>
         <geometry>
-          <mesh filename="file://$(find wuji_description)/meshes/hand2/left/l_digit_proximal.STL" scale="1 ${direction} 1"/>
-        </geometry>
-        <material name="">
-          <color rgba="1 1 1 1"/>
-        </material>
-      </visual>
-      <collision>
-        <origin xyz="0 0 0" rpy="0 0 0"/>
-        <geometry>
-          <mesh filename="file://$(find wuji_description)/meshes/hand2/left/l_digit_proximal.STL" scale="1 ${direction} 1"/>
+          <mesh filename="package://wuji_description/meshes/hand2/left/l_digit_proximal.glb" scale="1 ${direction} 1"/>
+        </geometry>
+      </visual>
+      <collision>
+        <origin xyz="0 0 0" rpy="0 0 0"/>
+        <geometry>
+          <mesh filename="package://wuji_description/meshes/hand2/left/l_digit_proximal.glb" scale="1 ${direction} 1"/>
         </geometry>
       </collision>
@@ -278,14 +255,11 @@
         <origin xyz="0 0 0" rpy="0 0 0"/>
         <geometry>
-          <mesh filename="file://$(find wuji_description)/meshes/hand2/left/l_digit_proximal_abd.STL" scale="1 ${direction} 1"/>
-        </geometry>
-        <material name="">
-          <color rgba="1 1 1 1"/>
-        </material>
-      </visual>
-      <collision>
-        <origin xyz="0 0 0" rpy="0 0 0"/>
-        <geometry>
-          <mesh filename="file://$(find wuji_description)/meshes/hand2/left/l_digit_proximal_abd.STL" scale="1 ${direction} 1"/>
+          <mesh filename="package://wuji_description/meshes/hand2/left/l_digit_proximal_abd.glb" scale="1 ${direction} 1"/>
+        </geometry>
+      </visual>
+      <collision>
+        <origin xyz="0 0 0" rpy="0 0 0"/>
+        <geometry>
+          <mesh filename="package://wuji_description/meshes/hand2/left/l_digit_proximal_abd.glb" scale="1 ${direction} 1"/>
         </geometry>
       </collision>
@@ -309,14 +283,11 @@
         <origin xyz="0 0 0" rpy="0 0 0"/>
         <geometry>
-          <mesh filename="file://$(find wuji_description)/meshes/hand2/left/l_digit_middle.STL" scale="1 ${direction} 1"/>
-        </geometry>
-        <material name="">
-          <color rgba="1 1 1 1"/>
-        </material>
-      </visual>
-      <collision>
-        <origin xyz="0 0 0" rpy="0 0 0"/>
-        <geometry>
-          <mesh filename="file://$(find wuji_description)/meshes/hand2/left/l_digit_middle.STL" scale="1 ${direction} 1"/>
+          <mesh filename="package://wuji_description/meshes/hand2/left/l_digit_middle.glb" scale="1 ${direction} 1"/>
+        </geometry>
+      </visual>
+      <collision>
+        <origin xyz="0 0 0" rpy="0 0 0"/>
+        <geometry>
+          <mesh filename="package://wuji_description/meshes/hand2/left/l_digit_middle.glb" scale="1 ${direction} 1"/>
         </geometry>
       </collision>
@@ -340,14 +311,11 @@
         <origin xyz="0 0 0" rpy="0 0 0"/>
         <geometry>
-          <mesh filename="file://$(find wuji_description)/meshes/hand2/left/l_digit_distal.STL" scale="1 ${direction} 1"/>
-        </geometry>
-        <material name="">
-          <color rgba="0.792156862745098 0.819607843137255 0.933333333333333 1"/>
-        </material>
-      </visual>
-      <collision>
-        <origin xyz="0 0 0" rpy="0 0 0"/>
-        <geometry>
-          <mesh filename="file://$(find wuji_description)/meshes/hand2/left/l_digit_distal.STL" scale="1 ${direction} 1"/>
+          <mesh filename="package://wuji_description/meshes/hand2/left/l_digit_distal.glb" scale="1 ${direction} 1"/>
+        </geometry>
+      </visual>
+      <collision>
+        <origin xyz="0 0 0" rpy="0 0 0"/>
+        <geometry>
+          <mesh filename="package://wuji_description/meshes/hand2/left/l_digit_distal.glb" scale="1 ${direction} 1"/>
         </geometry>
       </collision>
@@ -377,14 +345,11 @@
         <origin xyz="0 0 0" rpy="0 0 0"/>
         <geometry>
-          <mesh filename="file://$(find wuji_description)/meshes/hand2/left/l_digit_tip_sensor_frame.STL" scale="1 ${direction} 1"/>
-        </geometry>
-        <material name="">
-          <color rgba="0.55 0.78 0.95 1"/>
-        </material>
-      </visual>
-      <collision>
-        <origin xyz="0 0 0" rpy="0 0 0"/>
-        <geometry>
-          <mesh filename="file://$(find wuji_description)/meshes/hand2/left/l_digit_tip_sensor_frame.STL" scale="1 ${direction} 1"/>
+          <mesh filename="package://wuji_description/meshes/hand2/left/l_digit_tip_sensor_frame.glb" scale="1 ${direction} 1"/>
+        </geometry>
+      </visual>
+      <collision>
+        <origin xyz="0 0 0" rpy="0 0 0"/>
+        <geometry>
+          <mesh filename="package://wuji_description/meshes/hand2/left/l_digit_tip_sensor_frame.glb" scale="1 ${direction} 1"/>
         </geometry>
       </collision>
@@ -404,14 +369,11 @@
         <origin xyz="0 0 0" rpy="0 0 0"/>
         <geometry>
-          <mesh filename="file://$(find wuji_description)/meshes/hand2/left/l_digit_proximal.STL" scale="1 ${direction} 1"/>
-        </geometry>
-        <material name="">
-          <color rgba="1 1 1 1"/>
-        </material>
-      </visual>
-      <collision>
-        <origin xyz="0 0 0" rpy="0 0 0"/>
-        <geometry>
-          <mesh filename="file://$(find wuji_description)/meshes/hand2/left/l_digit_proximal.STL" scale="1 ${direction} 1"/>
+          <mesh filename="package://wuji_description/meshes/hand2/left/l_digit_proximal.glb" scale="1 ${direction} 1"/>
+        </geometry>
+      </visual>
+      <collision>
+        <origin xyz="0 0 0" rpy="0 0 0"/>
+        <geometry>
+          <mesh filename="package://wuji_description/meshes/hand2/left/l_digit_proximal.glb" scale="1 ${direction} 1"/>
         </geometry>
       </collision>
@@ -435,14 +397,11 @@
         <origin xyz="0 0 0" rpy="0 0 0"/>
         <geometry>
-          <mesh filename="file://$(find wuji_description)/meshes/hand2/left/l_digit_proximal_abd.STL" scale="1 ${direction} 1"/>
-        </geometry>
-        <material name="">
-          <color rgba="1 1 1 1"/>
-        </material>
-      </visual>
-      <collision>
-        <origin xyz="0 0 0" rpy="0 0 0"/>
-        <geometry>
-          <mesh filename="file://$(find wuji_description)/meshes/hand2/left/l_digit_proximal_abd.STL" scale="1 ${direction} 1"/>
+          <mesh filename="package://wuji_description/meshes/hand2/left/l_digit_proximal_abd.glb" scale="1 ${direction} 1"/>
+        </geometry>
+      </visual>
+      <collision>
+        <origin xyz="0 0 0" rpy="0 0 0"/>
+        <geometry>
+          <mesh filename="package://wuji_description/meshes/hand2/left/l_digit_proximal_abd.glb" scale="1 ${direction} 1"/>
         </geometry>
       </collision>
@@ -466,14 +425,11 @@
         <origin xyz="0 0 0" rpy="0 0 0"/>
         <geometry>
-          <mesh filename="file://$(find wuji_description)/meshes/hand2/left/l_digit_middle.STL" scale="1 ${direction} 1"/>
-        </geometry>
-        <material name="">
-          <color rgba="1 1 1 1"/>
-        </material>
-      </visual>
-      <collision>
-        <origin xyz="0 0 0" rpy="0 0 0"/>
-        <geometry>
-          <mesh filename="file://$(find wuji_description)/meshes/hand2/left/l_digit_middle.STL" scale="1 ${direction} 1"/>
+          <mesh filename="package://wuji_description/meshes/hand2/left/l_digit_middle.glb" scale="1 ${direction} 1"/>
+        </geometry>
+      </visual>
+      <collision>
+        <origin xyz="0 0 0" rpy="0 0 0"/>
+        <geometry>
+          <mesh filename="package://wuji_description/meshes/hand2/left/l_digit_middle.glb" scale="1 ${direction} 1"/>
         </geometry>
       </collision>
@@ -497,14 +453,11 @@
         <origin xyz="0 0 0" rpy="0 0 0"/>
         <geometry>
-          <mesh filename="file://$(find wuji_description)/meshes/hand2/left/l_digit_distal.STL" scale="1 ${direction} 1"/>
-        </geometry>
-        <material name="">
-          <color rgba="0.792156862745098 0.819607843137255 0.933333333333333 1"/>
-        </material>
-      </visual>
-      <collision>
-        <origin xyz="0 0 0" rpy="0 0 0"/>
-        <geometry>
-          <mesh filename="file://$(find wuji_description)/meshes/hand2/left/l_digit_distal.STL" scale="1 ${direction} 1"/>
+          <mesh filename="package://wuji_description/meshes/hand2/left/l_digit_distal.glb" scale="1 ${direction} 1"/>
+        </geometry>
+      </visual>
+      <collision>
+        <origin xyz="0 0 0" rpy="0 0 0"/>
+        <geometry>
+          <mesh filename="package://wuji_description/meshes/hand2/left/l_digit_distal.glb" scale="1 ${direction} 1"/>
         </geometry>
       </collision>
@@ -534,14 +487,11 @@
         <origin xyz="0 0 0" rpy="0 0 0"/>
         <geometry>
-          <mesh filename="file://$(find wuji_description)/meshes/hand2/left/l_digit_tip_sensor_frame.STL" scale="1 ${direction} 1"/>
-        </geometry>
-        <material name="">
-          <color rgba="0.55 0.78 0.95 1"/>
-        </material>
-      </visual>
-      <collision>
-        <origin xyz="0 0 0" rpy="0 0 0"/>
-        <geometry>
-          <mesh filename="file://$(find wuji_description)/meshes/hand2/left/l_digit_tip_sensor_frame.STL" scale="1 ${direction} 1"/>
+          <mesh filename="package://wuji_description/meshes/hand2/left/l_digit_tip_sensor_frame.glb" scale="1 ${direction} 1"/>
+        </geometry>
+      </visual>
+      <collision>
+        <origin xyz="0 0 0" rpy="0 0 0"/>
+        <geometry>
+          <mesh filename="package://wuji_description/meshes/hand2/left/l_digit_tip_sensor_frame.glb" scale="1 ${direction} 1"/>
         </geometry>
       </collision>
@@ -561,14 +511,11 @@
         <origin xyz="0 0 0" rpy="0 0 0"/>
         <geometry>
-          <mesh filename="file://$(find wuji_description)/meshes/hand2/left/l_digit_proximal.STL" scale="1 ${direction} 1"/>
-        </geometry>
-        <material name="">
-          <color rgba="1 1 1 1"/>
-        </material>
-      </visual>
-      <collision>
-        <origin xyz="0 0 0" rpy="0 0 0"/>
-        <geometry>
-          <mesh filename="file://$(find wuji_description)/meshes/hand2/left/l_digit_proximal.STL" scale="1 ${direction} 1"/>
+          <mesh filename="package://wuji_description/meshes/hand2/left/l_digit_proximal.glb" scale="1 ${direction} 1"/>
+        </geometry>
+      </visual>
+      <collision>
+        <origin xyz="0 0 0" rpy="0 0 0"/>
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