Commit message: Accept optional rw_rate on Freedom, Inspire, and XHand1 side systems.
Omit the ros2_control attribute when unset so controller_manager rate remains the default.

Co-authored-by: Cursor <cursoragent@cursor.com>

File: dexhands/freedom_description/xacro/ros2_control/side_systems.xacro (robot description, xacro)
@@ -3,36 +3,52 @@
   <xacro:include filename="$(find freedom_description)/xacro/ros2_control/freedomv1.xacro"/>
   <xacro:include filename="$(find freedom_description)/xacro/ros2_control/freedomv2.xacro"/>
-  <xacro:macro name="freedom_rs485_side_system" params="side serial_port slave_id:=auto baudrate:=115200 type:=freedomv1 command_speed:=100">
-    <ros2_control name="${type}_${side}_system" type="system">
-      <hardware>
-        <plugin>modbus_ros2_control/FreedomRS485Hardware</plugin>
-        <param name="serial_port">${serial_port}</param>
-        <param name="hand_side">${side}</param>
-        <param name="slave_id">${slave_id}</param>
-        <param name="baudrate">${baudrate}</param>
-        <param name="protocol_version">${type}</param>
-        <param name="command_speed">${command_speed}</param>
-        <param name="read_feedback">true</param>
-        <param name="feedback_timeout_ms">50</param>
-      </hardware>
-      <xacro:if value="${type == 'freedomv2' or type == 'freedom_v2'}">
-        <xacro:freedomv2_interfaces name="${side}_hand"/>
-      </xacro:if>
-      <xacro:unless value="${type == 'freedomv2' or type == 'freedom_v2'}">
+  <xacro:macro name="side_ros2_control_system" params="name rw_rate:='' *contents">
+    <xacro:if value="${rw_rate != ''}">
+      <ros2_control name="${name}" type="system" rw_rate="${rw_rate}">
+        <xacro:insert_block name="contents"/>
+      </ros2_control>
+    </xacro:if>
+    <xacro:unless value="${rw_rate != ''}">
+      <ros2_control name="${name}" type="system">
+        <xacro:insert_block name="contents"/>
+      </ros2_control>
+    </xacro:unless>
+  </xacro:macro>
+  <xacro:macro name="freedom_rs485_side_system" params="side serial_port slave_id:=auto baudrate:=115200 type:=freedomv1 command_speed:=100 rw_rate:=''">
+    <xacro:side_ros2_control_system name="${type}_${side}_system" rw_rate="${rw_rate}">
+      <contents>
+        <hardware>
+          <plugin>modbus_ros2_control/FreedomRS485Hardware</plugin>
+          <param name="serial_port">${serial_port}</param>
+          <param name="hand_side">${side}</param>
+          <param name="slave_id">${slave_id}</param>
+          <param name="baudrate">${baudrate}</param>
+          <param name="protocol_version">${type}</param>
+          <param name="command_speed">${command_speed}</param>
+          <param name="read_feedback">true</param>
+          <param name="feedback_timeout_ms">50</param>
+        </hardware>
+        <xacro:if value="${type == 'freedomv2' or type == 'freedom_v2'}">
+          <xacro:freedomv2_interfaces name="${side}_hand"/>
+        </xacro:if>
+        <xacro:unless value="${type == 'freedomv2' or type == 'freedom_v2'}">
+          <xacro:freedom_interfaces name="${side}_hand"/>
+        </xacro:unless>
+      </contents>
+    </xacro:side_ros2_control_system>
+  </xacro:macro>
+  <xacro:macro name="freedom_can_side_system" params="side can_interface device_id rw_rate:=''">
+    <xacro:side_ros2_control_system name="freedom_v1_${side}_can_system" rw_rate="${rw_rate}">
+      <contents>
+        <hardware>
+          <plugin>can_ros2_control/FreedomCanHardware</plugin>
+          <param name="can_interface">${can_interface}</param>
+          <param name="device_id">${device_id}</param>
+          <param name="read_feedback">true</param>
+          <param name="feedback_timeout_ms">1</param>
+        </hardware>
         <xacro:freedom_interfaces name="${side}_hand"/>
-      </xacro:unless>
-    </ros2_control>
-  </xacro:macro>
-  <xacro:macro name="freedom_can_side_system" params="side can_interface device_id">
-    <ros2_control name="freedom_v1_${side}_can_system" type="system">
-      <hardware>
-        <plugin>can_ros2_control/FreedomCanHardware</plugin>
-        <param name="can_interface">${can_interface}</param>
-        <param name="device_id">${device_id}</param>
-        <param name="read_feedback">true</param>
-        <param name="feedback_timeout_ms">1</param>
-      </hardware>
-      <xacro:freedom_interfaces name="${side}_hand"/>
-    </ros2_control>
+      </contents>
+    </xacro:side_ros2_control_system>
   </xacro:macro>
 </robot>

File: dexhands/xhand1_description/xacro/ros2_control/side_systems.xacro (robot description, xacro)
@@ -100,19 +100,33 @@
     </joint>
   </xacro:macro>
-  <xacro:macro name="xhand1_rs485_side_system" params="side serial_port baudrate:=3000000 host_id:=0xFE hand_id:=0">
-    <ros2_control name="xhand1_${side}_system" type="system">
-      <hardware>
-        <plugin>modbus_ros2_control/XHand1RS485Hardware</plugin>
-        <param name="serial_port">${serial_port}</param>
-        <param name="baudrate">${baudrate}</param>
-        <param name="host_id">${host_id}</param>
-        <param name="hand_id">${hand_id}</param>
-        <param name="require_initial_feedback">true</param>
-        <param name="feedback_timeout_ms">50</param>
-        <param name="background_period_ms">12</param>
-        <param name="control_mode">3</param>
-      </hardware>
-      <xacro:xhand1_interfaces name="${side}_hand"/>
-    </ros2_control>
+  <xacro:macro name="side_ros2_control_system" params="name rw_rate:='' *contents">
+    <xacro:if value="${rw_rate != ''}">
+      <ros2_control name="${name}" type="system" rw_rate="${rw_rate}">
+        <xacro:insert_block name="contents"/>
+      </ros2_control>
+    </xacro:if>
+    <xacro:unless value="${rw_rate != ''}">
+      <ros2_control name="${name}" type="system">
+        <xacro:insert_block name="contents"/>
+      </ros2_control>
+    </xacro:unless>
+  </xacro:macro>
+  <xacro:macro name="xhand1_rs485_side_system" params="side serial_port baudrate:=3000000 host_id:=0xFE hand_id:=0 rw_rate:=''">
+    <xacro:side_ros2_control_system name="xhand1_${side}_system" rw_rate="${rw_rate}">
+      <contents>
+        <hardware>
+          <plugin>modbus_ros2_control/XHand1RS485Hardware</plugin>
+          <param name="serial_port">${serial_port}</param>
+          <param name="baudrate">${baudrate}</param>
+          <param name="host_id">${host_id}</param>
+          <param name="hand_id">${hand_id}</param>
+          <param name="require_initial_feedback">true</param>
+          <param name="feedback_timeout_ms">50</param>
+          <param name="background_period_ms">12</param>
+          <param name="control_mode">3</param>
+        </hardware>
+        <xacro:xhand1_interfaces name="${side}_hand"/>
+      </contents>
+    </xacro:side_ros2_control_system>
   </xacro:macro>
 </robot>

File: gripper/inspire_description/xacro/ros2_control/side_systems.xacro (robot description, xacro)
@@ -3,39 +3,55 @@
   <xacro:include filename="$(find inspire_description)/xacro/ros2_control/RH56E2.xacro"/>
   <xacro:include filename="$(find inspire_description)/xacro/ros2_control/RH56F2.xacro"/>
-  <xacro:macro name="inspire_rs485_side_system" params="side serial_port baudrate:=115200 slave_id:=auto read_feedback:=true hand_type:=inspire_e2">
-    <ros2_control name="${hand_type}_${side}_system" type="system">
-      <hardware>
-        <plugin>modbus_ros2_control/InspireHandHardware</plugin>
-        <param name="serial_port">${serial_port}</param>
-        <param name="hand_side">${side}</param>
-        <param name="baudrate">${baudrate}</param>
-        <param name="slave_id">${slave_id}</param>
-        <param name="read_feedback">${read_feedback}</param>
-      </hardware>
-      <xacro:if value="${hand_type == 'inspire_e2'}">
-        <xacro:inspire_rh56e2_interfaces name="${side}_hand"/>
-      </xacro:if>
-      <xacro:if value="${hand_type == 'inspire_f2'}">
-        <xacro:inspire_rh56f2_interfaces name="${side}_hand"/>
-      </xacro:if>
-    </ros2_control>
+  <xacro:macro name="side_ros2_control_system" params="name rw_rate:='' *contents">
+    <xacro:if value="${rw_rate != ''}">
+      <ros2_control name="${name}" type="system" rw_rate="${rw_rate}">
+        <xacro:insert_block name="contents"/>
+      </ros2_control>
+    </xacro:if>
+    <xacro:unless value="${rw_rate != ''}">
+      <ros2_control name="${name}" type="system">
+        <xacro:insert_block name="contents"/>
+      </ros2_control>
+    </xacro:unless>
   </xacro:macro>
-  <xacro:macro name="inspire_canfd_side_system" params="side can_interface hand_id:=auto read_feedback:=true hand_type:=inspire_e2">
-    <ros2_control name="${hand_type}_${side}_canfd_system" type="system">
-      <hardware>
-        <plugin>can_ros2_control/InspireCanfdHardware</plugin>
-        <param name="can_interface">${can_interface}</param>
-        <param name="hand_side">${side}</param>
-        <param name="hand_id">${hand_id}</param>
-        <param name="read_feedback">${read_feedback}</param>
-        <param name="feedback_timeout_ms">2</param>
-      </hardware>
-      <xacro:if value="${hand_type == 'inspire_e2'}">
-        <xacro:inspire_rh56e2_interfaces name="${side}_hand"/>
-      </xacro:if>
-      <xacro:if value="${hand_type == 'inspire_f2'}">
-        <xacro:inspire_rh56f2_interfaces name="${side}_hand"/>
-      </xacro:if>
-    </ros2_control>
+  <xacro:macro name="inspire_rs485_side_system" params="side serial_port baudrate:=115200 slave_id:=auto read_feedback:=true hand_type:=inspire_e2 rw_rate:=''">
+    <xacro:side_ros2_control_system name="${hand_type}_${side}_system" rw_rate="${rw_rate}">
+      <contents>
+        <hardware>
+          <plugin>modbus_ros2_control/InspireHandHardware</plugin>
+          <param name="serial_port">${serial_port}</param>
+          <param name="hand_side">${side}</param>
+          <param name="baudrate">${baudrate}</param>
+          <param name="slave_id">${slave_id}</param>
+          <param name="read_feedback">${read_feedback}</param>
+        </hardware>
+        <xacro:if value="${hand_type == 'inspire_e2'}">
+          <xacro:inspire_rh56e2_interfaces name="${side}_hand"/>
+        </xacro:if>
+        <xacro:if value="${hand_type == 'inspire_f2'}">
+          <xacro:inspire_rh56f2_interfaces name="${side}_hand"/>
+        </xacro:if>
+      </contents>
+    </xacro:side_ros2_control_system>
+  </xacro:macro>
+  <xacro:macro name="inspire_canfd_side_system" params="side can_interface hand_id:=auto read_feedback:=true hand_type:=inspire_e2 rw_rate:=''">
+    <xacro:side_ros2_control_system name="${hand_type}_${side}_canfd_system" rw_rate="${rw_rate}">
+      <contents>
+        <hardware>
+          <plugin>can_ros2_control/InspireCanfdHardware</plugin>
+          <param name="can_interface">${can_interface}</param>
+          <param name="hand_side">${side}</param>
+          <param name="hand_id">${hand_id}</param>
+          <param name="read_feedback">${read_feedback}</param>
+          <param name="feedback_timeout_ms">2</param>
+        </hardware>
+        <xacro:if value="${hand_type == 'inspire_e2'}">
+          <xacro:inspire_rh56e2_interfaces name="${side}_hand"/>
+        </xacro:if>
+        <xacro:if value="${hand_type == 'inspire_f2'}">
+          <xacro:inspire_rh56f2_interfaces name="${side}_hand"/>
+        </xacro:if>
+      </contents>
+    </xacro:side_ros2_control_system>
   </xacro:macro>
 </robot>
