Commit message: Share side_ros2_control_system from robot_common_launch.
Keep one optional-rw_rate wrapper so each EE package does not copy the same xacro helper.

File: dexhands/freedom_description/xacro/ros2_control/side_systems.xacro (robot description, xacro)
@@ -1,18 +1,7 @@
 <?xml version="1.0"?>
 <robot xmlns:xacro="http://www.ros.org/wiki/xacro">
+  <xacro:include filename="$(find robot_common_launch)/xacro/ros2_control/side_system.xacro"/>
   <xacro:include filename="$(find freedom_description)/xacro/ros2_control/freedomv1.xacro"/>
   <xacro:include filename="$(find freedom_description)/xacro/ros2_control/freedomv2.xacro"/>
-  <xacro:macro name="side_ros2_control_system" params="name rw_rate:='' *contents">
-    <xacro:if value="${rw_rate != ''}">
-      <ros2_control name="${name}" type="system" rw_rate="${rw_rate}">
-        <xacro:insert_block name="contents"/>
-      </ros2_control>
-    </xacro:if>
-    <xacro:unless value="${rw_rate != ''}">
-      <ros2_control name="${name}" type="system">
-        <xacro:insert_block name="contents"/>
-      </ros2_control>
-    </xacro:unless>
-  </xacro:macro>
   <xacro:macro name="freedom_rs485_side_system" params="side serial_port slave_id:=auto baudrate:=115200 type:=freedomv1 command_speed:=100 rw_rate:=''">
     <xacro:side_ros2_control_system name="${type}_${side}_system" rw_rate="${rw_rate}">

File: dexhands/linkerhand_description/xacro/ros2_control/side_systems.xacro (robot description, xacro)
@@ -1,18 +1,7 @@
 <?xml version="1.0"?>
 <robot xmlns:xacro="http://www.ros.org/wiki/xacro">
+  <xacro:include filename="$(find robot_common_launch)/xacro/ros2_control/side_system.xacro"/>
   <xacro:include filename="$(find linkerhand_description)/xacro/ros2_control/o6.xacro"/>
   <xacro:include filename="$(find linkerhand_description)/xacro/ros2_control/o7.xacro"/>
-  <xacro:macro name="side_ros2_control_system" params="name rw_rate:='' *contents">
-    <xacro:if value="${rw_rate != ''}">
-      <ros2_control name="${name}" type="system" rw_rate="${rw_rate}">
-        <xacro:insert_block name="contents"/>
-      </ros2_control>
-    </xacro:if>
-    <xacro:unless value="${rw_rate != ''}">
-      <ros2_control name="${name}" type="system">
-        <xacro:insert_block name="contents"/>
-      </ros2_control>
-    </xacro:unless>
-  </xacro:macro>
   <xacro:macro name="side_usb_hand_system" params="side hand_type serial_port rw_rate:=''">
     <xacro:property name="usb_hand_system_name" value="${str('linkerhand_7' if hand_type == 'linkerhand_o7' else 'linkerhand_6')}"/>

File: dexhands/theohand_description/xacro/ros2_control/side_systems.xacro (robot description, xacro)
@@ -1,17 +1,6 @@
 <?xml version="1.0"?>
 <robot xmlns:xacro="http://www.ros.org/wiki/xacro">
+  <xacro:include filename="$(find robot_common_launch)/xacro/ros2_control/side_system.xacro"/>
   <xacro:include filename="$(find theohand_description)/xacro/ros2_control/std16a.xacro"/>
-  <xacro:macro name="side_ros2_control_system" params="name rw_rate:='' *contents">
-    <xacro:if value="${rw_rate != ''}">
-      <ros2_control name="${name}" type="system" rw_rate="${rw_rate}">
-        <xacro:insert_block name="contents"/>
-      </ros2_control>
-    </xacro:if>
-    <xacro:unless value="${rw_rate != ''}">
-      <ros2_control name="${name}" type="system">
-        <xacro:insert_block name="contents"/>
-      </ros2_control>
-    </xacro:unless>
-  </xacro:macro>
   <xacro:macro name="theohand_usb_side_system" params="side serial_port baudrate:=115200 slave_id:=auto rw_rate:=''">
     <xacro:property name="theohand_slave_id" value="${2 if side == 'left' and slave_id == 'auto' else 1 if side == 'right' and slave_id == 'auto' else slave_id}"/>

File: dexhands/xhand1_description/xacro/ros2_control/side_systems.xacro (robot description, xacro)
@@ -1,4 +1,5 @@
 <?xml version="1.0"?>
 <robot xmlns:xacro="http://www.ros.org/wiki/xacro">
+  <xacro:include filename="$(find robot_common_launch)/xacro/ros2_control/side_system.xacro"/>
   <xacro:macro name="xhand1_interfaces" params="name">
     <xacro:property name="prefix" value="${name + '_' if name else ''}"/>
@@ -100,16 +101,4 @@
     </joint>
   </xacro:macro>
-  <xacro:macro name="side_ros2_control_system" params="name rw_rate:='' *contents">
-    <xacro:if value="${rw_rate != ''}">
-      <ros2_control name="${name}" type="system" rw_rate="${rw_rate}">
-        <xacro:insert_block name="contents"/>
-      </ros2_control>
-    </xacro:if>
-    <xacro:unless value="${rw_rate != ''}">
-      <ros2_control name="${name}" type="system">
-        <xacro:insert_block name="contents"/>
-      </ros2_control>
-    </xacro:unless>
-  </xacro:macro>
   <xacro:macro name="xhand1_rs485_side_system" params="side serial_port baudrate:=3000000 host_id:=0xFE hand_id:=0 rw_rate:=''">
     <xacro:side_ros2_control_system name="xhand1_${side}_system" rw_rate="${rw_rate}">

File: gripper/changingtek_description/xacro/ros2_control/side_systems.xacro (robot description, xacro)
@@ -1,16 +1,5 @@
 <?xml version="1.0"?>
 <robot xmlns:xacro="http://www.ros.org/wiki/xacro">
-  <xacro:macro name="side_ros2_control_system" params="name rw_rate:='' *contents">
-    <xacro:if value="${rw_rate != ''}">
-      <ros2_control name="${name}" type="system" rw_rate="${rw_rate}">
-        <xacro:insert_block name="contents"/>
-      </ros2_control>
-    </xacro:if>
-    <xacro:unless value="${rw_rate != ''}">
-      <ros2_control name="${name}" type="system">
-        <xacro:insert_block name="contents"/>
-      </ros2_control>
-    </xacro:unless>
-  </xacro:macro>
+  <xacro:include filename="$(find robot_common_launch)/xacro/ros2_control/side_system.xacro"/>
   <xacro:macro name="changingtek_usb_side_system" params="side variant serial_port rw_rate:=''">
     <xacro:side_ros2_control_system name="changingtek_${side}_system" rw_rate="${rw_rate}">

File: gripper/inspire_description/xacro/ros2_control/side_systems.xacro (robot description, xacro)
@@ -1,18 +1,7 @@
 <?xml version="1.0"?>
 <robot xmlns:xacro="http://www.ros.org/wiki/xacro">
+  <xacro:include filename="$(find robot_common_launch)/xacro/ros2_control/side_system.xacro"/>
   <xacro:include filename="$(find inspire_description)/xacro/ros2_control/RH56E2.xacro"/>
   <xacro:include filename="$(find inspire_description)/xacro/ros2_control/RH56F2.xacro"/>
-  <xacro:macro name="side_ros2_control_system" params="name rw_rate:='' *contents">
-    <xacro:if value="${rw_rate != ''}">
-      <ros2_control name="${name}" type="system" rw_rate="${rw_rate}">
-        <xacro:insert_block name="contents"/>
-      </ros2_control>
-    </xacro:if>
-    <xacro:unless value="${rw_rate != ''}">
-      <ros2_control name="${name}" type="system">
-        <xacro:insert_block name="contents"/>
-      </ros2_control>
-    </xacro:unless>
-  </xacro:macro>
   <xacro:macro name="inspire_rs485_side_system" params="side serial_port baudrate:=115200 slave_id:=auto read_feedback:=true hand_type:=inspire_e2 rw_rate:=''">
     <xacro:side_ros2_control_system name="${hand_type}_${side}_system" rw_rate="${rw_rate}">

File: gripper/jodell_description/xacro/ros2_control/side_systems.xacro (robot description, xacro)
@@ -1,16 +1,5 @@
 <?xml version="1.0"?>
 <robot xmlns:xacro="http://www.ros.org/wiki/xacro">
-  <xacro:macro name="side_ros2_control_system" params="name rw_rate:='' *contents">
-    <xacro:if value="${rw_rate != ''}">
-      <ros2_control name="${name}" type="system" rw_rate="${rw_rate}">
-        <xacro:insert_block name="contents"/>
-      </ros2_control>
-    </xacro:if>
-    <xacro:unless value="${rw_rate != ''}">
-      <ros2_control name="${name}" type="system">
-        <xacro:insert_block name="contents"/>
-      </ros2_control>
-    </xacro:unless>
-  </xacro:macro>
+  <xacro:include filename="$(find robot_common_launch)/xacro/ros2_control/side_system.xacro"/>
   <xacro:macro name="jodell_usb_side_system" params="side serial_port rw_rate:=''">
     <xacro:side_ros2_control_system name="jodell_${side}_system" rw_rate="${rw_rate}">
