Commit message: Unwrap side-system contents so ros2_control can parse the URDF.
*contents leaves a <contents> tag in the expanded robot_description; **contents inserts only the children.

Co-authored-by: Cursor <cursoragent@cursor.com>

File: robot_common_launch/xacro/ros2_control/side_system.xacro (robot description, xacro)
@@ -1,6 +1,7 @@
 <?xml version="1.0"?>
 <robot xmlns:xacro="http://www.ros.org/wiki/xacro">
-	<!-- Optional ros2_control rw_rate: omit the attribute when empty so CM rate is used. -->
-	<xacro:macro name="side_ros2_control_system" params="name rw_rate:='' *contents">
+	<!-- Optional ros2_control rw_rate: omit the attribute when empty so CM rate is used.
+	     Use **contents (not *contents): insert_block must unwrap <contents>, or URDF keeps that tag. -->
+	<xacro:macro name="side_ros2_control_system" params="name rw_rate:='' **contents">
 		<xacro:if value="${rw_rate != ''}">
 			<ros2_control name="${name}" type="system" rw_rate="${rw_rate}">
