Commit message: update param

File: dexhands/wuji_description/xacro/ros2_control/hand.xacro (robot description, xacro)
@@ -30,5 +30,5 @@
     </joint>
     <xacro:include filename="$(find wuji_description)/xacro/hand.xacro"/>
-    <ros2_control name="wuji_hand_system" type="system">
+    <ros2_control name="wuji_hand_system" type="system" rw_rate="200">
         <hardware>
             <xacro:if value="${'$(arg ros2_control_hardware_type)' == 'gz'}">

File: dexhands/wuji_description/xacro/ros2_control/hands2.xacro (robot description, xacro)
@@ -30,6 +30,6 @@
     <child link="right_hand_hand_base"/>
   </joint>
-  <xacro:macro name="wuji_hand2_side_system" params="side hand_side device_address serial_number">
-    <ros2_control name="wuji_hand2_${side}_system" type="system">
+  <xacro:macro name="wuji_hand2_side_system" params="side hand_side device_address serial_number rw_rate:=200">
+    <ros2_control name="wuji_hand2_${side}_system" type="system" rw_rate="${rw_rate}">
       <hardware>
         <xacro:if value="${'$(arg ros2_control_hardware_type)' == 'gz'}">

Commit message: update xacro

File: dexhands/wuji_description/xacro/ros2_control/hand.xacro (robot description, xacro)
@@ -6,15 +6,4 @@
     <xacro:arg name="ros2_control_hardware_type" default="mock_components"/>
     <xacro:arg name="use_mount" default="false"/>
-    <!-- Real HI (wuji_ros2_control) — unused for mock/gz/isaac -->
-    <xacro:arg name="device_address" default=""/>
-    <xacro:arg name="serial_number" default=""/>
-    <xacro:arg name="mit_kp" default="3.0"/>
-    <xacro:arg name="mit_kd" default="0.05"/>
-    <xacro:arg name="effort_limit" default="1.5"/>
-    <xacro:arg name="read_feedback" default="true"/>
-    <xacro:arg name="require_initial_feedback" default="true"/>
-    <xacro:arg name="command_deadband" default="0.0"/>
-    <xacro:arg name="connect_timeout_ms" default="5000"/>
-    <xacro:arg name="enable_timeout_s" default="5.0"/>
     <link name="world"/>
     <joint name="world_fixed" type="fixed">
@@ -54,16 +43,7 @@
                     <param name="hand_side">right</param>
                 </xacro:unless>
-                <param name="device_address">$(arg device_address)</param>
-                <xacro:if value="${'$(arg serial_number)' != ''}">
-                    <param name="serial_number">$(arg serial_number)</param>
-                </xacro:if>
-                <param name="mit_kp">$(arg mit_kp)</param>
-                <param name="mit_kd">$(arg mit_kd)</param>
-                <param name="effort_limit">$(arg effort_limit)</param>
-                <param name="read_feedback">$(arg read_feedback)</param>
-                <param name="require_initial_feedback">$(arg require_initial_feedback)</param>
-                <param name="command_deadband">$(arg command_deadband)</param>
-                <param name="connect_timeout_ms">$(arg connect_timeout_ms)</param>
-                <param name="enable_timeout_s">$(arg enable_timeout_s)</param>
+                <param name="mit_kp">3.0</param>
+                <param name="mit_kd">0.05</param>
+                <param name="effort_limit">1.5</param>
             </xacro:if>
         </hardware>

File: dexhands/wuji_description/xacro/ros2_control/hands2.xacro (robot description, xacro)
@@ -3,16 +3,4 @@
 <robot name="Wuji_hands2" xmlns:xacro="http://www.ros.org/wiki/xacro">
   <xacro:arg name="ros2_control_hardware_type" default="mock_components"/>
-  <xacro:arg name="device_address_left" default=""/>
-  <xacro:arg name="device_address_right" default=""/>
-  <xacro:arg name="serial_number_left" default=""/>
-  <xacro:arg name="serial_number_right" default=""/>
-  <xacro:arg name="mit_kp" default="3.0"/>
-  <xacro:arg name="mit_kd" default="0.05"/>
-  <xacro:arg name="effort_limit" default="1.5"/>
-  <xacro:arg name="read_feedback" default="true"/>
-  <xacro:arg name="require_initial_feedback" default="true"/>
-  <xacro:arg name="command_deadband" default="0.0"/>
-  <xacro:arg name="connect_timeout_ms" default="5000"/>
-  <xacro:arg name="enable_timeout_s" default="5.0"/>
   <xacro:include filename="$(find wuji_description)/xacro/hand2.xacro"/>
   <xacro:include filename="$(find wuji_description)/xacro/ros2_control/hand2.xacro"/>
@@ -30,5 +18,5 @@
     <child link="right_hand_hand_base"/>
   </joint>
-  <xacro:macro name="wuji_hand2_side_system" params="side hand_side device_address serial_number rw_rate:=200">
+  <xacro:macro name="wuji_hand2_side_system" params="side rw_rate:=200">
     <ros2_control name="wuji_hand2_${side}_system" type="system" rw_rate="${rw_rate}">
       <hardware>
@@ -48,17 +36,8 @@
         <xacro:if value="${'$(arg ros2_control_hardware_type)' == 'real'}">
           <plugin>wuji_ros2_control/WujiHand2Hardware</plugin>
-          <param name="hand_side">${hand_side}</param>
-          <param name="device_address">${device_address}</param>
-          <xacro:if value="${serial_number != ''}">
-            <param name="serial_number">${serial_number}</param>
-          </xacro:if>
-          <param name="mit_kp">$(arg mit_kp)</param>
-          <param name="mit_kd">$(arg mit_kd)</param>
-          <param name="effort_limit">$(arg effort_limit)</param>
-          <param name="read_feedback">$(arg read_feedback)</param>
-          <param name="require_initial_feedback">$(arg require_initial_feedback)</param>
-          <param name="command_deadband">$(arg command_deadband)</param>
-          <param name="connect_timeout_ms">$(arg connect_timeout_ms)</param>
-          <param name="enable_timeout_s">$(arg enable_timeout_s)</param>
+          <param name="hand_side">${side}</param>
+          <param name="mit_kp">3.0</param>
+          <param name="mit_kd">0.05</param>
+          <param name="effort_limit">1.5</param>
         </xacro:if>
       </hardware>
@@ -66,11 +45,5 @@
     </ros2_control>
   </xacro:macro>
-  <xacro:wuji_hand2_side_system
-    side="left" hand_side="left"
-    device_address="$(arg device_address_left)"
-    serial_number="$(arg serial_number_left)"/>
-  <xacro:wuji_hand2_side_system
-    side="right" hand_side="right"
-    device_address="$(arg device_address_right)"
-    serial_number="$(arg serial_number_right)"/>
+  <xacro:wuji_hand2_side_system side="left"/>
+  <xacro:wuji_hand2_side_system side="right"/>
 </robot>
